Commit message: perseus_description: Add CAN bus and h/w  config arguments
Exposing these as xacro arguments allows selecting multiple launch configurations without modifying raw `*.xacro` files.

File: software/ros_ws/src/perseus/description/urdf/perseus.urdf.xacro (robot description, xacro)
@@ -2,5 +2,13 @@
 <robot xmlns:xacro="http://www.ros.org/wiki/xacro" name="perseus">
   <xacro:arg name="prefix" default="" />
+  <xacro:arg name="can_bus" default="can0" />
   <xacro:arg name="use_mock_hardware" default="false" />
+  <xacro:arg name="use_legacy_hardware" default="true" />
+  <xacro:property name="use_legacy_hardware" value="$(arg use_legacy_hardware)" />
+  <xacro:property name="real_hardware_plugin"
+    value="${'perseus_hardware/McbSystemHardware' if use_legacy_hardware else 'perseus_hardware/VescSystemHardware'}" />
+  <xacro:property name="use_mock_hardware" value="$(arg use_mock_hardware)" />
+  <xacro:property name="hardware_plugin"
+    value="${'mock_components/GenericSystem' if use_mock_hardware else real_hardware_plugin}" />
   <!-- Import URDF description -->
   <xacro:include filename="$(find perseus_description)/urdf/perseus.urdf.xacro" />
@@ -11,4 +19,4 @@
   <!-- Instantiate the description and the ROS2 control information -->
   <xacro:perseus prefix="$(arg prefix)" />
-  <xacro:perseus_ros2_control name="Perseus" prefix="$(arg prefix)" use_mock_hardware="$(arg use_mock_hardware)"/>
+  <xacro:perseus_ros2_control name="Perseus" prefix="$(arg prefix)" can_bus="$(arg can_bus)" hardware_plugin="${hardware_plugin}"/>
 </robot>

File: software/ros_ws/src/perseus_description/ros2_control/perseus.ros2_control.xacro (robot description, xacro)
@@ -1,18 +1,17 @@
 <?xml version="1.0"?>
 <robot xmlns:xacro="http://www.ros.org/wiki/xacro">
-  <xacro:macro name="perseus_ros2_control" params="name prefix use_mock_hardware">
+  <xacro:macro name="perseus_ros2_control" params="name prefix can_bus hardware_plugin">
+    <xacro:property name="is_mock" value="${hardware_plugin == 'mock_components/GenericSystem'}"/>
     <ros2_control name="${name}" type="system">
-      <xacro:unless value="${use_mock_hardware}">
-        <hardware>
-          <plugin>perseus_hardware/VescSystemHardware</plugin>
-          <param name="can_bus">vcan0</param>
-        </hardware>
-      </xacro:unless>
-      <xacro:if value="${use_mock_hardware}">
-        <hardware>
-          <plugin>mock_components/GenericSystem</plugin>
+      <hardware>
+        <plugin>${hardware_plugin}</plugin>
+        <xacro:unless value="${is_mock}">
+          <param name="can_bus">${can_bus}</param>
+        </xacro:unless>
+        <xacro:if value="${is_mock}">
+          <!-- Enable velocity -> position integration over time -->
           <param name="calculate_dynamics">true</param>
-        </hardware>
-      </xacro:if>
+        </xacro:if>
+      </hardware>
       <joint name="${prefix}front_left_wheel_joint">
         <param name="id">0</param>
