Commit message: perseus_description: Add current+temperature state interfaces
Also macro-fied the definitions to avoid copy-pasting everything

File: software/ros_ws/src/perseus_description/ros2_control/perseus.ros2_control.xacro (robot description, xacro)
@@ -14,28 +14,18 @@
         </xacro:if>
       </hardware>
-      <joint name="${prefix}front_left_wheel_joint">
-        <param name="id">0</param>
-        <command_interface name="velocity"/>
-        <state_interface name="position"/>
-        <state_interface name="velocity"/>
-      </joint>
-      <joint name="${prefix}front_right_wheel_joint">
-        <param name="id">1</param>
-        <command_interface name="velocity"/>
-        <state_interface name="position"/>
-        <state_interface name="velocity"/>
-      </joint>
-      <joint name="${prefix}rear_left_wheel_joint">
-        <param name="id">2</param>
-        <command_interface name="velocity"/>
-        <state_interface name="position"/>
-        <state_interface name="velocity"/>
-      </joint>
-      <joint name="${prefix}rear_right_wheel_joint">
-        <param name="id">3</param>
-        <command_interface name="velocity"/>
-        <state_interface name="position"/>
-        <state_interface name="velocity"/>
-      </joint>
+      <xacro:macro name="ros2_control_joint" params="name id">
+        <joint name="${prefix}${name}_wheel_joint">
+          <param name="id">${id}</param>
+          <command_interface name="velocity"/>
+          <state_interface name="position"/>
+          <state_interface name="velocity"/>
+          <state_interface name="current"/>
+          <state_interface name="temperature"/>
+        </joint>
+      </xacro:macro>
+      <xacro:ros2_control_joint name="front_left" id="0"/>
+      <xacro:ros2_control_joint name="front_right" id="1"/>
+      <xacro:ros2_control_joint name="rear_left" id="2"/>
+      <xacro:ros2_control_joint name="rear_right" id="3"/>
     </ros2_control>
   </xacro:macro>

Commit message: feat: Implement running simulation using `gz`
- Created `perseus_simulation` package
- Refactored `perseus` package to remove `bringup` folder
- Modularised launch files for individual logical components
- Add `nixGL` and `nix-gl-host` to flake inputs for running RViz and Gazebo
- Clean up `ros2_control` description
- Occasional Nix code/comment cleanup
- Properly split simulation/non-sim workspaces so Gazebo is no longer included by default

Co-authored-by: Nigel H-S <1388693+DingoOz@users.noreply.github.com>

File: software/ros_ws/src/perseus_description/ros2_control/perseus.ros2_control.xacro (robot description, xacro)
@@ -1,16 +1,11 @@
 <?xml version="1.0"?>
 <robot xmlns:xacro="http://www.ros.org/wiki/xacro">
-  <xacro:macro name="perseus_ros2_control" params="name prefix can_bus hardware_plugin">
-    <xacro:property name="is_mock" value="${hardware_plugin == 'mock_components/GenericSystem'}"/>
+  <xacro:macro name="perseus_ros2_control" params="namespace:='' name prefix can_bus:='can0' hardware_plugin">
     <ros2_control name="${name}" type="system">
       <hardware>
         <plugin>${hardware_plugin}</plugin>
-        <xacro:unless value="${is_mock}">
-          <param name="can_bus">${can_bus}</param>
-        </xacro:unless>
-        <xacro:if value="${is_mock}">
-          <!-- Enable velocity -> position integration over time -->
-          <param name="calculate_dynamics">true</param>
-        </xacro:if>
+        <param name="can_bus">${can_bus}</param>
+        <!-- Enable velocity -> position integration over time for mock hardware -->
+        <param name="calculate_dynamics">true</param>
       </hardware>
       <xacro:macro name="ros2_control_joint" params="name id">
@@ -29,4 +24,15 @@
       <xacro:ros2_control_joint name="rear_right" id="3"/>
     </ros2_control>
+    <gazebo>
+      <plugin filename="libgz_ros2_control-system.so"
+        name="gz_ros2_control::GazeboSimROS2ControlPlugin">
+        <ros>
+          <namespace>${namespace}</namespace>
+          <!-- <remapping>/diff_drive_base_controller/cmd_vel:=/cmd_vel</remapping> -->
+        </ros>
+        <parameters>$(find perseus)/config/perseus_controllers.yaml</parameters>
+        <parameters>$(find perseus_simulation)/config/ros2_control_sim.yaml</parameters>
+      </plugin>
+    </gazebo>
   </xacro:macro>
 </robot>

Commit message: fix: Don't include gazebo information if not in sim

File: software/ros_ws/src/perseus_description/ros2_control/perseus.ros2_control.xacro (robot description, xacro)
@@ -24,15 +24,18 @@
       <xacro:ros2_control_joint name="rear_right" id="3"/>
     </ros2_control>
-    <gazebo>
-      <plugin filename="libgz_ros2_control-system.so"
-        name="gz_ros2_control::GazeboSimROS2ControlPlugin">
-        <ros>
-          <namespace>${namespace}</namespace>
-          <!-- <remapping>/diff_drive_base_controller/cmd_vel:=/cmd_vel</remapping> -->
-        </ros>
-        <parameters>$(find perseus)/config/perseus_controllers.yaml</parameters>
-        <parameters>$(find perseus_simulation)/config/ros2_control_sim.yaml</parameters>
-      </plugin>
-    </gazebo>
+    <xacro:property name="is_sim" value='${hardware_plugin == "gz_ros2_control/GazeboSimSystem"}' />
+    <xacro:if value="${is_sim}">
+      <gazebo>
+        <plugin filename="libgz_ros2_control-system.so"
+          name="gz_ros2_control::GazeboSimROS2ControlPlugin">
+          <ros>
+            <namespace>${namespace}</namespace>
+            <!-- <remapping>/diff_drive_base_controller/cmd_vel:=/cmd_vel</remapping> -->
+          </ros>
+          <parameters>$(find perseus)/config/perseus_controllers.yaml</parameters>
+          <parameters>$(find perseus_simulation)/config/ros2_control_sim.yaml</parameters>
+        </plugin>
+      </gazebo>
+    </xacro:if>
   </xacro:macro>
 </robot>
