File: hardware/dc-motor-driver/dc-motor-driver.kicad_pcb (KiCad board)
At the start: 2 copper layers, 100 x 90 mm, 73 parts, among them J1 DE9, J10 MOT, J12 MOT, J14 MOT, J2 VIN, J4 MOT, J6 MOT, J8 MOT, U1 DRV8874PWPR, U2 DRV8874PWPR, U3 DRV8874PWPR, U4 DRV8874PWPR, U5 DRV8874PWPR, U6 DRV8874PWPR

Commit message: feat: Routing progress
Connections:
- PCB1 pad 18: unconnected-(PCB1-A10-Pad18) -> /BANK2_ILIM
- PCB1 pad 19: /BANK2_ILIM -> /BANK3_ILIM
- R11 pad 1: /Driver_5/I_LIM -> /BANK3_ILIM
- R12 pad 1: /Driver_6/I_LIM -> /BANK3_ILIM
Routing:
- net +3V3: track 9.14 -> 182.8 mm, vias 6 -> 7
- net /BANK3_ILIM: track 0.00 -> 98.7 mm, vias 0 -> 4
- net /BANK1_~{FLT}: track 35.3 -> 128.8 mm, vias 2 -> 6
- net /BANK3_I_SENSE: track 17.0 -> 109.7 mm, vias 1 -> 4
- net /BANK1_I_SENSE: track 44.6 -> 133.6 mm, vias 2 -> 3
- net /BANK2_ILIM: track 25.6 -> 114.3 mm, vias 2 -> 5
- net /BANK2_I_SENSE: track 44.0 -> 129.5 mm, vias 2 -> 4
- net /BANK2_~{FLT}: track 35.3 -> 117.7 mm, vias 2 -> 6
- net VCC: track 134.3 -> 201.9 mm
- net Net-(PCB1-CAN_H): track 0.00 -> 53.5 mm
- net /BANK1_ILIM: track 25.6 -> 75.0 mm, vias 2 -> 4
- net Net-(PCB1-CAN_L): track 0.00 -> 47.5 mm
- net /~{SLEEP}: track 187.3 -> 155.3 mm, vias 7 -> 6
- net /MOT1_IN1: track 73.0 -> 58.3 mm, vias 2 -> 3
- net /MOT1_IN2: track 74.6 -> 60.9 mm, vias 2 -> 3
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
Commit message: feat: Layout done
Parts:
- added C37: 100n, Capacitor_SMD:C_0603_1608Metric, F.Cu at (146.1, 65.6)
- added D1: BAT54SWF, Package_TO_SOT_SMD:SOT-323_SC-70, F.Cu at (149.2, 65.7)
- added H1: MountingHole_Pad, MountingHole:MountingHole_3mm_Pad, F.Cu at (188.0, 57.0)
- added H2: MountingHole_Pad, MountingHole:MountingHole_3mm_Pad, F.Cu at (188.0, 115.0)
- added H3: MountingHole_Pad, MountingHole:MountingHole_3mm_Pad, F.Cu at (122.0, 57.0)
- added H4: MountingHole_Pad, MountingHole:MountingHole_3mm_Pad, F.Cu at (140.0, 115.0)
- added H5: MountingHole_Pad, MountingHole:MountingHole_3mm_Pad, F.Cu at (104.0, 104.0)
- added J5: MOT, TerminalBlock_4Ucon:TerminalBlock_4Ucon_1x02_P3.50mm_Horizontal, F.Cu at (151.3, 54.7)
- added R16: 1k, Resistor_SMD:R_0603_1608Metric, F.Cu at (153.4, 60.3)
- added R17: 10k, Resistor_SMD:R_0603_1608Metric, F.Cu at (152.5, 65.1)
- added U7: BV1HB045EFJ-CE2, Package_SO:HTSOP-8-1EP_3.9x4.9mm_P1.27mm_EP2.4x3.2mm_ThermalVias, F.Cu at (148.9, 61.4)
- moved C26 5.03 mm to (123.0, 64.2), turned to 180 degrees
Connections:
- net Net-(PCB1-CAN_H) renamed /CAN+
- net Net-(PCB1-CAN_L) renamed /CAN-
- PCB1 pad 15: unconnected-(PCB1-A7-Pad15) -> /MAGNET_I_SENSE
- PCB1 pad 17: unconnected-(PCB1-A9-Pad17) -> /MAGNET_CTL
Routing:
- net /MAGNET_CTL: track 0.00 -> 50.7 mm, vias 0 -> 2
- net /MAGNET_I_SENSE: track 0.00 -> 48.2 mm, vias 0 -> 2
- net VCC: track 201.9 -> 235.4 mm, vias 0 -> 1
- net GND: track 57.3 -> 73.9 mm, vias 54 -> 214
- net /MOT6_IN1: track 21.8 -> 36.2 mm
- net /MOT6_IN2: track 23.3 -> 34.9 mm
- net Net-(J5-Pin_2): track 0.00 -> 9.24 mm
- net Net-(U7-SENSE): track 0.00 -> 8.79 mm
- net +3V3: track 182.8 -> 189.6 mm
- net /~{SLEEP}: track 155.3 -> 160.7 mm, vias 6 -> 8
- net /BANK3_I_SENSE: track 109.7 -> 113.5 mm, vias 4 -> 3
- net /BANK2_ILIM: track 114.3 -> 117.0 mm
- net /MOT5_IN2: track 55.0 -> 56.2 mm

Commit message: added silkscreens to PCB and confirmed PCB ready for manufacturing
Parts:
- added REF**: Smolhaj_Scale_0.1, Symbol:Smolhaj_Scale_0.1, F.Cu at (176.0, 52.0)
- J5: value MOT -> MAG
Routing:
- net GND: vias 214 -> 154
Other:
- board text added: "- +"
- board text added: "Actuator Driver V0R1"
- board text added: "JCN MRB"
