File: hardware/dc-motor-driver/dc-motor-driver.kicad_sch (KiCad schematic)
At the start: 7 parts, among them J1 DE9, J2 VIN

Commit message: feat: Layout done
Parts:
- added C37: 100n, Capacitor_SMD:C_0603_1608Metric, symbol Capacitor:C_100n_50V_0603
- added D1: BAT54SWF, Package_TO_SOT_SMD:SOT-323_SC-70, symbol Semiconductor_Diodes:BAT54SWF
- added H1, H2, H3, H4, H5: MountingHole_Pad, MountingHole:MountingHole_3mm_Pad, symbol Mechanical:MountingHole_Pad
- added J5: MOT, TerminalBlock_4Ucon:TerminalBlock_4Ucon_1x02_P3.50mm_Horizontal, symbol Connector:Screw_Terminal_01x02
- added R16: 1k, Resistor_SMD:R_0603_1608Metric, symbol Resistor:R_1k_0603
- added R17: 10k, Resistor_SMD:R_0603_1608Metric, symbol Resistor:R_10k_0603
- added U7: BV1HB045EFJ-CE2, Package_SO:HTSOP-8-1EP_3.9x4.9mm_P1.27mm_EP2.4x3.2mm_ThermalVias, symbol PMIC, Load Switches & Drivers:BV1HB045EFJ-CE2
Connections:
- net +3V3: now also D1.2 (K)
- net GND: now also C37.2, D1.1 (A), H1.1, H2.1, H3.1, H4.1, H5.1, J5.1 (Pin_1), R16.2, U7.1 (GND)
- net VCC: now also C37.1, U7.3 (SEN), U7.9 (VBB)
- net MAGNET_I_SENSE: now reaches PCB1.15 (A7)
- net MAGNET_I_SENSE: now also D1.3 (COM), R17.2
- net MAGNET_CTL: now reaches PCB1.17 (A9)
- net MAGNET_CTL: now also U7.2 (IN)
- net CAN+: now reaches J1.7, J1.8, PCB1.7 (CAN_H)
- net CAN-: now reaches J1.1, J1.2, PCB1.8 (CAN_L)
- new net: J5.2 (Pin_2), U7.5 (OUT_1), U7.6 (OUT_2), U7.7 (OUT_3), U7.8 (OUT_4)
- new net: R16.1, R17.1, U7.4 (SENSE)
Other:
- company: (none) -> QUTRC
- title: (none) -> DC Motor Driver
- moved on the sheet: R13, R14, R15

Commit message: added silkscreens to PCB and confirmed PCB ready for manufacturing
Parts:
- J5: value MOT -> MAG
Connections:
- no-connect marks 5 -> 14
Changed lines of the file:
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@@
+	)
+	(no_connect
+		(at 129.54 96.52)
+	)
+	(no_connect
+		(at 175.26 93.98)
+	)
+	(no_connect
+		(at 129.54 91.44)
 	)
 	(no_connect
@@
 	)
 	(no_connect
+		(at 129.54 101.6)
+	)
+	(no_connect
 		(at 107.95 93.98)
 	)
@@
 	)
 	(no_connect
+		(at 175.26 91.44)
+	)
+	(no_connect
+		(at 175.26 88.9)
+	)
+	(no_connect
+		(at 129.54 93.98)
+	)
+	(no_connect
+		(at 129.54 99.06)
+	)
+	(no_connect
 		(at 107.95 101.6)
+	)
+	(no_connect
+		(at 175.26 96.52)
 	)
 	(no_connect
@@
 			)
 		)
-		(property "Value" "MOT"
+		(property "Value" "MAG"
 			(at 271.145 90.1701 0)
 			(effects
