File: hardware/dc-motor-driver/dc-motor-driver.kicad_sch (KiCad schematic)
At the start: 18 parts, among them J1 DE9, J2 VIN, J5 MAG, U7 BV1HB045EFJ-CE2

Commit message: Removed EOL mosfet
Parts:
- removed C37: 100n, Capacitor_SMD:C_0603_1608Metric, symbol Capacitor:C_100n_50V_0603
- removed D1: BAT54SWF, Package_TO_SOT_SMD:SOT-323_SC-70, symbol Semiconductor_Diodes:BAT54SWF
- removed R16: 1k, Resistor_SMD:R_0603_1608Metric, symbol Resistor:R_1k_0603
- removed R17: 10k, Resistor_SMD:R_0603_1608Metric, symbol Resistor:R_10k_0603
- removed U7: BV1HB045EFJ-CE2, Package_SO:HTSOP-8-1EP_3.9x4.9mm_P1.27mm_EP2.4x3.2mm_ThermalVias, symbol PMIC, Load Switches & Drivers:BV1HB045EFJ-CE2
- added C19: 100u, Capacitor_SMD:CP_Elec_6.3x7.7, symbol Capacitor:C_100u_35V
- added Q1: CSD16301Q2, Package_SON:Texas_DQK, symbol Transistor_FET:CSD16301Q2
Connections:
- net GND: now also C19.2
- net MAGNET_CTL: now also Q1.3 (G)
- net VCC: now also C19.1, Q1.1 (D), Q1.2 (D), Q1.5 (D), Q1.6 (D), Q1.8 (D)
- net at J5.2 (Pin_2): now also Q1.4 (S), Q1.7 (S)
- net MAGNET_I_SENSE: no longer names the net of PCB1.15 (A7)
Other:
- moved on the sheet: J5

Commit message: Added new mosfet and silkscreen, DRC and ERC passing
Parts:
- removed C19: 100u, Capacitor_SMD:CP_Elec_6.3x7.7, symbol Capacitor:C_100u_35V
Connections:
- net GND: now also J2.2 (Pin_2), J5.2 (Pin_2); no longer J2.1 (Pin_1), J5.1 (Pin_1)
- net VCC: now also J2.1 (Pin_1); no longer J2.2 (Pin_2)
- net at Q1.4 (S), Q1.7 (S): now also J5.1 (Pin_1); no longer J5.2 (Pin_2)
- no-connect marks 14 -> 16
Other:
- moved on the sheet: J5
