Commit message: perseus_lite: Complete fix for URDF links and frames

File: software/ros_ws/src/perseus_lite_description/urdf/perseus_lite.urdf.xacro (robot description, xacro)
@@ -10,5 +10,5 @@
     <xacro:chassis />
     <joint name="${prefix}chassis_joint" type="fixed">
-      <origin xyz="0.21 0.0 0.35" rpy="0.0 0.0 -${pi/2}"/>
+      <origin xyz="0.0 0.0 0.20" rpy="0.0 0.0 0.0"/>
       <parent link="${prefix}base_link"/>
       <child link="${prefix}chassis"/>
@@ -17,9 +17,9 @@
     <!-- LEFT -->
     <xacro:rocker side="left">
-      <origin xyz="-0.275 -0.075 0.05" rpy="0.0 0.0 ${-pi/2}"/>
+      <origin xyz="0.0 0.14 0.0" rpy="0.0 0.0 0.0"/>
     </xacro:rocker>
     <!-- RIGHT -->
     <xacro:rocker side="right">
-      <origin xyz="0.275 -0.075 0.05" rpy="0.0 0.0 ${-pi/2}"/>
+      <origin xyz="0.0 -0.14 0.0" rpy="0.0 0.0 0.0"/>
     </xacro:rocker>
     <xacro:sensors>

File: software/ros_ws/src/perseus_lite_description/urdf/rocker.urdf.xacro (robot description, xacro)
@@ -38,8 +38,8 @@
     <xacro:motor_wheel end="front">
       <xacro:if value="${side == 'left'}">
-        <origin xyz="-0.3 -0.225 -0.25" rpy="0.0 0.0 ${-pi/2}"/>
+        <origin xyz="0.15 0.22 -0.13" rpy="0.0 0.0 0.0"/>
       </xacro:if>
       <xacro:if value="${side == 'right'}">
-        <origin xyz="-0.3 0.225 -0.25" rpy="0.0 0.0 ${pi/2}"/>
+        <origin xyz="0.15 -0.22 -0.13" rpy="0.0 0.0 0.0"/>
       </xacro:if>
     </xacro:motor_wheel>
@@ -47,8 +47,8 @@
     <xacro:motor_wheel end="rear">
       <xacro:if value="${side == 'left'}">
-        <origin xyz="0.55 -0.225 -0.25" rpy="0.0 0.0 ${-pi/2}"/>
+        <origin xyz="-0.33 0.22 -0.13" rpy="0.0 0.0 0.0"/>
       </xacro:if>
       <xacro:if value="${side == 'right'}">
-        <origin xyz="0.55 0.225 -0.25" rpy="0.0 0.0 ${pi/2}"/>
+        <origin xyz="-0.33 -0.22 -0.13" rpy="0.0 0.0 0.0"/>
       </xacro:if>
     </xacro:motor_wheel>

File: software/ros_ws/src/perseus_lite_description/urdf/sensors.urdf.xacro (robot description, xacro)
@@ -25,7 +25,7 @@
     </link>
     <joint name="${prefix}c1_lidar_joint" type="fixed">
-        <parent link="${prefix}base_link"/>
+        <parent link="${prefix}chassis"/>
         <child link="${prefix}c1_lidar_frame"/>
-        <origin xyz="0.2 0.4 0.35" rpy="0 0 0"/>
+        <origin xyz="0.0 0.22 0.0" rpy="0 0 0"/>
     </joint>
     <gazebo reference="${prefix}c1_lidar_frame">
@@ -76,7 +76,7 @@
     </link>
     <joint name="${prefix}imu_joint" type="fixed">
-        <parent link="${prefix}base_link"/>
+        <parent link="${prefix}chassis"/>
         <child link="${prefix}imu_link"/>
-        <origin xyz="0.0 0.0 0.1" rpy="0 0 0"/>
+        <origin xyz="0.0 0.0 0.02" rpy="0 0 0"/>
     </joint>
     <gazebo reference="${prefix}imu_link">

File: software/ros_ws/src/perseus_lite_description/urdf/wheel.urdf.xacro (robot description, xacro)
@@ -24,5 +24,5 @@
     <joint name="${prefix}${end}_${side}_wheel_joint" type="continuous">
       <xacro:if value="${side == 'left'}">
-        <axis xyz="0 -1 0" rpy="0 0 0"/>
+        <axis xyz="0 1 0" rpy="0 0 0"/>
       </xacro:if>
       <xacro:if value="${side == 'right'}">
@@ -31,5 +31,5 @@
       <parent link="${prefix}${end}_${side}_motor"/>
       <child link="${prefix}${end}_${side}_wheel"/>
-      <origin xyz="-0.0625 0.0 0.0" rpy="0.0 0.0 ${-pi/2}"/>
+      <origin xyz="-0.0625 0.0 0.0" rpy="0.0 0.0 0.0"/>
       <dynamics damping="0.5" friction="0.5"/>
     </joint>

Commit message: perseus_lite: additional tweaks to URDF and nav yamls

File: software/ros_ws/src/perseus_lite_description/urdf/perseus_lite.urdf.xacro (robot description, xacro)
@@ -10,5 +10,5 @@
     <xacro:chassis />
     <joint name="${prefix}chassis_joint" type="fixed">
-      <origin xyz="0.0 0.0 0.20" rpy="0.0 0.0 0.0"/>
+      <origin xyz="0.21 0.0 0.35" rpy="0.0 0.0 0"/>
       <parent link="${prefix}base_link"/>
       <child link="${prefix}chassis"/>
@@ -17,9 +17,9 @@
     <!-- LEFT -->
     <xacro:rocker side="left">
-      <origin xyz="0.0 0.14 0.0" rpy="0.0 0.0 0.0"/>
+      <origin xyz="-0.275 -0.075 0.05" rpy="0.0 0.0 ${-pi/2}"/>
     </xacro:rocker>
     <!-- RIGHT -->
     <xacro:rocker side="right">
-      <origin xyz="0.0 -0.14 0.0" rpy="0.0 0.0 0.0"/>
+      <origin xyz="0.275 -0.075 0.05" rpy="0.0 0.0 ${-pi/2}"/>
     </xacro:rocker>
     <xacro:sensors>

File: software/ros_ws/src/perseus_lite_description/urdf/rocker.urdf.xacro (robot description, xacro)
@@ -38,8 +38,8 @@
     <xacro:motor_wheel end="front">
       <xacro:if value="${side == 'left'}">
-        <origin xyz="0.15 0.22 -0.13" rpy="0.0 0.0 0.0"/>
+        <origin xyz="-0.3 -0.225 -0.25" rpy="0.0 0.0 0.0"/>
       </xacro:if>
       <xacro:if value="${side == 'right'}">
-        <origin xyz="0.15 -0.22 -0.13" rpy="0.0 0.0 0.0"/>
+        <origin xyz="-0.3 0.225 -0.25" rpy="0.0 0.0 ${pi/2}"/>
       </xacro:if>
     </xacro:motor_wheel>
@@ -47,8 +47,8 @@
     <xacro:motor_wheel end="rear">
       <xacro:if value="${side == 'left'}">
-        <origin xyz="-0.33 0.22 -0.13" rpy="0.0 0.0 0.0"/>
+        <origin xyz="0.55 -0.225 -0.25" rpy="0.0 0.0 ${-pi/2}"/>
       </xacro:if>
       <xacro:if value="${side == 'right'}">
-        <origin xyz="-0.33 -0.22 -0.13" rpy="0.0 0.0 0.0"/>
+        <origin xyz="0.55 0.225 -0.25" rpy="0.0 0.0 ${pi/2}"/>
       </xacro:if>
     </xacro:motor_wheel>

Commit message: perseus_lite: wheels in URDF now correctly aligned

File: software/ros_ws/src/perseus_lite_description/urdf/perseus_lite.urdf.xacro (robot description, xacro)
@@ -10,5 +10,5 @@
     <xacro:chassis />
     <joint name="${prefix}chassis_joint" type="fixed">
-      <origin xyz="0.21 0.0 0.35" rpy="0.0 0.0 0"/>
+      <origin xyz="0.0 0.0 0.35" rpy="0.0 0.0 0"/>
       <parent link="${prefix}base_link"/>
       <child link="${prefix}chassis"/>

File: software/ros_ws/src/perseus_lite_description/urdf/wheel.urdf.xacro (robot description, xacro)
@@ -12,11 +12,11 @@
         <origin xyz="0.0 0.0 0.0" rpy="0.0 0.0 0.0"/>
         <geometry>
-          <mesh scale="0.05 0.05 0.05" filename="file://$(find perseus_lite_description)/meshes/wheel.dae"/>
+          <mesh scale="0.1 0.1 0.1" filename="file://$(find perseus_lite_description)/meshes/wheel.dae"/>
         </geometry>
       </visual>
       <collision>
-        <origin xyz="0.0 -0.00375 0.0" rpy="1.570796 0.0 0.0"/>
+        <origin xyz="0.0 -0.0075 0.0" rpy="1.570796 0.0 0.0"/>
         <geometry>
-          <cylinder length="0.02875" radius="0.03625" />
+          <cylinder length="0.0575" radius="0.0725" />
         </geometry>
       </collision>
@@ -24,12 +24,12 @@
     <joint name="${prefix}${end}_${side}_wheel_joint" type="continuous">
       <xacro:if value="${side == 'left'}">
-        <axis xyz="0 1 0" rpy="0 0 0"/>
+        <axis xyz="0 0 1"/>
       </xacro:if>
       <xacro:if value="${side == 'right'}">
-        <axis xyz="0 -1 0" rpy="0 0 0"/>
+        <axis xyz="0 0 -1"/>
       </xacro:if>
       <parent link="${prefix}${end}_${side}_motor"/>
       <child link="${prefix}${end}_${side}_wheel"/>
-      <origin xyz="-0.03125 0.0 0.0" rpy="0.0 0.0 0.0"/>
+      <origin xyz="-0.0625 0.0 0.0" rpy="0.0 ${pi/2} 0.0"/>
       <dynamics damping="0.5" friction="0.5"/>
     </joint>

Commit message: perseus_lite: updated URDF before roatation fix

File: software/ros_ws/src/perseus_lite_description/urdf/perseus_lite.urdf.xacro (robot description, xacro)
@@ -10,5 +10,5 @@
     <xacro:chassis />
     <joint name="${prefix}chassis_joint" type="fixed">
-      <origin xyz="0.0 0.0 0.35" rpy="0.0 0.0 0"/>
+      <origin xyz="0.0 0.0 0.15" rpy="0.0 0.0 ${-pi/2}"/>
       <parent link="${prefix}base_link"/>
       <child link="${prefix}chassis"/>
