Commit message: perseus_lite: corrected the scaled inertia of the chassis

File: software/ros_ws/src/perseus_lite_description/urdf/chassis.urdf.xacro (robot description, xacro)
@@ -5,10 +5,11 @@
     <!-- CHASSIS -->
     <link name="${prefix}chassis">
-      <inertial>
+       <inertial>
         <!-- Scaled inertial properties for Perseus Lite -->
         <origin xyz="0.0 -0.08550236602 0.07366242988" rpy="0 0 0"/>
         <mass value="1.38449701513"/> <!-- Scaled by 0.5 -->
-        <inertia ixx="0.021308" iyy="0.011578" izz="0.028045"
-                 ixy="0.0" iyz="0.000676" ixz="-0.0"/>
+        <!-- Updated inertia values using square scaling factor (0.5^2 = 0.25) -->
+        <inertia ixx="0.005327" iyy="0.002894" izz="0.007011"
+                 ixy="0.0" iyz="0.000169" ixz="-0.0"/>
       </inertial>
       <visual>

Commit message: TF realignment part way complete

File: software/ros_ws/src/perseus_lite_description/urdf/chassis.urdf.xacro (robot description, xacro)
@@ -14,5 +14,5 @@
       </inertial>
       <visual>
-        <origin xyz="0.0 0.0 0.0" rpy="0 0.0 0.0"/>
+        <origin xyz="0.0 0.0 0.0" rpy="0 0.0 ${-pi/2}"/>
         <geometry>
           <mesh scale="0.05 0.05 0.05" filename="file://$(find perseus_lite_description)/meshes/chassis.dae"/>
@@ -20,5 +20,5 @@
       </visual>
       <collision>
-        <origin xyz="0.0 -0.15 0.05" rpy="0 0.0 0.0"/>
+        <origin xyz="0.0 -0.15 0.05" rpy="0 0.0 ${-pi/2}"/>
         <geometry>
           <box size="0.2375 0.2625 0.1" />

File: software/ros_ws/src/perseus_lite_description/urdf/motor_wheel.urdf.xacro (robot description, xacro)
@@ -11,5 +11,5 @@
       </inertial>
       <visual>
-        <origin xyz="-0.1325 0.0 0.0" rpy="0.0 0.0 ${pi}"/>
+        <origin xyz="-0.1325 0.0 0.0" rpy="0.0 0.0 ${pi/2}"/>
         <geometry>
           <mesh scale="0.05 0.05 0.05" filename="file://$(find perseus_lite_description)/meshes/gearbox.dae"/>
@@ -18,5 +18,5 @@
       </visual>
       <collision>
-        <origin xyz="-0.15 0.0 0.0" rpy="0.0 0.0 0.0"/>
+        <origin xyz="-0.15 0.0 0.0" rpy="0.0 0.0 ${-pi/2}"/>
         <geometry>
           <box size="0.05 0.05 0.0375" />

File: software/ros_ws/src/perseus_lite_description/urdf/perseus_lite.urdf.xacro (robot description, xacro)
@@ -10,5 +10,5 @@
     <xacro:chassis />
     <joint name="${prefix}chassis_joint" type="fixed">
-      <origin xyz="0.0 0.0 0.15" rpy="0.0 0.0 ${-pi/2}"/>
+      <origin xyz="0.0 0.0 0.15" rpy="0.0 0.0 0.0"/>
       <parent link="${prefix}base_link"/>
       <child link="${prefix}chassis"/>
@@ -17,9 +17,9 @@
     <!-- LEFT -->
     <xacro:rocker side="left">
-      <origin xyz="-0.1375 -0.0375 0.025" rpy="0.0 0.0 ${-pi/2}"/>
+      <origin xyz="-0.0375 0.1375 0.025" rpy="0.0 0.0 0.0"/>
     </xacro:rocker>
     <!-- RIGHT -->
     <xacro:rocker side="right">
-      <origin xyz="0.1375 -0.0375 0.025" rpy="0.0 0.0 ${-pi/2}"/>
+      <origin xyz="-0.0375 -0.1375 0.025" rpy="0.0 0.0 0.0"/>
     </xacro:rocker>
     <xacro:sensors>

File: software/ros_ws/src/perseus_lite_description/urdf/rocker.urdf.xacro (robot description, xacro)
@@ -18,5 +18,5 @@
       </inertial>
       <visual>
-        <origin xyz="0.0 0.0 0.0" rpy="0.0 0.0 0.0"/>
+        <origin xyz="0.0 0.0 0.0" rpy="0.0 0.0 ${pi}"/>
         <geometry>
           <mesh scale="0.05 0.05 0.05" filename="file://$(find perseus_lite_description)/meshes/rocker_${side}.dae"/>
@@ -24,5 +24,5 @@
       </visual>
       <collision>
-        <origin xyz="0.1 0.0 -0.025" rpy="0.0 0.3 0.0"/>
+        <origin xyz="0.1 0.0 -0.025" rpy="0.0 0.3 ${pi}"/>
         <geometry>
           <box size="0.2 0.025 0.015" />

File: software/ros_ws/src/perseus_lite_description/urdf/wheel.urdf.xacro (robot description, xacro)
@@ -10,5 +10,5 @@
       </inertial>
       <visual>
-        <origin xyz="0.0 0.0 0.0" rpy="0.0 0.0 0.0"/>
+        <origin xyz="0.0 0.0 0.0" rpy="0.0 0.0 ${-pi/2}"/>
         <geometry>
           <mesh scale="0.1 0.1 0.1" filename="file://$(find perseus_lite_description)/meshes/wheel.dae"/>
@@ -16,5 +16,5 @@
       </visual>
       <collision>
-        <origin xyz="0.0 -0.0075 0.0" rpy="1.570796 0.0 0.0"/>
+        <origin xyz="0.0 -0.0075 0.0" rpy="1.570796 0.0 ${-pi/2}"/>
         <geometry>
           <cylinder length="0.0575" radius="0.0725" />

Commit message: perseus_lite: improved URDF, x axis aligned

File: software/ros_ws/src/perseus_lite_description/urdf/chassis.urdf.xacro (robot description, xacro)
@@ -48,5 +48,5 @@
     </link>
     <joint name="${prefix}flange_bearing_joint" type="fixed">
-      <origin xyz="0.0 -0.3 0.05" rpy="0 ${-pi/2} ${pi/2}"/>
+      <origin xyz="-0.3 -0.0 0.05" rpy="0 ${-pi/2} 0.0"/>
       <parent link="${prefix}chassis"/>
       <child link="${prefix}flange_bearing"/>

File: software/ros_ws/src/perseus_lite_description/urdf/motor_wheel.urdf.xacro (robot description, xacro)
@@ -2,14 +2,14 @@
 <robot name="motor_wheel" xmlns:xacro="http://www.ros.org/wiki/xacro">
   <xacro:include filename="$(find perseus_lite_description)/urdf/wheel.urdf.xacro"/>
+  <!-- MOTOR JOINT -->
   <xacro:macro name="motor_wheel" params="prefix:=^ side:=^ end *origin">
     <link name="${prefix}${end}_${side}_motor">
       <inertial>
-        <!-- moving origin has no perceivable impact-->
-        <origin xyz="0.0 0.0 0.0" rpy="0.0 0.0 0.0"/>
+        <origin xyz="0.0 0.1 0.0" rpy="0.0 0.0 0.0"/>
         <mass value="2.6182895"/>
         <inertia ixx="0.00125" iyy="0.00125" izz="0.00125" ixy="0.0" iyz="0.0" ixz="0.0"/> <!-- TEMP -->
       </inertial>
       <visual>
-        <origin xyz="-0.1325 0.0 0.0" rpy="0.0 0.0 ${pi/2}"/>
+        <origin xyz="-0.0 0.0 0.0" rpy="0.0 0.0 ${pi/2}"/>
         <geometry>
           <mesh scale="0.05 0.05 0.05" filename="file://$(find perseus_lite_description)/meshes/gearbox.dae"/>
@@ -18,5 +18,5 @@
       </visual>
       <collision>
-        <origin xyz="-0.15 0.0 0.0" rpy="0.0 0.0 ${-pi/2}"/>
+        <origin xyz="-0.0 0.0 0.0" rpy="0.0 0.0 ${pi/2}"/>
         <geometry>
           <box size="0.05 0.05 0.0375" />

File: software/ros_ws/src/perseus_lite_description/urdf/rocker.urdf.xacro (robot description, xacro)
@@ -38,8 +38,8 @@
     <xacro:motor_wheel end="front">
       <xacro:if value="${side == 'left'}">
-        <origin xyz="-0.17 -0.1 -0.1" rpy="0.0 0.0 ${-pi/2}"/>
+        <origin xyz="0.17 -0.04 -0.1" rpy="0.0 0.0 ${pi}"/>
       </xacro:if>
       <xacro:if value="${side == 'right'}">
-        <origin xyz="-0.17 0.1 -0.1" rpy="0.0 0.0 ${pi/2}"/>
+        <origin xyz="0.17 0.04 -0.1" rpy="0.0 0.0 0.0"/>
       </xacro:if>
     </xacro:motor_wheel>
@@ -47,8 +47,8 @@
     <xacro:motor_wheel end="rear">
       <xacro:if value="${side == 'left'}">
-        <origin xyz="0.31 -0.1 -0.1" rpy="0.0 0.0 ${-pi/2}"/>
+        <origin xyz="-0.30 -0.04 -0.1" rpy="0.0 0.0 ${pi}"/>
       </xacro:if>
       <xacro:if value="${side == 'right'}">
-        <origin xyz="0.31 0.1 -0.1" rpy="0.0 0.0 ${pi/2}"/>
+        <origin xyz="-0.30 0.04 -0.1" rpy="0.0 0.0 0.0"/>
       </xacro:if>
     </xacro:motor_wheel>

File: software/ros_ws/src/perseus_lite_description/urdf/wheel.urdf.xacro (robot description, xacro)
@@ -22,4 +22,5 @@
       </collision>
     </link>
+    <!-- WHEEL -->
     <joint name="${prefix}${end}_${side}_wheel_joint" type="continuous">
       <xacro:if value="${side == 'left'}">
@@ -31,5 +32,5 @@
       <parent link="${prefix}${end}_${side}_motor"/>
       <child link="${prefix}${end}_${side}_wheel"/>
-      <origin xyz="-0.0625 0.0 0.0" rpy="0.0 ${pi/2} 0.0"/>
+      <origin xyz="0.0 -0.09 0.0" rpy="0.0 ${pi/2} ${-pi/2}"/>
       <dynamics damping="0.5" friction="0.5"/>
     </joint>

Commit message: perseus-lite(description): Changes to macros
- removed some large mesh files by using macros
- updated the dependency from p-l to perseus-description in the process

File: software/ros_ws/src/perseus_lite_description/urdf/chassis.urdf.xacro (robot description, xacro)
@@ -16,5 +16,5 @@
         <origin xyz="0.0 0.0 0.0" rpy="0 0.0 ${-pi/2}"/>
         <geometry>
-          <mesh scale="0.05 0.05 0.05" filename="file://$(find perseus_lite_description)/meshes/chassis.dae"/>
+          <mesh scale="0.05 0.05 0.05" filename="file://$(find perseus_description)/meshes/chassis.dae"/>
         </geometry>
       </visual>
@@ -37,5 +37,5 @@
         <origin xyz="0.0 0.0 0.0" rpy="0 0 0"/>
         <geometry>
-          <mesh scale="0.05 0.05 0.05" filename="file://$(find perseus_lite_description)/meshes/flange_bearing.dae"/>
+          <mesh scale="0.05 0.05 0.05" filename="file://$(find perseus_description)/meshes/flange_bearing.dae"/>
         </geometry>
       </visual>
@@ -43,5 +43,5 @@
         <origin xyz="0.0 0.0 0.0" rpy="0 0 0"/>
         <geometry>
-          <mesh scale="0.05 0.05 0.05" filename="file://$(find perseus_lite_description)/meshes/flange_bearing.dae"/>
+          <mesh scale="0.05 0.05 0.05" filename="file://$(find perseus_description)/meshes/flange_bearing.dae"/>
         </geometry>
       </collision>
@@ -63,5 +63,5 @@
         <origin xyz="0.0 0.0 0.0" rpy="0.0 0.0 0.0"/>
         <geometry>
-          <mesh scale="0.05 0.05 0.05" filename="file://$(find perseus_lite_description)/meshes/differential_bar.dae"/>
+          <mesh scale="0.05 0.05 0.05" filename="file://$(find perseus_description)/meshes/differential_bar.dae"/>
         </geometry>
       </visual>

File: software/ros_ws/src/perseus_lite_description/urdf/motor_wheel.urdf.xacro (robot description, xacro)
@@ -13,5 +13,5 @@
         <origin xyz="-0.0 0.0 0.0" rpy="0.0 0.0 ${pi/2}"/>
         <geometry>
-          <mesh scale="0.05 0.05 0.05" filename="file://$(find perseus_lite_description)/meshes/gearbox.dae"/>
+          <mesh scale="0.05 0.05 0.05" filename="file://$(find perseus_description)/meshes/gearbox.dae"/>
         </geometry>
         <!-- <material name="white"/> -->

File: software/ros_ws/src/perseus_lite_description/urdf/rocker.urdf.xacro (robot description, xacro)
@@ -20,5 +20,5 @@
         <origin xyz="0.0 0.0 0.0" rpy="0.0 0.0 ${pi}"/>
         <geometry>
-          <mesh scale="0.05 0.05 0.05" filename="file://$(find perseus_lite_description)/meshes/rocker_${side}.dae"/>
+          <mesh scale="0.05 0.05 0.05" filename="file://$(find perseus_description)/meshes/rocker_${side}.dae"/>
         </geometry>
       </visual>
