Commit message: perseus_lite: updated speed values

File: software/ros_ws/src/perseus_lite_description/urdf/wheel.urdf.xacro (robot description, xacro)
@@ -25,5 +25,5 @@
     <joint name="${prefix}${end}_${side}_wheel_joint" type="continuous">
       <xacro:if value="${side == 'left'}">
-        <axis xyz="0 0 1"/>
+        <axis xyz="0 0 -1"/>
       </xacro:if>
       <xacro:if value="${side == 'right'}">

Commit message: p-l: Correction for wheel direction in URDF to fix turning

File: software/ros_ws/src/perseus_lite_description/urdf/wheel.urdf.xacro (robot description, xacro)
@@ -28,5 +28,5 @@
       </xacro:if>
       <xacro:if value="${side == 'right'}">
-        <axis xyz="0 0 -1"/>
+        <axis xyz="0 0 1"/>
       </xacro:if>
       <parent link="${prefix}${end}_${side}_motor"/>

Commit message: updating URDF to fix lack of turning

File: software/ros_ws/src/perseus_lite_description/urdf/wheel.urdf.xacro (robot description, xacro)
@@ -28,5 +28,5 @@
       </xacro:if>
       <xacro:if value="${side == 'right'}">
-        <axis xyz="0 0 1"/>
+        <axis xyz="0 0 -1"/>
       </xacro:if>
       <parent link="${prefix}${end}_${side}_motor"/>
