Commit message: perseus_lite: improved URDF motor position

File: software/ros_ws/src/perseus_lite_description/urdf/motor_wheel.urdf.xacro (robot description, xacro)
@@ -7,19 +7,19 @@
         <!-- moving origin has no perceivable impact-->
         <origin xyz="0.0 0.0 0.0" rpy="0.0 0.0 0.0"/>
-        <mass value="5.236579"/>
-        <inertia ixx="0.01" iyy="0.01" izz="0.01" ixy="0.0" iyz="0.0" ixz="0.0"/> <!-- TEMP -->
+        <mass value="2.6182895"/>
+        <inertia ixx="0.00125" iyy="0.00125" izz="0.00125" ixy="0.0" iyz="0.0" ixz="0.0"/> <!-- TEMP -->
       </inertial>
       <visual>
-        <origin xyz="-0.265 0.0 0.0" rpy="0.0 0.0 ${pi}"/>
+        <origin xyz="-0.1325 0.0 0.0" rpy="0.0 0.0 ${pi}"/>
         <geometry>
-          <mesh scale="0.1 0.1 0.1" filename="file://$(find perseus_lite_description)/meshes/gearbox.dae"/>
+          <mesh scale="0.05 0.05 0.05" filename="file://$(find perseus_lite_description)/meshes/gearbox.dae"/>
         </geometry>
         <!-- <material name="white"/> -->
       </visual>
       <collision>
-        <origin xyz="-0.3 0.0 0.0" rpy="0.0 0.0 0.0"/>
+        <origin xyz="-0.15 0.0 0.0" rpy="0.0 0.0 0.0"/>
         <geometry>
-          <box size="0.1 0.1 0.075" />
-          <!--mesh scale="0.1 0.1 0.1" filename="file://$(find perseus_lite_description)/meshes/gearbox.dae"/-->
+          <box size="0.05 0.05 0.0375" />
+          <!--mesh scale="0.05 0.05 0.05" filename="file://$(find perseus_lite_description)/meshes/gearbox.dae"/-->
         </geometry>
       </collision>

File: software/ros_ws/src/perseus_lite_description/urdf/perseus_lite.urdf.xacro (robot description, xacro)
@@ -17,9 +17,9 @@
     <!-- LEFT -->
     <xacro:rocker side="left">
-      <origin xyz="-0.275 -0.075 0.05" rpy="0.0 0.0 ${-pi/2}"/>
+      <origin xyz="-0.1375 -0.0375 0.025" rpy="0.0 0.0 ${-pi/2}"/>
     </xacro:rocker>
     <!-- RIGHT -->
     <xacro:rocker side="right">
-      <origin xyz="0.275 -0.075 0.05" rpy="0.0 0.0 ${-pi/2}"/>
+      <origin xyz="0.1375 -0.0375 0.025" rpy="0.0 0.0 ${-pi/2}"/>
     </xacro:rocker>
     <xacro:sensors>

File: software/ros_ws/src/perseus_lite_description/urdf/rocker.urdf.xacro (robot description, xacro)
@@ -6,25 +6,25 @@
     <link name="${prefix}${side}_rocker">
       <inertial>
-        <origin xyz="0.011819187400851083 -0.08337339654014758 -0.06739096070989994" rpy="0.0 0.0 0.0"/>
+        <origin xyz="0.005909593700425542 -0.04168669827007379 -0.03369548035494997" rpy="0.0 0.0 0.0"/>
         <!-- RIGHT -->
         <xacro:if value="${side == 'right'}">
-          <inertia ixx="0.078224" iyy="0.009964" izz="0.076528" ixy="0.003701" iyz="-0.006846" ixz="0.00298"/>
+          <inertia ixx="0.009778" iyy="0.0012455" izz="0.009566" ixy="0.000462625" iyz="-0.00085575" ixz="0.0003725"/>
         </xacro:if>
         <!-- LEFT -->
         <xacro:if value="${side == 'left'}">
-          <inertia ixx="0.078224" iyy="0.009964" izz="0.076528" ixy="0.003701" iyz="-0.006846" ixz="0.00298"/>
+          <inertia ixx="0.009778" iyy="0.0012455" izz="0.009566" ixy="0.000462625" iyz="-0.00085575" ixz="0.0003725"/>
         </xacro:if>
-        <mass value="1.2546142039512485"/>
+        <mass value="0.6273071019756242"/>
       </inertial>
       <visual>
         <origin xyz="0.0 0.0 0.0" rpy="0.0 0.0 0.0"/>
         <geometry>
-          <mesh scale="0.1 0.1 0.1" filename="file://$(find perseus_lite_description)/meshes/rocker_${side}.dae"/>
+          <mesh scale="0.05 0.05 0.05" filename="file://$(find perseus_lite_description)/meshes/rocker_${side}.dae"/>
         </geometry>
       </visual>
       <collision>
-        <origin xyz="0.2 0.0 -0.05" rpy="0.0 0.3 0.0"/>
+        <origin xyz="0.1 0.0 -0.025" rpy="0.0 0.3 0.0"/>
         <geometry>
-          <box size="0.4 0.05 0.03" />
+          <box size="0.2 0.025 0.015" />
         </geometry>
       </collision>
@@ -38,8 +38,8 @@
     <xacro:motor_wheel end="front">
       <xacro:if value="${side == 'left'}">
-        <origin xyz="-0.3 -0.225 -0.25" rpy="0.0 0.0 0.0"/>
+        <origin xyz="-0.17 -0.1 -0.1" rpy="0.0 0.0 ${-pi/2}"/>
       </xacro:if>
       <xacro:if value="${side == 'right'}">
-        <origin xyz="-0.3 0.225 -0.25" rpy="0.0 0.0 ${pi/2}"/>
+        <origin xyz="-0.17 0.1 -0.1" rpy="0.0 0.0 ${pi/2}"/>
       </xacro:if>
     </xacro:motor_wheel>
@@ -47,8 +47,8 @@
     <xacro:motor_wheel end="rear">
       <xacro:if value="${side == 'left'}">
-        <origin xyz="0.55 -0.225 -0.25" rpy="0.0 0.0 ${-pi/2}"/>
+        <origin xyz="0.31 -0.1 -0.1" rpy="0.0 0.0 ${-pi/2}"/>
       </xacro:if>
       <xacro:if value="${side == 'right'}">
-        <origin xyz="0.55 0.225 -0.25" rpy="0.0 0.0 ${pi/2}"/>
+        <origin xyz="0.31 0.1 -0.1" rpy="0.0 0.0 ${pi/2}"/>
       </xacro:if>
     </xacro:motor_wheel>

File: software/ros_ws/src/perseus_lite_description/urdf/wheel.urdf.xacro (robot description, xacro)
@@ -16,7 +16,7 @@
       </visual>
       <collision>
-        <origin xyz="0.0 -0.0075 0.0" rpy="1.570796 0.0 0.0"/>
+        <origin xyz="0.0 -0.00375 0.0" rpy="1.570796 0.0 0.0"/>
         <geometry>
-          <cylinder length="0.0575" radius="0.0725" />
+          <cylinder length="0.02875" radius="0.03625" />
         </geometry>
       </collision>
@@ -31,5 +31,5 @@
       <parent link="${prefix}${end}_${side}_motor"/>
       <child link="${prefix}${end}_${side}_wheel"/>
-      <origin xyz="-0.0625 0.0 0.0" rpy="0.0 0.0 0.0"/>
+      <origin xyz="-0.03125 0.0 0.0" rpy="0.0 0.0 0.0"/>
       <dynamics damping="0.5" friction="0.5"/>
     </joint>

Commit message: fix(perseus-lite): Align URDF wheel joints with Perseus conventions
- Change wheel rotation axis from Z to Y axis to match Perseus model
- Differentiate left/right wheel joint axes (left: -Y, right: +Y) to
  fix rviz2 visualization matching physical servo rotation direction
- Mirror motor visual/collision orientations for left vs right sides
- Remove compensating pi rotations from motor joint origins
- Wrap robot_description in ParameterValue to fix YAML parsing errors

File: software/ros_ws/src/perseus_lite_description/urdf/motor_wheel.urdf.xacro (robot description, xacro)
@@ -6,20 +6,28 @@
     <link name="${prefix}${end}_${side}_motor">
       <inertial>
-        <origin xyz="0.0 0.1 0.0" rpy="0.0 0.0 0.0"/>
+        <origin xyz="0.0 0.0 0.0" rpy="0.0 0.0 0.0"/>
         <mass value="2.6182895"/>
-        <inertia ixx="0.00125" iyy="0.00125" izz="0.00125" ixy="0.0" iyz="0.0" ixz="0.0"/> <!-- TEMP -->
+        <inertia ixx="0.00125" iyy="0.00125" izz="0.00125" ixy="0.0" iyz="0.0" ixz="0.0"/>
       </inertial>
       <visual>
-        <origin xyz="-0.0 0.0 0.0" rpy="0.0 0.0 ${pi/2}"/>
+        <xacro:if value="${side == 'left'}">
+          <origin xyz="0.0 0.0 0.0" rpy="0.0 0.0 ${-pi/2}"/>
+        </xacro:if>
+        <xacro:if value="${side == 'right'}">
+          <origin xyz="0.0 0.0 0.0" rpy="0.0 0.0 ${pi/2}"/>
+        </xacro:if>
         <geometry>
           <mesh scale="0.05 0.05 0.05" filename="file://$(find perseus_description)/meshes/gearbox.dae"/>
         </geometry>
-        <!-- <material name="white"/> -->
       </visual>
       <collision>
-        <origin xyz="-0.0 0.0 0.0" rpy="0.0 0.0 ${pi/2}"/>
+        <xacro:if value="${side == 'left'}">
+          <origin xyz="0.0 0.0 0.0" rpy="0.0 0.0 ${pi/2}"/>
+        </xacro:if>
+        <xacro:if value="${side == 'right'}">
+          <origin xyz="0.0 0.0 0.0" rpy="0.0 0.0 ${-pi/2}"/>
+        </xacro:if>
         <geometry>
           <box size="0.05 0.05 0.0375" />
-          <!--mesh scale="0.05 0.05 0.05" filename="file://$(find perseus_lite_description)/meshes/gearbox.dae"/-->
         </geometry>
       </collision>

File: software/ros_ws/src/perseus_lite_description/urdf/rocker.urdf.xacro (robot description, xacro)
@@ -38,5 +38,5 @@
     <xacro:motor_wheel end="front">
       <xacro:if value="${side == 'left'}">
-        <origin xyz="0.17 -0.04 -0.1" rpy="0.0 0.0 ${pi}"/>
+        <origin xyz="0.17 -0.04 -0.1" rpy="0.0 0.0 0.0"/>
       </xacro:if>
       <xacro:if value="${side == 'right'}">
@@ -47,5 +47,5 @@
     <xacro:motor_wheel end="rear">
       <xacro:if value="${side == 'left'}">
-        <origin xyz="-0.30 -0.04 -0.1" rpy="0.0 0.0 ${pi}"/>
+        <origin xyz="-0.30 -0.04 -0.1" rpy="0.0 0.0 0.0"/>
       </xacro:if>
       <xacro:if value="${side == 'right'}">

File: software/ros_ws/src/perseus_lite_description/urdf/wheel.urdf.xacro (robot description, xacro)
@@ -1,14 +1,24 @@
 <?xml version="1.0"?>
 <robot name="wheel" xmlns:xacro="http://ros.org/wiki/xacro">
+  <xacro:property name="wheel_radius" value="0.0725"/>
+  <xacro:property name="wheel_length" value="0.0575"/>
+  <xacro:property name="wheel_mass" value="0.005"/>
+  <xacro:property name="wheels_y_offset" value="0.09"/>
   <xacro:macro name="wheel" params="prefix:=^ side:=^ end:=^">
     <link name="${prefix}${end}_${side}_wheel">
       <inertial>
         <origin xyz="0.0 0.0 0.0" rpy="0.0 0.0 0.0"/>
-        <mass value="0.005"/>  <!-- Scaled mass -->
+        <mass value="${wheel_mass}"/>
         <inertia ixx="0.006434" iyy="0.003644" izz="0.003644"
                  ixy="0.0" iyz="0.0" ixz="0.0"/>
       </inertial>
       <visual>
-        <origin xyz="0.0 0.0 0.0" rpy="0.0 0.0 ${-pi/2}"/>
+        <!-- Rotate mesh so tread pattern faces outward -->
+        <xacro:if value="${side == 'left'}">
+          <origin xyz="0.0 0.0 0.0" rpy="0.0 0.0 ${pi}"/>
+        </xacro:if>
+        <xacro:if value="${side == 'right'}">
+          <origin xyz="0.0 0.0 0.0" rpy="0.0 0.0 0.0"/>
+        </xacro:if>
         <geometry>
           <mesh scale="0.1 0.1 0.1" filename="file://$(find perseus_lite_description)/meshes/wheel.dae"/>
@@ -16,22 +26,24 @@
       </visual>
       <collision>
-        <origin xyz="0.0 -0.0075 0.0" rpy="1.570796 0.0 ${-pi/2}"/>
+        <!-- Rotate cylinder 90° around X to align with Y axis (wheel axle) -->
+        <origin xyz="0.0 0.0 0.0" rpy="${pi/2} 0.0 0.0"/>
         <geometry>
-          <cylinder length="0.0575" radius="0.0725" />
+          <cylinder radius="${wheel_radius}" length="${wheel_length}"/>
         </geometry>
       </collision>
     </link>
-    <!-- WHEEL -->
+    <!-- WHEEL JOINT -->
     <joint name="${prefix}${end}_${side}_wheel_joint" type="continuous">
+      <parent link="${prefix}${end}_${side}_motor"/>
+      <child link="${prefix}${end}_${side}_wheel"/>
       <xacro:if value="${side == 'left'}">
-        <axis xyz="0 0 -1"/>
+        <origin xyz="0.0 ${wheels_y_offset} 0.0" rpy="0.0 0.0 0.0"/>
+        <axis xyz="0 -1 0"/>
       </xacro:if>
       <xacro:if value="${side == 'right'}">
-        <axis xyz="0 0 -1"/>
+        <origin xyz="0.0 ${-wheels_y_offset} 0.0" rpy="0.0 0.0 0.0"/>
+        <axis xyz="0 1 0"/>
       </xacro:if>
-      <parent link="${prefix}${end}_${side}_motor"/>
-      <child link="${prefix}${end}_${side}_wheel"/>
-      <origin xyz="0.0 -0.09 0.0" rpy="0.0 ${pi/2} ${-pi/2}"/>
-      <dynamics damping="0.5" friction="0.5"/>
+      <dynamics damping="0.2" friction="0.3"/>
     </joint>
   <transmission name="${prefix}${end}_${side}_wheel_trans">
