Commit message: perseus_lite: updated URDF and nav2 launch

File: software/ros_ws/src/perseus_lite_description/urdf/sensors.urdf.xacro (robot description, xacro)
@@ -52,4 +52,84 @@
         </sensor>
     </gazebo>
+    <!-- IMU Sensor -->
+    <link name="${prefix}imu_link">
+        <inertial>
+            <mass value="0.001"/>
+            <origin xyz="0 0 0" rpy="0 0 0"/>
+            <inertia ixx="0.0001" ixy="0" ixz="0"
+                     iyy="0.0001" iyz="0"
+                     izz="0.0001"/>
+        </inertial>
+        <visual>
+            <origin xyz="0 0 0" rpy="0 0 0"/>
+            <geometry>
+                <box size="0.02 0.02 0.01"/>
+            </geometry>
+            <material name="blue"/>
+        </visual>
+        <collision>
+            <origin xyz="0 0 0" rpy="0 0 0"/>
+            <geometry>
+                <box size="0.02 0.02 0.01"/>
+            </geometry>
+        </collision>
+    </link>
+    <joint name="${prefix}imu_joint" type="fixed">
+        <parent link="${prefix}base_link"/>
+        <child link="${prefix}imu_link"/>
+        <origin xyz="0.0 0.0 0.1" rpy="0 0 0"/>
+    </joint>
+    <gazebo reference="${prefix}imu_link">
+        <material>Gazebo/Blue</material>
+        <sensor name="imu" type="imu">
+            <pose>0 0 0 0 0 0</pose>
+            <always_on>true</always_on>
+            <update_rate>100</update_rate>
+            <topic>imu/data</topic>
+            <frame>${prefix}imu_link</frame>
+            <imu>
+                <angular_velocity>
+                    <x>
+                        <noise type="gaussian">
+                            <mean>0.0</mean>
+                            <stddev>2e-4</stddev>
+                        </noise>
+                    </x>
+                    <y>
+                        <noise type="gaussian">
+                            <mean>0.0</mean>
+                            <stddev>2e-4</stddev>
+                        </noise>
+                    </y>
+                    <z>
+                        <noise type="gaussian">
+                            <mean>0.0</mean>
+                            <stddev>2e-4</stddev>
+                        </noise>
+                    </z>
+                </angular_velocity>
+                <linear_acceleration>
+                    <x>
+                        <noise type="gaussian">
+                            <mean>0.0</mean>
+                            <stddev>1.7e-2</stddev>
+                        </noise>
+                    </x>
+                    <y>
+                        <noise type="gaussian">
+                            <mean>0.0</mean>
+                            <stddev>1.7e-2</stddev>
+                        </noise>
+                    </y>
+                    <z>
+                        <noise type="gaussian">
+                            <mean>0.0</mean>
+                            <stddev>1.7e-2</stddev>
+                        </noise>
+                    </z>
+                </linear_acceleration>
+            </imu>
+        </sensor>
+    </gazebo>
   </xacro:macro>
 </robot>

Commit message: fix(perseus-lite): Fix lidar mount transform and servo velocity scaling
Correct the lidar URDF to reflect the actual mounting (centered, flipped
upside-down) and rework the STS3215 velocity conversion to use the full
15-bit protocol range with proper RPM scaling. Also disable servo
acceleration ramping for more responsive control.

File: software/ros_ws/src/perseus_lite_description/urdf/sensors.urdf.xacro (robot description, xacro)
@@ -27,5 +27,6 @@
         <parent link="${prefix}chassis"/>
         <child link="${prefix}c1_lidar_frame"/>
-        <origin xyz="0.0 0.22 0.0" rpy="0 0 0"/>
+        <!-- Lidar mounted at center of chassis, underneath, flipped upside down -->
+        <origin xyz="0.0 0.0 -0.04" rpy="${pi} 0 0"/>
     </joint>
     <gazebo reference="${prefix}c1_lidar_frame">

Commit message: feat(perseus-lite): Add Logitech C920 camera support
Add v4l2_camera node to publish camera images on the ROS network from
the front-mounted C920 USB webcam. Includes URDF camera_link and
camera_optical_frame, and adds v4l2-camera to Nix and package deps.

File: software/ros_ws/src/perseus_lite_description/urdf/sensors.urdf.xacro (robot description, xacro)
@@ -133,4 +133,40 @@
         </sensor>
     </gazebo>
+    <!-- Camera (Logitech C920) -->
+    <link name="${prefix}camera_link">
+        <inertial>
+            <mass value="0.162"/>
+            <origin xyz="0 0 0" rpy="0 0 0"/>
+            <inertia ixx="0.0001" ixy="0" ixz="0"
+                     iyy="0.0001" iyz="0"
+                     izz="0.0001"/>
+        </inertial>
+        <visual>
+            <origin xyz="0 0 0" rpy="0 0 0"/>
+            <geometry>
+                <box size="0.03 0.094 0.024"/>
+            </geometry>
+            <material name="grey"/>
+        </visual>
+        <collision>
+            <origin xyz="0 0 0" rpy="0 0 0"/>
+            <geometry>
+                <box size="0.03 0.094 0.024"/>
+            </geometry>
+        </collision>
+    </link>
+    <joint name="${prefix}camera_joint" type="fixed">
+        <parent link="${prefix}chassis"/>
+        <child link="${prefix}camera_link"/>
+        <!-- Mounted on top of chassis, front-facing -->
+        <origin xyz="0.08 0.0 0.04" rpy="0 0 0"/>
+    </joint>
+    <link name="${prefix}camera_optical_frame"/>
+    <joint name="${prefix}camera_optical_joint" type="fixed">
+        <parent link="${prefix}camera_link"/>
+        <child link="${prefix}camera_optical_frame"/>
+        <!-- Rotate to optical frame convention: Z-forward, X-right, Y-down -->
+        <origin xyz="0 0 0" rpy="${-pi/2} 0 ${-pi/2}"/>
+    </joint>
   </xacro:macro>
 </robot>
