Commit message: Enhance camera integration and simulation configurations
- Add RGB camera sensor configuration to camera_rgb.urdf.xacro
- Update gz_bridge.yaml to include camera topics for ROS-Gazebo communication
- Enable shadows for the sun light in perseus_arc_world.world
- Remove unused turtlebot3_dqn_stage2.world file
- Delete outdated CHANGELOG.rst from perseus_teleop package

File: software/ros_ws/src/perseus_description/urdf/camera_rgb.urdf.xacro (robot description, xacro)
@@ -1,3 +1,5 @@
 <?xml version="1.0"?>
+<!-- 0.220 0 0.4 -->
+<!-- <box size="0.020 0.07 0.03"/>  -->
 <robot name="camera_rgb" xmlns:xacro="http://ros.org/wiki/xacro">
   <xacro:macro name="camera_rgb" params="prefix:=^">
@@ -15,4 +17,33 @@
         </visual>
     </link>
+    <joint name="camera_optical_joint" type="fixed">
+        <parent link="camera_link"/>
+        <child link="camera_link_optical"/>
+        <origin xyz="0 0 0" rpy="${-pi/2} 0 ${-pi/2}"/>
+    </joint>
+    <link name="camera_link_optical"></link>
+    <gazebo reference="camera_link">
+        <material>Gazebo/Black</material>
+        <sensor name="camera" type="camera">
+            <pose> 0 0 0 0 0 0 </pose>
+            <visualize>true</visualize>
+            <update_rate>10</update_rate>
+            <camera>
+                <camera_info_topic>camera/camera_info</camera_info_topic>
+                <horizontal_fov>1.089</horizontal_fov>
+                <image>
+                    <format>R8G8B8</format>
+                    <width>640</width>
+                    <height>480</height>
+                </image>
+                <clip>
+                    <near>0.05</near>
+                    <far>8.0</far>
+                </clip>
+            </camera>
+            <topic>camera/image_raw</topic>
+            <gz_frame_id>camera_link_optical</gz_frame_id>
+        </sensor>
+    </gazebo>
   </xacro:macro>
 </robot>

Commit message: Update camera RGB URDF configuration for improved simulation accuracy

File: software/ros_ws/src/perseus_description/urdf/camera_rgb.urdf.xacro (robot description, xacro)
@@ -24,5 +24,5 @@
     <link name="camera_link_optical"></link>
     <gazebo reference="camera_link">
-        <material>Gazebo/Black</material>
+        <material>Gazebo/Red</material>
         <sensor name="camera" type="camera">
             <pose> 0 0 0 0 0 0 </pose>

Commit message: just some random adjustment

File: software/ros_ws/src/perseus_description/urdf/camera_rgb.urdf.xacro (robot description, xacro)
@@ -39,5 +39,5 @@
                 <clip>
                     <near>0.05</near>
-                    <far>8.0</far>
+                    <far>100</far>
                 </clip>
             </camera>

File: software/ros_ws/src/perseus_description/urdf/sensors.urdf.xacro (robot description, xacro)
@@ -8,5 +8,5 @@
                 <cylinder radius="0.06" length="0.06"/>
             </geometry>
-            <material name="black"/>
+            <material name="red"/>
         </visual>
         <collision>
@@ -81,5 +81,5 @@
             <visualize>true</visualize>
             <update_rate>10</update_rate>
-            <topic>scan</topic>
+            <topic>scan2</topic>
             <ray>
                 <scan>

Commit message: fix: Rename robot and sensor types in camera_rgb.urdf.xacro to reflect depth camera configuration

File: software/ros_ws/src/perseus_description/urdf/camera_rgb.urdf.xacro (robot description, xacro)
@@ -2,6 +2,6 @@
 <!-- 0.220 0 0.4 -->
 <!-- <box size="0.020 0.07 0.03"/>  -->
-<robot name="camera_rgb" xmlns:xacro="http://ros.org/wiki/xacro">
-  <xacro:macro name="camera_rgb" params="prefix:=^">
+<robot name="camera_depth" xmlns:xacro="http://ros.org/wiki/xacro">
+  <xacro:macro name="camera_depth" params="prefix:=^">
     <joint name="camera_joint" type="fixed">
         <parent link="base_link"/>
@@ -25,5 +25,5 @@
     <gazebo reference="camera_link">
         <material>Gazebo/Red</material>
-        <sensor name="camera" type="camera">
+        <sensor name="depth_camera" type="depth_camera">
             <pose> 0 0 0 0 0 0 </pose>
             <visualize>true</visualize>
@@ -37,4 +37,9 @@
                     <height>480</height>
                 </image>
+                <depth_camera>
+                    <output>
+                        <type>depth</type>
+                    </output>
+                </depth_camera>
                 <clip>
                     <near>0.05</near>
@@ -43,4 +48,6 @@
             </camera>
             <topic>camera/image_raw</topic>
+            <depth_camera_topic>camera/depth/image_raw</depth_camera_topic>
+            <point_cloud_topic>camera/points</point_cloud_topic>
             <gz_frame_id>camera_link_optical</gz_frame_id>
         </sensor>
