Commit message: feat: update configurations for 2D and 3D SLAM integration, enhance EKF settings, and add launch files

File: software/ros_ws/src/perseus_description/urdf/flange_bearing.urdf.xacro (robot description, xacro)
@@ -35,5 +35,5 @@
     </visual>
     <collision>
-    <origin xyz="0.0 0.0 -0.01" rpy="0.0 0.0 0.0"/>
+    <origin xyz="0.0 0.0 0.0" rpy="${-pi/2} 0 ${-pi/2}"/>
     <geometry>
         <mesh scale="${0.1/scale_factor} ${0.1/scale_factor}  ${0.1/scale_factor}" filename="file://$(find perseus_description)/meshes/differential_bar.dae"/>

File: software/ros_ws/src/perseus_description/urdf/motor_wheel.urdf.xacro (robot description, xacro)
@@ -4,5 +4,5 @@
     <inertial>
       <!-- moving origin has no perceivable impact-->
-      <origin xyz="0.0 0.0 0.0" rpy="0.0 0.0 0.0"/>
+      <origin xyz="0 0.0 0.0" rpy="0.0 0.0 ${pi/2}"/>
       <mass value="1"/>
       <inertia ixx="0.01" iyy="0.01" izz="0.01" ixy="0.0" iyz="0.0" ixz="0.0"/> <!-- TEMP -->
@@ -16,5 +16,5 @@
     </visual>
     <collision>
-      <origin xyz="-0.3 0.0 0.0" rpy="0.0 0.0 ${pi/2}"/>
+      <origin xyz="0 0.0 0.0" rpy="0.0 0.0 ${pi/2}"/>
       <geometry>
         <mesh scale="${0.1/scale_factor} ${0.1/scale_factor}  ${0.1/scale_factor}" filename="file://$(find perseus_description)/meshes/gearbox.dae"/>
@@ -25,5 +25,5 @@
     <inertial>
       <!-- moving origin has no perceivable impact-->
-      <origin xyz="0.0 0.0 0.0" rpy="0.0 0.0 0.0"/>
+      <origin xyz="0 0.0 0.0" rpy="0.0 0.0 ${pi/2}"/>
       <mass value="1"/>
       <inertia ixx="0.01" iyy="0.01" izz="0.01" ixy="0.0" iyz="0.0" ixz="0.0"/> <!-- TEMP -->
@@ -37,5 +37,5 @@
     </visual>
     <collision>
-      <origin xyz="-0.3 0.0 0.0" rpy="0.0 0.0 ${pi/2}"/>
+      <origin xyz="0 0.0 0.0" rpy="0.0 0.0 ${pi/2}"/>
       <geometry>
         <mesh scale="${0.1/scale_factor} ${0.1/scale_factor}  ${0.1/scale_factor}" filename="file://$(find perseus_description)/meshes/gearbox.dae"/>

File: software/ros_ws/src/perseus_description/urdf/perseus.urdf.xacro (robot description, xacro)
@@ -30,4 +30,10 @@
     <!-- An empty base_link to attach everything to -->
     <link name="${prefix}base_link"/>
+    <link name="${prefix}base_footprint"/>  <!-- 2D footprint for SLAM & navigation -->
+    <joint name="${prefix}base_to_footprint" type="fixed">
+      <origin xyz="0 0 0" rpy="0 0 0"/>
+      <parent link="${prefix}chassis"/>
+      <child link="${prefix}base_footprint"/>
+    </joint>
     <joint name="${prefix}chassis_joint" type="fixed"> <!-- Joint Connect base_link and chassis -->
       <origin xyz="0.3 0.0 ${chassis_z_offset/scale_factor}" rpy="0 0.0 0.0"/>

File: software/ros_ws/src/perseus_description/urdf/sensors.urdf.xacro (robot description, xacro)
@@ -41,5 +41,5 @@
   </material>
   <sensor name="${prefix}lidar_sensor" type="gpu_lidar">
-    <topic>scan</topic>
+    <topic>scan_3d</topic>
     <update_rate>50</update_rate>
     <always_on>false</always_on>
@@ -77,5 +77,5 @@
   </material>
   <sensor name="${prefix}laser_2d_sensor" type="gpu_lidar">
-    <topic>scan_2d</topic>
+    <topic>scan</topic>
     <update_rate>50</update_rate>
     <always_on>true</always_on>

Commit message: refactor: Update flange_bearing properties and remove obsolete models from the simulation

File: software/ros_ws/src/perseus_description/urdf/flange_bearing.urdf.xacro (robot description, xacro)
@@ -1,7 +1,10 @@
 <?xml version="1.0"?>
 <robot name="flange_bearing" xmlns:xacro="http://ros.org/wiki/xacro">
-<xacro:property name="bar_length" value="0.22"/>
+<xacro:property name="bar_length" value="0.5"/>
 <xacro:property name="bar_width" value="0.03"/>
 <xacro:property name="bar_height" value="0.03"/>
+<xacro:property name="bearing_length" value="0.2"/>
+<xacro:property name="bearing_width" value="0.03"/>
+<xacro:property name="bearing_height" value="0.03"/>
 <!-- Flange Bearing -->
 <link name="${prefix}flange_bearing">
@@ -20,5 +23,5 @@
     <origin xyz="0.0 0.0 0.0" rpy="0 0 0"/>
     <geometry>
-        <mesh scale="${0.1/scale_factor} ${0.1/scale_factor}  ${0.1/scale_factor}" filename="file://$(find perseus_description)/meshes/flange_bearing.dae"/>
+        <box size="${bar_length/scale_factor} ${bar_width/scale_factor} ${bar_height/scale_factor}"/>
     </geometry>
     </collision>

Commit message: Add ArUco markers models and textures for Perseus simulation
- Created model.config and model.sdf for aruco_markers4 and aruco_markers5, defining their properties and visual representations.
- Added textures for aruco_markers4 and aruco_markers5.
- Introduced cubes model with multiple colored cubes, including model.config and model.sdf files.
- Added obstacles model with multiple cylindrical obstacles, including model.config and model.sdf files.

File: software/ros_ws/src/perseus_description/urdf/flange_bearing.urdf.xacro (robot description, xacro)
@@ -7,9 +7,10 @@
 <xacro:property name="bearing_width" value="0.03"/>
 <xacro:property name="bearing_height" value="0.03"/>
+<xacro:property name="bearing_mass" value="2.7689940302592726"/>  <!-- Kg -->
 <!-- Flange Bearing -->
 <link name="${prefix}flange_bearing">
     <inertial>
     <origin xyz="0.0 0.0 0.0" rpy="0 0 0"/>
-    <mass value="1.327488734939265"/>
+    <mass value="${bearing_mass}"/>
     <inertia ixx="0.001313" iyy="0.001699" izz="0.000647" ixy="0.0" iyz="0.0" ixz="-0.0"/>
     </inertial>
@@ -21,5 +22,5 @@
     </visual>
     <collision>
-    <origin xyz="0.0 0.0 0.0" rpy="0 0 0"/>
+    <origin xyz="0.0 0.0 0.0" rpy="${-pi/2} 0 ${pi/2}"/>
     <geometry>
         <box size="${bar_length/scale_factor} ${bar_width/scale_factor} ${bar_height/scale_factor}"/>
@@ -32,5 +33,5 @@
         <origin xyz="0 0 0.0" rpy="0.0 0.0 0.0"/>
         <mass value="0.9172649518127158"/>
-        <inertia ixx="0.00036" iyy="0.018339" izz="0.018134" ixy="3e-06" iyz="-0.0" ixz="0.0"/>
+        <xacro:box_inertia m="${chassis_mass}" x="${chassis_length/scale_factor}" y="${chassis_width/scale_factor}" z="${chassis_height/scale_factor}"/>
     </inertial>
     <visual>

File: software/ros_ws/src/perseus_description/urdf/perseus.urdf.xacro (robot description, xacro)
@@ -35,4 +35,5 @@
     <xacro:include filename="$(find perseus_description)/urdf/wheel.urdf.xacro"/>
     <xacro:include filename="$(find perseus_description)/urdf/sensors.urdf.xacro"/>
+    <xacro:include filename="$(find perseus_description)/urdf/camera_depth.urdf.xacro" />
     <!-- An empty base_link to attach everything to -->
     <link name="${prefix}base_link"/>
@@ -110,4 +111,14 @@
       <origin xyz="0 0 -0.04" rpy="0 ${PI} 0"/>
     </joint>
+    <joint name="${prefix}laser_2d_joint" type="fixed">
+      <parent link="${prefix}chassis"/>
+      <child link="${prefix}laser_2d_frame"/>
+      <origin xyz="-0.15 0 0.25" rpy="0 0 0"/>
+    </joint>
+    <joint name="${prefix}camera_joint" type="fixed">
+        <parent link="${prefix}chassis"/>
+        <child link="${prefix}camera_link"/>
+        <origin xyz="0.01 0 0.18" rpy="0 0 0"/>
+    </joint>
   </xacro:macro>
 </robot>

File: software/ros_ws/src/perseus_description/urdf/sensors.urdf.xacro (robot description, xacro)
@@ -1,4 +1,5 @@
 <?xml version="1.0"?>
 <robot name="lidar" xmlns:xacro="http://ros.org/wiki/xacro">
+<!-- 3D LIDAR (Existing - Livox MID-360) -->
 <link name="${prefix}laser_frame">
     <visual>
@@ -15,4 +16,21 @@
     </collision>
 </link>
+<!-- 2D LIDAR -->
+<link name="${prefix}laser_2d_frame">
+    <visual>
+        <origin xyz="0 0 0"/>
+        <geometry>
+            <cylinder radius="0.04" length="0.04"/>
+        </geometry>
+        <material name="blue">
+            <color rgba="0.0 0.0 1.0 1.0"/>
+        </material>
+    </visual>
+    <collision>
+        <geometry>
+            <cylinder radius="0.04" length="0.04"/>
+        </geometry>
+    </collision>
+</link>
 <!-- Simulating the Livox MID-360 -->
 <gazebo reference="${prefix}laser_frame">
@@ -23,7 +41,7 @@
   </material>
   <sensor name="${prefix}lidar_sensor" type="gpu_lidar">
-    <topic>scan</topic>
-    <update_rate>10</update_rate>
-    <always_on>true</always_on>
+    <topic>scan_3d</topic>
+    <update_rate>50</update_rate>
+    <always_on>false</always_on>
     <visualize>false</visualize>
     <ray>
@@ -51,3 +69,39 @@
   </sensor>
 </gazebo>
+<!-- 2D LIDAR SENSOR (Traditional 2D Laser Scanner) -->
+<gazebo reference="${prefix}laser_2d_frame">
+  <material>
+    <ambient>0.0 0.0 1.0 1</ambient>
+    <diffuse>0.0 0.0 1.0 1</diffuse>
+    <specular>0.0 0.0 1.0 1</specular>
+  </material>
+  <sensor name="${prefix}laser_2d_sensor" type="gpu_lidar">
+    <topic>scan</topic>
+    <update_rate>10</update_rate>
+    <always_on>true</always_on>
+    <visualize>false</visualize>
+    <ray>
+      <scan>
+        <horizontal>
+          <samples>720</samples>
+          <resolution>1</resolution>
+          <min_angle>-3.14159</min_angle>
+          <max_angle>3.14159</max_angle>
+        </horizontal>
+        <!-- Single horizontal plane for 2D scanning -->
+        <vertical>
+          <samples>1</samples>
+          <min_angle>0.0</min_angle>
+          <max_angle>0.0</max_angle>
+        </vertical>
+      </scan>
+      <range>
+        <min>0.05</min>
+        <max>200.0</max>
+        <resolution>0.01</resolution>
+      </range>
+    </ray>
+    <gz_frame_id>laser_2d_frame</gz_frame_id>
+  </sensor>
+</gazebo>
 </robot>

Commit message: refactor: Update inertial properties for flange bearing and replace inertia with box inertia calculation

File: software/ros_ws/src/perseus_description/urdf/flange_bearing.urdf.xacro (robot description, xacro)
@@ -11,7 +11,7 @@
 <link name="${prefix}flange_bearing">
     <inertial>
-    <origin xyz="0.0 0.0 0.0" rpy="0 0 0"/>
+    <origin xyz="0.0 0.0 0.0" rpy="${-pi/2} 0 ${pi/2}"/>
     <mass value="${bearing_mass}"/>
-    <inertia ixx="0.001313" iyy="0.001699" izz="0.000647" ixy="0.0" iyz="0.0" ixz="-0.0"/>
+    <xacro:box_inertia m="${bearing_mass}" x="${bearing_length/scale_factor}" y="${bearing_width/scale_factor}" z="${bearing_height/scale_factor}"/>
     </inertial>
     <visual>
