Commit message: fix(urdf): adjust motor wheel and rocker arm origins and orientations for left and right sides

File: software/ros_ws/src/perseus_description/urdf/motor_wheel.urdf.xacro (robot description, xacro)
@@ -11,5 +11,10 @@
       </inertial>
       <visual>
-        <origin xyz="-0.265 0.0 0.0" rpy="0.0 0.0 ${pi}"/>
+        <xacro:if value="${side == 'left'}">
+          <origin xyz="0 0.0 0.0" rpy="0.0 0.0 ${-pi/2}"/>
+        </xacro:if>
+        <xacro:if value="${side == 'right'}">
+          <origin xyz="0 0.0 0.0" rpy="0.0 0.0 ${pi/2}"/>
+        </xacro:if>
         <geometry>
           <mesh scale="0.1 0.1 0.1" filename="file://$(find perseus_description)/meshes/gearbox.dae"/>
@@ -18,5 +23,5 @@
       </visual>
       <collision>
-        <origin xyz="-0.3 0.0 0.0" rpy="0.0 0.0 0.0"/>
+        <origin xyz="-0.3 0.0 0.0" rpy="0.0 0.0 ${pi/2}"/>
         <geometry>
           <box size="0.1 0.1 0.075" />

File: software/ros_ws/src/perseus_description/urdf/perseus.urdf.xacro (robot description, xacro)
@@ -23,9 +23,9 @@
     <!-- LEFT -->
     <xacro:rocker side="left">
-      <origin xyz="-0.275 -0.075 0.05" rpy="0.0 0.0 ${-pi/2}"/>
+      <origin xyz="-0.075 0.275 0.05" rpy="0.0 0.0 0"/>
     </xacro:rocker>
     <!-- RIGHT -->
     <xacro:rocker side="right">
-      <origin xyz="0.275 -0.075 0.05" rpy="0.0 0.0 ${-pi/2}"/>
+      <origin xyz="-0.075 -0.275 0.05" rpy="0.0 0.0 0.0"/>
     </xacro:rocker>
     <xacro:sensors>

File: software/ros_ws/src/perseus_description/urdf/rocker.urdf.xacro (robot description, xacro)
@@ -6,5 +6,5 @@
     <link name="${prefix}${side}_rocker">
       <inertial>
-        <origin xyz="0.011819187400851083 -0.08337339654014758 -0.06739096070989994" rpy="0.0 0.0 0.0"/>
+        <origin xyz="0.0 -0.0 -0.0" rpy="0 0 0"/>
         <!-- RIGHT -->
         <xacro:if value="${side == 'right'}">
@@ -18,5 +18,5 @@
       </inertial>
       <visual>
-        <origin xyz="0.0 0.0 0.0" rpy="0.0 0.0 0.0"/>
+        <origin xyz="0.0 0.0 0.0" rpy="0.0 0.0 ${pi}"/>
         <geometry>
           <mesh scale="0.1 0.1 0.1" filename="file://$(find perseus_description)/meshes/rocker_${side}.dae"/>
@@ -26,5 +26,5 @@
         <origin xyz="0.2 0.0 -0.05" rpy="0.0 0.3 0.0"/>
         <geometry>
-          <box size="0.4 0.05 0.03" />
+          <mesh scale="0.1 0.1 0.1" filename="file://$(find perseus_description)/meshes/rocker_${side}.dae"/>
         </geometry>
       </collision>
@@ -38,8 +38,8 @@
     <xacro:motor_wheel end="front">
       <xacro:if value="${side == 'left'}">
-        <origin xyz="-0.3 -0.225 -0.25" rpy="0.0 0.0 ${-pi/2}"/>
+        <origin xyz="0.3 -0.035 -0.25" rpy="0.0 0.0 0"/>
       </xacro:if>
       <xacro:if value="${side == 'right'}">
-        <origin xyz="-0.3 0.225 -0.25" rpy="0.0 0.0 ${pi/2}"/>
+        <origin xyz="0.3 0.035 -0.25" rpy="0.0 0.0 0"/>
       </xacro:if>
     </xacro:motor_wheel>
@@ -47,8 +47,8 @@
     <xacro:motor_wheel end="rear">
       <xacro:if value="${side == 'left'}">
-        <origin xyz="0.55 -0.225 -0.25" rpy="0.0 0.0 ${-pi/2}"/>
+        <origin xyz="-0.55 -0.035 -0.25" rpy="0.0 0.0 0.0"/>
       </xacro:if>
       <xacro:if value="${side == 'right'}">
-        <origin xyz="0.55 0.225 -0.25" rpy="0.0 0.0 ${pi/2}"/>
+        <origin xyz="-0.55 0.035 -0.25" rpy="0.0 0.0 0.0"/>
       </xacro:if>
     </xacro:motor_wheel>

Commit message: refactor: Improve formatting and structure of Nix package files for better readability

File: software/ros_ws/src/perseus_description/urdf/motor_wheel.urdf.xacro (robot description, xacro)
@@ -6,5 +6,10 @@
       <inertial>
         <!-- moving origin has no perceivable impact-->
-        <origin xyz="0.0 0.0 0.0" rpy="0.0 0.0 0.0"/>
+        <xacro:if value="${side == 'left'}">
+          <origin xyz="0 0.0 0.0" rpy="0.0 0.0 ${-pi/2}"/>
+        </xacro:if>
+        <xacro:if value="${side == 'right'}">
+          <origin xyz="0 0.0 0.0" rpy="0.0 0.0 ${pi/2}"/>
+        </xacro:if>
         <mass value="5.236579"/>
         <inertia ixx="0.01" iyy="0.01" izz="0.01" ixy="0.0" iyz="0.0" ixz="0.0"/> <!-- TEMP -->

Commit message: Refactor URDF and XACRO files for motor, rocker, and wheel components to improve structure and add dynamic properties for better simulation accuracy.

File: software/ros_ws/src/perseus_description/urdf/motor_wheel.urdf.xacro (robot description, xacro)
@@ -5,87 +5,58 @@
   <xacro:property name="collision_motor_width" value="0.1"/>  <!-- m -->
   <xacro:property name="collision_motor_height" value="0.075"/>  <!-- m -->
-  <link name="${prefix}front_right_motor">
-    <inertial>
-      <!-- moving origin has no perceivable impact-->
-      <origin xyz="0.0 0.0 0.0" rpy="0.0 0.0 0.0"/>
-      <mass value="${motor_mass}"/>
-      <inertia ixx="0.01" iyy="0.01" izz="0.01" ixy="0.0" iyz="0.0" ixz="0.0"/> <!-- TEMP -->
-    </inertial>
-    <visual>
-      <origin xyz="0 0.0 0.0" rpy="0.0 0.0 ${pi/2}"/>
-      <geometry>
-        <mesh scale="0.1 0.1  0.1" filename="file://$(find perseus_description)/meshes/gearbox.dae"/>
-      </geometry>
-      <!-- <material name="white"/> -->
-    </visual>
-    <collision>
-      <origin xyz="0.0 0.0 0.0" rpy="0.0 0.0 ${pi/2}"/>
-      <geometry>
-        <box size="${collision_motor_length} ${collision_motor_width} ${collision_motor_height}" />
-      </geometry>
-    </collision>
-  </link>
-  <link name="${prefix}rear_right_motor">
-    <inertial>
-      <!-- moving origin has no perceivable impact-->
-      <origin xyz="0.0 0.0 0.0" rpy="0.0 0.0 0.0"/>
-      <mass value="${motor_mass}"/>
-      <inertia ixx="0.01" iyy="0.01" izz="0.01" ixy="0.0" iyz="0.0" ixz="0.0"/> <!-- TEMP -->
-    </inertial>
-    <visual>
-      <origin xyz="0 0.0 0.0" rpy="0.0 0.0 ${pi/2}"/>
-      <geometry>
-        <mesh scale="0.1 0.1  0.1" filename="file://$(find perseus_description)/meshes/gearbox.dae"/>
-      </geometry>
-      <!-- <material name="white"/> -->
-    </visual>
-    <collision>
-      <origin xyz="0.0 0.0 0.0" rpy="0.0 0.0 ${pi/2}"/>
-      <geometry>
-        <box size="${collision_motor_length} ${collision_motor_width} ${collision_motor_height}" />
-      </geometry>
-    </collision>
-  </link>
-  <link name="${prefix}front_left_motor">
-    <inertial>
-      <!-- moving origin has no perceivable impact-->
-      <origin xyz="0.0 0.0 0.0" rpy="0.0 0.0 0.0"/>
-      <mass value="${motor_mass}"/>
-      <inertia ixx="0.01" iyy="0.01" izz="0.01" ixy="0.0" iyz="0.0" ixz="0.0"/> <!-- TEMP -->
-    </inertial>
-    <visual>
-      <origin xyz="0 0.0 0.0" rpy="0.0 0.0 ${-pi/2}"/>
-      <geometry>
-        <mesh scale="0.1 0.1  0.1" filename="file://$(find perseus_description)/meshes/gearbox.dae"/>
-      </geometry>
-      <!-- <material name="white"/> -->
-    </visual>
-    <collision>
-      <origin xyz="0 0.0 0.0" rpy="0.0 0.0 ${-pi/2}"/>
-      <geometry>
-        <box size="${collision_motor_length} ${collision_motor_width} ${collision_motor_height}" />
-      </geometry>
-    </collision>
-  </link>
-  <link name="${prefix}rear_left_motor">
-    <inertial>
-      <!-- moving origin has no perceivable impact-->
-      <origin xyz="0.0 0.0 0.0" rpy="0.0 0.0 0.0"/>
-      <mass value="${motor_mass}"/>
-      <inertia ixx="0.01" iyy="0.01" izz="0.01" ixy="0.0" iyz="0.0" ixz="0.0"/> <!-- TEMP -->
-    </inertial>
-    <visual>
-      <origin xyz="0 0.0 0.0" rpy="0.0 0.0 ${-pi/2}"/>
-      <geometry>
-        <mesh scale="0.1 0.1  0.1" filename="file://$(find perseus_description)/meshes/gearbox.dae"/>
-      </geometry>
-      <!-- <material name="white"/> -->
-    </visual>
-    <collision>
-      <origin xyz="0 0.0 0.0" rpy="0.0 0.0 ${-pi/2}"/>
-      <geometry>
-        <box size="${collision_motor_length} ${collision_motor_width} ${collision_motor_height}" />
-      </geometry>
-    </collision>
-  </link>
+  <xacro:macro name="motor" params="prefix:=^ side:=^ end:=^">
+    <link name="${prefix}${end}_${side}_motor">
+      <inertial>
+        <!-- moving origin has no perceivable impact-->
+        <origin xyz="0.0 0.0 0.0" rpy="0.0 0.0 0.0"/>
+        <mass value="${motor_mass}"/>
+        <inertia ixx="0.01" iyy="0.01" izz="0.01" ixy="0.0" iyz="0.0" ixz="0.0"/> <!-- TEMP -->
+      </inertial>
+      <visual>
+        <xacro:if value="${side == 'left'}">
+          <origin xyz="0 0.0 0.0" rpy="0.0 0.0 ${pi/2}"/>
+        </xacro:if>
+        <xacro:if value="${side == 'right'}">
+          <origin xyz="0 0.0 0.0" rpy="0.0 0.0 ${-pi/2}"/>
+        </xacro:if>
+        <geometry>
+          <mesh scale="0.1 0.1  0.1" filename="file://$(find perseus_description)/meshes/gearbox.dae"/>
+        </geometry>
+        <!-- <material name="white"/> -->
+      </visual>
+      <collision>
+        <xacro:if value="${side == 'left'}">
+          <origin xyz="0.0 0.0 0.0" rpy="0.0 0.0 ${pi/2}"/>
+        </xacro:if>
+        <xacro:if value="${side == 'right'}">
+          <origin xyz="0.0 0.0 0.0" rpy="0.0 0.0 ${-pi/2}"/>
+        </xacro:if>
+        <geometry>
+          <box size="${collision_motor_length} ${collision_motor_width} ${collision_motor_height}" />
+        </geometry>
+      </collision>
+    </link>
+    <joint name="${prefix}${end}_${side}_motor_joint" type="fixed">
+      <parent link="${prefix}${side}_rocker"/>
+      <child link="${prefix}${end}_${side}_motor"/>
+      <xacro:if value="${end == 'front'}">
+        <xacro:if value="${side == 'left'}">
+          <origin xyz="${front_motors_x_offset} -${motors_y_offset} ${motors_z_offset}" rpy="0.0 0.0 0.0"/>
+        </xacro:if>
+        <xacro:if value="${side == 'right'}">
+          <origin xyz="${front_motors_x_offset} ${motors_y_offset} ${motors_z_offset}" rpy="0.0 0.0 0.0"/>
+        </xacro:if>
+      </xacro:if>
+      <xacro:if value="${end == 'rear'}">
+        <xacro:if value="${side == 'left'}">
+          <origin xyz="${rear_motors_x_offset} -${motors_y_offset} ${motors_z_offset}" rpy="0.0 0.0 0.0"/>
+        </xacro:if>
+        <xacro:if value="${side == 'right'}">
+          <origin xyz="${rear_motors_x_offset} ${motors_y_offset} ${motors_z_offset}" rpy="0.0 0.0 0.0"/>
+        </xacro:if>
+      </xacro:if>
+    </joint>
+  <!-- ADD 1 WHEEL FOR EACH MOTOR -->
+  <xacro:wheel prefix="" side="${side}"  end="${end}"/>
+  </xacro:macro>
 </robot>

File: software/ros_ws/src/perseus_description/urdf/perseus.urdf.xacro (robot description, xacro)
@@ -2,5 +2,20 @@
 <robot xmlns:xacro="http://ros.org/wiki/xacro">
   <xacro:macro name="perseus" params="prefix">
-    <!-- Constants for robot dimensions -->
+    <xacro:property name="front_motors_x_offset" value="0.3"/>
+    <xacro:property name="rear_motors_x_offset" value="-0.55"/>
+    <!-- Rocker properties -->
+    <xacro:property name="rocker_mass" value="0.5"/>
+    <xacro:property name="rocker_length" value="${(front_motors_x_offset-rear_motors_x_offset)*1/2}"/>  <!-- Use positive absolute value -->
+    <xacro:property name="rocker_width" value="0.03"/>
+    <xacro:property name="rocker_collision_x_offset" value="-0.10"/>
+    <xacro:property name="rocker_height" value="0.2"/>
+    <xacro:property name="rocker_base_distance" value="0.275" />
+    <xacro:property name="rocker_x_offset" value="0.075"/>
+    <xacro:property name="rocker_y_offset" value="0.05"/>
+    <!-- Wheels Properties -->
+    <xacro:property name="wheel_mass" value="1.0"/>
+    <xacro:property name="wheels_y_offset" value="0.125"/>
+    <xacro:property name="wheel_radius" value="0.15"/>
+    <xacro:property name="wheel_length" value="0.14"/>
     <!-- Chassis Properties -->
     <xacro:property name="base_mass" value="0.3" /> <!-- arbitrary value for base mass -->
@@ -8,32 +23,31 @@
     <xacro:property name="chassis_length" value="0.6" />
     <xacro:property name="chassis_height" value="0.2" />
-    <xacro:property name="chassis_z_offset" value="0.35" /> <!-- Space btw top of beam and the each joint -->
+    <xacro:property name="chassis_z_offset" value="${rocker_height + wheel_radius}" /> <!-- Space btw top of beam and the each joint -->
     <!-- Flange Bearing Properties -->
-    <xacro:property name="flange_bearing_z_offset" value="0.1"/>
-    <!-- Rocker Properties -->
-    <xacro:property name="rocker_base_distance" value="0.275" />
-    <xacro:property name="rocker_x_offset" value="0.075"/>
-    <xacro:property name="rocker_y_offset" value="0.05"/>
+    <xacro:property name="flange_bearing_z_offset" value="${chassis_height/2}"/>
     <!-- Motors Properties -->
     <xacro:property name="motors_y_offset" value="0.035"/>
     <xacro:property name="motors_z_offset" value="-0.25"/>
-    <xacro:property name="front_motors_x_offset" value="0.3"/>
-    <xacro:property name="rear_motors_x_offset" value="-0.55"/>
-    <!-- Wheels Properties -->
-    <xacro:property name="wheels_y_offset" value="0.125"/>
-    <xacro:property name="wheel_mass" value="1.0"/>
-    <xacro:property name="wheel_radius" value="0.15"/>
-    <xacro:property name="wheel_length" value="0.14"/>
+    <xacro:property name="motor_mass" value="5.236579"/>  <!-- Kg -->
+    <xacro:property name="collision_motor_length" value="0.1"/>  <!-- m -->
+    <xacro:property name="collision_motor_width" value="0.1"/>  <!-- m -->
+    <xacro:property name="collision_motor_height" value="0.075"/>  <!-- m -->
     <!-- ADD COMPONENTS -->
     <xacro:include filename="$(find perseus_description)/urdf/inertia_macros.xacro"/>
     <xacro:include filename="$(find perseus_description)/urdf/chassis.urdf.xacro"/>
     <xacro:include filename="$(find perseus_description)/urdf/flange_bearing.urdf.xacro"/>
+    <xacro:include filename="$(find perseus_description)/urdf/wheel.urdf.xacro"/>
+    <xacro:include filename="$(find perseus_description)/urdf/motor_wheel.urdf.xacro"/>
     <xacro:include filename="$(find perseus_description)/urdf/rocker.urdf.xacro"/>
-    <xacro:include filename="$(find perseus_description)/urdf/motor_wheel.urdf.xacro"/>
-    <xacro:include filename="$(find perseus_description)/urdf/wheel.urdf.xacro"/>
     <xacro:include filename="$(find perseus_description)/urdf/sensors.urdf.xacro"/>
     <xacro:include filename="$(find perseus_description)/urdf/camera_depth.urdf.xacro" />
     <!-- An empty base_link to attach everything to -->
     <link name="${prefix}base_link"/>
+    <joint name="base_footprint_joint" type="fixed">
+        <parent link="base_link"/>
+        <child link="base_footprint"/>
+        <origin xyz="0 0 0" rpy="0 0 0"/>
+    </joint>
+    <link name="${prefix}base_footprint"/>
     <joint name="${prefix}chassis_joint" type="fixed"> <!-- Joint Connect base_link and chassis -->
       <origin xyz="0 0.0 ${chassis_z_offset}" rpy="0.0 0.0 0.0"/>
@@ -41,38 +55,11 @@
       <child link="${prefix}chassis"/>
     </joint>
+    <!-- ADD 2 ROCKERS (INCLUDING 4 MOTORS + 4 WHEELS) -->
+    <xacro:rocker prefix="" side="left"/>
+    <xacro:rocker prefix="" side="right"/>
     <joint name="${prefix}flange_bearing_joint" type="fixed">
       <origin xyz="${-chassis_length} 0.0 ${flange_bearing_z_offset}" rpy="0 0 0"/>
       <parent link="${prefix}chassis"/>
       <child link="${prefix}flange_bearing"/>
-    </joint>
-    <joint name="${prefix}left_rocker_joint" type="fixed">
-      <origin xyz="${-rocker_x_offset} ${rocker_base_distance} ${rocker_y_offset} " rpy="0 0 0"/>
-      <parent link="${prefix}chassis"/>
-      <child link="${prefix}left_rocker"/>
-    </joint>
-    <joint name="${prefix}right_rocker_joint" type="fixed">
-      <origin xyz="${-rocker_x_offset} ${-rocker_base_distance} ${rocker_y_offset} " rpy="0 0 0"/>
-      <parent link="${prefix}chassis"/>
-      <child link="${prefix}right_rocker"/>
-    </joint>
-    <joint name="${prefix}front_left_motor_joint" type="fixed">
-      <parent link="${prefix}left_rocker"/>
-      <child link="${prefix}front_left_motor"/>
-      <origin xyz="${front_motors_x_offset} -${motors_y_offset} ${motors_z_offset}" rpy="0.0 0.0 0"/>
-    </joint>
-    <joint name="${prefix}rear_left_motor_joint" type="fixed">
-      <parent link="${prefix}left_rocker"/>
-      <child link="${prefix}rear_left_motor"/>
-      <origin xyz="${rear_motors_x_offset} -${motors_y_offset} ${motors_z_offset}" rpy="0.0 0.0 0.0"/>
-    </joint>
-    <joint name="${prefix}front_right_motor_joint" type="fixed">
-      <parent link="${prefix}right_rocker"/>
-      <child link="${prefix}front_right_motor"/>
-      <origin xyz="${front_motors_x_offset} ${motors_y_offset} ${motors_z_offset}" rpy="0.0 0.0 0"/>
-    </joint>
-    <joint name="${prefix}rear_right_motor_joint" type="fixed">
-      <parent link="${prefix}right_rocker"/>
-      <child link="${prefix}rear_right_motor"/>
-      <origin xyz="${rear_motors_x_offset} ${motors_y_offset} ${motors_z_offset}" rpy="0.0 0.0 0.0"/>
     </joint>
     <joint name="${prefix}laser_joint" type="fixed">

File: software/ros_ws/src/perseus_description/urdf/rocker.urdf.xacro (robot description, xacro)
@@ -1,15 +1,9 @@
 <?xml version="1.0"?>
 <robot name="rocker" xmlns:xacro="http://ros.org/wiki/xacro">
-  <!-- Rocker properties - Fix negative values -->
-  <xacro:property name="rocker_mass" value="0.5"/>
-  <xacro:property name="rocker_length" value="0.85"/>  <!-- Use positive absolute value -->
-  <xacro:property name="rocker_height" value="0.05"/>  <!-- Use positive value -->
-  <xacro:property name="rocker_width" value="0.03"/>
-  <xacro:property name="rocker_collision_x_offset" value="-0.10"/>
-  <xacro:property name="rocker_collision_z_offset" value="-0.2"/>
-  <!-- LEFT ROCKER LINK -->
-  <link name="${prefix}left_rocker">
+  <!-- ROCKER LINK -->
+  <xacro:macro name="rocker" params="prefix:=^ side:=^">
+  <link name="${prefix}${side}_rocker">
     <inertial>
-      <origin xyz="${rocker_collision_x_offset} 0.0 ${rocker_collision_z_offset}" rpy="0.0 0.0 0.0"/>
+      <origin xyz="${rocker_collision_x_offset} 0.0 -${rocker_height}" rpy="0.0 0.0 0.0"/>
       <mass value="${rocker_mass}"/>
       <xacro:box_inertia m="${rocker_mass}"
@@ -21,10 +15,14 @@
       <origin xyz="0.0 0.0 0.0" rpy="0.0 0.0 ${pi}"/>
       <geometry>
-        <mesh scale="0.1 0.1 0.1"
-              filename="file://$(find perseus_description)/meshes/rocker_left.dae"/>
+      <xacro:if value="${side == 'left'}">
+        <mesh scale="0.1 0.1 0.1" filename="file://$(find perseus_description)/meshes/rocker_left.dae"/>
+      </xacro:if>
+      <xacro:if value="${side == 'right'}">
+        <mesh scale="0.1 0.1 0.1" filename="file://$(find perseus_description)/meshes/rocker_right.dae"/>
+      </xacro:if>
       </geometry>
     </visual>
     <collision>
-      <origin xyz="${rocker_collision_x_offset} 0.0 ${rocker_collision_z_offset}" rpy="0.0 0.0 0.0"/>
+      <origin xyz="${rocker_collision_x_offset} 0.0 -${rocker_height}" rpy="0.0 0.0 0.0"/>
       <geometry>
         <box size="${rocker_length} ${rocker_width} ${rocker_height}"/>
@@ -32,27 +30,17 @@
     </collision>
   </link>
-  <!-- RIGHT ROCKER LINK -->
-  <link name="${prefix}right_rocker">
-    <inertial>
-      <origin xyz="${rocker_collision_x_offset} 0.0 ${rocker_collision_z_offset}" rpy="0.0 0.0 0.0"/>
-      <mass value="${rocker_mass}"/>
-      <xacro:box_inertia m="${rocker_mass}"
-                         x="${rocker_length}"
-                         y="${rocker_width}"
-                         z="${rocker_height}"/>
-    </inertial>
-    <visual>
-      <origin xyz="0.0 0.0 0.0" rpy="0.0 0.0 ${pi}"/>
-      <geometry>
-        <mesh scale="0.1 0.1 0.1"
-              filename="file://$(find perseus_description)/meshes/rocker_right.dae"/>
-      </geometry>
-    </visual>
-    <collision>
-      <origin xyz="${rocker_collision_x_offset} 0.0 ${rocker_collision_z_offset}" rpy="0.0 0.0 0.0"/>
-      <geometry>
-        <box size="${rocker_length} ${rocker_width} ${rocker_height}"/>
-      </geometry>
-    </collision>
-  </link>
+  <joint name="${prefix}${side}_rocker_joint" type="fixed">
+    <xacro:if value="${side == 'left'}">
+      <origin xyz="${-rocker_x_offset} ${rocker_base_distance} ${rocker_y_offset} " rpy="0 0 0"/>
+    </xacro:if>
+    <xacro:if value="${side == 'right'}">
+      <origin xyz="${-rocker_x_offset} -${rocker_base_distance} ${rocker_y_offset} " rpy="0 0 0"/>
+    </xacro:if>
+    <parent link="${prefix}chassis"/>
+    <child link="${prefix}${side}_rocker"/>
+  </joint>
+  <!-- ADD 2 MOTORS FOR EACH SIDE -->
+  <xacro:motor prefix="" side="${side}"  end="front"/>
+  <xacro:motor prefix="" side="${side}"  end="rear"/>
+  </xacro:macro>
 </robot>

File: software/ros_ws/src/perseus_description/urdf/wheel.urdf.xacro (robot description, xacro)
@@ -76,7 +76,7 @@
   </gazebo>
 </xacro:macro>
-<xacro:wheel prefix="" side="left"  end="front"/>
+<!-- <xacro:wheel prefix="" side="left"  end="front"/>
 <xacro:wheel prefix="" side="left"  end="rear"/>
 <xacro:wheel prefix="" side="right" end="front"/>
-<xacro:wheel prefix="" side="right" end="rear"/>
+<xacro:wheel prefix="" side="right" end="rear"/> -->
 </robot>

Commit message: Remove unnecessary properties for motor mass and collision dimensions in motor_wheel.urdf.xacro

File: software/ros_ws/src/perseus_description/urdf/motor_wheel.urdf.xacro (robot description, xacro)
@@ -1,8 +1,4 @@
 <?xml version="1.0"?>
 <robot name="motor_wheel" xmlns:xacro="http://www.ros.org/wiki/xacro">
-  <xacro:property name="motor_mass" value="5.236579"/>  <!-- Kg -->
-  <xacro:property name="collision_motor_length" value="0.1"/>  <!-- m -->
-  <xacro:property name="collision_motor_width" value="0.1"/>  <!-- m -->
-  <xacro:property name="collision_motor_height" value="0.075"/>  <!-- m -->
   <xacro:macro name="motor" params="prefix:=^ side:=^ end:=^">
     <link name="${prefix}${end}_${side}_motor">
