Commit message: Fix wheel and motor orientation for left and right sides in URDF files to ensure correct simulation behavior.

File: software/ros_ws/src/perseus_description/urdf/motor_wheel.urdf.xacro (robot description, xacro)
@@ -11,8 +11,8 @@
       <visual>
         <xacro:if value="${side == 'left'}">
-          <origin xyz="0 0.0 0.0" rpy="0.0 0.0 ${pi/2}"/>
+          <origin xyz="0 0.0 0.0" rpy="0.0 0.0 ${-pi/2}"/>
         </xacro:if>
         <xacro:if value="${side == 'right'}">
-          <origin xyz="0 0.0 0.0" rpy="0.0 0.0 ${-pi/2}"/>
+          <origin xyz="0 0.0 0.0" rpy="0.0 0.0 ${pi/2}"/>
         </xacro:if>
         <geometry>

File: software/ros_ws/src/perseus_description/urdf/wheel.urdf.xacro (robot description, xacro)
@@ -8,5 +8,5 @@
       </xacro:if>
       <xacro:if value="${side == 'right'}">
-        <origin xyz="0.0 0.0  0.0" rpy="0.0 0.0 0.0"/>
+        <origin xyz="0.0 0.0  0.0" rpy="0.0 0.0 -${pi}"/>
       </xacro:if>
       <mass value="${wheel_mass}"/>
@@ -18,5 +18,5 @@
       </xacro:if>
       <xacro:if value="${side == 'right'}">
-        <origin xyz="0.0 0.0  0.0" rpy="0.0 0.0 0.0"/>
+        <origin xyz="0.0 0.0  0.0" rpy="0.0 0.0 -${pi}"/>
       </xacro:if>
       <geometry>
@@ -29,5 +29,5 @@
       </xacro:if>
         <xacro:if value="${side == 'right'}">
-      <origin xyz="0.0 0.0 0.0" rpy="${pi/2} 0.0 0.0"/>
+      <origin xyz="0.0 0.0 0.0" rpy="${pi/2} 0.0 -${pi}"/>
       </xacro:if>
       <geometry>
@@ -61,5 +61,5 @@
                   so that the rover can turn (skid steer) -->
                   <!-- forward coefficient of friction -->
-                  <mu>0.3</mu>
+                  <mu>100</mu>
                   <!-- perpendicular coefficient of friction -->
                   <mu2>1</mu2>
