Commit message: Made URDF REP-103/REP-105 aligned,ready for Nav2 integration
- wheel.urdf.xacro - Unified wheel axis to -Y for REP-103 compliance (positive velocity = forward)
- inertia_macros.xacro - Added cylinder_inertia_y macro for Y-axis aligned cylinders
- wheel.urdf.xacro - using cylinder inertia, and friction tuned [mu=1.5, mu2=0.2]
- xbox_controller.py - Negated joystick axes for ROS convention, removed conditional rotation inversion
- All controller YAMLs - Negative scaling for forward/turn to match ROS convention

File: software/ros_ws/src/perseus_description/urdf/inertia_macros.xacro (robot description, xacro)
@@ -9,5 +9,5 @@
       ixy="0" iyz="0" ixz="0"/>
   </xacro:macro>
-  <!-- Cylinder inertia macro -->
+  <!-- Cylinder inertia macro (axis along Z) -->
   <xacro:macro name="cylinder_inertia" params="m radius length">
     <inertia
@@ -15,4 +15,12 @@
       iyy="${m*(3*radius*radius+length*length)/12}"
       izz="${m*radius*radius/2}"
+      ixy="0" iyz="0" ixz="0"/>
+  </xacro:macro>
+  <!-- Cylinder inertia macro (axis along Y) - use for wheels -->
+  <xacro:macro name="cylinder_inertia_y" params="m radius length">
+    <inertia
+      ixx="${m*(3*radius*radius+length*length)/12}"
+      iyy="${m*radius*radius/2}"
+      izz="${m*(3*radius*radius+length*length)/12}"
       ixy="0" iyz="0" ixz="0"/>
   </xacro:macro>

File: software/ros_ws/src/perseus_description/urdf/wheel.urdf.xacro (robot description, xacro)
@@ -4,31 +4,24 @@
   <link name="${prefix}${end}_${side}_wheel">
     <inertial>
+      <origin xyz="0.0 0.0 0.0" rpy="0.0 0.0 0.0"/>
+      <mass value="${wheel_mass}"/>
+      <!-- Use Y-axis aligned cylinder inertia since wheels rotate around Y axis -->
+      <xacro:cylinder_inertia_y m="${wheel_mass}" radius="${wheel_radius}" length="${wheel_length}"/>
+    </inertial>
+    <visual>
+      <!-- Rotate mesh so tread pattern faces outward -->
       <xacro:if value="${side == 'left'}">
-        <origin xyz="0.0 0.0  0.0" rpy="0.0 0.0 ${pi}"/>
+        <origin xyz="0.0 0.0 0.0" rpy="0.0 0.0 ${pi}"/>
       </xacro:if>
       <xacro:if value="${side == 'right'}">
-        <origin xyz="0.0 0.0  0.0" rpy="0.0 0.0 -${pi}"/>
-      </xacro:if>
-      <mass value="${wheel_mass}"/>
-      <xacro:cylinder_inertia m="${wheel_mass}" radius="${wheel_radius}" length="${wheel_length}"/>
-    </inertial>
-    <visual>
-      <xacro:if value="${side == 'left'}">
-        <origin xyz="0.0 0.0  0.0" rpy="0.0 0.0 ${pi}"/>
-      </xacro:if>
-      <xacro:if value="${side == 'right'}">
-        <origin xyz="0.0 0.0  0.0" rpy="0.0 0.0 -${pi}"/>
+        <origin xyz="0.0 0.0 0.0" rpy="0.0 0.0 0.0"/>
       </xacro:if>
       <geometry>
-        <mesh scale="0.1 0.1  0.1" filename="file://$(find perseus_description)/meshes/wheel.dae"/>
+        <mesh scale="0.1 0.1 0.1" filename="file://$(find perseus_description)/meshes/wheel.dae"/>
       </geometry>
     </visual>
     <collision>
-      <xacro:if value="${side == 'left'}">
-        <origin xyz="0.0 0.0 0.0" rpy="${pi/2} 0.0 ${pi}"/>
-      </xacro:if>
-        <xacro:if value="${side == 'right'}">
-      <origin xyz="0.0 0.0 0.0" rpy="${pi/2} 0.0 -${pi}"/>
-      </xacro:if>
+      <!-- Rotate cylinder 90° around X to align with Y axis (wheel axle) -->
+      <origin xyz="0.0 0.0 0.0" rpy="${pi/2} 0.0 0.0"/>
       <geometry>
         <cylinder radius="${wheel_radius}" length="${wheel_length}"/>
@@ -37,15 +30,15 @@
   </link>
   <joint name="${prefix}${end}_${side}_wheel_joint" type="continuous">
+    <parent link="${prefix}${end}_${side}_motor"/>
+    <child link="${prefix}${end}_${side}_wheel"/>
     <xacro:if value="${side == 'left'}">
-      <origin xyz="0 ${wheels_y_offset} 0.0" rpy="0.0 0.0 0"/>
-      <axis xyz="0 1 0" rpy="0 0 0"/>
+      <origin xyz="0.0 ${wheels_y_offset} 0.0" rpy="0.0 0.0 0.0"/>
     </xacro:if>
     <xacro:if value="${side == 'right'}">
-      <origin xyz="0 ${-wheels_y_offset} 0.0" rpy="0.0 0.0 ${pi}"/>
-      <axis xyz="0 -1 0" rpy="0 0 0"/>
+      <origin xyz="0.0 ${-wheels_y_offset} 0.0" rpy="0.0 0.0 0.0"/>
     </xacro:if>
+    <!-- Axis -Y: positive velocity = forward motion (standard ROS/diff_drive convention) -->
+    <axis xyz="0 -1 0"/>
     <dynamics damping="0.2" friction="0.3"/>
-    <parent link="${prefix}${end}_${side}_motor"/>
-    <child link="${prefix}${end}_${side}_wheel"/>
   </joint>
   <gazebo reference="${prefix}${end}_${side}_wheel">
@@ -58,15 +51,14 @@
               <ode>
                   <!--
-                  In this case, the wheels need lower sideways than forwards coefficients of friction
-                  so that the rover can turn (skid steer) -->
-                  <!-- forward coefficient of friction -->
-                  <mu>100</mu>
-                  <!-- perpendicular coefficient of friction -->
-                  <mu2>1</mu2>
-                  <!--
-                  However, since mu/mu2 are normally relative to world coordinates,
-                  the rover would only be able to turn 90 degrees either way before they swapped, making turning impossible.
-                  To solve this, we need to specify the direction that mu/mu2 are relative to.
+                  Skid-steer friction setup:
+                  - mu: friction in fdir1 direction (forward/backward rolling)
+                  - mu2: friction perpendicular to fdir1 (sideways sliding for turning)
+                  - fdir1: primary friction direction in link frame
                   -->
+                  <!-- Forward/backward friction - high to grip and drive -->
+                  <mu>1.5</mu>
+                  <!-- Sideways friction - low to allow skid steering -->
+                  <mu2>0.2</mu2>
+                  <!-- fdir1 points forward (X) in link frame -->
                   <fdir1>1 0 0</fdir1>
               </ode>
