Commit message: persues_simulation: addded readme and tuned wheel attributes
- Lowered friction to allow for turning
- Added a very basic readme with basic commands

File: software/ros_ws/src/perseus_description/urdf/wheel.urdf.xacro (robot description, xacro)
@@ -6,5 +6,5 @@
         <origin xyz="0.0 0.0 0.0" rpy="0.0 0.0 0.0"/>
         <mass value="1.0"/>
-        <inertia ixx="0.051473" iyy="0.029155" izz="0.029154" ixy="0.0" iyz="0.0" ixz="0.0"/>
+        <inertia ixx="0.04" iyy="0.02" izz="0.02" ixy="0.0" iyz="0.0" ixz="0.0"/>
       </inertial>
       <visual>
@@ -19,4 +19,9 @@
           <cylinder length="0.115" radius="0.145" />
         </geometry>
+        <contact>
+          <lateral_friction value="0.8"/>
+          <rolling_friction value="0.1"/>
+          <spinning_friction value="0.1"/>
+        </contact>
       </collision>
     </link>
@@ -31,5 +36,5 @@
       <child link="${prefix}${end}_${side}_wheel"/>
       <origin xyz="-0.125 0.0 0.0" rpy="0.0 0.0 ${-pi/2}"/>
-      <dynamics damping="1.0" friction="1.0"/>
+      <dynamics damping="0.2" friction="0.3"/>
     </joint>
   </xacro:macro>

Commit message: fix: Correctly define simulated wheel friction

File: software/ros_ws/src/perseus_description/urdf/wheel.urdf.xacro (robot description, xacro)
@@ -19,11 +19,33 @@
           <cylinder length="0.115" radius="0.145" />
         </geometry>
-        <contact>
-          <lateral_friction value="0.8"/>
-          <rolling_friction value="0.1"/>
-          <spinning_friction value="0.1"/>
-        </contact>
       </collision>
     </link>
+    <!-- we need to use the gazebo tag to add in properties normally only found in SDF files -->
+    <gazebo reference="${prefix}${end}_${side}_wheel">
+      <!-- TODO: Fix the material tag (this isn't the proper way to do it, and spits out warnings) -->
+      <material>Gazebo/Orange</material>
+      <!-- see http://sdformat.org/spec?ver=1.12&elem=collision -->
+      <collision>
+        <surface>
+            <friction>
+                <ode>
+                    <!--
+                    In this case, the wheels need lower sideways than forwards coefficients of friction
+                    so that the rover can turn (skid steer) -->
+                    <!-- forward coefficient of friction -->
+                    <mu>1</mu>
+                    <!-- perpendicular coefficient of friction -->
+                    <mu2>0.3</mu2>
+                    <!--
+                    However, since mu/mu2 are normally relative to world coordinates,
+                    the rover would only be able to turn 90 degrees either way before they swapped, making turning impossible.
+                    To solve this, we need to specify the direction that mu/mu2 are relative to.
+                    -->
+                    <fdir1>1 0 0</fdir1>
+                </ode>
+            </friction>
+        </surface>
+      </collision>
+    </gazebo>
     <joint name="${prefix}${end}_${side}_wheel_joint" type="continuous">
       <xacro:if value="${side == 'left'}">

Commit message: refactor: Update wheel URDF properties and adjust origin positions for left and right wheels

File: software/ros_ws/src/perseus_description/urdf/wheel.urdf.xacro (robot description, xacro)
@@ -2,12 +2,27 @@
 <robot name="wheel" xmlns:xacro="http://ros.org/wiki/xacro">
   <xacro:macro name="wheel" params="prefix:=^ side:=^ end:=^">
+    <!-- WHEEL PROPERTIES -->
+      <xacro:property name="track_width" value="0.1" />
+      <xacro:property name="wheel_radius" value="0.05" />
+      <xacro:property name="wheel_mass" value="1.0" />
+      <xacro:property name="wheel_base" value="1.0" />
     <link name="${prefix}${end}_${side}_wheel">
       <inertial>
-        <origin xyz="0.0 0.0 0.0" rpy="0.0 0.0 0.0"/>
+        <xacro:if value="${side == 'left'}">
+          <origin xyz="0.0 0.125  0.0" rpy="0.0 0.0 0"/>
+        </xacro:if>
+        <xacro:if value="${side == 'right'}">
+          <origin xyz="0.0 -0.125  0.0" rpy="0.0 0.0 0.0"/>
+        </xacro:if>
         <mass value="1.0"/>
         <inertia ixx="0.04" iyy="0.02" izz="0.02" ixy="0.0" iyz="0.0" ixz="0.0"/>
       </inertial>
       <visual>
-        <origin xyz="0.0 0.0 0.0" rpy="0.0 0.0 0.0"/>
+        <xacro:if value="${side == 'left'}">
+          <origin xyz="0.0 0.125  0.0" rpy="0.0 0.0 ${pi}"/>
+        </xacro:if>
+        <xacro:if value="${side == 'right'}">
+          <origin xyz="0.0 -0.125  0.0" rpy="0.0 0.0 0.0"/>
+        </xacro:if>
         <geometry>
           <mesh scale="0.1 0.1 0.1" filename="file://$(find perseus_description)/meshes/wheel.dae"/>
@@ -15,7 +30,12 @@
       </visual>
       <collision>
-        <origin xyz="0.0 -0.015 0.0" rpy="1.570796 0.0 0.0"/>
+        <xacro:if value="${side == 'left'}">
+          <origin xyz="0.0 0.0 0.0" rpy="0.0 0.0 ${pi}"/>
+        </xacro:if>
+        <xacro:if value="${side == 'right'}">
+          <origin xyz="0.0 0.0 0.0" rpy="0.0 0.0 0.0"/>
+        </xacro:if>
         <geometry>
-          <cylinder length="0.115" radius="0.145" />
+          <mesh scale="0.1 0.1 0.1" filename="file://$(find perseus_description)/meshes/wheel.dae"/>
         </geometry>
       </collision>
@@ -57,5 +77,5 @@
       <parent link="${prefix}${end}_${side}_motor"/>
       <child link="${prefix}${end}_${side}_wheel"/>
-      <origin xyz="-0.125 0.0 0.0" rpy="0.0 0.0 ${-pi/2}"/>
+      <origin xyz="0.0 0 0.0" rpy="0.0 0.0 0"/>
       <dynamics damping="0.2" friction="0.3"/>
     </joint>

Commit message: fix: Correct axis direction for right wheel in URDF definition

File: software/ros_ws/src/perseus_description/urdf/wheel.urdf.xacro (robot description, xacro)
@@ -73,5 +73,5 @@
       </xacro:if>
       <xacro:if value="${side == 'right'}">
-        <axis xyz="0 -1 0" rpy="0 0 0"/>
+        <axis xyz="0 1 0" rpy="0 0 0"/>
       </xacro:if>
       <parent link="${prefix}${end}_${side}_motor"/>

Commit message: fix: Correct wheel joint axis and origin orientation for right side

File: software/ros_ws/src/perseus_description/urdf/wheel.urdf.xacro (robot description, xacro)
@@ -53,9 +53,9 @@
       </xacro:if>
       <xacro:if value="${side == 'right'}">
-        <axis xyz="0 -1 0" rpy="0 0 0"/>
+        <axis xyz="0 1 0" rpy="0 0 0"/>
       </xacro:if>
       <parent link="${prefix}${end}_${side}_motor"/>
       <child link="${prefix}${end}_${side}_wheel"/>
-      <origin xyz="-0.125 0.0 0.0" rpy="0.0 0.0 ${-pi/2}"/>
+      <origin xyz="-0.125 0.0 0.0" rpy="0.0 0.0 0"/>
       <dynamics damping="0.2" friction="0.3"/>
     </joint>

Commit message: fix: Correct wheel joint axis and origin orientation for right side

File: software/ros_ws/src/perseus_description/urdf/wheel.urdf.xacro (robot description, xacro)
@@ -77,5 +77,5 @@
       <parent link="${prefix}${end}_${side}_motor"/>
       <child link="${prefix}${end}_${side}_wheel"/>
-      <origin xyz="0.0 0 0.0" rpy="0.0 0.0 0"/>
+      <origin xyz="0.125 0.0 0.0" rpy="0.0 0.0 0"/>
       <dynamics damping="0.2" friction="0.3"/>
     </joint>

Commit message: fix: Update joint origin position for wheel to correct alignment

File: software/ros_ws/src/perseus_description/urdf/wheel.urdf.xacro (robot description, xacro)
@@ -77,5 +77,5 @@
       <parent link="${prefix}${end}_${side}_motor"/>
       <child link="${prefix}${end}_${side}_wheel"/>
-      <origin xyz="-0.125 0.0 0.0" rpy="0.0 0.0 0"/>
+      <origin xyz="0 0 0.0" rpy="0.0 0.0 0"/>
       <dynamics damping="0.2" friction="0.3"/>
     </joint>

Commit message: corrected URDF, generic and xbox controller and the telop diag TUI

File: software/ros_ws/src/perseus_description/urdf/wheel.urdf.xacro (robot description, xacro)
@@ -38,6 +38,6 @@
       <origin xyz="0.0 ${-wheels_y_offset} 0.0" rpy="0.0 0.0 0.0"/>
     </xacro:if>
-    <!-- Axis -Y: positive velocity = forward motion (standard ROS/diff_drive convention) -->
-    <axis xyz="0 -1 0"/>
+    <!-- Axis +Y: positive velocity = forward motion (ROS REP-103 convention) -->
+    <axis xyz="0 1 0"/>
     <dynamics damping="0.2" friction="0.3"/>
   </joint>
