Commit message: perseus_description: added the m2m2 lidar to the xacro

File: software/ros_ws/src/perseus_description/urdf/sensors.urdf.xacro (robot description, xacro)
@@ -20,4 +20,32 @@
         <child link="${prefix}laser_frame"/>
         <origin xyz="0 0 0.23" rpy="0 0 0"/>
+    </joint>
+    <!-- M2M2 Lidar -->
+    <link name="${prefix}m2m2_lidar_frame">
+        <inertial>
+            <mass value="0.165"/>
+            <origin xyz="0 0 0" rpy="0 0 0"/>
+            <inertia ixx="0.0001" ixy="0" ixz="0"
+                     iyy="0.0001" iyz="0"
+                     izz="0.0001"/>
+        </inertial>
+        <visual>
+            <origin xyz="0 0 0" rpy="0 0 0"/>
+            <geometry>
+                <box size="0.055 0.055 0.080"/>
+            </geometry>
+            <material name="grey"/>
+        </visual>
+        <collision>
+            <origin xyz="0 0 0" rpy="0 0 0"/>
+            <geometry>
+                <box size="0.055 0.055 0.080"/>
+            </geometry>
+        </collision>
+    </link>
+    <joint name="${prefix}m2m2_lidar_joint" type="fixed">
+        <parent link="${prefix}base_link"/>
+        <child link="${prefix}m2m2_lidar_frame"/>
+        <origin xyz="0.2 0.4 0.35" rpy="0 0 0"/>
     </joint>
     <gazebo reference="${prefix}laser_frame">

Commit message: fix: Rotate m2m2 90deg CW

File: software/ros_ws/src/perseus_description/urdf/sensors.urdf.xacro (robot description, xacro)
@@ -47,5 +47,5 @@
         <parent link="${prefix}base_link"/>
         <child link="${prefix}m2m2_lidar_frame"/>
-        <origin xyz="0.2 0.4 0.35" rpy="0 0 0"/>
+        <origin xyz="0.2 0.4 0.35" rpy="0 0 -1.57"/>
     </joint>
     <gazebo reference="${prefix}laser_frame">

Commit message: feat: Livox config + URDF

File: software/ros_ws/src/perseus_description/urdf/sensors.urdf.xacro (robot description, xacro)
@@ -49,4 +49,31 @@
         <origin xyz="0.2 0.4 0.35" rpy="0 0 0"/>
     </joint>
+        <link name="${prefix}livox_frame">
+        <inertial>
+            <mass value="0.165"/>
+            <origin xyz="0 0 0" rpy="0 0 0"/>
+            <inertia ixx="0.0001" ixy="0" ixz="0"
+                     iyy="0.0001" iyz="0"
+                     izz="0.0001"/>
+        </inertial>
+        <visual>
+            <origin xyz="0 0 0" rpy="0 0 0"/>
+            <geometry>
+                <box size="0.055 0.055 0.080"/>
+            </geometry>
+            <material name="grey"/>
+        </visual>
+        <collision>
+            <origin xyz="0 0 0" rpy="0 0 0"/>
+            <geometry>
+                <box size="0.055 0.055 0.080"/>
+            </geometry>
+        </collision>
+    </link>
+    <joint name="${prefix}livox_joint" type="fixed">
+        <parent link="${prefix}base_link"/>
+        <child link="${prefix}livox_frame"/>
+	<origin xyz="0.8 0 1.1" rpy="${pi} 0 0"/>
+    </joint>
     <gazebo reference="${prefix}m2m2_lidar_frame">
         <material>Gazebo/Black</material>

Commit message: fix: Update laser frame material and joint parent link

File: software/ros_ws/src/perseus_description/urdf/sensors.urdf.xacro (robot description, xacro)
@@ -8,5 +8,5 @@
                 <cylinder radius="0.06" length="0.06"/>
             </geometry>
-            <material name="black"/>
+            <material name="red"/>
         </visual>
         <collision>
@@ -17,7 +17,7 @@
     </link>
     <joint name="${prefix}laser_joint" type="fixed">
-        <parent link="${prefix}chassis"/>
+        <parent link="${prefix}base_link"/>
         <child link="${prefix}laser_frame"/>
-        <origin xyz="0 0 0.23" rpy="0 0 0"/>
+        <origin xyz="0.220 0 0.4" rpy="0 0 0"/>
     </joint>
     <link name="${prefix}m2m2_lidar_frame">
@@ -75,6 +75,6 @@
 	<origin xyz="0.8 0 1.1" rpy="${pi} 0 0"/>
     </joint>
-    <gazebo reference="${prefix}m2m2_lidar_frame">
-        <material>Gazebo/Black</material>
+    <gazebo reference="${prefix}laser_frame">
+        <material>Gazebo/Red</material>
         <sensor name="laser" type="gpu_lidar">
             <pose>0 0 0 0 0 0</pose>

Commit message: fix: Correct laser joint origin height in URDF

File: software/ros_ws/src/perseus_description/urdf/sensors.urdf.xacro (robot description, xacro)
@@ -19,5 +19,5 @@
         <parent link="${prefix}base_link"/>
         <child link="${prefix}laser_frame"/>
-        <origin xyz="0.220 0 0.4" rpy="0 0 0"/>
+        <origin xyz="0.220 0 0.6" rpy="0 0 0"/>
     </joint>
     <link name="${prefix}m2m2_lidar_frame">

Commit message: fix: update navigation parameters and include waypoints bridge for improved robot control and simulation

File: software/ros_ws/src/perseus_description/urdf/sensors.urdf.xacro (robot description, xacro)
@@ -117,13 +117,26 @@
 </gazebo>
 <gazebo reference="${prefix}livox_frame">
-    <material>Gazebo/Grey</material>
-    <sensor name="${prefix}lidar_imu" type="imu">
-        <always_on>1</always_on>
-        <update_rate>10</update_rate>
-        <visualize>true</visualize>
-        <topic>scan_3d/imu</topic>
-        <!-- Add frame id to imu sensor (achieving correct frame association)-->
-        <gz_frame_id>${prefix}livox_frame</gz_frame_id>
-    </sensor>
+  <material>Gazebo/Grey</material>
+  <sensor name="${prefix}lidar_imu" type="imu">
+    <always_on>1</always_on>
+    <update_rate>200</update_rate>
+    <visualize>true</visualize>
+    <topic>scan_3d/imu</topic>
+    <gz_frame_id>${prefix}livox_frame</gz_frame_id>
+    <imu>
+      <angular_velocity>
+        <z>
+          <noise type="gaussian">
+            <!-- white noise -->
+            <mean>0.0</mean>
+            <stddev>0.005512</stddev>
+            <!-- constant bias (offset) -->
+            <bias_mean>-0.015635</bias_mean>
+            <bias_stddev>0.0</bias_stddev>
+          </noise>
+        </z>
+      </angular_velocity>
+    </imu>
+  </sensor>
 </gazebo>
 </robot>
