Commit message: fix: Update camera frame references and transform logic in ArUco detector node

File: software/ros_ws/src/perseus_description/urdf/camera_depth.urdf.xacro (robot description, xacro)
@@ -20,5 +20,5 @@
         <parent link="camera_link"/>
         <child link="camera_link_optical"/>
-        <origin xyz="0 0 0" rpy="${-pi/2} 0 ${-pi/2}"/>
+        <origin xyz="0 0 0" rpy="0 0 0"/>
     </joint>
     <link name="camera_link_optical"></link>

Commit message: feat: disable 2D mode and enable full 3D odometry in EKF configuration

File: software/ros_ws/src/perseus_description/urdf/camera_depth.urdf.xacro (robot description, xacro)
@@ -3,5 +3,4 @@
 <!-- <box size="0.020 0.07 0.03"/>  -->
 <robot name="camera_depth" xmlns:xacro="http://ros.org/wiki/xacro">
-  <xacro:macro name="camera_depth" params="prefix">
     <link name="${prefix}camera_link">
         <visual>
@@ -41,4 +40,3 @@
         </sensor>
     </gazebo>
-  </xacro:macro>
 </robot>

Commit message: Refactor URDF files to improve properties and dimensions for various components, including camera, chassis, flange bearing, rocker, and wheels. Update sensor configurations in gz_bridge.yaml for better topic management.

File: software/ros_ws/src/perseus_description/urdf/camera_depth.urdf.xacro (robot description, xacro)
@@ -1,10 +1,17 @@
 <?xml version="1.0"?>
-<!-- 0.220 0 0.4 -->
-<!-- <box size="0.020 0.07 0.03"/>  -->
 <robot name="camera_depth" xmlns:xacro="http://ros.org/wiki/xacro">
+    <xacro:property name="camera_mass" value="0.1"/>
+    <xacro:property name="camera_width" value="0.07"/>
+    <xacro:property name="camera_height" value="0.03"/>
+    <xacro:property name="camera_depth" value="0.020"/>
     <link name="${prefix}camera_link">
+        <inertial>
+            <origin xyz="0 0 0" rpy="0 0 0"/>
+            <mass value="${camera_mass}"/>
+            <xacro:box_inertia m="${camera_mass}" x="${camera_depth}" y="${camera_width}" z="${camera_height}"/>
+        </inertial>
         <visual>
             <geometry>
-                <box size="0.020 0.07 0.03"/>
+                <box size="${camera_depth} ${camera_width} ${camera_height}"/>
             </geometry>
             <material name="red"/>
@@ -22,5 +29,5 @@
             <pose> 0 0 0 0 0 0 </pose>
             <visualize>true</visualize>
-            <update_rate>100</update_rate>
+            <update_rate>30</update_rate>
             <always_on>true</always_on>
             <camera>
@@ -35,4 +42,5 @@
                 </clip>
             </camera>
+            <topic>/perseus/rgbd_camera</topic>
             <gz_frame_id>${prefix}camera_link_optical</gz_frame_id>
             <min_depth>0.05</min_depth>

File: software/ros_ws/src/perseus_description/urdf/chassis.urdf.xacro (robot description, xacro)
@@ -4,19 +4,19 @@
   <link name="${prefix}chassis">
     <inertial>
-      <origin xyz="${-chassis_length/scale_factor*0.5} 0.0 ${chassis_height/scale_factor*0.5}" rpy="0 0.0 0.0"/>
+      <origin xyz="${-chassis_length*0.5} 0.0 ${chassis_height*0.5}" rpy="0 0.0 0.0"/>
       <mass value="${chassis_mass}"/>
-      <xacro:box_inertia m="${chassis_mass}" x="${chassis_length/scale_factor}" y="${chassis_width/scale_factor}" z="${chassis_height/scale_factor}"/>
+      <xacro:box_inertia m="${chassis_mass}" x="${chassis_length}" y="${chassis_width}" z="${chassis_height}"/>
     </inertial>
     <visual>
       <origin xyz="0.0 0.0 0.0" rpy="0 0.0 -${pi/2}"/>
       <geometry>
-        <mesh scale="${0.1/scale_factor} ${0.1/scale_factor}  ${0.1/scale_factor}" filename="file://$(find perseus_description)/meshes/chassis.dae"/>
+        <mesh scale="${0.1} ${0.1}  ${0.1}" filename="file://$(find perseus_description)/meshes/chassis.dae"/>
       </geometry>
     </visual>
     <collision>
-      <origin xyz="${-chassis_length/scale_factor*0.5} 0.0 ${chassis_height/scale_factor*0.5}" rpy="0 0.0 0"/>
+      <origin xyz="${-chassis_length*0.5} 0.0 ${chassis_height*0.5}" rpy="0 0.0 0"/>
       <!-- Modified to make collision more simple, chassis mesh replaced with box -->
       <geometry>
-        <box size="${chassis_length/scale_factor} ${chassis_width/scale_factor} ${chassis_height/scale_factor}"/>
+        <box size="${chassis_length} ${chassis_width} ${chassis_height}"/>
       </geometry>
     </collision>

File: software/ros_ws/src/perseus_description/urdf/flange_bearing.urdf.xacro (robot description, xacro)
@@ -1,7 +1,8 @@
 <?xml version="1.0"?>
 <robot name="flange_bearing" xmlns:xacro="http://ros.org/wiki/xacro">
-<xacro:property name="bar_length" value="0.5"/>
+<xacro:property name="bar_length" value="0.58"/>
 <xacro:property name="bar_width" value="0.03"/>
 <xacro:property name="bar_height" value="0.03"/>
+<xacro:property name="bar_mass" value="0.917264951812715"/>
 <xacro:property name="bearing_length" value="0.2"/>
 <xacro:property name="bearing_width" value="0.03"/>
@@ -13,10 +14,10 @@
     <origin xyz="0.0 0.0 0.0" rpy="${-pi/2} 0 ${pi/2}"/>
     <mass value="${bearing_mass}"/>
-    <xacro:box_inertia m="${bearing_mass}" x="${bearing_length/scale_factor}" y="${bearing_width/scale_factor}" z="${bearing_height/scale_factor}"/>
+    <xacro:box_inertia m="${bearing_mass}" x="${bearing_length}" y="${bearing_width}" z="${bearing_height}"/>
     </inertial>
     <visual>
     <origin xyz="0.0 0.0 0.0" rpy="${-pi/2} 0 ${pi/2}"/>
     <geometry>
-        <mesh scale="${0.1/scale_factor} ${0.1/scale_factor}  ${0.1/scale_factor}" filename="file://$(find perseus_description)/meshes/flange_bearing.dae"/>
+        <mesh scale="${0.1} ${0.1}  ${0.1}" filename="file://$(find perseus_description)/meshes/flange_bearing.dae"/>
     </geometry>
     </visual>
@@ -24,5 +25,5 @@
     <origin xyz="0.0 0.0 0.0" rpy="${-pi/2} 0 ${pi/2}"/>
     <geometry>
-        <box size="${bar_length/scale_factor} ${bar_width/scale_factor} ${bar_height/scale_factor}"/>
+        <box size="${bar_length} ${bar_width} ${bar_height}"/>
     </geometry>
     </collision>
@@ -32,11 +33,11 @@
     <inertial>
         <origin xyz="0 0 0.0" rpy="0.0 0.0 0.0"/>
-        <mass value="0.9172649518127158"/>
-        <xacro:box_inertia m="${chassis_mass}" x="${chassis_length/scale_factor}" y="${chassis_width/scale_factor}" z="${chassis_height/scale_factor}"/>
+        <mass value="${bar_mass}"/>
+        <xacro:box_inertia m="${bar_mass}" x="${bar_length}" y="${bar_width}" z="${bar_height}"/>
     </inertial>
     <visual>
     <origin xyz="0.0 0.0 0.0" rpy="${-pi/2} 0 ${-pi/2}"/>
     <geometry>
-        <mesh scale="${0.1/scale_factor} ${0.1/scale_factor}  ${0.1/scale_factor}" filename="file://$(find perseus_description)/meshes/differential_bar.dae"/>
+        <mesh scale=  "${0.1} ${0.1}  ${0.1}" filename="file://$(find perseus_description)/meshes/differential_bar.dae"/>
     </geometry>
     </visual>
@@ -44,10 +45,10 @@
     <origin xyz="0.0 0.0 0.0" rpy="${-pi/2} 0 ${-pi/2}"/>
     <geometry>
-        <box size="${bar_length/scale_factor} ${bar_width/scale_factor} ${bar_height/scale_factor}"/>
+        <box size="${bar_length} ${bar_width} ${bar_height}"/>
     </geometry>
     </collision>
 </link>
 <joint name="${prefix}differential_bar_joint" type="fixed">
-    <origin xyz="${-0.05/scale_factor} 0.0 0.0" rpy="0 0.0 0"/>
+    <origin xyz="${-0.05} 0.0 0.0" rpy="0 0.0 0"/>
     <axis xyz="0.0 0.0 1.0"/>
     <parent link="${prefix}flange_bearing"/>

File: software/ros_ws/src/perseus_description/urdf/motor_wheel.urdf.xacro (robot description, xacro)
@@ -15,5 +15,5 @@
       <origin xyz="0 0.0 0.0" rpy="0.0 0.0 ${pi/2}"/>
       <geometry>
-        <mesh scale="${0.1/scale_factor} ${0.1/scale_factor}  ${0.1/scale_factor}" filename="file://$(find perseus_description)/meshes/gearbox.dae"/>
+        <mesh scale="${0.1} ${0.1}  ${0.1}" filename="file://$(find perseus_description)/meshes/gearbox.dae"/>
       </geometry>
       <!-- <material name="white"/> -->
@@ -22,5 +22,5 @@
       <origin xyz="0.0 0.0 0.0" rpy="0.0 0.0 ${pi/2}"/>
       <geometry>
-        <box size="${collision_motor_length/scale_factor} ${collision_motor_width/scale_factor} ${collision_motor_height/scale_factor}" />
+        <box size="${collision_motor_length} ${collision_motor_width} ${collision_motor_height}" />
       </geometry>
     </collision>
@@ -36,5 +36,5 @@
       <origin xyz="0 0.0 0.0" rpy="0.0 0.0 ${pi/2}"/>
       <geometry>
-        <mesh scale="${0.1/scale_factor} ${0.1/scale_factor}  ${0.1/scale_factor}" filename="file://$(find perseus_description)/meshes/gearbox.dae"/>
+        <mesh scale="${0.1} ${0.1}  ${0.1}" filename="file://$(find perseus_description)/meshes/gearbox.dae"/>
       </geometry>
       <!-- <material name="white"/> -->
@@ -43,5 +43,5 @@
       <origin xyz="0.0 0.0 0.0" rpy="0.0 0.0 ${pi/2}"/>
       <geometry>
-        <box size="${collision_motor_length/scale_factor} ${collision_motor_width/scale_factor} ${collision_motor_height/scale_factor}" />
+        <box size="${collision_motor_length} ${collision_motor_width} ${collision_motor_height}" />
       </geometry>
     </collision>
@@ -57,5 +57,5 @@
       <origin xyz="0 0.0 0.0" rpy="0.0 0.0 ${-pi/2}"/>
       <geometry>
-        <mesh scale="${0.1/scale_factor} ${0.1/scale_factor}  ${0.1/scale_factor}" filename="file://$(find perseus_description)/meshes/gearbox.dae"/>
+        <mesh scale="${0.1} ${0.1}  ${0.1}" filename="file://$(find perseus_description)/meshes/gearbox.dae"/>
       </geometry>
       <!-- <material name="white"/> -->
@@ -64,5 +64,5 @@
       <origin xyz="0 0.0 0.0" rpy="0.0 0.0 ${-pi/2}"/>
       <geometry>
-        <box size="${collision_motor_length/scale_factor} ${collision_motor_width/scale_factor} ${collision_motor_height/scale_factor}" />
+        <box size="${collision_motor_length} ${collision_motor_width} ${collision_motor_height}" />
       </geometry>
     </collision>
@@ -78,5 +78,5 @@
       <origin xyz="0 0.0 0.0" rpy="0.0 0.0 ${-pi/2}"/>
       <geometry>
-        <mesh scale="${0.1/scale_factor} ${0.1/scale_factor}  ${0.1/scale_factor}" filename="file://$(find perseus_description)/meshes/gearbox.dae"/>
+        <mesh scale="${0.1} ${0.1}  ${0.1}" filename="file://$(find perseus_description)/meshes/gearbox.dae"/>
       </geometry>
       <!-- <material name="white"/> -->
@@ -85,5 +85,5 @@
       <origin xyz="0 0.0 0.0" rpy="0.0 0.0 ${-pi/2}"/>
       <geometry>
-        <box size="${collision_motor_length/scale_factor} ${collision_motor_width/scale_factor} ${collision_motor_height/scale_factor}" />
+        <box size="${collision_motor_length} ${collision_motor_width} ${collision_motor_height}" />
       </geometry>
     </collision>

File: software/ros_ws/src/perseus_description/urdf/perseus.urdf.xacro (robot description, xacro)
@@ -3,6 +3,4 @@
   <xacro:macro name="perseus" params="prefix">
     <!-- Constants for robot dimensions -->
-    <xacro:property name="scale_factor" value="1"/>  <!-- 1 for Perseus and 2 for Perseu_Lite -->
-    <xacro:property name="PI" value="3.1415926535897931"/>
     <!-- Chassis Properties -->
     <xacro:property name="base_mass" value="0.3" /> <!-- arbitrary value for base mass -->
@@ -39,20 +37,20 @@
     <link name="${prefix}base_link"/>
     <joint name="${prefix}chassis_joint" type="fixed"> <!-- Joint Connect base_link and chassis -->
-      <origin xyz="0 0.0 ${chassis_z_offset/scale_factor}" rpy="0.0 0.0 0.0"/>
+      <origin xyz="0 0.0 ${chassis_z_offset}" rpy="0.0 0.0 0.0"/>
       <parent link="${prefix}base_link"/>
       <child link="${prefix}chassis"/>
     </joint>
     <joint name="${prefix}flange_bearing_joint" type="fixed">
-      <origin xyz="${-chassis_length/scale_factor} 0.0 ${flange_bearing_z_offset/scale_factor}" rpy="0 0 0"/>
+      <origin xyz="${-chassis_length} 0.0 ${flange_bearing_z_offset}" rpy="0 0 0"/>
       <parent link="${prefix}chassis"/>
       <child link="${prefix}flange_bearing"/>
     </joint>
     <joint name="${prefix}left_rocker_joint" type="fixed">
-      <origin xyz="${-rocker_x_offset/scale_factor} ${rocker_base_distance/scale_factor} ${rocker_y_offset/scale_factor} " rpy="0 0 0"/>
+      <origin xyz="${-rocker_x_offset} ${rocker_base_distance} ${rocker_y_offset} " rpy="0 0 0"/>
       <parent link="${prefix}chassis"/>
       <child link="${prefix}left_rocker"/>
     </joint>
     <joint name="${prefix}right_rocker_joint" type="fixed">
-      <origin xyz="${-rocker_x_offset/scale_factor} ${-rocker_base_distance/scale_factor} ${rocker_y_offset/scale_factor} " rpy="0 0 0"/>
+      <origin xyz="${-rocker_x_offset} ${-rocker_base_distance} ${rocker_y_offset} " rpy="0 0 0"/>
       <parent link="${prefix}chassis"/>
       <child link="${prefix}right_rocker"/>
@@ -61,20 +59,20 @@
       <parent link="${prefix}left_rocker"/>
       <child link="${prefix}front_left_motor"/>
-      <origin xyz="${front_motors_x_offset/scale_factor} -${motors_y_offset/scale_factor} ${motors_z_offset/scale_factor}" rpy="0.0 0.0 0"/>
+      <origin xyz="${front_motors_x_offset} -${motors_y_offset} ${motors_z_offset}" rpy="0.0 0.0 0"/>
     </joint>
     <joint name="${prefix}rear_left_motor_joint" type="fixed">
       <parent link="${prefix}left_rocker"/>
       <child link="${prefix}rear_left_motor"/>
-      <origin xyz="${rear_motors_x_offset/scale_factor} -${motors_y_offset/scale_factor} ${motors_z_offset/scale_factor}" rpy="0.0 0.0 0.0"/>
+      <origin xyz="${rear_motors_x_offset} -${motors_y_offset} ${motors_z_offset}" rpy="0.0 0.0 0.0"/>
     </joint>
     <joint name="${prefix}front_right_motor_joint" type="fixed">
       <parent link="${prefix}right_rocker"/>
       <child link="${prefix}front_right_motor"/>
-      <origin xyz="${front_motors_x_offset/scale_factor} ${motors_y_offset/scale_factor} ${motors_z_offset/scale_factor}" rpy="0.0 0.0 0"/>
+      <origin xyz="${front_motors_x_offset} ${motors_y_offset} ${motors_z_offset}" rpy="0.0 0.0 0"/>
     </joint>
     <joint name="${prefix}rear_right_motor_joint" type="fixed">
       <parent link="${prefix}right_rocker"/>
       <child link="${prefix}rear_right_motor"/>
-      <origin xyz="${rear_motors_x_offset/scale_factor} ${motors_y_offset/scale_factor} ${motors_z_offset/scale_factor}" rpy="0.0 0.0 0.0"/>
+      <origin xyz="${rear_motors_x_offset} ${motors_y_offset} ${motors_z_offset}" rpy="0.0 0.0 0.0"/>
     </joint>
     <joint name="${prefix}front_left_wheel_joint" type="continuous">
@@ -82,5 +80,5 @@
       <parent link="${prefix}front_left_motor"/>
       <child link="${prefix}front_left_wheel"/>
-      <origin xyz="0 ${wheels_y_offset/scale_factor} 0.0" rpy="0.0 0.0 0"/>
+      <origin xyz="0 ${wheels_y_offset} 0.0" rpy="0.0 0.0 0"/>
       <dynamics damping="0.2" friction="0.3"/>
     </joint>
@@ -89,5 +87,5 @@
       <parent link="${prefix}rear_left_motor"/>
       <child link="${prefix}rear_left_wheel"/>
-      <origin xyz="0 ${wheels_y_offset/scale_factor} 0.0" rpy="0.0 0.0 0"/>
+      <origin xyz="0 ${wheels_y_offset} 0.0" rpy="0.0 0.0 0"/>
       <dynamics damping="0.2" friction="0.3"/>
     </joint>
@@ -96,5 +94,5 @@
       <parent link="${prefix}front_right_motor"/>
       <child link="${prefix}front_right_wheel"/>
-      <origin xyz="0 -${wheels_y_offset/scale_factor} 0.0" rpy="0.0 0.0 0"/>
+      <origin xyz="0 -${wheels_y_offset} 0.0" rpy="0.0 0.0 0"/>
       <dynamics damping="0.2" friction="0.3"/>
     </joint>
@@ -103,5 +101,5 @@
       <parent link="${prefix}rear_right_motor"/>
       <child link="${prefix}rear_right_wheel"/>
-      <origin xyz="0 -${wheels_y_offset/scale_factor} 0.0" rpy="0.0 0.0 0"/>
+      <origin xyz="0 -${wheels_y_offset} 0.0" rpy="0.0 0.0 0"/>
       <dynamics damping="0.2" friction="0.3"/>
     </joint>
@@ -109,5 +107,5 @@
       <parent link="${prefix}chassis"/>
       <child link="${prefix}laser_frame"/>
-      <origin xyz="0 0 -0.04" rpy="0 ${PI} 0"/>
+      <origin xyz="0 0 -0.04" rpy="0 ${pi} 0"/>
     </joint>
     <joint name="${prefix}laser_2d_joint" type="fixed">

File: software/ros_ws/src/perseus_description/urdf/rocker.urdf.xacro (robot description, xacro)
@@ -11,5 +11,5 @@
   <link name="${prefix}left_rocker">
     <inertial>
-      <origin xyz="${rocker_collision_x_offset/scale_factor} 0.0 ${rocker_collision_z_offset/scale_factor}" rpy="0.0 0.0 0.0"/>
+      <origin xyz="${rocker_collision_x_offset} 0.0 ${rocker_collision_z_offset}" rpy="0.0 0.0 0.0"/>
       <mass value="${rocker_mass}"/>
       <xacro:box_inertia m="${rocker_mass}"
@@ -21,12 +21,12 @@
       <origin xyz="0.0 0.0 0.0" rpy="0.0 0.0 ${pi}"/>
       <geometry>
-        <mesh scale="${0.1/scale_factor} ${0.1/scale_factor} ${0.1/scale_factor}"
+        <mesh scale="${0.1} ${0.1} ${0.1}"
               filename="file://$(find perseus_description)/meshes/rocker_left.dae"/>
       </geometry>
     </visual>
     <collision>
-      <origin xyz="${rocker_collision_x_offset/scale_factor} 0.0 ${rocker_collision_z_offset/scale_factor}" rpy="0.0 0.0 0.0"/>
+      <origin xyz="${rocker_collision_x_offset} 0.0 ${rocker_collision_z_offset}" rpy="0.0 0.0 0.0"/>
       <geometry>
-        <box size="${rocker_length/scale_factor} ${rocker_width/scale_factor} ${rocker_height/scale_factor}"/>
+        <box size="${rocker_length} ${rocker_width} ${rocker_height}"/>
       </geometry>
     </collision>
@@ -35,5 +35,5 @@
   <link name="${prefix}right_rocker">
     <inertial>
-      <origin xyz="${rocker_collision_x_offset/scale_factor} 0.0 ${rocker_collision_z_offset/scale_factor}" rpy="0.0 0.0 0.0"/>
+      <origin xyz="${rocker_collision_x_offset} 0.0 ${rocker_collision_z_offset}" rpy="0.0 0.0 0.0"/>
       <mass value="${rocker_mass}"/>
       <xacro:box_inertia m="${rocker_mass}"
@@ -45,12 +45,12 @@
       <origin xyz="0.0 0.0 0.0" rpy="0.0 0.0 ${pi}"/>
       <geometry>
-        <mesh scale="${0.1/scale_factor} ${0.1/scale_factor} ${0.1/scale_factor}"
+        <mesh scale="${0.1} ${0.1} ${0.1}"
               filename="file://$(find perseus_description)/meshes/rocker_right.dae"/>
       </geometry>
     </visual>
     <collision>
-      <origin xyz="${rocker_collision_x_offset/scale_factor} 0.0 ${rocker_collision_z_offset/scale_factor}" rpy="0.0 0.0 0.0"/>
+      <origin xyz="${rocker_collision_x_offset} 0.0 ${rocker_collision_z_offset}" rpy="0.0 0.0 0.0"/>
       <geometry>
-        <box size="${rocker_length/scale_factor} ${rocker_width/scale_factor} ${rocker_height/scale_factor}"/>
+        <box size="${rocker_length} ${rocker_width} ${rocker_height}"/>
       </geometry>
     </collision>

File: software/ros_ws/src/perseus_description/urdf/sensors.urdf.xacro (robot description, xacro)
@@ -1,10 +1,21 @@
 <?xml version="1.0"?>
 <robot name="lidar" xmlns:xacro="http://ros.org/wiki/xacro">
+<xacro:property name="laser_2d_mass" value="0.1"/>
+<xacro:property name="laser_2d_radius" value="0.04"/>
+<xacro:property name="laser_2d_length" value="0.04"/>
+<xacro:property name="laser_3d_mass" value="0.2"/>
+<xacro:property name="laser_3d_radius" value="0.06"/>
+<xacro:property name="laser_3d_length" value="0.06"/>
 <!-- 3D LIDAR (Existing - Livox MID-360) -->
 <link name="${prefix}laser_frame">
+    <inertial>
+        <origin xyz="0 0 0"/>
+        <mass value="${laser_3d_mass}"/>
+        <xacro:box_inertia m="${laser_3d_mass}" x="${laser_3d_length}" y="${laser_3d_radius}" z="${laser_3d_radius}"/>
+    </inertial>
     <visual>
         <origin xyz="0 0 0"/>
         <geometry>
-            <cylinder radius="0.06" length="0.06"/>
+            <cylinder radius="${laser_3d_radius}" length="${laser_3d_length}"/>
         </geometry>
         <material name="black"/>
@@ -12,5 +23,5 @@
     <collision>
         <geometry>
-            <cylinder radius="0.06" length="0.06"/>
+            <cylinder radius="${laser_3d_radius}" length="${laser_3d_length}"/>
         </geometry>
     </collision>
@@ -18,8 +29,13 @@
 <!-- 2D LIDAR -->
 <link name="${prefix}laser_2d_frame">
+    <inertial>
+        <origin xyz="0 0 0"/>
+        <mass value="${laser_2d_mass}"/>
+        <xacro:box_inertia m="${laser_2d_mass}" x="${laser_2d_length}" y="${laser_2d_radius}" z="${laser_2d_radius}"/>
+    </inertial>
     <visual>
         <origin xyz="0 0 0"/>
         <geometry>
-            <cylinder radius="0.04" length="0.04"/>
+            <cylinder radius="${laser_2d_radius}" length="${laser_2d_length}"/>
         </geometry>
         <material name="blue">

File: software/ros_ws/src/perseus_description/urdf/wheel.urdf.xacro (robot description, xacro)
@@ -10,5 +10,5 @@
     <origin xyz="0.0 0.0  0.0" rpy="0.0 0.0 ${pi}"/>
     <geometry>
-      <mesh scale="${0.1/scale_factor} ${0.1/scale_factor}  ${0.1/scale_factor}" filename="file://$(find perseus_description)/meshes/wheel.dae"/>
+      <mesh scale="${0.1} ${0.1}  ${0.1}" filename="file://$(find perseus_description)/meshes/wheel.dae"/>
     </geometry>
   </visual>
@@ -16,5 +16,5 @@
     <origin xyz="0.0 0.0 0.0" rpy="${pi/2} 0.0 ${pi}"/>
     <geometry>
-      <cylinder radius="${wheel_radius/scale_factor}" length="${wheel_length/scale_factor}"/>
+      <cylinder radius="${wheel_radius}" length="${wheel_length}"/>
     </geometry>
   </collision>
@@ -29,5 +29,5 @@
       <origin xyz="0.0 0.0  0.0" rpy="0.0 0.0 0.0"/>
     <geometry>
-      <mesh scale="${0.1/scale_factor} ${0.1/scale_factor}  ${0.1/scale_factor}" filename="file://$(find perseus_description)/meshes/wheel.dae"/>
+      <mesh scale="${0.1} ${0.1}  ${0.1}" filename="file://$(find perseus_description)/meshes/wheel.dae"/>
     </geometry>
   </visual>
@@ -35,5 +35,5 @@
     <origin xyz="0.0 0.0 0.0" rpy="${pi/2} 0.0 0.0"/>
     <geometry>
-      <cylinder radius="${wheel_radius/scale_factor}" length="${wheel_length/scale_factor}"/>
+      <cylinder radius="${wheel_radius}" length="${wheel_length}"/>
     </geometry>
   </collision>
@@ -48,5 +48,5 @@
       <origin xyz="0.0 0.0  0.0" rpy="0.0 0.0 ${pi}"/>
     <geometry>
-      <mesh scale="${0.1/scale_factor} ${0.1/scale_factor}  ${0.1/scale_factor}" filename="file://$(find perseus_description)/meshes/wheel.dae"/>
+      <mesh scale="${0.1} ${0.1}  ${0.1}" filename="file://$(find perseus_description)/meshes/wheel.dae"/>
     </geometry>
   </visual>
@@ -54,5 +54,5 @@
     <origin xyz="0.0 0.0 0.0" rpy="${pi/2} 0.0 ${pi}"/>
     <geometry>
-      <cylinder radius="${wheel_radius/scale_factor}" length="${wheel_length/scale_factor}"/>
+      <cylinder radius="${wheel_radius}" length="${wheel_length}"/>
     </geometry>
   </collision>
@@ -67,5 +67,5 @@
       <origin xyz="0.0 0.0  0.0" rpy="0.0 0.0 0.0"/>
     <geometry>
-      <mesh scale="${0.1/scale_factor} ${0.1/scale_factor}  ${0.1/scale_factor}" filename="file://$(find perseus_description)/meshes/wheel.dae"/>
+      <mesh scale="${0.1} ${0.1}  ${0.1}" filename="file://$(find perseus_description)/meshes/wheel.dae"/>
     </geometry>
   </visual>
@@ -73,5 +73,5 @@
     <origin xyz="0.0 0.0 0.0" rpy="${pi/2} 0.0 0.0"/>
     <geometry>
-      <cylinder radius="${wheel_radius/scale_factor}" length="${wheel_length/scale_factor}"/>
+      <cylinder radius="${wheel_radius}" length="${wheel_length}"/>
     </geometry>
   </collision>
