Commit message: Refactor URDF files to standardize mesh scale formatting and improve collision definitions for various components including camera, chassis, flange bearing, motor wheel, rocker, and wheel.

File: software/ros_ws/src/perseus_description/urdf/camera_depth.urdf.xacro (robot description, xacro)
@@ -17,4 +17,9 @@
             <material name="red"/>
         </visual>
+        <collision>
+            <geometry>
+                <box size="${camera_depth} ${camera_width} ${camera_height}"/>
+            </geometry>
+        </collision>
     </link>
     <joint name="${prefix}camera_optical_joint" type="fixed">

File: software/ros_ws/src/perseus_description/urdf/chassis.urdf.xacro (robot description, xacro)
@@ -11,5 +11,5 @@
       <origin xyz="0.0 0.0 0.0" rpy="0 0.0 -${pi/2}"/>
       <geometry>
-        <mesh scale="${0.1} ${0.1}  ${0.1}" filename="file://$(find perseus_description)/meshes/chassis.dae"/>
+        <mesh scale="0.1 0.1  0.1" filename="file://$(find perseus_description)/meshes/chassis.dae"/>
       </geometry>
     </visual>

File: software/ros_ws/src/perseus_description/urdf/flange_bearing.urdf.xacro (robot description, xacro)
@@ -19,5 +19,5 @@
     <origin xyz="0.0 0.0 0.0" rpy="${-pi/2} 0 ${pi/2}"/>
     <geometry>
-        <mesh scale="${0.1} ${0.1}  ${0.1}" filename="file://$(find perseus_description)/meshes/flange_bearing.dae"/>
+        <mesh scale="0.1 0.1  0.1" filename="file://$(find perseus_description)/meshes/flange_bearing.dae"/>
     </geometry>
     </visual>
@@ -39,5 +39,5 @@
     <origin xyz="0.0 0.0 0.0" rpy="${-pi/2} 0 ${-pi/2}"/>
     <geometry>
-        <mesh scale=  "${0.1} ${0.1}  ${0.1}" filename="file://$(find perseus_description)/meshes/differential_bar.dae"/>
+        <mesh scale=  "0.1 0.1  0.1" filename="file://$(find perseus_description)/meshes/differential_bar.dae"/>
     </geometry>
     </visual>

File: software/ros_ws/src/perseus_description/urdf/motor_wheel.urdf.xacro (robot description, xacro)
@@ -15,5 +15,5 @@
       <origin xyz="0 0.0 0.0" rpy="0.0 0.0 ${pi/2}"/>
       <geometry>
-        <mesh scale="${0.1} ${0.1}  ${0.1}" filename="file://$(find perseus_description)/meshes/gearbox.dae"/>
+        <mesh scale="0.1 0.1  0.1" filename="file://$(find perseus_description)/meshes/gearbox.dae"/>
       </geometry>
       <!-- <material name="white"/> -->
@@ -36,5 +36,5 @@
       <origin xyz="0 0.0 0.0" rpy="0.0 0.0 ${pi/2}"/>
       <geometry>
-        <mesh scale="${0.1} ${0.1}  ${0.1}" filename="file://$(find perseus_description)/meshes/gearbox.dae"/>
+        <mesh scale="0.1 0.1  0.1" filename="file://$(find perseus_description)/meshes/gearbox.dae"/>
       </geometry>
       <!-- <material name="white"/> -->
@@ -57,5 +57,5 @@
       <origin xyz="0 0.0 0.0" rpy="0.0 0.0 ${-pi/2}"/>
       <geometry>
-        <mesh scale="${0.1} ${0.1}  ${0.1}" filename="file://$(find perseus_description)/meshes/gearbox.dae"/>
+        <mesh scale="0.1 0.1  0.1" filename="file://$(find perseus_description)/meshes/gearbox.dae"/>
       </geometry>
       <!-- <material name="white"/> -->
@@ -78,5 +78,5 @@
       <origin xyz="0 0.0 0.0" rpy="0.0 0.0 ${-pi/2}"/>
       <geometry>
-        <mesh scale="${0.1} ${0.1}  ${0.1}" filename="file://$(find perseus_description)/meshes/gearbox.dae"/>
+        <mesh scale="0.1 0.1  0.1" filename="file://$(find perseus_description)/meshes/gearbox.dae"/>
       </geometry>
       <!-- <material name="white"/> -->

File: software/ros_ws/src/perseus_description/urdf/perseus.urdf.xacro (robot description, xacro)
@@ -76,32 +76,4 @@
       <origin xyz="${rear_motors_x_offset} ${motors_y_offset} ${motors_z_offset}" rpy="0.0 0.0 0.0"/>
     </joint>
-    <joint name="${prefix}front_left_wheel_joint" type="continuous">
-      <axis xyz="0 1 0" rpy="0 0 0"/>
-      <parent link="${prefix}front_left_motor"/>
-      <child link="${prefix}front_left_wheel"/>
-      <origin xyz="0 ${wheels_y_offset} 0.0" rpy="0.0 0.0 0"/>
-      <dynamics damping="0.2" friction="0.3"/>
-    </joint>
-    <joint name="${prefix}rear_left_wheel_joint" type="continuous">
-      <axis xyz="0 1 0" rpy="0 0 0"/>
-      <parent link="${prefix}rear_left_motor"/>
-      <child link="${prefix}rear_left_wheel"/>
-      <origin xyz="0 ${wheels_y_offset} 0.0" rpy="0.0 0.0 0"/>
-      <dynamics damping="0.2" friction="0.3"/>
-    </joint>
-    <joint name="${prefix}front_right_wheel_joint" type="continuous">
-      <axis xyz="0 1 0" rpy="0 0 0"/>
-      <parent link="${prefix}front_right_motor"/>
-      <child link="${prefix}front_right_wheel"/>
-      <origin xyz="0 -${wheels_y_offset} 0.0" rpy="0.0 0.0 0"/>
-      <dynamics damping="0.2" friction="0.3"/>
-    </joint>
-    <joint name="${prefix}rear_right_wheel_joint" type="continuous">
-      <axis xyz="0 1 0" rpy="0 0 0"/>
-      <parent link="${prefix}rear_right_motor"/>
-      <child link="${prefix}rear_right_wheel"/>
-      <origin xyz="0 -${wheels_y_offset} 0.0" rpy="0.0 0.0 0"/>
-      <dynamics damping="0.2" friction="0.3"/>
-    </joint>
     <joint name="${prefix}laser_joint" type="fixed">
       <parent link="${prefix}chassis"/>

File: software/ros_ws/src/perseus_description/urdf/rocker.urdf.xacro (robot description, xacro)
@@ -21,5 +21,5 @@
       <origin xyz="0.0 0.0 0.0" rpy="0.0 0.0 ${pi}"/>
       <geometry>
-        <mesh scale="${0.1} ${0.1} ${0.1}"
+        <mesh scale="0.1 0.1 0.1"
               filename="file://$(find perseus_description)/meshes/rocker_left.dae"/>
       </geometry>
@@ -45,5 +45,5 @@
       <origin xyz="0.0 0.0 0.0" rpy="0.0 0.0 ${pi}"/>
       <geometry>
-        <mesh scale="${0.1} ${0.1} ${0.1}"
+        <mesh scale="0.1 0.1 0.1"
               filename="file://$(find perseus_description)/meshes/rocker_right.dae"/>
       </geometry>

File: software/ros_ws/src/perseus_description/urdf/wheel.urdf.xacro (robot description, xacro)
@@ -1,183 +1,82 @@
 <?xml version="1.0"?>
 <robot name="wheel" xmlns:xacro="http://ros.org/wiki/xacro">
-<link name="${prefix}front_left_wheel">
-  <inertial>
-    <origin xyz="0.0 0.0  0.0" rpy="0.0 0.0 ${pi}"/>
-    <mass value="${wheel_mass}"/>
-    <xacro:cylinder_inertia m="${wheel_mass}" radius="${wheel_radius}" length="${wheel_length}"/>
-  </inertial>
-  <visual>
-    <origin xyz="0.0 0.0  0.0" rpy="0.0 0.0 ${pi}"/>
-    <geometry>
-      <mesh scale="${0.1} ${0.1}  ${0.1}" filename="file://$(find perseus_description)/meshes/wheel.dae"/>
-    </geometry>
-  </visual>
-  <collision>
-    <origin xyz="0.0 0.0 0.0" rpy="${pi/2} 0.0 ${pi}"/>
-    <geometry>
-      <cylinder radius="${wheel_radius}" length="${wheel_length}"/>
-    </geometry>
-  </collision>
-</link>
-<link name="${prefix}front_right_wheel">
-  <inertial>
-    <origin xyz="0.0 0.0  0.0" rpy="0.0 0.0 0.0"/>
-    <mass value="${wheel_mass}"/>
-    <xacro:cylinder_inertia m="${wheel_mass}" radius="${wheel_radius}" length="${wheel_length}"/>
-  </inertial>
-  <visual>
-      <origin xyz="0.0 0.0  0.0" rpy="0.0 0.0 0.0"/>
-    <geometry>
-      <mesh scale="${0.1} ${0.1}  ${0.1}" filename="file://$(find perseus_description)/meshes/wheel.dae"/>
-    </geometry>
-  </visual>
-  <collision>
-    <origin xyz="0.0 0.0 0.0" rpy="${pi/2} 0.0 0.0"/>
-    <geometry>
-      <cylinder radius="${wheel_radius}" length="${wheel_length}"/>
-    </geometry>
-  </collision>
-</link>
-<link name="${prefix}rear_left_wheel">
-  <inertial>
-    <origin xyz="0.0 0.0  0.0" rpy="0.0 0.0 ${pi}"/>
-    <mass value="${wheel_mass}"/>
-    <xacro:cylinder_inertia m="${wheel_mass}" radius="${wheel_radius}" length="${wheel_length}"/>
-  </inertial>
-  <visual>
-      <origin xyz="0.0 0.0  0.0" rpy="0.0 0.0 ${pi}"/>
-    <geometry>
-      <mesh scale="${0.1} ${0.1}  ${0.1}" filename="file://$(find perseus_description)/meshes/wheel.dae"/>
-    </geometry>
-  </visual>
-  <collision>
-    <origin xyz="0.0 0.0 0.0" rpy="${pi/2} 0.0 ${pi}"/>
-    <geometry>
-      <cylinder radius="${wheel_radius}" length="${wheel_length}"/>
-    </geometry>
-  </collision>
-</link>
-<link name="${prefix}rear_right_wheel">
-  <inertial>
-    <origin xyz="0.0 0.0 0.0" rpy="0.0 0.0 0.0"/>
-    <mass value="${wheel_mass}"/>
-    <xacro:cylinder_inertia m="${wheel_mass}" radius="${wheel_radius}" length="${wheel_length}"/>
-  </inertial>
-  <visual>
-      <origin xyz="0.0 0.0  0.0" rpy="0.0 0.0 0.0"/>
-    <geometry>
-      <mesh scale="${0.1} ${0.1}  ${0.1}" filename="file://$(find perseus_description)/meshes/wheel.dae"/>
-    </geometry>
-  </visual>
-  <collision>
-    <origin xyz="0.0 0.0 0.0" rpy="${pi/2} 0.0 0.0"/>
-    <geometry>
-      <cylinder radius="${wheel_radius}" length="${wheel_length}"/>
-    </geometry>
-  </collision>
-</link>
-<gazebo reference="${prefix}front_left_wheel">
-  <!-- TODO: Fix the material tag (this isn't the proper way to do it, and spits out warnings) -->
-  <material>Gazebo/Orange</material>
-  <!-- see http://sdformat.org/spec?ver=1.12&elem=collision -->
-  <collision>
-    <surface>
-        <friction>
-            <ode>
-                <!--
-                In this case, the wheels need lower sideways than forwards coefficients of friction
-                so that the rover can turn (skid steer) -->
-                <!-- forward coefficient of friction -->
-                <mu>0.3</mu>
-                <!-- perpendicular coefficient of friction -->
-                <mu2>1</mu2>
-                <!--
-                However, since mu/mu2 are normally relative to world coordinates,
-                the rover would only be able to turn 90 degrees either way before they swapped, making turning impossible.
-                To solve this, we need to specify the direction that mu/mu2 are relative to.
-                -->
-                <fdir1>1 0 0</fdir1>
-            </ode>
-        </friction>
-    </surface>
-  </collision>
-</gazebo>
-<gazebo reference="${prefix}front_right_wheel">
-  <!-- TODO: Fix the material tag (this isn't the proper way to do it, and spits out warnings) -->
-  <material>Gazebo/Orange</material>
-  <!-- see http://sdformat.org/spec?ver=1.12&elem=collision -->
-  <collision>
-    <surface>
-        <friction>
-            <ode>
-                <!--
-                In this case, the wheels need lower sideways than forwards coefficients of friction
-                so that the rover can turn (skid steer) -->
-                <!-- forward coefficient of friction -->
-                <mu>0.3</mu>
-                <!-- perpendicular coefficient of friction -->
-                <mu2>1</mu2>
-                <!--
-                However, since mu/mu2 are normally relative to world coordinates,
-                the rover would only be able to turn 90 degrees either way before they swapped, making turning impossible.
-                To solve this, we need to specify the direction that mu/mu2 are relative to.
-                -->
-                <fdir1>1 0 0</fdir1>
-            </ode>
-        </friction>
-    </surface>
-  </collision>
-</gazebo>
-<gazebo reference="${prefix}rear_right_wheel">
-  <!-- TODO: Fix the material tag (this isn't the proper way to do it, and spits out warnings) -->
-  <material>Gazebo/Orange</material>
-  <!-- see http://sdformat.org/spec?ver=1.12&elem=collision -->
-  <collision>
-    <surface>
-        <friction>
-            <ode>
-                <!--
-                In this case, the wheels need lower sideways than forwards coefficients of friction
-                so that the rover can turn (skid steer) -->
-                <!-- forward coefficient of friction -->
-                <mu>0.3</mu>
-                <!-- perpendicular coefficient of friction -->
-                <mu2>1</mu2>
-                <!--
-                However, since mu/mu2 are normally relative to world coordinates,
-                the rover would only be able to turn 90 degrees either way before they swapped, making turning impossible.
-                To solve this, we need to specify the direction that mu/mu2 are relative to.
-                -->
-                <fdir1>1 0 0</fdir1>
-            </ode>
-        </friction>
-    </surface>
-  </collision>
-</gazebo>
-<gazebo reference="${prefix}rear_left_wheel">
-  <!-- TODO: Fix the material tag (this isn't the proper way to do it, and spits out warnings) -->
-  <material>Gazebo/Orange</material>
-  <!-- see http://sdformat.org/spec?ver=1.12&elem=collision -->
-  <collision>
-    <surface>
-        <friction>
-            <ode>
-                <!--
-                In this case, the wheels need lower sideways than forwards coefficients of friction
-                so that the rover can turn (skid steer) -->
-                <!-- forward coefficient of friction -->
-                <mu>0.3</mu>
-                <!-- perpendicular coefficient of friction -->
-                <mu2>1</mu2>
-                <!--
-                However, since mu/mu2 are normally relative to world coordinates,
-                the rover would only be able to turn 90 degrees either way before they swapped, making turning impossible.
-                To solve this, we need to specify the direction that mu/mu2 are relative to.
-                -->
-                <fdir1>1 0 0</fdir1>
-            </ode>
-        </friction>
-    </surface>
-  </collision>
-</gazebo>
+<xacro:macro name="wheel" params="prefix:=^ side:=^ end:=^">
+  <link name="${prefix}${end}_${side}_wheel">
+    <inertial>
+      <xacro:if value="${side == 'left'}">
+        <origin xyz="0.0 0.0  0.0" rpy="0.0 0.0 ${pi}"/>
+      </xacro:if>
+      <xacro:if value="${side == 'right'}">
+        <origin xyz="0.0 0.0  0.0" rpy="0.0 0.0 0.0"/>
+      </xacro:if>
+      <mass value="${wheel_mass}"/>
+      <xacro:cylinder_inertia m="${wheel_mass}" radius="${wheel_radius}" length="${wheel_length}"/>
+    </inertial>
+    <visual>
+      <xacro:if value="${side == 'left'}">
+        <origin xyz="0.0 0.0  0.0" rpy="0.0 0.0 ${pi}"/>
+      </xacro:if>
+      <xacro:if value="${side == 'right'}">
+        <origin xyz="0.0 0.0  0.0" rpy="0.0 0.0 0.0"/>
+      </xacro:if>
+      <geometry>
+        <mesh scale="0.1 0.1  0.1" filename="file://$(find perseus_description)/meshes/wheel.dae"/>
+      </geometry>
+    </visual>
+    <collision>
+      <xacro:if value="${side == 'left'}">
+        <origin xyz="0.0 0.0 0.0" rpy="${pi/2} 0.0 ${pi}"/>
+      </xacro:if>
+        <xacro:if value="${side == 'right'}">
+      <origin xyz="0.0 0.0 0.0" rpy="${pi/2} 0.0 0.0"/>
+      </xacro:if>
+      <geometry>
+        <cylinder radius="${wheel_radius}" length="${wheel_length}"/>
+      </geometry>
+    </collision>
+  </link>
+  <joint name="${prefix}${end}_${side}_wheel_joint" type="continuous">
+    <xacro:if value="${side == 'left'}">
+      <origin xyz="0 ${wheels_y_offset} 0.0" rpy="0.0 0.0 0"/>
+      <axis xyz="0 1 0" rpy="0 0 0"/>
+    </xacro:if>
+    <xacro:if value="${side == 'right'}">
+      <origin xyz="0 ${-wheels_y_offset} 0.0" rpy="0.0 0.0 ${pi}"/>
+      <axis xyz="0 -1 0" rpy="0 0 0"/>
+    </xacro:if>
+    <dynamics damping="0.2" friction="0.3"/>
+    <parent link="${prefix}${end}_${side}_motor"/>
+    <child link="${prefix}${end}_${side}_wheel"/>
+  </joint>
+  <gazebo reference="${prefix}${end}_${side}_wheel">
+    <!-- TODO: Fix the material tag (this isn't the proper way to do it, and spits out warnings) -->
+    <material>Gazebo/Orange</material>
+    <!-- see http://sdformat.org/spec?ver=1.12&elem=collision -->
+    <collision>
+      <surface>
+          <friction>
+              <ode>
+                  <!--
+                  In this case, the wheels need lower sideways than forwards coefficients of friction
+                  so that the rover can turn (skid steer) -->
+                  <!-- forward coefficient of friction -->
+                  <mu>0.3</mu>
+                  <!-- perpendicular coefficient of friction -->
+                  <mu2>1</mu2>
+                  <!--
+                  However, since mu/mu2 are normally relative to world coordinates,
+                  the rover would only be able to turn 90 degrees either way before they swapped, making turning impossible.
+                  To solve this, we need to specify the direction that mu/mu2 are relative to.
+                  -->
+                  <fdir1>1 0 0</fdir1>
+              </ode>
+          </friction>
+      </surface>
+    </collision>
+  </gazebo>
+</xacro:macro>
+<xacro:wheel prefix="" side="left"  end="front"/>
+<xacro:wheel prefix="" side="left"  end="rear"/>
+<xacro:wheel prefix="" side="right" end="front"/>
+<xacro:wheel prefix="" side="right" end="rear"/>
 </robot>

Commit message: Refactor URDF and XACRO files to remove unnecessary properties for camera, flange bearing, motor wheel, and sensors, improving overall structure and clarity.

File: software/ros_ws/src/perseus_description/urdf/camera_depth.urdf.xacro (robot description, xacro)
@@ -1,8 +1,4 @@
 <?xml version="1.0"?>
 <robot name="camera_depth" xmlns:xacro="http://ros.org/wiki/xacro">
-    <xacro:property name="camera_mass" value="0.1"/>
-    <xacro:property name="camera_width" value="0.07"/>
-    <xacro:property name="camera_height" value="0.03"/>
-    <xacro:property name="camera_depth" value="0.020"/>
     <link name="${prefix}camera_link">
         <inertial>

File: software/ros_ws/src/perseus_description/urdf/flange_bearing.urdf.xacro (robot description, xacro)
@@ -1,12 +1,4 @@
 <?xml version="1.0"?>
 <robot name="flange_bearing" xmlns:xacro="http://ros.org/wiki/xacro">
-<xacro:property name="bar_length" value="0.58"/>
-<xacro:property name="bar_width" value="0.03"/>
-<xacro:property name="bar_height" value="0.03"/>
-<xacro:property name="bar_mass" value="0.917264951812715"/>
-<xacro:property name="bearing_length" value="0.2"/>
-<xacro:property name="bearing_width" value="0.03"/>
-<xacro:property name="bearing_height" value="0.03"/>
-<xacro:property name="bearing_mass" value="2.7689940302592726"/>  <!-- Kg -->
 <!-- Flange Bearing -->
 <link name="${prefix}flange_bearing">

File: software/ros_ws/src/perseus_description/urdf/perseus.urdf.xacro (robot description, xacro)
@@ -2,6 +2,13 @@
 <robot xmlns:xacro="http://ros.org/wiki/xacro">
   <xacro:macro name="perseus" params="prefix">
+    <!-- Motors Properties -->
+    <xacro:property name="motors_y_offset" value="0.035"/>
+    <xacro:property name="motors_z_offset" value="-0.25"/>
     <xacro:property name="front_motors_x_offset" value="0.3"/>
     <xacro:property name="rear_motors_x_offset" value="-0.55"/>
+    <xacro:property name="motor_mass" value="5.236579"/>  <!-- Kg -->
+    <xacro:property name="collision_motor_length" value="0.1"/>  <!-- m -->
+    <xacro:property name="collision_motor_width" value="0.1"/>  <!-- m -->
+    <xacro:property name="collision_motor_height" value="0.075"/>  <!-- m -->
     <!-- Rocker properties -->
     <xacro:property name="rocker_mass" value="0.5"/>
@@ -25,12 +32,26 @@
     <xacro:property name="chassis_z_offset" value="${rocker_height + wheel_radius}" /> <!-- Space btw top of beam and the each joint -->
     <!-- Flange Bearing Properties -->
+    <xacro:property name="bearing_mass" value="2.7689940302592726"/>  <!-- Kg -->
     <xacro:property name="flange_bearing_z_offset" value="${chassis_height/2}"/>
-    <!-- Motors Properties -->
-    <xacro:property name="motors_y_offset" value="0.035"/>
-    <xacro:property name="motors_z_offset" value="-0.25"/>
-    <xacro:property name="motor_mass" value="5.236579"/>  <!-- Kg -->
-    <xacro:property name="collision_motor_length" value="0.1"/>  <!-- m -->
-    <xacro:property name="collision_motor_width" value="0.1"/>  <!-- m -->
-    <xacro:property name="collision_motor_height" value="0.075"/>  <!-- m -->
+    <xacro:property name="bearing_length" value="0.2"/>
+    <xacro:property name="bearing_width" value="0.03"/>
+    <xacro:property name="bearing_height" value="0.03"/>
+    <!-- Differential Bar Properties -->
+    <xacro:property name="bar_mass" value="0.917264951812715"/>
+    <xacro:property name="bar_length" value="0.58"/>
+    <xacro:property name="bar_width" value="0.03"/>
+    <xacro:property name="bar_height" value="0.03"/>
+    <!-- Depth Camera Properties -->
+    <xacro:property name="camera_mass" value="0.1"/>
+    <xacro:property name="camera_width" value="0.07"/>
+    <xacro:property name="camera_height" value="0.03"/>
+    <xacro:property name="camera_depth" value="0.020"/>
+    <!-- 2D and 3D LIDAR Properties -->
+    <xacro:property name="laser_2d_mass" value="0.1"/>
+    <xacro:property name="laser_2d_radius" value="0.04"/>
+    <xacro:property name="laser_2d_length" value="0.04"/>
+    <xacro:property name="laser_3d_mass" value="0.2"/>
+    <xacro:property name="laser_3d_radius" value="0.06"/>
+    <xacro:property name="laser_3d_length" value="0.06"/>
     <!-- ADD COMPONENTS -->
     <xacro:include filename="$(find perseus_description)/urdf/inertia_macros.xacro"/>

File: software/ros_ws/src/perseus_description/urdf/sensors.urdf.xacro (robot description, xacro)
@@ -1,10 +1,4 @@
 <?xml version="1.0"?>
 <robot name="lidar" xmlns:xacro="http://ros.org/wiki/xacro">
-<xacro:property name="laser_2d_mass" value="0.1"/>
-<xacro:property name="laser_2d_radius" value="0.04"/>
-<xacro:property name="laser_2d_length" value="0.04"/>
-<xacro:property name="laser_3d_mass" value="0.2"/>
-<xacro:property name="laser_3d_radius" value="0.06"/>
-<xacro:property name="laser_3d_length" value="0.06"/>
 <!-- 3D LIDAR (Existing - Livox MID-360) -->
 <link name="${prefix}laser_frame">

File: software/ros_ws/src/perseus_description/urdf/wheel.urdf.xacro (robot description, xacro)
@@ -76,7 +76,3 @@
   </gazebo>
 </xacro:macro>
-<!-- <xacro:wheel prefix="" side="left"  end="front"/>
-<xacro:wheel prefix="" side="left"  end="rear"/>
-<xacro:wheel prefix="" side="right" end="front"/>
-<xacro:wheel prefix="" side="right" end="rear"/> -->
 </robot>
