Commit message: Add inertia macros and refactor URDF files for Perseus robot
- Introduced inertia macros in `inertia_macros.xacro` for box, cylinder, and sphere inertia calculations.
- Refactored `motor_wheel.urdf.xacro` to use a macro for motor and wheel definitions, reducing redundancy.
- Updated `perseus.urdf.xacro` to include new properties for motors, rockers, and sensors, and streamlined component inclusion.
- Modified `rocker.urdf.xacro` to implement a macro for rocker links and associated motors.
- Enhanced `sensors.urdf.xacro` to include inertial properties for LIDAR components.
- Simplified `wheel.urdf.xacro` by creating a macro for wheel definitions, including inertia calculations.
- Adjusted `gz_bridge.yaml` to change Gazebo topic names for better integration with ROS.

File: software/ros_ws/src/perseus_description/urdf/camera_depth.urdf.xacro (robot description, xacro)
@@ -1,13 +1,21 @@
 <?xml version="1.0"?>
-<!-- 0.220 0 0.4 -->
-<!-- <box size="0.020 0.07 0.03"/>  -->
 <robot name="camera_depth" xmlns:xacro="http://ros.org/wiki/xacro">
     <link name="${prefix}camera_link">
+        <inertial>
+            <origin xyz="0 0 0" rpy="0 0 0"/>
+            <mass value="${camera_mass}"/>
+            <xacro:box_inertia m="${camera_mass}" x="${camera_depth}" y="${camera_width}" z="${camera_height}"/>
+        </inertial>
         <visual>
             <geometry>
-                <box size="0.020 0.07 0.03"/>
+                <box size="${camera_depth} ${camera_width} ${camera_height}"/>
             </geometry>
             <material name="red"/>
         </visual>
+        <collision>
+            <geometry>
+                <box size="${camera_depth} ${camera_width} ${camera_height}"/>
+            </geometry>
+        </collision>
     </link>
     <joint name="${prefix}camera_optical_joint" type="fixed">
@@ -22,5 +30,5 @@
             <pose> 0 0 0 0 0 0 </pose>
             <visualize>true</visualize>
-            <update_rate>100</update_rate>
+            <update_rate>10</update_rate>
             <always_on>true</always_on>
             <camera>
@@ -35,4 +43,5 @@
                 </clip>
             </camera>
+            <topic>/perseus/rgbd_camera</topic>
             <gz_frame_id>${prefix}camera_link_optical</gz_frame_id>
             <min_depth>0.05</min_depth>

File: software/ros_ws/src/perseus_description/urdf/chassis.urdf.xacro (robot description, xacro)
@@ -2,20 +2,20 @@
 <robot name="chassis" xmlns:xacro="http://ros.org/wiki/xacro">
   <link name="${prefix}chassis">
-  <inertial>
-    <origin xyz="0 0 0" rpy="0 0 0"/>
-    <mass value="0.2"/>
-    <inertia ixx="0.00014" iyy="0.00014" izz="0.00025" ixy="0.0" iyz="0.0" ixz="0.0"/>
-  </inertial>
+    <inertial>
+      <origin xyz="${-chassis_length*0.5} 0.0 ${chassis_height*0.5}" rpy="0 0.0 0.0"/>
+      <mass value="${chassis_mass}"/>
+      <xacro:box_inertia m="${chassis_mass}" x="${chassis_length}" y="${chassis_width}" z="${chassis_height}"/>
+    </inertial>
     <visual>
       <origin xyz="0.0 0.0 0.0" rpy="0 0.0 -${pi/2}"/>
       <geometry>
-        <mesh scale="${0.1/scale_factor} ${0.1/scale_factor}  ${0.1/scale_factor}" filename="file://$(find perseus_description)/meshes/chassis.dae"/>
+        <mesh scale="0.1 0.1  0.1" filename="file://$(find perseus_description)/meshes/chassis.dae"/>
       </geometry>
     </visual>
     <collision>
-      <origin xyz="0.0 0.0 0.0" rpy="0 0.0 -${pi/2}"/>
+      <origin xyz="${-chassis_length*0.5} 0.0 ${chassis_height*0.5}" rpy="0 0.0 0"/>
       <!-- Modified to make collision more simple, chassis mesh replaced with box -->
       <geometry>
-        <mesh scale="${0.1/scale_factor} ${0.1/scale_factor}  ${0.1/scale_factor}" filename="file://$(find perseus_description)/meshes/chassis.dae"/>
+        <box size="${chassis_length} ${chassis_width} ${chassis_height}"/>
       </geometry>
     </collision>
@@ -28,4 +28,5 @@
           <visualize>true</visualize>
           <topic>imu</topic>
+          <!-- Add frame id to imu sensor (achieving correct frame association)-->
           <gz_frame_id>${prefix}base_link</gz_frame_id>
       </sensor>

File: software/ros_ws/src/perseus_description/urdf/flange_bearing.urdf.xacro (robot description, xacro)
@@ -4,18 +4,18 @@
 <link name="${prefix}flange_bearing">
     <inertial>
-    <origin xyz="0.0 0.0 0.0" rpy="0 0 0"/>
-    <mass value="1"/>
-    <inertia ixx="0.001313" iyy="0.001699" izz="0.000647" ixy="0.0" iyz="0.0" ixz="-0.0"/>
+    <origin xyz="0.0 0.0 0.0" rpy="${-pi/2} 0 ${pi/2}"/>
+    <mass value="${bearing_mass}"/>
+    <xacro:box_inertia m="${bearing_mass}" x="${bearing_length}" y="${bearing_width}" z="${bearing_height}"/>
     </inertial>
     <visual>
     <origin xyz="0.0 0.0 0.0" rpy="${-pi/2} 0 ${pi/2}"/>
     <geometry>
-        <mesh scale="${0.1/scale_factor} ${0.1/scale_factor}  ${0.1/scale_factor}" filename="file://$(find perseus_description)/meshes/flange_bearing.dae"/>
+        <mesh scale="0.1 0.1  0.1" filename="file://$(find perseus_description)/meshes/flange_bearing.dae"/>
     </geometry>
     </visual>
     <collision>
-    <origin xyz="0.0 0.0 0.0" rpy="0 0 0"/>
+    <origin xyz="0.0 0.0 0.0" rpy="${-pi/2} 0 ${pi/2}"/>
     <geometry>
-        <mesh scale="${0.1/scale_factor} ${0.1/scale_factor}  ${0.1/scale_factor}" filename="file://$(find perseus_description)/meshes/flange_bearing.dae"/>
+        <box size="${bar_length} ${bar_width} ${bar_height}"/>
     </geometry>
     </collision>
@@ -25,11 +25,11 @@
     <inertial>
         <origin xyz="0 0 0.0" rpy="0.0 0.0 0.0"/>
-        <mass value="0.9172649518127158"/>
-        <inertia ixx="0.00036" iyy="0.018339" izz="0.018134" ixy="3e-06" iyz="-0.0" ixz="0.0"/>
+        <mass value="${bar_mass}"/>
+        <xacro:box_inertia m="${bar_mass}" x="${bar_length}" y="${bar_width}" z="${bar_height}"/>
     </inertial>
     <visual>
     <origin xyz="0.0 0.0 0.0" rpy="${-pi/2} 0 ${-pi/2}"/>
     <geometry>
-        <mesh scale="${0.1/scale_factor} ${0.1/scale_factor}  ${0.1/scale_factor}" filename="file://$(find perseus_description)/meshes/differential_bar.dae"/>
+        <mesh scale=  "0.1 0.1  0.1" filename="file://$(find perseus_description)/meshes/differential_bar.dae"/>
     </geometry>
     </visual>
@@ -37,10 +37,10 @@
     <origin xyz="0.0 0.0 0.0" rpy="${-pi/2} 0 ${-pi/2}"/>
     <geometry>
-        <mesh scale="${0.1/scale_factor} ${0.1/scale_factor}  ${0.1/scale_factor}" filename="file://$(find perseus_description)/meshes/differential_bar.dae"/>
+        <box size="${bar_length} ${bar_width} ${bar_height}"/>
     </geometry>
     </collision>
 </link>
 <joint name="${prefix}differential_bar_joint" type="fixed">
-    <origin xyz="${-0.05/scale_factor} 0.0 0.0" rpy="0 0.0 0"/>
+    <origin xyz="${-0.05} 0.0 0.0" rpy="0 0.0 0"/>
     <axis xyz="0.0 0.0 1.0"/>
     <parent link="${prefix}flange_bearing"/>

File: software/ros_ws/src/perseus_description/urdf/motor_wheel.urdf.xacro (robot description, xacro)
@@ -1,87 +1,58 @@
 <?xml version="1.0"?>
 <robot name="motor_wheel" xmlns:xacro="http://www.ros.org/wiki/xacro">
-  <link name="${prefix}front_right_motor">
-    <inertial>
-      <!-- moving origin has no perceivable impact-->
-      <origin xyz="0 0.0 0.0" rpy="0.0 0.0 ${pi/2}"/>
-      <mass value="1"/>
-      <inertia ixx="0.01" iyy="0.01" izz="0.01" ixy="0.0" iyz="0.0" ixz="0.0"/> <!-- TEMP -->
-    </inertial>
-    <visual>
-      <origin xyz="0 0.0 0.0" rpy="0.0 0.0 ${pi/2}"/>
-      <geometry>
-        <mesh scale="${0.1/scale_factor} ${0.1/scale_factor}  ${0.1/scale_factor}" filename="file://$(find perseus_description)/meshes/gearbox.dae"/>
-      </geometry>
-      <!-- <material name="white"/> -->
-    </visual>
-    <collision>
-      <origin xyz="0 0.0 0.0" rpy="0.0 0.0 ${pi/2}"/>
-      <geometry>
-        <mesh scale="${0.1/scale_factor} ${0.1/scale_factor}  ${0.1/scale_factor}" filename="file://$(find perseus_description)/meshes/gearbox.dae"/>
-      </geometry>
-    </collision>
-  </link>
-  <link name="${prefix}rear_right_motor">
-    <inertial>
-      <!-- moving origin has no perceivable impact-->
-      <origin xyz="0 0.0 0.0" rpy="0.0 0.0 ${pi/2}"/>
-      <mass value="1"/>
-      <inertia ixx="0.01" iyy="0.01" izz="0.01" ixy="0.0" iyz="0.0" ixz="0.0"/> <!-- TEMP -->
-    </inertial>
-    <visual>
-      <origin xyz="0 0.0 0.0" rpy="0.0 0.0 ${pi/2}"/>
-      <geometry>
-        <mesh scale="${0.1/scale_factor} ${0.1/scale_factor}  ${0.1/scale_factor}" filename="file://$(find perseus_description)/meshes/gearbox.dae"/>
-      </geometry>
-      <!-- <material name="white"/> -->
-    </visual>
-    <collision>
-      <origin xyz="0 0.0 0.0" rpy="0.0 0.0 ${pi/2}"/>
-      <geometry>
-        <mesh scale="${0.1/scale_factor} ${0.1/scale_factor}  ${0.1/scale_factor}" filename="file://$(find perseus_description)/meshes/gearbox.dae"/>
-      </geometry>
-    </collision>
-  </link>
-  <link name="${prefix}front_left_motor">
-    <inertial>
-      <!-- moving origin has no perceivable impact-->
-      <origin xyz="0.0 0.0 0.0" rpy="0.0 0.0 0.0"/>
-      <mass value="1"/>
-      <inertia ixx="0.01" iyy="0.01" izz="0.01" ixy="0.0" iyz="0.0" ixz="0.0"/> <!-- TEMP -->
-    </inertial>
-    <visual>
-      <origin xyz="0 0.0 0.0" rpy="0.0 0.0 ${-pi/2}"/>
-      <geometry>
-        <mesh scale="${0.1/scale_factor} ${0.1/scale_factor}  ${0.1/scale_factor}" filename="file://$(find perseus_description)/meshes/gearbox.dae"/>
-      </geometry>
-      <!-- <material name="white"/> -->
-    </visual>
-    <collision>
-      <origin xyz="0 0.0 0.0" rpy="0.0 0.0 ${-pi/2}"/>
-      <geometry>
-        <mesh scale="${0.1/scale_factor} ${0.1/scale_factor}  ${0.1/scale_factor}" filename="file://$(find perseus_description)/meshes/gearbox.dae"/>
-      </geometry>
-    </collision>
-  </link>
-  <link name="${prefix}rear_left_motor">
-    <inertial>
-      <!-- moving origin has no perceivable impact-->
-      <origin xyz="0.0 0.0 0.0" rpy="0.0 0.0 0.0"/>
-      <mass value="1"/>
-      <inertia ixx="0.01" iyy="0.01" izz="0.01" ixy="0.0" iyz="0.0" ixz="0.0"/> <!-- TEMP -->
-    </inertial>
-    <visual>
-      <origin xyz="0 0.0 0.0" rpy="0.0 0.0 ${-pi/2}"/>
-      <geometry>
-        <mesh scale="${0.1/scale_factor} ${0.1/scale_factor}  ${0.1/scale_factor}" filename="file://$(find perseus_description)/meshes/gearbox.dae"/>
-      </geometry>
-      <!-- <material name="white"/> -->
-    </visual>
-    <collision>
-      <origin xyz="0 0.0 0.0" rpy="0.0 0.0 ${-pi/2}"/>
-      <geometry>
-        <mesh scale="${0.1/scale_factor} ${0.1/scale_factor}  ${0.1/scale_factor}" filename="file://$(find perseus_description)/meshes/gearbox.dae"/>
-      </geometry>
-    </collision>
-  </link>
+  <xacro:macro name="motor" params="prefix:=^ side:=^ end:=^">
+    <link name="${prefix}${end}_${side}_motor">
+      <inertial>
+        <!-- moving origin has no perceivable impact-->
+        <origin xyz="0.0 0.0 0.0" rpy="0.0 0.0 0.0"/>
+        <mass value="${motor_mass}"/>
+        <inertia ixx="0.01" iyy="0.01" izz="0.01" ixy="0.0" iyz="0.0" ixz="0.0"/> <!-- TEMP -->
+      </inertial>
+      <visual>
+        <xacro:if value="${side == 'left'}">
+          <origin xyz="0 0.0 0.0" rpy="0.0 0.0 ${-pi/2}"/>
+        </xacro:if>
+        <xacro:if value="${side == 'right'}">
+          <origin xyz="0 0.0 0.0" rpy="0.0 0.0 ${pi/2}"/>
+        </xacro:if>
+        <geometry>
+          <mesh scale="0.1 0.1  0.1" filename="file://$(find perseus_description)/meshes/gearbox.dae"/>
+        </geometry>
+        <!-- <material name="white"/> -->
+      </visual>
+      <collision>
+        <xacro:if value="${side == 'left'}">
+          <origin xyz="0.0 0.0 0.0" rpy="0.0 0.0 ${pi/2}"/>
+        </xacro:if>
+        <xacro:if value="${side == 'right'}">
+          <origin xyz="0.0 0.0 0.0" rpy="0.0 0.0 ${-pi/2}"/>
+        </xacro:if>
+        <geometry>
+          <box size="${collision_motor_length} ${collision_motor_width} ${collision_motor_height}" />
+        </geometry>
+      </collision>
+    </link>
+    <joint name="${prefix}${end}_${side}_motor_joint" type="fixed">
+      <parent link="${prefix}${side}_rocker"/>
+      <child link="${prefix}${end}_${side}_motor"/>
+      <xacro:if value="${end == 'front'}">
+        <xacro:if value="${side == 'left'}">
+          <origin xyz="${front_motors_x_offset} -${motors_y_offset} ${motors_z_offset}" rpy="0.0 0.0 0.0"/>
+        </xacro:if>
+        <xacro:if value="${side == 'right'}">
+          <origin xyz="${front_motors_x_offset} ${motors_y_offset} ${motors_z_offset}" rpy="0.0 0.0 0.0"/>
+        </xacro:if>
+      </xacro:if>
+      <xacro:if value="${end == 'rear'}">
+        <xacro:if value="${side == 'left'}">
+          <origin xyz="${rear_motors_x_offset} -${motors_y_offset} ${motors_z_offset}" rpy="0.0 0.0 0.0"/>
+        </xacro:if>
+        <xacro:if value="${side == 'right'}">
+          <origin xyz="${rear_motors_x_offset} ${motors_y_offset} ${motors_z_offset}" rpy="0.0 0.0 0.0"/>
+        </xacro:if>
+      </xacro:if>
+    </joint>
+  <!-- ADD 1 WHEEL FOR EACH MOTOR -->
+  <xacro:wheel prefix="" side="${side}"  end="${end}"/>
+  </xacro:macro>
 </robot>
