Commit message: Add inertia macros and refactor URDF files for Perseus robot
- Introduced inertia macros in `inertia_macros.xacro` for box, cylinder, and sphere inertia calculations.
- Refactored `motor_wheel.urdf.xacro` to use a macro for motor and wheel definitions, reducing redundancy.
- Updated `perseus.urdf.xacro` to include new properties for motors, rockers, and sensors, and streamlined component inclusion.
- Modified `rocker.urdf.xacro` to implement a macro for rocker links and associated motors.
- Enhanced `sensors.urdf.xacro` to include inertial properties for LIDAR components.
- Simplified `wheel.urdf.xacro` by creating a macro for wheel definitions, including inertia calculations.
- Adjusted `gz_bridge.yaml` to change Gazebo topic names for better integration with ROS.

File: software/ros_ws/src/perseus_description/urdf/perseus.urdf.xacro (robot description, xacro)
@@ -2,110 +2,90 @@
 <robot xmlns:xacro="http://ros.org/wiki/xacro">
   <xacro:macro name="perseus" params="prefix">
-    <!-- Constants for robot dimensions -->
-    <xacro:property name="scale_factor" value="1"/>  <!-- 1 for Perseus and 2 for Perseu_Lite -->
-    <xacro:property name="PI" value="3.1415926535897931"/>
-    <xacro:property name="base_mass" value="0.3" /> <!-- arbitrary value for base mass -->
-    <xacro:property name="chassis_width" value="0.1" />
+    <!-- Motors Properties -->
+    <xacro:property name="motors_y_offset" value="0.035"/>
+    <xacro:property name="motors_z_offset" value="-0.25"/>
+    <xacro:property name="front_motors_x_offset" value="0.3"/>
+    <xacro:property name="rear_motors_x_offset" value="-0.55"/>
+    <xacro:property name="motor_mass" value="5.236579"/>  <!-- Kg -->
+    <xacro:property name="collision_motor_length" value="0.1"/>  <!-- m -->
+    <xacro:property name="collision_motor_width" value="0.1"/>  <!-- m -->
+    <xacro:property name="collision_motor_height" value="0.075"/>  <!-- m -->
+    <!-- Rocker properties -->
+    <xacro:property name="rocker_mass" value="0.5"/>
+    <xacro:property name="rocker_length" value="${(front_motors_x_offset-rear_motors_x_offset)*1/2}"/>  <!-- Use positive absolute value -->
+    <xacro:property name="rocker_width" value="0.03"/>
+    <xacro:property name="rocker_collision_x_offset" value="-0.10"/>
+    <xacro:property name="rocker_height" value="0.2"/>
+    <xacro:property name="rocker_base_distance" value="0.275" />
+    <xacro:property name="rocker_x_offset" value="0.075"/>
+    <xacro:property name="rocker_y_offset" value="0.05"/>
+    <!-- Wheels Properties -->
+    <xacro:property name="wheel_mass" value="1.0"/>
+    <xacro:property name="wheels_y_offset" value="0.125"/>
+    <xacro:property name="wheel_radius" value="0.15"/>
+    <xacro:property name="wheel_length" value="0.14"/>
+    <!-- Chassis Properties -->
+    <xacro:property name="chassis_mass" value="2.7689940302592726"/>  <!-- Kg -->
+    <xacro:property name="chassis_width" value="0.45" />
     <xacro:property name="chassis_length" value="0.6" />
-    <xacro:property name="chassis_height" value="0.05" />
-    <xacro:property name="chassis_z_offset" value="0.35" /> <!-- Space btw top of beam and the each joint -->
-    <xacro:property name="flange_bearing_z_offset" value="0.1"/>  <!-- 1 for Perseus and 2 for Perseu_Lite -->
-    <xacro:property name="rocker_base_distance" value="0.275" />
-    <xacro:property name="rocker_x_offset" value="0.075"/>  <!-- 1 for Perseus and 2 for Perseu_Lite -->
-    <xacro:property name="rocker_y_offset" value="0.05"/>  <!-- 1 for Perseus and 2 for Perseu_Lite -->
-    <xacro:property name="motors_y_offset" value="0.035"/>  <!-- 1 for Perseus and 2 for Perseu_Lite -->
-    <xacro:property name="motors_z_offset" value="-0.25"/>  <!-- 1 for Perseus and 2 for Perseu_Lite -->
-    <xacro:property name="front_motors_x_offset" value="0.3"/>  <!-- 1 for Perseus and 2 for Perseu_Lite -->
-    <xacro:property name="rear_motors_x_offset" value="-0.55"/>  <!-- 1 for Perseus and 2 for Perseu_Lite -->
-    <xacro:property name="wheels_y_offset" value="0.125"/>
+    <xacro:property name="chassis_height" value="0.2" />
+    <xacro:property name="chassis_z_offset" value="${rocker_height + wheel_radius}" /> <!-- Space btw top of beam and the each joint -->
+    <!-- Flange Bearing Properties -->
+    <xacro:property name="bearing_mass" value="2.7689940302592726"/>  <!-- Kg -->
+    <xacro:property name="flange_bearing_z_offset" value="${chassis_height/2}"/>
+    <xacro:property name="bearing_length" value="0.2"/>
+    <xacro:property name="bearing_width" value="0.03"/>
+    <xacro:property name="bearing_height" value="0.03"/>
+    <!-- Differential Bar Properties -->
+    <xacro:property name="bar_mass" value="0.917264951812715"/>
+    <xacro:property name="bar_length" value="0.58"/>
+    <xacro:property name="bar_width" value="0.03"/>
+    <xacro:property name="bar_height" value="0.03"/>
+    <!-- Depth Camera Properties -->
+    <xacro:property name="camera_mass" value="0.1"/>
+    <xacro:property name="camera_width" value="0.07"/>
+    <xacro:property name="camera_height" value="0.03"/>
+    <xacro:property name="camera_depth" value="0.020"/>
+    <!-- 2D and 3D LIDAR Properties -->
+    <xacro:property name="laser_2d_mass" value="0.1"/>
+    <xacro:property name="laser_2d_radius" value="0.04"/>
+    <xacro:property name="laser_2d_length" value="0.04"/>
+    <xacro:property name="laser_3d_mass" value="0.2"/>
+    <xacro:property name="laser_3d_radius" value="0.06"/>
+    <xacro:property name="laser_3d_length" value="0.06"/>
     <!-- ADD COMPONENTS -->
+    <xacro:include filename="$(find perseus_description)/urdf/inertia_macros.xacro"/>
     <xacro:include filename="$(find perseus_description)/urdf/chassis.urdf.xacro"/>
     <xacro:include filename="$(find perseus_description)/urdf/flange_bearing.urdf.xacro"/>
+    <xacro:include filename="$(find perseus_description)/urdf/wheel.urdf.xacro"/>
+    <xacro:include filename="$(find perseus_description)/urdf/motor_wheel.urdf.xacro"/>
     <xacro:include filename="$(find perseus_description)/urdf/rocker.urdf.xacro"/>
-    <xacro:include filename="$(find perseus_description)/urdf/motor_wheel.urdf.xacro"/>
-    <xacro:include filename="$(find perseus_description)/urdf/wheel.urdf.xacro"/>
     <xacro:include filename="$(find perseus_description)/urdf/sensors.urdf.xacro"/>
     <xacro:include filename="$(find perseus_description)/urdf/camera_depth.urdf.xacro" />
-    <!-- <xacro:camera_depth prefix="$(prefix)" /> -->
     <!-- An empty base_link to attach everything to -->
     <link name="${prefix}base_link"/>
-    <link name="${prefix}base_footprint"/>  <!-- 2D footprint for SLAM & navigation -->
-    <joint name="${prefix}base_to_footprint" type="fixed">
-      <origin xyz="0 0 0" rpy="0 0 0"/>
-      <parent link="${prefix}chassis"/>
-      <child link="${prefix}base_footprint"/>
-    </joint>
     <joint name="${prefix}chassis_joint" type="fixed"> <!-- Joint Connect base_link and chassis -->
-      <origin xyz="0.3 0.0 ${chassis_z_offset/scale_factor}" rpy="0 0.0 0.0"/>
+      <origin xyz="0 0.0 ${chassis_z_offset}" rpy="0.0 0.0 0.0"/>
       <parent link="${prefix}base_link"/>
       <child link="${prefix}chassis"/>
     </joint>
+    <link name="${prefix}base_footprint"/>
+    <joint name="base_footprint_joint" type="fixed">
+        <parent link="${prefix}base_link"/>
+        <child link="${prefix}base_footprint"/>
+        <origin xyz="0 0 0" rpy="0 0 0"/>
+    </joint>
+    <!-- ADD 2 ROCKERS (INCLUDING 4 MOTORS + 4 WHEELS) -->
+    <xacro:rocker prefix="" side="left"/>
+    <xacro:rocker prefix="" side="right"/>
     <joint name="${prefix}flange_bearing_joint" type="fixed">
-      <origin xyz="${-chassis_length/scale_factor} 0.0 ${flange_bearing_z_offset/scale_factor}" rpy="0 0 0"/>
+      <origin xyz="${-chassis_length} 0.0 ${flange_bearing_z_offset}" rpy="0 0 0"/>
       <parent link="${prefix}chassis"/>
       <child link="${prefix}flange_bearing"/>
-    </joint>
-    <joint name="${prefix}left_rocker_joint" type="fixed">
-      <origin xyz="${-rocker_x_offset/scale_factor} ${rocker_base_distance/scale_factor} ${rocker_y_offset/scale_factor} " rpy="0 0 0"/>
-      <parent link="${prefix}chassis"/>
-      <child link="${prefix}left_rocker"/>
-    </joint>
-    <joint name="${prefix}right_rocker_joint" type="fixed">
-      <origin xyz="${-rocker_x_offset/scale_factor} ${-rocker_base_distance/scale_factor} ${rocker_y_offset/scale_factor} " rpy="0 0 0"/>
-      <parent link="${prefix}chassis"/>
-      <child link="${prefix}right_rocker"/>
-    </joint>
-    <joint name="${prefix}front_left_motor_joint" type="fixed">
-      <parent link="${prefix}left_rocker"/>
-      <child link="${prefix}front_left_motor"/>
-      <origin xyz="${front_motors_x_offset/scale_factor} -${motors_y_offset/scale_factor} ${motors_z_offset/scale_factor}" rpy="0.0 0.0 0"/>
-    </joint>
-    <joint name="${prefix}rear_left_motor_joint" type="fixed">
-      <parent link="${prefix}left_rocker"/>
-      <child link="${prefix}rear_left_motor"/>
-      <origin xyz="${rear_motors_x_offset/scale_factor} -${motors_y_offset/scale_factor} ${motors_z_offset/scale_factor}" rpy="0.0 0.0 0.0"/>
-    </joint>
-    <joint name="${prefix}front_right_motor_joint" type="fixed">
-      <parent link="${prefix}right_rocker"/>
-      <child link="${prefix}front_right_motor"/>
-      <origin xyz="${front_motors_x_offset/scale_factor} ${motors_y_offset/scale_factor} ${motors_z_offset/scale_factor}" rpy="0.0 0.0 0"/>
-    </joint>
-    <joint name="${prefix}rear_right_motor_joint" type="fixed">
-      <parent link="${prefix}right_rocker"/>
-      <child link="${prefix}rear_right_motor"/>
-      <origin xyz="${rear_motors_x_offset/scale_factor} ${motors_y_offset/scale_factor} ${motors_z_offset/scale_factor}" rpy="0.0 0.0 0.0"/>
-    </joint>
-    <joint name="${prefix}front_left_wheel_joint" type="continuous">
-      <axis xyz="0 1 0" rpy="0 0 0"/>
-      <parent link="${prefix}front_left_motor"/>
-      <child link="${prefix}front_left_wheel"/>
-      <origin xyz="0 ${wheels_y_offset/scale_factor} 0.0" rpy="0.0 0.0 0"/>
-      <dynamics damping="0.2" friction="0.3"/>
-    </joint>
-    <joint name="${prefix}rear_left_wheel_joint" type="continuous">
-      <axis xyz="0 1 0" rpy="0 0 0"/>
-      <parent link="${prefix}rear_left_motor"/>
-      <child link="${prefix}rear_left_wheel"/>
-      <origin xyz="0 ${wheels_y_offset/scale_factor} 0.0" rpy="0.0 0.0 0"/>
-      <dynamics damping="0.2" friction="0.3"/>
-    </joint>
-    <joint name="${prefix}front_right_wheel_joint" type="continuous">
-      <axis xyz="0 1 0" rpy="0 0 0"/>
-      <parent link="${prefix}front_right_motor"/>
-      <child link="${prefix}front_right_wheel"/>
-      <origin xyz="0 -${wheels_y_offset/scale_factor} 0.0" rpy="0.0 0.0 0"/>
-      <dynamics damping="0.2" friction="0.3"/>
-    </joint>
-    <joint name="${prefix}rear_right_wheel_joint" type="continuous">
-      <axis xyz="0 1 0" rpy="0 0 0"/>
-      <parent link="${prefix}rear_right_motor"/>
-      <child link="${prefix}rear_right_wheel"/>
-      <origin xyz="0 -${wheels_y_offset/scale_factor} 0.0" rpy="0.0 0.0 0"/>
-      <dynamics damping="0.2" friction="0.3"/>
     </joint>
     <joint name="${prefix}laser_joint" type="fixed">
       <parent link="${prefix}chassis"/>
       <child link="${prefix}laser_frame"/>
-      <origin xyz="0 0 -0.035" rpy="0 ${PI} 0"/>
+      <origin xyz="0 0 -0.04" rpy="0 ${pi} 0"/>
     </joint>
     <joint name="${prefix}laser_2d_joint" type="fixed">

File: software/ros_ws/src/perseus_description/urdf/rocker.urdf.xacro (robot description, xacro)
@@ -1,35 +1,46 @@
 <?xml version="1.0"?>
 <robot name="rocker" xmlns:xacro="http://ros.org/wiki/xacro">
-  <link name="${prefix}left_rocker">
-    <!-- <inertial>
-    </inertial> -->
+  <!-- ROCKER LINK -->
+  <xacro:macro name="rocker" params="prefix:=^ side:=^">
+  <link name="${prefix}${side}_rocker">
+    <inertial>
+      <origin xyz="${rocker_collision_x_offset} 0.0 -${rocker_height}" rpy="0.0 0.0 0.0"/>
+      <mass value="${rocker_mass}"/>
+      <xacro:box_inertia m="${rocker_mass}"
+                         x="${rocker_length}"
+                         y="${rocker_width}"
+                         z="${rocker_height}"/>
+    </inertial>
     <visual>
       <origin xyz="0.0 0.0 0.0" rpy="0.0 0.0 ${pi}"/>
       <geometry>
-        <mesh scale="${0.1/scale_factor} ${0.1/scale_factor}  ${0.1/scale_factor}" filename="file://$(find perseus_description)/meshes/rocker_left.dae"/>
+      <xacro:if value="${side == 'left'}">
+        <mesh scale="0.1 0.1 0.1" filename="file://$(find perseus_description)/meshes/rocker_left.dae"/>
+      </xacro:if>
+      <xacro:if value="${side == 'right'}">
+        <mesh scale="0.1 0.1 0.1" filename="file://$(find perseus_description)/meshes/rocker_right.dae"/>
+      </xacro:if>
       </geometry>
     </visual>
     <collision>
-      <origin xyz="0.0 0.0 0.0" rpy="0.0 0.0 ${pi}"/>
+      <origin xyz="${rocker_collision_x_offset} 0.0 -${rocker_height}" rpy="0.0 0.0 0.0"/>
       <geometry>
-        <mesh scale="${0.1/scale_factor} ${0.1/scale_factor}  ${0.1/scale_factor}" filename="file://$(find perseus_description)/meshes/rocker_left.dae"/>
+        <box size="${rocker_length} ${rocker_width} ${rocker_height}"/>
       </geometry>
     </collision>
   </link>
-  <link name="${prefix}right_rocker">
-    <!-- <inertial>
-    </inertial> -->
-    <visual>
-      <origin xyz="0.0 0.0 0.0" rpy="0.0 0.0 ${pi}"/>
-      <geometry>
-        <mesh scale="${0.1/scale_factor} ${0.1/scale_factor}  ${0.1/scale_factor}" filename="file://$(find perseus_description)/meshes/rocker_right.dae"/>
-      </geometry>
-    </visual>
-    <collision>
-      <origin xyz="0.0 0.0 0.0" rpy="0.0 0.0 ${pi}"/>
-      <geometry>
-        <mesh scale="${0.1/scale_factor} ${0.1/scale_factor}  ${0.1/scale_factor}" filename="file://$(find perseus_description)/meshes/rocker_right.dae"/>
-      </geometry>
-    </collision>
-  </link>
+  <joint name="${prefix}${side}_rocker_joint" type="fixed">
+    <xacro:if value="${side == 'left'}">
+      <origin xyz="${-rocker_x_offset} ${rocker_base_distance} ${rocker_y_offset} " rpy="0 0 0"/>
+    </xacro:if>
+    <xacro:if value="${side == 'right'}">
+      <origin xyz="${-rocker_x_offset} -${rocker_base_distance} ${rocker_y_offset} " rpy="0 0 0"/>
+    </xacro:if>
+    <parent link="${prefix}chassis"/>
+    <child link="${prefix}${side}_rocker"/>
+  </joint>
+  <!-- ADD 2 MOTORS FOR EACH SIDE -->
+  <xacro:motor prefix="" side="${side}"  end="front"/>
+  <xacro:motor prefix="" side="${side}"  end="rear"/>
+  </xacro:macro>
 </robot>

File: software/ros_ws/src/perseus_description/urdf/sensors.urdf.xacro (robot description, xacro)
@@ -3,8 +3,13 @@
 <!-- 3D LIDAR (Existing - Livox MID-360) -->
 <link name="${prefix}laser_frame">
+    <inertial>
+        <origin xyz="0 0 0"/>
+        <mass value="${laser_3d_mass}"/>
+        <xacro:box_inertia m="${laser_3d_mass}" x="${laser_3d_length}" y="${laser_3d_radius}" z="${laser_3d_radius}"/>
+    </inertial>
     <visual>
         <origin xyz="0 0 0"/>
         <geometry>
-            <cylinder radius="0.06" length="0.06"/>
+            <cylinder radius="${laser_3d_radius}" length="${laser_3d_length}"/>
         </geometry>
         <material name="black"/>
@@ -12,5 +17,5 @@
     <collision>
         <geometry>
-            <cylinder radius="0.06" length="0.06"/>
+            <cylinder radius="${laser_3d_radius}" length="${laser_3d_length}"/>
         </geometry>
     </collision>
@@ -18,8 +23,13 @@
 <!-- 2D LIDAR -->
 <link name="${prefix}laser_2d_frame">
+    <inertial>
+        <origin xyz="0 0 0"/>
+        <mass value="${laser_2d_mass}"/>
+        <xacro:box_inertia m="${laser_2d_mass}" x="${laser_2d_length}" y="${laser_2d_radius}" z="${laser_2d_radius}"/>
+    </inertial>
     <visual>
         <origin xyz="0 0 0"/>
         <geometry>
-            <cylinder radius="0.04" length="0.04"/>
+            <cylinder radius="${laser_2d_radius}" length="${laser_2d_length}"/>
         </geometry>
         <material name="blue">
