Commit message: Add inertia macros and refactor URDF files for Perseus robot
- Introduced inertia macros in `inertia_macros.xacro` for box, cylinder, and sphere inertia calculations.
- Refactored `motor_wheel.urdf.xacro` to use a macro for motor and wheel definitions, reducing redundancy.
- Updated `perseus.urdf.xacro` to include new properties for motors, rockers, and sensors, and streamlined component inclusion.
- Modified `rocker.urdf.xacro` to implement a macro for rocker links and associated motors.
- Enhanced `sensors.urdf.xacro` to include inertial properties for LIDAR components.
- Simplified `wheel.urdf.xacro` by creating a macro for wheel definitions, including inertia calculations.
- Adjusted `gz_bridge.yaml` to change Gazebo topic names for better integration with ROS.

File: software/ros_ws/src/perseus_description/urdf/wheel.urdf.xacro (robot description, xacro)
@@ -1,135 +1,70 @@
 <?xml version="1.0"?>
 <robot name="wheel" xmlns:xacro="http://ros.org/wiki/xacro">
-<link name="${prefix}front_left_wheel">
-  <inertial>
-    <origin xyz="0 0 0" rpy="0 0 0"/>
-    <mass value="0.2"/>
-    <inertia ixx="0.00014" iyy="0.00014" izz="0.00025" ixy="0.0" iyz="0.0" ixz="0.0"/>
-  </inertial>
-  <visual>
-    <origin xyz="0.0 0.0  0.0" rpy="0.0 0.0 ${pi}"/>
-    <geometry>
-      <mesh scale="${0.1/scale_factor} ${0.1/scale_factor}  ${0.1/scale_factor}" filename="file://$(find perseus_description)/meshes/wheel.dae"/>
-    </geometry>
-  </visual>
-  <collision>
-    <origin xyz="0.0 0.0 0.0" rpy="0.0 0.0 ${pi}"/>
-    <geometry>
-      <mesh scale="${0.1/scale_factor} ${0.1/scale_factor}  ${0.1/scale_factor}" filename="file://$(find perseus_description)/meshes/wheel.dae"/>
-    </geometry>
-  </collision>
-</link>
-<link name="${prefix}front_right_wheel">
-  <inertial>
-    <origin xyz="0 0 0" rpy="0 0 0"/>
-    <mass value="0.2"/>
-    <inertia ixx="0.00014" iyy="0.00014" izz="0.00025" ixy="0.0" iyz="0.0" ixz="0.0"/>
-  </inertial>
-  <visual>
-      <origin xyz="0.0 0.0  0.0" rpy="0.0 0.0 0.0"/>
-    <geometry>
-      <mesh scale="${0.1/scale_factor} ${0.1/scale_factor}  ${0.1/scale_factor}" filename="file://$(find perseus_description)/meshes/wheel.dae"/>
-    </geometry>
-  </visual>
-  <collision>
-    <origin xyz="0.0 0.0 0.0" rpy="0.0 0.0 0.0"/>
-    <geometry>
-      <mesh scale="${0.1/scale_factor} ${0.1/scale_factor}  ${0.1/scale_factor}" filename="file://$(find perseus_description)/meshes/wheel.dae"/>
-    </geometry>
-  </collision>
-</link>
-<link name="${prefix}rear_left_wheel">
-  <inertial>
-    <origin xyz="0 0 0" rpy="0 0 0"/>
-    <mass value="0.2"/>
-    <inertia ixx="0.00014" iyy="0.00014" izz="0.00025" ixy="0.0" iyz="0.0" ixz="0.0"/>
-  </inertial>
-  <visual>
-      <origin xyz="0.0 0.0  0.0" rpy="0.0 0.0 ${pi}"/>
-    <geometry>
-      <mesh scale="${0.1/scale_factor} ${0.1/scale_factor}  ${0.1/scale_factor}" filename="file://$(find perseus_description)/meshes/wheel.dae"/>
-    </geometry>
-  </visual>
-  <collision>
-    <origin xyz="0.0 0.0 0.0" rpy="0.0 0.0 ${pi}"/>
-    <geometry>
-      <mesh scale="${0.1/scale_factor} ${0.1/scale_factor}  ${0.1/scale_factor}" filename="file://$(find perseus_description)/meshes/wheel.dae"/>
-    </geometry>
-  </collision>
-</link>
-<link name="${prefix}rear_right_wheel">
-  <inertial>
-    <origin xyz="0 0 0" rpy="0 0 0"/>
-    <mass value="0.2"/>
-    <inertia ixx="0.00014" iyy="0.00014" izz="0.00025" ixy="0.0" iyz="0.0" ixz="0.0"/>
-  </inertial>
-  <visual>
-      <origin xyz="0.0 0.0  0.0" rpy="0.0 0.0 0.0"/>
-    <geometry>
-      <mesh scale="${0.1/scale_factor} ${0.1/scale_factor}  ${0.1/scale_factor}" filename="file://$(find perseus_description)/meshes/wheel.dae"/>
-    </geometry>
-  </visual>
-  <collision>
-    <origin xyz="0.0 0.0 0.0" rpy="0.0 0.0 0.0"/>
-    <geometry>
-      <mesh scale="${0.1/scale_factor} ${0.1/scale_factor}  ${0.1/scale_factor}" filename="file://$(find perseus_description)/meshes/wheel.dae"/>
-    </geometry>
-  </collision>
-</link>
-<gazebo reference="${prefix}front_left_wheel">
-  <material>Gazebo/Orange</material>
-  <collision>
-    <surface>
-        <friction>
-            <ode>
-                <mu>0.01</mu>
-                <mu2>0.01</mu2>
-                <fdir1>1 0 0</fdir1>
-            </ode>
-        </friction>
-    </surface>
-  </collision>
-</gazebo>
-<gazebo reference="${prefix}front_right_wheel">
-  <material>Gazebo/Orange</material>
-  <collision>
-    <surface>
-        <friction>
-            <ode>
-                <mu>0.01</mu>
-                <mu2>0.01</mu2>
-                <fdir1>1 0 0</fdir1>
-            </ode>
-        </friction>
-    </surface>
-  </collision>
-</gazebo>
-<gazebo reference="${prefix}rear_right_wheel">
-  <material>Gazebo/Orange</material>
-  <collision>
-    <surface>
-        <friction>
-            <ode>
-                <mu>0.01</mu>
-                <mu2>0.01</mu2>
-                <fdir1>1 0 0</fdir1>
-            </ode>
-        </friction>
-    </surface>
-  </collision>
-</gazebo>
-<gazebo reference="${prefix}rear_left_wheel">
-  <material>Gazebo/Orange</material>
-  <collision>
-    <surface>
-        <friction>
-            <ode>
-                <mu>0.01</mu>
-                <mu2>0.01</mu2>
-                <fdir1>1 0 0</fdir1>
-            </ode>
-        </friction>
-    </surface>
-  </collision>
-</gazebo>
+<xacro:macro name="wheel" params="prefix:=^ side:=^ end:=^">
+  <link name="${prefix}${end}_${side}_wheel">
+    <inertial>
+      <origin xyz="0.0 0.0 0.0" rpy="0.0 0.0 0.0"/>
+      <mass value="${wheel_mass}"/>
+      <!-- Use Y-axis aligned cylinder inertia since wheels rotate around Y axis -->
+      <xacro:cylinder_inertia_y m="${wheel_mass}" radius="${wheel_radius}" length="${wheel_length}"/>
+    </inertial>
+    <visual>
+      <!-- Rotate mesh so tread pattern faces outward -->
+      <xacro:if value="${side == 'left'}">
+        <origin xyz="0.0 0.0 0.0" rpy="0.0 0.0 ${pi}"/>
+      </xacro:if>
+      <xacro:if value="${side == 'right'}">
+        <origin xyz="0.0 0.0 0.0" rpy="0.0 0.0 0.0"/>
+      </xacro:if>
+      <geometry>
+        <mesh scale="0.1 0.1 0.1" filename="file://$(find perseus_description)/meshes/wheel.dae"/>
+      </geometry>
+    </visual>
+    <collision>
+      <!-- Rotate cylinder 90° around X to align with Y axis (wheel axle) -->
+      <origin xyz="0.0 0.0 0.0" rpy="${pi/2} 0.0 0.0"/>
+      <geometry>
+        <cylinder radius="${wheel_radius}" length="${wheel_length}"/>
+      </geometry>
+    </collision>
+  </link>
+  <joint name="${prefix}${end}_${side}_wheel_joint" type="continuous">
+    <parent link="${prefix}${end}_${side}_motor"/>
+    <child link="${prefix}${end}_${side}_wheel"/>
+    <xacro:if value="${side == 'left'}">
+      <origin xyz="0.0 ${wheels_y_offset} 0.0" rpy="0.0 0.0 0.0"/>
+    </xacro:if>
+    <xacro:if value="${side == 'right'}">
+      <origin xyz="0.0 ${-wheels_y_offset} 0.0" rpy="0.0 0.0 0.0"/>
+    </xacro:if>
+    <!-- Axis -Y: positive velocity = forward motion (standard ROS/diff_drive convention) -->
+    <axis xyz="0 1 0"/>
+    <dynamics damping="0.2" friction="0.3"/>
+  </joint>
+  <gazebo reference="${prefix}${end}_${side}_wheel">
+    <!-- TODO: Fix the material tag (this isn't the proper way to do it, and spits out warnings) -->
+    <material>Gazebo/Orange</material>
+    <!-- see http://sdformat.org/spec?ver=1.12&elem=collision -->
+    <collision>
+      <surface>
+          <friction>
+              <ode>
+                  <!--
+                  Skid-steer friction setup:
+                  - mu: friction in fdir1 direction (forward/backward rolling)
+                  - mu2: friction perpendicular to fdir1 (sideways sliding for turning)
+                  - fdir1: primary friction direction in link frame
+                  -->
+                  <!-- Forward/backward friction - high to grip and drive -->
+                  <mu>1.5</mu>
+                  <!-- Sideways friction - low to allow skid steering -->
+                  <mu2>0.2</mu2>
+                  <!-- fdir1 points forward (X) in link frame -->
+                  <fdir1>1 0 0</fdir1>
+              </ode>
+          </friction>
+      </surface>
+    </collision>
+  </gazebo>
+</xacro:macro>
 </robot>

Commit message: Refactor SLAM Toolbox parameters, add autonomy launch file, and implement behavior tree nodes
- Updated slam_toolbox_params.yaml to modify frame names, mapping parameters, and resolution settings.
- Created autonomy.launch.py to launch SLAM and navigation stacks together.
- Added simulation map files (sim_map.pgm, sim_map.yaml, sim_map_serial.data, sim_map_serial.posegraph) for testing.
- Introduced perseus_bt_nodes package with behavior tree nodes: GetGoalFromGoals, IncrementIndex, and PopFirstGoal.
- Updated camera depth URDF to correct joint orientations.
- Increased IMU sensor update rate in chassis URDF.
- Added realsense_params.yaml for configuring RealSense camera parameters.
- Created realsense.launch.py to launch RealSense camera with parameters.
- Modified gazebo.launch.py to streamline the launch process with nixGL.
- Updated teleop widget in web UI to publish to '/cmd_vel_out' instead of '/web_vel'.

File: software/ros_ws/src/perseus_description/urdf/camera_depth.urdf.xacro (robot description, xacro)
@@ -22,5 +22,5 @@
         <parent link="${prefix}camera_link"/>
         <child link="${prefix}camera_link_optical"/>
-        <origin xyz="0 0 0" rpy="0 0 0"/>
+        <origin xyz="0 0 0" rpy="-1.57079632679 0 -1.57079632679"/>
     </joint>
     <link name="${prefix}camera_link_optical"></link>

File: software/ros_ws/src/perseus_description/urdf/chassis.urdf.xacro (robot description, xacro)
@@ -25,5 +25,5 @@
       <sensor name="imu_sensor" type="imu">
           <always_on>1</always_on>
-          <update_rate>10</update_rate>
+          <update_rate>50</update_rate>
           <visualize>true</visualize>
           <topic>imu</topic>

Commit message: Feat: Update URDF and configuration for camera and lidar integration to meet with current topics name, position and orientation.

File: software/ros_ws/src/perseus_description/urdf/camera_depth.urdf.xacro (robot description, xacro)
@@ -22,5 +22,5 @@
         <parent link="${prefix}camera_link"/>
         <child link="${prefix}camera_link_optical"/>
-        <origin xyz="0 0 0" rpy="0 0 0"/>
+        <origin xyz="0 0 0" rpy="-1.57079632679 0 -1.57079632679"/>
     </joint>
     <link name="${prefix}camera_link_optical"></link>
@@ -44,5 +44,5 @@
             </camera>
             <topic>/perseus/rgbd_camera</topic>
-            <gz_frame_id>${prefix}camera_link_optical</gz_frame_id>
+            <gz_frame_id>${prefix}camera_link</gz_frame_id>
             <min_depth>0.05</min_depth>
             <max_depth>100.0</max_depth>

File: software/ros_ws/src/perseus_description/urdf/perseus.urdf.xacro (robot description, xacro)
@@ -44,14 +44,14 @@
     <!-- Depth Camera Properties -->
     <xacro:property name="camera_mass" value="0.1"/>
-    <xacro:property name="camera_width" value="0.07"/>
+    <xacro:property name="camera_width" value="0.12"/>
     <xacro:property name="camera_height" value="0.03"/>
-    <xacro:property name="camera_depth" value="0.020"/>
+    <xacro:property name="camera_depth" value="0.025"/>
     <!-- 2D and 3D LIDAR Properties -->
     <xacro:property name="laser_2d_mass" value="0.1"/>
     <xacro:property name="laser_2d_radius" value="0.04"/>
     <xacro:property name="laser_2d_length" value="0.04"/>
-    <xacro:property name="laser_3d_mass" value="0.2"/>
-    <xacro:property name="laser_3d_radius" value="0.06"/>
-    <xacro:property name="laser_3d_length" value="0.06"/>
+    <xacro:property name="livox_mass" value="0.2"/>
+    <xacro:property name="livox_radius" value="0.04"/>
+    <xacro:property name="livox_length" value="0.04"/>
     <!-- ADD COMPONENTS -->
     <xacro:include filename="$(find perseus_description)/urdf/inertia_macros.xacro"/>
@@ -86,6 +86,6 @@
     <joint name="${prefix}laser_joint" type="fixed">
       <parent link="${prefix}chassis"/>
-      <child link="${prefix}laser_frame"/>
-      <origin xyz="0 0 -0.04" rpy="0 ${pi} 0"/>
+      <child link="${prefix}livox_frame"/>
+      <origin xyz="-0.27 -0.04 -0.04" rpy="0 ${pi} ${pi}"/>
     </joint>
     <joint name="${prefix}laser_2d_joint" type="fixed">
@@ -97,5 +97,5 @@
         <parent link="${prefix}chassis"/>
         <child link="${prefix}camera_link"/>
-        <origin xyz="0.01 0 0.18" rpy="0 0 0"/>
+        <origin xyz="0.145 0 0.34" rpy="0 0.174533 0"/>
     </joint>
   </xacro:macro>

File: software/ros_ws/src/perseus_description/urdf/sensors.urdf.xacro (robot description, xacro)
@@ -2,14 +2,14 @@
 <robot name="lidar" xmlns:xacro="http://ros.org/wiki/xacro">
 <!-- 3D LIDAR (Existing - Livox MID-360) -->
-<link name="${prefix}laser_frame">
+<link name="${prefix}livox_frame">
     <inertial>
         <origin xyz="0 0 0"/>
-        <mass value="${laser_3d_mass}"/>
-        <xacro:box_inertia m="${laser_3d_mass}" x="${laser_3d_length}" y="${laser_3d_radius}" z="${laser_3d_radius}"/>
+        <mass value="${livox_mass}"/>
+        <xacro:box_inertia m="${livox_mass}" x="${livox_length}" y="${livox_radius}" z="${livox_radius}"/>
     </inertial>
     <visual>
         <origin xyz="0 0 0"/>
         <geometry>
-            <cylinder radius="${laser_3d_radius}" length="${laser_3d_length}"/>
+            <cylinder radius="${livox_radius}" length="${livox_length}"/>
         </geometry>
         <material name="black"/>
@@ -17,5 +17,5 @@
     <collision>
         <geometry>
-            <cylinder radius="${laser_3d_radius}" length="${laser_3d_length}"/>
+            <cylinder radius="${livox_radius}" length="${livox_length}"/>
         </geometry>
     </collision>
@@ -44,5 +44,5 @@
 </link>
 <!-- Simulating the Livox MID-360 -->
-<gazebo reference="${prefix}laser_frame">
+<gazebo reference="${prefix}livox_frame">
   <material>
     <ambient>0.1 0.1 0.1 1</ambient>
@@ -76,5 +76,5 @@
       </range>
     </ray>
-    <gz_frame_id>laser_frame</gz_frame_id>
+    <gz_frame_id>${prefix}livox_frame</gz_frame_id>
   </sensor>
 </gazebo>
@@ -112,6 +112,17 @@
       </range>
     </ray>
-    <gz_frame_id>laser_2d_frame</gz_frame_id>
+    <gz_frame_id>${prefix}laser_2d_frame</gz_frame_id>
   </sensor>
 </gazebo>
+<gazebo reference="${prefix}livox_frame">
+    <material>Gazebo/Grey</material>
+    <sensor name="${prefix}lidar_imu" type="imu">
+        <always_on>1</always_on>
+        <update_rate>10</update_rate>
+        <visualize>true</visualize>
+        <topic>scan_3d/imu</topic>
+        <!-- Add frame id to imu sensor (achieving correct frame association)-->
+        <gz_frame_id>${prefix}livox_frame</gz_frame_id>
+    </sensor>
+</gazebo>
 </robot>

Commit message: Refactor autonomy package and update configurations
- Added example command for navigating through poses in README.md.
- Updated EKF parameters to use the correct IMU topic and added relative option.
- Modified navigation parameters to improve performance and removed docking server configuration.
- Adjusted local and global costmap parameters for better obstacle detection and inflation.
- Updated URDF files for the robot description, including changes to camera and LIDAR configurations.
- Enhanced vision parameters for ArUco detection, including camera info subscription.
- Implemented camera info handling in ArUco detector to dynamically update camera matrix and distortion coefficients.
- Updated pointcloud to laserscan launch file to reflect new topic names and target frames.

File: software/ros_ws/src/perseus_description/urdf/camera_depth.urdf.xacro (robot description, xacro)
@@ -44,5 +44,5 @@
             </camera>
             <topic>/perseus/rgbd_camera</topic>
-            <gz_frame_id>${prefix}camera_link_optical</gz_frame_id>
+            <gz_frame_id>${prefix}camera_link</gz_frame_id>
             <min_depth>0.05</min_depth>
             <max_depth>100.0</max_depth>

File: software/ros_ws/src/perseus_description/urdf/chassis.urdf.xacro (robot description, xacro)
@@ -25,5 +25,5 @@
       <sensor name="imu_sensor" type="imu">
           <always_on>1</always_on>
-          <update_rate>50</update_rate>
+          <update_rate>10</update_rate>
           <visualize>true</visualize>
           <topic>imu</topic>

File: software/ros_ws/src/perseus_description/urdf/perseus.urdf.xacro (robot description, xacro)
@@ -44,14 +44,14 @@
     <!-- Depth Camera Properties -->
     <xacro:property name="camera_mass" value="0.1"/>
-    <xacro:property name="camera_width" value="0.07"/>
+    <xacro:property name="camera_width" value="0.12"/>
     <xacro:property name="camera_height" value="0.03"/>
-    <xacro:property name="camera_depth" value="0.020"/>
+    <xacro:property name="camera_depth" value="0.025"/>
     <!-- 2D and 3D LIDAR Properties -->
     <xacro:property name="laser_2d_mass" value="0.1"/>
     <xacro:property name="laser_2d_radius" value="0.04"/>
     <xacro:property name="laser_2d_length" value="0.04"/>
-    <xacro:property name="laser_3d_mass" value="0.2"/>
-    <xacro:property name="laser_3d_radius" value="0.06"/>
-    <xacro:property name="laser_3d_length" value="0.06"/>
+    <xacro:property name="livox_mass" value="0.2"/>
+    <xacro:property name="livox_radius" value="0.04"/>
+    <xacro:property name="livox_length" value="0.04"/>
     <!-- ADD COMPONENTS -->
     <xacro:include filename="$(find perseus_description)/urdf/inertia_macros.xacro"/>
@@ -86,6 +86,6 @@
     <joint name="${prefix}laser_joint" type="fixed">
       <parent link="${prefix}chassis"/>
-      <child link="${prefix}laser_frame"/>
-      <origin xyz="0 0 -0.04" rpy="0 ${pi} 0"/>
+      <child link="${prefix}livox_frame"/>
+      <origin xyz="-0.27 -0.04 -0.04" rpy="0 ${pi} ${pi}"/>
     </joint>
     <joint name="${prefix}laser_2d_joint" type="fixed">
@@ -97,5 +97,5 @@
         <parent link="${prefix}chassis"/>
         <child link="${prefix}camera_link"/>
-        <origin xyz="0.01 0 0.18" rpy="0 0 0"/>
+        <origin xyz="0.145 0 0.34" rpy="0 0.174533 0"/>
     </joint>
   </xacro:macro>

File: software/ros_ws/src/perseus_description/urdf/sensors.urdf.xacro (robot description, xacro)
@@ -2,14 +2,14 @@
 <robot name="lidar" xmlns:xacro="http://ros.org/wiki/xacro">
 <!-- 3D LIDAR (Existing - Livox MID-360) -->
-<link name="${prefix}laser_frame">
+<link name="${prefix}livox_frame">
     <inertial>
         <origin xyz="0 0 0"/>
-        <mass value="${laser_3d_mass}"/>
-        <xacro:box_inertia m="${laser_3d_mass}" x="${laser_3d_length}" y="${laser_3d_radius}" z="${laser_3d_radius}"/>
+        <mass value="${livox_mass}"/>
+        <xacro:box_inertia m="${livox_mass}" x="${livox_length}" y="${livox_radius}" z="${livox_radius}"/>
     </inertial>
     <visual>
         <origin xyz="0 0 0"/>
         <geometry>
-            <cylinder radius="${laser_3d_radius}" length="${laser_3d_length}"/>
+            <cylinder radius="${livox_radius}" length="${livox_length}"/>
         </geometry>
         <material name="black"/>
@@ -17,5 +17,5 @@
     <collision>
         <geometry>
-            <cylinder radius="${laser_3d_radius}" length="${laser_3d_length}"/>
+            <cylinder radius="${livox_radius}" length="${livox_length}"/>
         </geometry>
     </collision>
@@ -44,5 +44,5 @@
 </link>
 <!-- Simulating the Livox MID-360 -->
-<gazebo reference="${prefix}laser_frame">
+<gazebo reference="${prefix}livox_frame">
   <material>
     <ambient>0.1 0.1 0.1 1</ambient>
@@ -53,6 +53,6 @@
     <topic>scan_3d</topic>
     <update_rate>50</update_rate>
-    <always_on>true</always_on>
-    <visualize>true</visualize>
+    <always_on>false</always_on>
+    <visualize>false</visualize>
     <ray>
       <scan>
@@ -72,9 +72,9 @@
       <range>
         <min>0.20</min>
-        <max>70.0</max>
+        <max>30.0</max>
         <resolution>0.013</resolution>
       </range>
     </ray>
-    <gz_frame_id>laser_frame</gz_frame_id>
+    <gz_frame_id>${prefix}livox_frame</gz_frame_id>
   </sensor>
 </gazebo>
@@ -112,6 +112,17 @@
       </range>
     </ray>
-    <gz_frame_id>laser_2d_frame</gz_frame_id>
+    <gz_frame_id>${prefix}laser_2d_frame</gz_frame_id>
   </sensor>
 </gazebo>
+<gazebo reference="${prefix}livox_frame">
+    <material>Gazebo/Grey</material>
+    <sensor name="${prefix}lidar_imu" type="imu">
+        <always_on>1</always_on>
+        <update_rate>10</update_rate>
+        <visualize>true</visualize>
+        <topic>scan_3d/imu</topic>
+        <!-- Add frame id to imu sensor (achieving correct frame association)-->
+        <gz_frame_id>${prefix}livox_frame</gz_frame_id>
+    </sensor>
+</gazebo>
 </robot>
