Commit message: Enhance RViz configuration and URDF models
- Updated RViz configuration to include new TF panel and additional frames (base_footprint, camera_link, camera_link_optical, livox_frame) with appropriate visibility settings.
- Adjusted marker scale and view parameters for improved visualization.
- Modified camera_depth.urdf.xacro to use a mesh for the camera representation instead of a box.
- Corrected the position of the livox_frame in perseus.urdf.xacro for better alignment.
- Updated sensors.urdf.xacro to include a mesh for the Livox MID-360 and adjusted its visual and collision origins.
- Simplified the gazebo launch process by removing unnecessary nix commands

File: software/ros_ws/src/perseus_description/urdf/camera_depth.urdf.xacro (robot description, xacro)
@@ -8,6 +8,7 @@
         </inertial>
         <visual>
+            <origin xyz="0.003 0 0" rpy="${pi/2} 0.0 ${pi/2}"/>
             <geometry>
-                <box size="${camera_depth} ${camera_width} ${camera_height}"/>
+                <mesh scale="1.0 1.0 1.0" filename="file://$(find perseus_description)/meshes/d455.dae"/>
             </geometry>
             <material name="red"/>

File: software/ros_ws/src/perseus_description/urdf/perseus.urdf.xacro (robot description, xacro)
@@ -87,5 +87,5 @@
       <parent link="${prefix}chassis"/>
       <child link="${prefix}livox_frame"/>
-      <origin xyz="-0.193 -0.047 -0.03375" rpy="0 ${pi} ${pi}"/>
+      <origin xyz="-0.173 -0.047 -0.03375" rpy="0 ${pi} ${pi}"/>
     </joint>
     <joint name="${prefix}laser_2d_joint" type="fixed">

File: software/ros_ws/src/perseus_description/urdf/sensors.urdf.xacro (robot description, xacro)
@@ -4,16 +4,17 @@
 <link name="${prefix}livox_frame">
     <inertial>
-        <origin xyz="0 0 0"/>
+        <origin xyz="0 0.0 0.0" rpy="${pi/2} 0.0 ${pi}"/>
         <mass value="${livox_mass}"/>
         <xacro:box_inertia m="${livox_mass}" x="${livox_length}" y="${livox_radius}" z="${livox_radius}"/>
     </inertial>
     <visual>
-        <origin xyz="0 0 0"/>
+        <origin xyz="0 0.0 -0.02" rpy="${pi/2} 0.0 0.0"/>
         <geometry>
-            <cylinder radius="${livox_radius}" length="${livox_length}"/>
+            <mesh scale="1.0 1.0  1.0" filename="file://$(find perseus_description)/meshes/mid-360.dae"/>
         </geometry>
         <material name="black"/>
     </visual>
     <collision>
+        <origin xyz="0 0.0 -0.02" rpy="0.0 0.0 0.0"/>
         <geometry>
             <cylinder radius="${livox_radius}" length="${livox_length}"/>

Commit message: chore: clean up empty code change sections in the changes log

File: software/ros_ws/src/perseus_description/urdf/camera_depth.urdf.xacro (robot description, xacro)
@@ -8,6 +8,7 @@
         </inertial>
         <visual>
+            <origin xyz="0.003 0 0" rpy="${pi/2} 0.0 ${pi/2}"/>
             <geometry>
-                <box size="${camera_depth} ${camera_width} ${camera_height}"/>
+                <mesh scale="1.0 1.0 1.0" filename="file://$(find perseus_description)/meshes/d455.dae"/>
             </geometry>
             <material name="red"/>
@@ -44,5 +45,5 @@
             </camera>
             <topic>/perseus/rgbd_camera</topic>
-            <gz_frame_id>${prefix}camera_link_optical</gz_frame_id>
+            <gz_frame_id>${prefix}camera_link</gz_frame_id>
             <min_depth>0.05</min_depth>
             <max_depth>100.0</max_depth>

File: software/ros_ws/src/perseus_description/urdf/perseus.urdf.xacro (robot description, xacro)
@@ -87,5 +87,5 @@
       <parent link="${prefix}chassis"/>
       <child link="${prefix}livox_frame"/>
-      <origin xyz="-0.27 -0.04 -0.04" rpy="0 ${pi} ${pi}"/>
+      <origin xyz="-0.173 0.047 -0.04375" rpy="0 ${pi} ${pi/2}"/>
     </joint>
     <joint name="${prefix}laser_2d_joint" type="fixed">
@@ -97,5 +97,5 @@
         <parent link="${prefix}chassis"/>
         <child link="${prefix}camera_link"/>
-        <origin xyz="0.145 0 0.34" rpy="0 0.174533 0"/>
+        <origin xyz="0.055 0 0.184" rpy="0 0.0 0"/>
     </joint>
   </xacro:macro>

File: software/ros_ws/src/perseus_description/urdf/sensors.urdf.xacro (robot description, xacro)
@@ -4,16 +4,17 @@
 <link name="${prefix}livox_frame">
     <inertial>
-        <origin xyz="0 0 0"/>
+        <origin xyz="0 0.0 0.0" rpy="${pi/2} 0.0 ${pi}"/>
         <mass value="${livox_mass}"/>
         <xacro:box_inertia m="${livox_mass}" x="${livox_length}" y="${livox_radius}" z="${livox_radius}"/>
     </inertial>
     <visual>
-        <origin xyz="0 0 0"/>
+        <origin xyz="0 0.0 -0.02" rpy="${pi/2} 0.0 ${pi}"/>
         <geometry>
-            <cylinder radius="${livox_radius}" length="${livox_length}"/>
+            <mesh scale="1.0 1.0  1.0" filename="file://$(find perseus_description)/meshes/mid-360.dae"/>
         </geometry>
         <material name="black"/>
     </visual>
     <collision>
+        <origin xyz="0 0.0 -0.02" rpy="0.0 0.0 0.0"/>
         <geometry>
             <cylinder radius="${livox_radius}" length="${livox_length}"/>

Commit message: feat: Add RealSense URDF and update related configurations

File: software/ros_ws/src/perseus_description/urdf/camera_depth.urdf.xacro (robot description, xacro)
@@ -1,32 +1,8 @@
 <?xml version="1.0"?>
-<robot name="camera_depth" xmlns:xacro="http://ros.org/wiki/xacro">
-    <link name="${prefix}camera_link">
-        <inertial>
-            <origin xyz="0 0 0" rpy="0 0 0"/>
-            <mass value="${camera_mass}"/>
-            <xacro:box_inertia m="${camera_mass}" x="${camera_depth}" y="${camera_width}" z="${camera_height}"/>
-        </inertial>
-        <visual>
-            <origin xyz="0.003 0 0" rpy="${pi/2} 0.0 ${pi/2}"/>
-            <geometry>
-                <mesh scale="1.0 1.0 1.0" filename="file://$(find perseus_description)/meshes/d455.dae"/>
-            </geometry>
-            <material name="red"/>
-        </visual>
-        <collision>
-            <geometry>
-                <box size="${camera_depth} ${camera_width} ${camera_height}"/>
-            </geometry>
-        </collision>
-    </link>
-    <joint name="${prefix}camera_optical_joint" type="fixed">
-        <parent link="${prefix}camera_link"/>
-        <child link="${prefix}camera_link_optical"/>
-        <origin xyz="0 0 0" rpy="-1.57079632679 0 -1.57079632679"/>
-    </joint>
-    <link name="${prefix}camera_link_optical"></link>
-    <gazebo reference="${prefix}camera_link">
+<robot name="camera_d455_gazebo" xmlns:xacro="http://ros.org/wiki/xacro">
+    <!-- RGB Color Camera -->
+    <gazebo reference="${prefix}camera_color_frame">
         <material>Gazebo/Red</material>
-        <sensor name="rgbd_camera" type="rgbd_camera">
+        <sensor name="rgb_camera" type="camera">
             <pose> 0 0 0 0 0 0 </pose>
             <visualize>true</visualize>
@@ -44,8 +20,75 @@
                 </clip>
             </camera>
-            <topic>/perseus/rgbd_camera</topic>
-            <gz_frame_id>${prefix}camera_link</gz_frame_id>
+            <topic>camera/camera/color/image_raw</topic>
+            <gz_frame_id>${prefix}camera_color_optical_frame</gz_frame_id>
+        </sensor>
+    </gazebo>
+    <gazebo reference="${prefix}camera_depth_frame">
+        <sensor name="rgbd_camera" type="rgbd_camera">
+            <pose>0 0 0 0 0 0</pose>
+            <visualize>false</visualize>
+            <update_rate>30</update_rate>
+            <always_on>true</always_on>
+            <camera>
+                <horizontal_fov>1.089</horizontal_fov>
+                <image>
+                    <width>640</width>
+                    <height>480</height>
+                </image>
+                <clip>
+                    <near>0.05</near>
+                    <far>10.0</far>
+                </clip>
+            </camera>
+            <topic>/camera/camera/depth</topic>
+            <gz_frame_id>${prefix}camera_depth_optical_frame</gz_frame_id>
             <min_depth>0.05</min_depth>
-            <max_depth>100.0</max_depth>
+            <max_depth>10.0</max_depth>
+        </sensor>
+    </gazebo>
+    <!-- Left IR Camera -->
+    <gazebo reference="${prefix}camera_infra1_frame">
+        <sensor name="ir_left_camera" type="camera">
+            <pose>0 0 0 0 0 0</pose>
+            <visualize>false</visualize>
+            <update_rate>30</update_rate>
+            <always_on>true</always_on>
+            <camera>
+                <horizontal_fov>1.089</horizontal_fov>
+                <image>
+                    <width>640</width>
+                    <height>480</height>
+                    <format>L_INT8</format>
+                </image>
+                <clip>
+                    <near>0.05</near>
+                    <far>100</far>
+                </clip>
+            </camera>
+            <topic>/camera/camera/infra1/image_raw</topic>
+            <gz_frame_id>${prefix}camera_infra1_optical_frame</gz_frame_id>
+        </sensor>
+    </gazebo>
+    <!-- Right IR Camera -->
+    <gazebo reference="${prefix}camera_infra2_frame">
+        <sensor name="ir_right_camera" type="camera">
+            <pose>0 0 0 0 0 0</pose>
+            <visualize>false</visualize>
+            <update_rate>30</update_rate>
+            <always_on>true</always_on>
+            <camera>
+                <horizontal_fov>1.089</horizontal_fov>
+                <image>
+                    <width>640</width>
+                    <height>480</height>
+                    <format>L_INT8</format>
+                </image>
+                <clip>
+                    <near>0.05</near>
+                    <far>100</far>
+                </clip>
+            </camera>
+            <topic>/camera/camera/infra2/image_raw</topic>
+            <gz_frame_id>${prefix}camera_infra2_optical_frame</gz_frame_id>
         </sensor>
     </gazebo>

File: software/ros_ws/src/perseus_description/urdf/perseus.urdf.xacro (robot description, xacro)
@@ -63,4 +63,5 @@
     <xacro:include filename="$(find perseus_description)/urdf/sensors.urdf.xacro"/>
     <xacro:include filename="$(find perseus_description)/urdf/camera_depth.urdf.xacro" />
+    <xacro:include filename="$(find realsense2_description)/urdf/_d455.urdf.xacro"/>
     <!-- An empty base_link to attach everything to -->
     <link name="${prefix}base_link"/>
@@ -94,9 +95,7 @@
       <origin xyz="-0.15 0 0.25" rpy="0 0 0"/>
     </joint>
-    <joint name="${prefix}camera_joint" type="fixed">
-        <parent link="${prefix}chassis"/>
-        <child link="${prefix}camera_link"/>
-        <origin xyz="0.055 0 0.184" rpy="0 0.0 0"/>
-    </joint>
+  <xacro:sensor_d455 parent="${prefix}chassis" use_nominal_extrinsics="true">
+    <origin xyz="0.055 0.0 0.184" rpy="0 0 0"/>
+  </xacro:sensor_d455>
   </xacro:macro>
 </robot>
