Commit message: perseus_description: Inherit xacro parameters
This reduces things like `prefix="${prefix}"` quite a lot

File: software/ros_ws/src/perseus_description/urdf/chassis.urdf.xacro (robot description, xacro)
@@ -2,5 +2,5 @@
 <robot name="chassis" xmlns:xacro="http://ros.org/wiki/xacro">
   <!-- Contains base rover chassis and balance bar -->
-  <xacro:macro name="chassis" params="prefix">
+  <xacro:macro name="chassis" params="prefix:=^">
     <!-- CHASSIS -->
     <link name="${prefix}chassis">
@@ -15,5 +15,4 @@
           <mesh scale="0.1 0.1 0.1" filename="file://$(find perseus_description)/meshes/chassis.dae"/>
         </geometry>
-        <!-- <material name="silver"/> -->
       </visual>
       <collision>
@@ -38,5 +37,4 @@
           <mesh scale="0.1 0.1 0.1" filename="file://$(find perseus_description)/meshes/flange_bearing.dae"/>
         </geometry>
-        <!-- <material name="blue"/> -->
       </visual>
       <collision>
@@ -64,10 +62,8 @@
           <mesh scale="0.1 0.1 0.1" filename="file://$(find perseus_description)/meshes/differential_bar.dae"/>
         </geometry>
-        <!-- <material name="red"/> -->
       </visual>
       <collision>
         <origin xyz="0.0 0.0 -0.01" rpy="0.0 0.0 0.0"/>
         <geometry>
-          <!-- close enough-->
           <box size="0.5 0.05 0.03" />
           <!--mesh scale="0.1 0.1 0.1" filename="file://$(find perseus_description)/meshes/differential_bar.dae"/-->

File: software/ros_ws/src/perseus_description/urdf/motor_wheel.urdf.xacro (robot description, xacro)
@@ -2,5 +2,5 @@
 <robot name="motor_wheel" xmlns:xacro="http://www.ros.org/wiki/xacro">
   <xacro:include filename="$(find perseus_description)/urdf/wheel.urdf.xacro"/>
-  <xacro:macro name="motor_wheel" params="prefix side end *origin">
+  <xacro:macro name="motor_wheel" params="prefix:=^ side:=^ end *origin">
     <link name="${prefix}${end}_${side}_motor">
       <inertial>
@@ -42,5 +42,5 @@
       </actuator>
     </transmission> -->
-    <xacro:wheel prefix="${prefix}" side="${side}" end="${end}"/>
+    <xacro:wheel />
   </xacro:macro>
 </robot>

File: software/ros_ws/src/perseus_description/urdf/perseus.urdf.xacro (robot description, xacro)
@@ -8,5 +8,5 @@
     <link name="${prefix}base_link"/>
     <!-- CHASSIS -->
-    <xacro:chassis prefix="${prefix}"/>
+    <xacro:chassis />
     <joint name="chassis_joint" type="fixed">
       <origin xyz="0.21 0.0 0.35" rpy="0.0 0.0 -${pi/2}"/>
@@ -16,9 +16,9 @@
     <!-- ROCKER ARMS -->
     <!-- LEFT -->
-    <xacro:rocker prefix="${prefix}" side="left">
+    <xacro:rocker side="left">
       <origin xyz="-0.275 -0.075 0.05" rpy="0.0 0.0 ${-pi/2}"/>
     </xacro:rocker>
     <!-- RIGHT -->
-    <xacro:rocker prefix="${prefix}" side="right">
+    <xacro:rocker side="right">
       <origin xyz="0.275 -0.075 0.05" rpy="0.0 0.0 ${-pi/2}"/>
     </xacro:rocker>

File: software/ros_ws/src/perseus_description/urdf/rocker.urdf.xacro (robot description, xacro)
@@ -2,17 +2,16 @@
 <robot name="rocker" xmlns:xacro="http://www.ros.org/wiki/xacro">
   <xacro:include filename="$(find perseus_description)/urdf/motor_wheel.urdf.xacro"/>
-  <xacro:macro name="rocker" params="prefix side *origin">
+  <xacro:macro name="rocker" params="prefix:=^ side *origin">
     <!-- ROCKER ARM -->
     <link name="${prefix}${side}_rocker">
       <inertial>
+        <origin xyz="0.011819187400851083 -0.08337339654014758 -0.06739096070989994" rpy="0.0 0.0 0.0"/>
         <!-- RIGHT -->
         <xacro:if value="${side == 'right'}">
-          <origin xyz="0.011819187400851083 -0.08337339654014758 -0.06739096070989994" rpy="0.0 0.0 0.0"/>
           <inertia ixx="0.078224" iyy="0.009964" izz="0.076528" ixy="0.003701" iyz="-0.006846" ixz="0.00298"/>
         </xacro:if>
         <!-- LEFT -->
         <xacro:if value="${side == 'left'}">
-          <origin xyz="0.011819187400851083 -0.08337339654014758 -0.06739096070989994" rpy="0.0 0.0 0.0"/>
-          <inertia ixx="0.078224" iyy="0.009964" izz="0.076528" ixy="-0.003701" iyz="-0.006845" ixz="-0.00298"/>
+          <inertia ixx="0.078224" iyy="0.009964" izz="0.076528" ixy="0.003701" iyz="-0.006846" ixz="0.00298"/>
         </xacro:if>
         <mass value="1.2546142039512485"/>
@@ -23,5 +22,4 @@
           <mesh scale="0.1 0.1 0.1" filename="file://$(find perseus_description)/meshes/rocker_${side}.dae"/>
         </geometry>
-        <!-- <material name="silver"/> -->
       </visual>
       <collision>
@@ -48,20 +46,15 @@
     </joint>
     <!-- FRONT MOTOR -->
-    <xacro:motor_wheel prefix="${prefix}" side="${side}" end="front">
+    <xacro:motor_wheel end="front">
       <xacro:if value="${side == 'left'}">
-        <!-- NHS: suspect this joint is the reason for the wheels turning backwards-->
-        <!--playing around with rotating in Z and manually placing offset for wheels-->
-        <!--ORIGINAL TEXT: origin xyz="-0.3 0.045 -0.25" rpy="0.0 0.0 ${pi/2}"/-->
         <origin xyz="-0.3 -0.225 -0.25" rpy="0.0 0.0 ${-pi/2}"/>
       </xacro:if>
       <xacro:if value="${side == 'right'}">
-        <!--ORIGINAL TEXT: origin xyz="-0.3 -0.045 -0.25" rpy="0.0 0.0 ${-pi/2}"/-->
         <origin xyz="-0.3 0.225 -0.25" rpy="0.0 0.0 ${pi/2}"/>
       </xacro:if>
     </xacro:motor_wheel>
     <!-- REAR MOTOR -->
-    <xacro:motor_wheel prefix="${prefix}" side="${side}" end="rear">
+    <xacro:motor_wheel end="rear">
       <xacro:if value="${side == 'left'}">
-        <!-- origin xyz="0.55 0.045 -0.25" rpy="0.0 0.0 ${pi/2}"/-->
         <origin xyz="0.55 -0.225 -0.25" rpy="0.0 0.0 ${-pi/2}"/>
       </xacro:if>

File: software/ros_ws/src/perseus_description/urdf/wheel.urdf.xacro (robot description, xacro)
@@ -1,5 +1,5 @@
 <?xml version="1.0"?>
 <robot name="wheel" xmlns:xacro="http://ros.org/wiki/xacro">
-  <xacro:macro name="wheel" params="prefix side end">
+  <xacro:macro name="wheel" params="prefix:=^ side:=^ end:=^">
     <link name="${prefix}${end}_${side}_wheel">
       <inertial>

Commit message: feat: Clean up description URDF
Co-authored-by: Nigel H-S <1388693+DingoOz@users.noreply.github.com>

File: software/ros_ws/src/perseus_description/urdf/chassis.urdf.xacro (robot description, xacro)
@@ -21,5 +21,4 @@
         <geometry>
           <box size="0.475 0.525 0.2" />
-          <!--mesh scale="0.1 0.1 0.1" filename="file://$(find perseus_description)/meshes/chassis.dae"/-->
         </geometry>
       </collision>
@@ -67,11 +66,7 @@
         <geometry>
           <box size="0.5 0.05 0.03" />
-          <!--mesh scale="0.1 0.1 0.1" filename="file://$(find perseus_description)/meshes/differential_bar.dae"/-->
         </geometry>
       </collision>
     </link>
-    <!-- <joint name="${prefix}differential_bar_joint" type="revolute"> -->
-      <!-- <limit upper="0.349066" lower="-0.349066" effort="100" velocity="100"/> -->
-      <!-- <dynamics damping="10.0" friction="10.0"/> -->
     <joint name="${prefix}differential_bar_joint" type="fixed">
       <origin xyz="0.0 0.0 0.05" rpy="${pi} 0.0 ${-pi/2}"/>

File: software/ros_ws/src/perseus_description/urdf/perseus.urdf.xacro (robot description, xacro)
@@ -9,5 +9,5 @@
     <!-- CHASSIS -->
     <xacro:chassis />
-    <joint name="chassis_joint" type="fixed">
+    <joint name="${prefix}chassis_joint" type="fixed">
       <origin xyz="0.21 0.0 0.35" rpy="0.0 0.0 -${pi/2}"/>
       <parent link="${prefix}base_link"/>

File: software/ros_ws/src/perseus_description/urdf/rocker.urdf.xacro (robot description, xacro)
@@ -27,21 +27,11 @@
         <geometry>
           <box size="0.4 0.05 0.03" />
-          <!--mesh scale="0.1 0.1 0.1" filename="file://$(find perseus_description)/meshes/rocker_${side}.dae"/-->
         </geometry>
       </collision>
     </link>
-    <joint name="${side}_rocker_joint" type="fixed"> <!-- revolute -->
-      <!-- <limit effort="100.0" lower="-0.24" upper="0.24" velocity="100.0"/>
-      <dynamics damping="0.1" friction="1.0"/> -->
+    <joint name="${prefix}${side}_rocker_joint" type="fixed">
       <xacro:insert_block name="origin"/>
-      <!-- <axis xyz="0 1 0"/> -->
-      <parent link="chassis"/>
-      <child link="${side}_rocker"/>
-      <!-- <xacro:if value="${side == 'right'}">
-        <mimic joint="flange_bearing_to_differential_bar"/>
-      </xacro:if>
-      <xacro:if value="${side == 'left'}">
-        <mimic joint="flange_bearing_to_differential_bar" multiplier="-1"/>
-      </xacro:if> -->
+      <parent link="${prefix}chassis"/>
+      <child link="${prefix}${side}_rocker"/>
     </joint>
     <!-- FRONT MOTOR -->

File: software/ros_ws/src/perseus_description/urdf/wheel.urdf.xacro (robot description, xacro)
@@ -5,5 +5,5 @@
       <inertial>
         <origin xyz="0.0 0.0 0.0" rpy="0.0 0.0 0.0"/>
-        <mass value="0.01"/>
+        <mass value="1.0"/>
         <inertia ixx="0.051473" iyy="0.029155" izz="0.029154" ixy="0.0" iyz="0.0" ixz="0.0"/>
       </inertial>
@@ -13,5 +13,4 @@
           <mesh scale="0.1 0.1 0.1" filename="file://$(find perseus_description)/meshes/wheel.dae"/>
         </geometry>
-        <!-- <material name="orange"></material> -->
       </visual>
       <collision>
@@ -19,5 +18,4 @@
         <geometry>
           <cylinder length="0.115" radius="0.145" />
-          <!--mesh scale="0.1 0.1 0.1" filename="file://$(find perseus_description)/meshes/wheel.dae"/-->
         </geometry>
       </collision>

Commit message: fix(urdf): update chassis and flange bearing collision geometry

File: software/ros_ws/src/perseus_description/urdf/chassis.urdf.xacro (robot description, xacro)
@@ -11,5 +11,5 @@
       </inertial>
       <visual>
-        <origin xyz="0.0 0.0 0.0" rpy="0 0.0 0.0"/>
+        <origin xyz="0.0 0.0 0.0" rpy="0 0.0 -${pi/2}"/>
         <geometry>
           <mesh scale="0.1 0.1 0.1" filename="file://$(find perseus_description)/meshes/chassis.dae"/>
@@ -17,8 +17,8 @@
       </visual>
       <collision>
-        <origin xyz="0.0 -0.3 0.1" rpy="0 0.0 0.0"/>
+        <origin xyz="0.0 0.0 0.0" rpy="0 0.0 -${pi/2}"/>
         <!-- Modified to make collision more simple, chassis mesh replaced with box -->
         <geometry>
-          <box size="0.475 0.525 0.2" />
+          <mesh scale="0.1 0.1 0.1" filename="file://$(find perseus_description)/meshes/chassis.dae"/>
         </geometry>
       </collision>
@@ -32,5 +32,5 @@
       </inertial>
       <visual>
-        <origin xyz="0.0 0.0 0.0" rpy="0 0 0"/>
+        <origin xyz="0.0 0.0 0.0" rpy="${-pi/2} 0 ${pi/2}"/>
         <geometry>
           <mesh scale="0.1 0.1 0.1" filename="file://$(find perseus_description)/meshes/flange_bearing.dae"/>
@@ -45,5 +45,5 @@
     </link>
     <joint name="${prefix}flange_bearing_joint" type="fixed">
-      <origin xyz="0.0 -0.6 0.1" rpy="0 ${-pi/2} ${pi/2}"/>
+      <origin xyz="-0.6 -0.0 0.1" rpy="0 0 0"/>
       <parent link="${prefix}chassis"/>
       <child link="${prefix}flange_bearing"/>
@@ -52,10 +52,10 @@
     <link name="${prefix}differential_bar">
       <inertial>
-        <origin xyz="-0.0012101129983653758 -0.04574872679422123 0.0" rpy="0.0 0.0 0.0"/>
+        <origin xyz="0 0 0.0" rpy="0.0 0.0 0.0"/>
         <mass value="0.9172649518127158"/>
         <inertia ixx="0.00036" iyy="0.018339" izz="0.018134" ixy="3e-06" iyz="-0.0" ixz="0.0"/>
       </inertial>
       <visual>
-        <origin xyz="0.0 0.0 0.0" rpy="0.0 0.0 0.0"/>
+        <origin xyz="0.0 0.0 0.0" rpy="${-pi/2} 0 ${-pi/2}"/>
         <geometry>
           <mesh scale="0.1 0.1 0.1" filename="file://$(find perseus_description)/meshes/differential_bar.dae"/>
@@ -70,5 +70,5 @@
     </link>
     <joint name="${prefix}differential_bar_joint" type="fixed">
-      <origin xyz="0.0 0.0 0.05" rpy="${pi} 0.0 ${-pi/2}"/>
+      <origin xyz="-0.05 0.0 0.0" rpy="0.0 0.0 0.0"/>
       <axis xyz="0.0 0.0 1.0"/>
       <parent link="${prefix}flange_bearing"/>

Commit message: fix(urdf): correct rpy values for differential bar joint origin

File: software/ros_ws/src/perseus_description/urdf/chassis.urdf.xacro (robot description, xacro)
@@ -70,5 +70,5 @@
     </link>
     <joint name="${prefix}differential_bar_joint" type="fixed">
-      <origin xyz="-0.05 0.0 0.0" rpy="0.0 0.0 0.0"/>
+      <origin xyz="-0.05 0.0 0.0" rpy="0 0.0 0"/>
       <axis xyz="0.0 0.0 1.0"/>
       <parent link="${prefix}flange_bearing"/>
