Commit message: Refactor URDF files for Perseus robot
- Updated rocker.urdf.xacro to simplify the definition of left and right rocker arms, removing unnecessary macros and including visual and collision elements directly.
- Revised wheel.urdf.xacro to define front and rear wheels without using macros, enhancing clarity and maintainability.
- Introduced a new chassis.urdf.xacro file to encapsulate the chassis structure, including inertial properties and visual/collision definitions.
- Created motor_wheel.urdf.xacro to define motor and wheel assemblies, streamlining the integration of wheel components.
- Added sensors.urdf.xacro to define laser and lidar sensors with appropriate joints and visual representations.
- Established perseus.materials.xacro to define materials used across the robot's components.
- Introduced a new perseus.urdf.xacro file to serve as the main entry point for the robot's URDF, integrating all components.
- Updated rviz configuration to enable visibility for all components, improving the visualization setup for simulation.

File: software/ros_ws/src/perseus_description/urdf/chassis.urdf.xacro (robot description, xacro)
@@ -1,78 +1,23 @@
 <?xml version="1.0"?>
 <robot name="chassis" xmlns:xacro="http://ros.org/wiki/xacro">
-  <!-- Contains base rover chassis and balance bar -->
-  <xacro:macro name="chassis" params="prefix:=^">
-    <!-- CHASSIS -->
-    <link name="${prefix}chassis">
-      <inertial>
-        <origin xyz="0.0 -0.17100473204 0.14732485976" rpy="0 0 0"/>
-        <mass value="2.7689940302592726"/>
-        <inertia ixx="0.170464" iyy="0.092623" izz="0.224359" ixy="0.0" iyz="0.005411" ixz="-0.0"/>
-      </inertial>
-      <visual>
-        <origin xyz="0.0 0.0 0.0" rpy="0 0.0 -${pi/2}"/>
-        <geometry>
-          <mesh scale="0.1 0.1 0.1" filename="file://$(find perseus_description)/meshes/chassis.dae"/>
-        </geometry>
-      </visual>
-      <collision>
-        <origin xyz="0.0 0.0 0.0" rpy="0 0.0 -${pi/2}"/>
-        <!-- Modified to make collision more simple, chassis mesh replaced with box -->
-        <geometry>
-          <mesh scale="0.1 0.1 0.1" filename="file://$(find perseus_description)/meshes/chassis.dae"/>
-        </geometry>
-      </collision>
-    </link>
-    <!-- Flange Bearing -->
-    <link name="${prefix}flange_bearing">
-      <inertial>
-        <origin xyz="0.0 0.0 0.0" rpy="0 0 0"/>
-        <mass value="1.327488734939265"/>
-        <inertia ixx="0.001313" iyy="0.001699" izz="0.000647" ixy="0.0" iyz="0.0" ixz="-0.0"/>
-      </inertial>
-      <visual>
-        <origin xyz="0.0 0.0 0.0" rpy="${-pi/2} 0 ${pi/2}"/>
-        <geometry>
-          <mesh scale="0.1 0.1 0.1" filename="file://$(find perseus_description)/meshes/flange_bearing.dae"/>
-        </geometry>
-      </visual>
-      <collision>
-        <origin xyz="0.0 0.0 0.0" rpy="0 0 0"/>
-        <geometry>
-          <mesh scale="0.1 0.1 0.1" filename="file://$(find perseus_description)/meshes/flange_bearing.dae"/>
-        </geometry>
-      </collision>
-    </link>
-    <joint name="${prefix}flange_bearing_joint" type="fixed">
-      <origin xyz="-0.6 -0.0 0.1" rpy="0 0 0"/>
-      <parent link="${prefix}chassis"/>
-      <child link="${prefix}flange_bearing"/>
-    </joint>
-    <!-- Balance/differential bar -->
-    <link name="${prefix}differential_bar">
-      <inertial>
-        <origin xyz="0 0 0.0" rpy="0.0 0.0 0.0"/>
-        <mass value="0.9172649518127158"/>
-        <inertia ixx="0.00036" iyy="0.018339" izz="0.018134" ixy="3e-06" iyz="-0.0" ixz="0.0"/>
-      </inertial>
-      <visual>
-        <origin xyz="0.0 0.0 0.0" rpy="${-pi/2} 0 ${-pi/2}"/>
-        <geometry>
-          <mesh scale="0.1 0.1 0.1" filename="file://$(find perseus_description)/meshes/differential_bar.dae"/>
-        </geometry>
-      </visual>
-      <collision>
-        <origin xyz="0.0 0.0 -0.01" rpy="0.0 0.0 0.0"/>
-        <geometry>
-          <box size="0.5 0.05 0.03" />
-        </geometry>
-      </collision>
-    </link>
-    <joint name="${prefix}differential_bar_joint" type="fixed">
-      <origin xyz="-0.05 0.0 0.0" rpy="0 0.0 0"/>
-      <axis xyz="0.0 0.0 1.0"/>
-      <parent link="${prefix}flange_bearing"/>
-      <child link="${prefix}differential_bar"/>
-    </joint>
-  </xacro:macro>
+  <link name="${prefix}chassis">
+    <!-- <inertial>
+      <origin xyz="0.0 -0.17100473204 0.14732485976" rpy="0 0 0"/>
+      <mass value="2.7689940302592726"/>
+      <inertia ixx="0.170464" iyy="0.092623" izz="0.224359" ixy="0.0" iyz="0.005411" ixz="-0.0"/>
+    </inertial> -->
+    <visual>
+      <origin xyz="0.0 0.0 0.0" rpy="0 0.0 -${pi/2}"/>
+      <geometry>
+        <mesh scale="${0.1/scale_factor} ${0.1/scale_factor}  ${0.1/scale_factor}" filename="file://$(find perseus_description)/meshes/chassis.dae"/>
+      </geometry>
+    </visual>
+    <collision>
+      <origin xyz="0.0 0.0 0.0" rpy="0 0.0 -${pi/2}"/>
+      <!-- Modified to make collision more simple, chassis mesh replaced with box -->
+      <geometry>
+        <mesh scale="${0.1/scale_factor} ${0.1/scale_factor}  ${0.1/scale_factor}" filename="file://$(find perseus_description)/meshes/chassis.dae"/>
+      </geometry>
+    </collision>
+  </link>
 </robot>

File: software/ros_ws/src/perseus_description/urdf/motor_wheel.urdf.xacro (robot description, xacro)
@@ -1,56 +1,71 @@
 <?xml version="1.0"?>
 <robot name="motor_wheel" xmlns:xacro="http://www.ros.org/wiki/xacro">
-  <xacro:include filename="$(find perseus_description)/urdf/wheel.urdf.xacro"/>
-  <xacro:macro name="motor_wheel" params="prefix:=^ side:=^ end *origin">
-    <link name="${prefix}${end}_${side}_motor">
-      <inertial>
-        <!-- moving origin has no perceivable impact-->
-        <xacro:if value="${side == 'left'}">
-          <origin xyz="0 0.0 0.0" rpy="0.0 0.0 ${-pi/2}"/>
-        </xacro:if>
-        <xacro:if value="${side == 'right'}">
-          <origin xyz="0 0.0 0.0" rpy="0.0 0.0 ${pi/2}"/>
-        </xacro:if>
-        <mass value="5.236579"/>
-        <inertia ixx="0.01" iyy="0.01" izz="0.01" ixy="0.0" iyz="0.0" ixz="0.0"/> <!-- TEMP -->
-      </inertial>
-      <visual>
-        <xacro:if value="${side == 'left'}">
-          <origin xyz="0 0.0 0.0" rpy="0.0 0.0 ${-pi/2}"/>
-        </xacro:if>
-        <xacro:if value="${side == 'right'}">
-          <origin xyz="0 0.0 0.0" rpy="0.0 0.0 ${pi/2}"/>
-        </xacro:if>
-        <geometry>
-          <mesh scale="0.1 0.1 0.1" filename="file://$(find perseus_description)/meshes/gearbox.dae"/>
-        </geometry>
-        <!-- <material name="white"/> -->
-      </visual>
-      <collision>
-        <origin xyz="-0.3 0.0 0.0" rpy="0.0 0.0 ${pi/2}"/>
-        <geometry>
-          <box size="0.1 0.1 0.075" />
-          <!--mesh scale="0.1 0.1 0.1" filename="file://$(find perseus_description)/meshes/gearbox.dae"/-->
-        </geometry>
-      </collision>
-    </link>
-    <!-- JOINT -->
-    <joint name="${prefix}${end}_${side}_motor_joint" type="fixed">
-      <parent link="${prefix}${side}_rocker"/>
-      <child link="${prefix}${end}_${side}_motor"/>
-      <xacro:insert_block name="origin"/>
-    </joint>
-    <!-- TRANSMISSION -->
-    <!-- <transmission name="gear_ratio">
-      <type>transmission_interface/SimpleTransmission</type>
-      <joint name="bogie_${prefix}_to_motor_${prefix}_${suffix}">
-        <hardwareInterface>EffortJointInterface</hardwareInterface>
-      </joint>
-      <actuator name="">
-        <mechanicalReduction>30</mechanicalReduction>
-        <hardwareInterface>EffortJointInterface</hardwareInterface>
-      </actuator>
-    </transmission> -->
-    <xacro:wheel />
-  </xacro:macro>
+  <link name="${prefix}front_right_motor">
+    <!-- <inertial>
+    </inertial> -->
+    <visual>
+      <origin xyz="0 0.0 0.0" rpy="0.0 0.0 ${pi/2}"/>
+      <geometry>
+        <mesh scale="${0.1/scale_factor} ${0.1/scale_factor}  ${0.1/scale_factor}" filename="file://$(find perseus_description)/meshes/gearbox.dae"/>
+      </geometry>
+      <!-- <material name="white"/> -->
+    </visual>
+    <collision>
+      <origin xyz="-0.3 0.0 0.0" rpy="0.0 0.0 ${pi/2}"/>
+      <geometry>
+        <mesh scale="${0.1/scale_factor} ${0.1/scale_factor}  ${0.1/scale_factor}" filename="file://$(find perseus_description)/meshes/gearbox.dae"/>
+      </geometry>
+    </collision>
+  </link>
+  <link name="${prefix}rear_right_motor">
+    <!-- <inertial>
+    </inertial> -->
+    <visual>
+      <origin xyz="0 0.0 0.0" rpy="0.0 0.0 ${pi/2}"/>
+      <geometry>
+        <mesh scale="${0.1/scale_factor} ${0.1/scale_factor}  ${0.1/scale_factor}" filename="file://$(find perseus_description)/meshes/gearbox.dae"/>
+      </geometry>
+      <!-- <material name="white"/> -->
+    </visual>
+    <collision>
+      <origin xyz="-0.3 0.0 0.0" rpy="0.0 0.0 ${pi/2}"/>
+      <geometry>
+        <mesh scale="${0.1/scale_factor} ${0.1/scale_factor}  ${0.1/scale_factor}" filename="file://$(find perseus_description)/meshes/gearbox.dae"/>
+      </geometry>
+    </collision>
+  </link>
+  <link name="${prefix}front_left_motor">
+    <!-- <inertial>
+    </inertial> -->
+    <visual>
+      <origin xyz="0 0.0 0.0" rpy="0.0 0.0 ${-pi/2}"/>
+      <geometry>
+        <mesh scale="${0.1/scale_factor} ${0.1/scale_factor}  ${0.1/scale_factor}" filename="file://$(find perseus_description)/meshes/gearbox.dae"/>
+      </geometry>
+      <!-- <material name="white"/> -->
+    </visual>
+    <collision>
+      <origin xyz="0 0.0 0.0" rpy="0.0 0.0 ${-pi/2}"/>
+      <geometry>
+        <mesh scale="${0.1/scale_factor} ${0.1/scale_factor}  ${0.1/scale_factor}" filename="file://$(find perseus_description)/meshes/gearbox.dae"/>
+      </geometry>
+    </collision>
+  </link>
+  <link name="${prefix}rear_left_motor">
+    <!-- <inertial>
+    </inertial> -->
+    <visual>
+      <origin xyz="0 0.0 0.0" rpy="0.0 0.0 ${-pi/2}"/>
+      <geometry>
+        <mesh scale="${0.1/scale_factor} ${0.1/scale_factor}  ${0.1/scale_factor}" filename="file://$(find perseus_description)/meshes/gearbox.dae"/>
+      </geometry>
+      <!-- <material name="white"/> -->
+    </visual>
+    <collision>
+      <origin xyz="0 0.0 0.0" rpy="0.0 0.0 ${-pi/2}"/>
+      <geometry>
+        <mesh scale="${0.1/scale_factor} ${0.1/scale_factor}  ${0.1/scale_factor}" filename="file://$(find perseus_description)/meshes/gearbox.dae"/>
+      </geometry>
+    </collision>
+  </link>
 </robot>

File: software/ros_ws/src/perseus_description/urdf/perseus.urdf.xacro (robot description, xacro)
@@ -2,33 +2,97 @@
 <robot xmlns:xacro="http://ros.org/wiki/xacro">
   <xacro:macro name="perseus" params="prefix">
-    <!-- Import components -->
+    <!-- Constants for robot dimensions -->
+    <xacro:property name="scale_factor" value="1"/>  <!-- 1 for Perseus and 2 for Perseu_Lite -->
+    <xacro:property name="PI" value="3.1415926535897931"/>
+    <xacro:property name="base_mass" value="0.3" /> <!-- arbitrary value for base mass -->
+    <xacro:property name="chassis_width" value="0.1" />
+    <xacro:property name="chassis_length" value="0.6" />
+    <xacro:property name="chassis_height" value="0.05" />
+    <xacro:property name="chassis_z_offset" value="0.35" /> <!-- Space btw top of beam and the each joint -->
+    <xacro:property name="flange_bearing_z_offset" value="0.1"/>  <!-- 1 for Perseus and 2 for Perseu_Lite -->
+    <xacro:property name="rocker_base_distance" value="0.275" />
+    <xacro:property name="rocker_x_offset" value="0.075"/>  <!-- 1 for Perseus and 2 for Perseu_Lite -->
+    <xacro:property name="rocker_y_offset" value="0.05"/>  <!-- 1 for Perseus and 2 for Perseu_Lite -->
+    <xacro:property name="motors_y_offset" value="0.035"/>  <!-- 1 for Perseus and 2 for Perseu_Lite -->
+    <xacro:property name="motors_z_offset" value="-0.25"/>  <!-- 1 for Perseus and 2 for Perseu_Lite -->
+    <xacro:property name="front_motors_x_offset" value="0.3"/>  <!-- 1 for Perseus and 2 for Perseu_Lite -->
+    <xacro:property name="rear_motors_x_offset" value="-0.55"/>  <!-- 1 for Perseus and 2 for Perseu_Lite -->
+    <xacro:property name="wheels_y_offset" value="0.125"/>
+    <!-- ADD COMPONENTS -->
     <xacro:include filename="$(find perseus_description)/urdf/chassis.urdf.xacro"/>
+    <xacro:include filename="$(find perseus_description)/urdf/flange_bearing.urdf.xacro"/>
     <xacro:include filename="$(find perseus_description)/urdf/rocker.urdf.xacro"/>
-    <xacro:include filename="$(find perseus_description)/urdf/sensors.urdf.xacro"/>
+    <xacro:include filename="$(find perseus_description)/urdf/motor_wheel.urdf.xacro"/>
+    <xacro:include filename="$(find perseus_description)/urdf/wheel.urdf.xacro"/>
+    <!-- An empty base_link to attach everything to -->
     <link name="${prefix}base_link"/>
-    <joint name="base_footprint_joint" type="fixed">
-        <parent link="base_link"/>
-        <child link="base_footprint"/>
-        <origin xyz="0 0 0" rpy="0 0 0"/>
-    </joint>
-    <link name="${prefix}base_footprint"/>
-    <!-- CHASSIS -->
-    <xacro:chassis />
-    <joint name="${prefix}chassis_joint" type="fixed">
-      <origin xyz="0.21 0.0 0.35" rpy="0.0 0.0 0.0"/>
+    <joint name="${prefix}chassis_joint" type="fixed"> <!-- Joint Connect base_link and chassis -->
+      <origin xyz="0 0.0 ${chassis_z_offset/scale_factor}" rpy="0.0 0.0 0.0"/>
       <parent link="${prefix}base_link"/>
       <child link="${prefix}chassis"/>
     </joint>
-    <!-- ROCKER ARMS -->
-    <!-- LEFT -->
-    <xacro:rocker side="left">
-      <origin xyz="-0.075 0.275 0.05" rpy="0.0 0.0 0"/>
-    </xacro:rocker>
-    <!-- RIGHT -->
-    <xacro:rocker side="right">
-      <origin xyz="-0.075 -0.275 0.05" rpy="0.0 0.0 0.0"/>
-    </xacro:rocker>
-    <xacro:sensors>
-    </xacro:sensors>
+    <joint name="${prefix}flange_bearing_joint" type="fixed">
+      <origin xyz="${-chassis_length/scale_factor} 0.0 ${flange_bearing_z_offset/scale_factor}" rpy="0 0 0"/>
+      <parent link="${prefix}chassis"/>
+      <child link="${prefix}flange_bearing"/>
+    </joint>
+    <joint name="${prefix}left_rocker_joint" type="fixed">
+      <origin xyz="${-rocker_x_offset/scale_factor} ${rocker_base_distance/scale_factor} ${rocker_y_offset/scale_factor} " rpy="0 0 0"/>
+      <parent link="${prefix}chassis"/>
+      <child link="${prefix}left_rocker"/>
+    </joint>
+    <joint name="${prefix}right_rocker_joint" type="fixed">
+      <origin xyz="${-rocker_x_offset/scale_factor} ${-rocker_base_distance/scale_factor} ${rocker_y_offset/scale_factor} " rpy="0 0 0"/>
+      <parent link="${prefix}chassis"/>
+      <child link="${prefix}right_rocker"/>
+    </joint>
+    <joint name="${prefix}front_left_motor_joint" type="fixed">
+      <parent link="${prefix}left_rocker"/>
+      <child link="${prefix}front_left_motor"/>
+      <origin xyz="${front_motors_x_offset/scale_factor} -${motors_y_offset/scale_factor} ${motors_z_offset/scale_factor}" rpy="0.0 0.0 0"/>
+    </joint>
+    <joint name="${prefix}rear_left_motor_joint" type="fixed">
+      <parent link="${prefix}left_rocker"/>
+      <child link="${prefix}rear_left_motor"/>
+      <origin xyz="${rear_motors_x_offset/scale_factor} -${motors_y_offset/scale_factor} ${motors_z_offset/scale_factor}" rpy="0.0 0.0 0.0"/>
+    </joint>
+    <joint name="${prefix}front_right_motor_joint" type="fixed">
+      <parent link="${prefix}right_rocker"/>
+      <child link="${prefix}front_right_motor"/>
+      <origin xyz="${front_motors_x_offset/scale_factor} ${motors_y_offset/scale_factor} ${motors_z_offset/scale_factor}" rpy="0.0 0.0 0"/>
+    </joint>
+    <joint name="${prefix}rear_right_motor_joint" type="fixed">
+      <parent link="${prefix}right_rocker"/>
+      <child link="${prefix}rear_right_motor"/>
+      <origin xyz="${rear_motors_x_offset/scale_factor} ${motors_y_offset/scale_factor} ${motors_z_offset/scale_factor}" rpy="0.0 0.0 0.0"/>
+    </joint>
+    <joint name="${prefix}front_left_wheel_joint" type="continuous">
+      <axis xyz="0 1 0" rpy="0 0 0"/>
+      <parent link="${prefix}front_left_motor"/>
+      <child link="${prefix}front_left_wheel"/>
+      <origin xyz="0 ${wheels_y_offset/scale_factor} 0.0" rpy="0.0 0.0 0"/>
+      <dynamics damping="0.2" friction="0.3"/>
+    </joint>
+    <joint name="${prefix}rear_left_wheel_joint" type="continuous">
+      <axis xyz="0 1 0" rpy="0 0 0"/>
+      <parent link="${prefix}rear_left_motor"/>
+      <child link="${prefix}rear_left_wheel"/>
+      <origin xyz="0 ${wheels_y_offset/scale_factor} 0.0" rpy="0.0 0.0 0"/>
+      <dynamics damping="0.2" friction="0.3"/>
+    </joint>
+    <joint name="${prefix}front_right_wheel_joint" type="continuous">
+      <axis xyz="0 1 0" rpy="0 0 0"/>
+      <parent link="${prefix}front_right_motor"/>
+      <child link="${prefix}front_right_wheel"/>
+      <origin xyz="0 -${wheels_y_offset/scale_factor} 0.0" rpy="0.0 0.0 0"/>
+      <dynamics damping="0.2" friction="0.3"/>
+    </joint>
+    <joint name="${prefix}rear_right_wheel_joint" type="continuous">
+      <axis xyz="0 1 0" rpy="0 0 0"/>
+      <parent link="${prefix}rear_right_motor"/>
+      <child link="${prefix}rear_right_wheel"/>
+      <origin xyz="0 -${wheels_y_offset/scale_factor} 0.0" rpy="0.0 0.0 0"/>
+      <dynamics damping="0.2" friction="0.3"/>
+    </joint>
   </xacro:macro>
 </robot>

File: software/ros_ws/src/perseus_description/urdf/rocker.urdf.xacro (robot description, xacro)
@@ -1,56 +1,35 @@
 <?xml version="1.0"?>
-<robot name="rocker" xmlns:xacro="http://www.ros.org/wiki/xacro">
-  <xacro:include filename="$(find perseus_description)/urdf/motor_wheel.urdf.xacro"/>
-  <xacro:macro name="rocker" params="prefix:=^ side *origin">
-    <!-- ROCKER ARM -->
-    <link name="${prefix}${side}_rocker">
-      <inertial>
-        <origin xyz="0.0 -0.0 -0.0" rpy="0 0 0"/>
-        <!-- RIGHT -->
-        <xacro:if value="${side == 'right'}">
-          <inertia ixx="0.078224" iyy="0.009964" izz="0.076528" ixy="0.003701" iyz="-0.006846" ixz="0.00298"/>
-        </xacro:if>
-        <!-- LEFT -->
-        <xacro:if value="${side == 'left'}">
-          <inertia ixx="0.078224" iyy="0.009964" izz="0.076528" ixy="0.003701" iyz="-0.006846" ixz="0.00298"/>
-        </xacro:if>
-        <mass value="1.2546142039512485"/>
-      </inertial>
-      <visual>
-        <origin xyz="0.0 0.0 0.0" rpy="0.0 0.0 ${pi}"/>
-        <geometry>
-          <mesh scale="0.1 0.1 0.1" filename="file://$(find perseus_description)/meshes/rocker_${side}.dae"/>
-        </geometry>
-      </visual>
-      <collision>
-        <origin xyz="0.2 0.0 -0.05" rpy="0.0 0.3 0.0"/>
-        <geometry>
-          <mesh scale="0.1 0.1 0.1" filename="file://$(find perseus_description)/meshes/rocker_${side}.dae"/>
-        </geometry>
-      </collision>
-    </link>
-    <joint name="${prefix}${side}_rocker_joint" type="fixed">
-      <xacro:insert_block name="origin"/>
-      <parent link="${prefix}chassis"/>
-      <child link="${prefix}${side}_rocker"/>
-    </joint>
-    <!-- FRONT MOTOR -->
-    <xacro:motor_wheel end="front">
-      <xacro:if value="${side == 'left'}">
-        <origin xyz="0.3 -0.035 -0.25" rpy="0.0 0.0 0"/>
-      </xacro:if>
-      <xacro:if value="${side == 'right'}">
-        <origin xyz="0.3 0.035 -0.25" rpy="0.0 0.0 0"/>
-      </xacro:if>
-    </xacro:motor_wheel>
-    <!-- REAR MOTOR -->
-    <xacro:motor_wheel end="rear">
-      <xacro:if value="${side == 'left'}">
-        <origin xyz="-0.55 -0.035 -0.25" rpy="0.0 0.0 0.0"/>
-      </xacro:if>
-      <xacro:if value="${side == 'right'}">
-        <origin xyz="-0.55 0.035 -0.25" rpy="0.0 0.0 0.0"/>
-      </xacro:if>
-    </xacro:motor_wheel>
-  </xacro:macro>
+<robot name="rocker" xmlns:xacro="http://ros.org/wiki/xacro">
+  <link name="${prefix}left_rocker">
+    <!-- <inertial>
+    </inertial> -->
+    <visual>
+      <origin xyz="0.0 0.0 0.0" rpy="0.0 0.0 ${pi}"/>
+      <geometry>
+        <mesh scale="${0.1/scale_factor} ${0.1/scale_factor}  ${0.1/scale_factor}" filename="file://$(find perseus_description)/meshes/rocker_left.dae"/>
+      </geometry>
+    </visual>
+    <collision>
+      <origin xyz="0.0 0.0 0.0" rpy="0.0 0.0 ${pi}"/>
+      <geometry>
+        <mesh scale="${0.1/scale_factor} ${0.1/scale_factor}  ${0.1/scale_factor}" filename="file://$(find perseus_description)/meshes/rocker_left.dae"/>
+      </geometry>
+    </collision>
+  </link>
+  <link name="${prefix}right_rocker">
+    <!-- <inertial>
+    </inertial> -->
+    <visual>
+      <origin xyz="0.0 0.0 0.0" rpy="0.0 0.0 ${pi}"/>
+      <geometry>
+        <mesh scale="${0.1/scale_factor} ${0.1/scale_factor}  ${0.1/scale_factor}" filename="file://$(find perseus_description)/meshes/rocker_right.dae"/>
+      </geometry>
+    </visual>
+    <collision>
+      <origin xyz="0.0 0.0 0.0" rpy="0.0 0.0 ${pi}"/>
+      <geometry>
+        <mesh scale="${0.1/scale_factor} ${0.1/scale_factor}  ${0.1/scale_factor}" filename="file://$(find perseus_description)/meshes/rocker_right.dae"/>
+      </geometry>
+    </collision>
+  </link>
 </robot>
