Commit message: Refactor URDF files for Perseus robot
- Updated rocker.urdf.xacro to simplify the definition of left and right rocker arms, removing unnecessary macros and including visual and collision elements directly.
- Revised wheel.urdf.xacro to define front and rear wheels without using macros, enhancing clarity and maintainability.
- Introduced a new chassis.urdf.xacro file to encapsulate the chassis structure, including inertial properties and visual/collision definitions.
- Created motor_wheel.urdf.xacro to define motor and wheel assemblies, streamlining the integration of wheel components.
- Added sensors.urdf.xacro to define laser and lidar sensors with appropriate joints and visual representations.
- Established perseus.materials.xacro to define materials used across the robot's components.
- Introduced a new perseus.urdf.xacro file to serve as the main entry point for the robot's URDF, integrating all components.
- Updated rviz configuration to enable visibility for all components, improving the visualization setup for simulation.

File: software/ros_ws/src/perseus_description/urdf/wheel.urdf.xacro (robot description, xacro)
@@ -1,83 +1,67 @@
 <?xml version="1.0"?>
 <robot name="wheel" xmlns:xacro="http://ros.org/wiki/xacro">
-  <xacro:macro name="wheel" params="prefix:=^ side:=^ end:=^">
-    <!-- WHEEL PROPERTIES -->
-      <xacro:property name="track_width" value="0.1" />
-      <xacro:property name="wheel_radius" value="0.05" />
-      <xacro:property name="wheel_mass" value="1.0" />
-      <xacro:property name="wheel_base" value="1.0" />
-    <link name="${prefix}${end}_${side}_wheel">
-      <inertial>
-        <xacro:if value="${side == 'left'}">
-          <origin xyz="0.0 0.125  0.0" rpy="0.0 0.0 0"/>
-        </xacro:if>
-        <xacro:if value="${side == 'right'}">
-          <origin xyz="0.0 -0.125  0.0" rpy="0.0 0.0 0.0"/>
-        </xacro:if>
-        <mass value="1.0"/>
-        <inertia ixx="0.04" iyy="0.02" izz="0.02" ixy="0.0" iyz="0.0" ixz="0.0"/>
-      </inertial>
-      <visual>
-        <xacro:if value="${side == 'left'}">
-          <origin xyz="0.0 0.125  0.0" rpy="0.0 0.0 ${pi}"/>
-        </xacro:if>
-        <xacro:if value="${side == 'right'}">
-          <origin xyz="0.0 -0.125  0.0" rpy="0.0 0.0 0.0"/>
-        </xacro:if>
-        <geometry>
-          <mesh scale="0.1 0.1 0.1" filename="file://$(find perseus_description)/meshes/wheel.dae"/>
-        </geometry>
-      </visual>
-      <collision>
-        <xacro:if value="${side == 'left'}">
-          <origin xyz="0.0 0.0 0.0" rpy="0.0 0.0 ${pi}"/>
-        </xacro:if>
-        <xacro:if value="${side == 'right'}">
-          <origin xyz="0.0 0.0 0.0" rpy="0.0 0.0 0.0"/>
-        </xacro:if>
-        <geometry>
-          <mesh scale="0.1 0.1 0.1" filename="file://$(find perseus_description)/meshes/wheel.dae"/>
-        </geometry>
-      </collision>
-    </link>
-    <!-- we need to use the gazebo tag to add in properties normally only found in SDF files -->
-    <gazebo reference="${prefix}${end}_${side}_wheel">
-      <!-- TODO: Fix the material tag (this isn't the proper way to do it, and spits out warnings) -->
-      <material>Gazebo/Orange</material>
-      <!-- see http://sdformat.org/spec?ver=1.12&elem=collision -->
-      <collision>
-        <surface>
-            <friction>
-                <ode>
-                    <!--
-                    In this case, the wheels need lower sideways than forwards coefficients of friction
-                    so that the rover can turn (skid steer) -->
-                    <!-- forward coefficient of friction -->
-                    <mu>1</mu>
-                    <!-- perpendicular coefficient of friction -->
-                    <mu2>0.3</mu2>
-                    <!--
-                    However, since mu/mu2 are normally relative to world coordinates,
-                    the rover would only be able to turn 90 degrees either way before they swapped, making turning impossible.
-                    To solve this, we need to specify the direction that mu/mu2 are relative to.
-                    -->
-                    <fdir1>1 0 0</fdir1>
-                </ode>
-            </friction>
-        </surface>
-      </collision>
-    </gazebo>
-    <joint name="${prefix}${end}_${side}_wheel_joint" type="continuous">
-      <xacro:if value="${side == 'left'}">
-        <axis xyz="0 1 0" rpy="0 0 0"/>
-      </xacro:if>
-      <xacro:if value="${side == 'right'}">
-        <axis xyz="0 1 0" rpy="0 0 0"/>
-      </xacro:if>
-      <parent link="${prefix}${end}_${side}_motor"/>
-      <child link="${prefix}${end}_${side}_wheel"/>
-      <origin xyz="0 0 0.0" rpy="0.0 0.0 0"/>
-      <dynamics damping="0.2" friction="0.3"/>
-    </joint>
-  </xacro:macro>
+<link name="${prefix}front_left_wheel">
+  <!-- <inertial>
+  </inertial> -->
+  <visual>
+    <origin xyz="0.0 0.0  0.0" rpy="0.0 0.0 ${pi}"/>
+    <geometry>
+      <mesh scale="${0.1/scale_factor} ${0.1/scale_factor}  ${0.1/scale_factor}" filename="file://$(find perseus_description)/meshes/wheel.dae"/>
+    </geometry>
+  </visual>
+  <collision>
+    <origin xyz="0.0 0.0 0.0" rpy="0.0 0.0 ${pi}"/>
+    <geometry>
+      <mesh scale="${0.1/scale_factor} ${0.1/scale_factor}  ${0.1/scale_factor}" filename="file://$(find perseus_description)/meshes/wheel.dae"/>
+    </geometry>
+  </collision>
+</link>
+<link name="${prefix}front_right_wheel">
+  <!-- <inertial>
+  </inertial> -->
+  <visual>
+      <origin xyz="0.0 0.0  0.0" rpy="0.0 0.0 0.0"/>
+    <geometry>
+      <mesh scale="${0.1/scale_factor} ${0.1/scale_factor}  ${0.1/scale_factor}" filename="file://$(find perseus_description)/meshes/wheel.dae"/>
+    </geometry>
+  </visual>
+  <collision>
+    <origin xyz="0.0 0.0 0.0" rpy="0.0 0.0 0.0"/>
+    <geometry>
+      <mesh scale="${0.1/scale_factor} ${0.1/scale_factor}  ${0.1/scale_factor}" filename="file://$(find perseus_description)/meshes/wheel.dae"/>
+    </geometry>
+  </collision>
+</link>
+<link name="${prefix}rear_left_wheel">
+  <!-- <inertial>
+  </inertial> -->
+  <visual>
+      <origin xyz="0.0 0.0  0.0" rpy="0.0 0.0 ${pi}"/>
+    <geometry>
+      <mesh scale="${0.1/scale_factor} ${0.1/scale_factor}  ${0.1/scale_factor}" filename="file://$(find perseus_description)/meshes/wheel.dae"/>
+    </geometry>
+  </visual>
+  <collision>
+    <origin xyz="0.0 0.0 0.0" rpy="0.0 0.0 ${pi}"/>
+    <geometry>
+      <mesh scale="${0.1/scale_factor} ${0.1/scale_factor}  ${0.1/scale_factor}" filename="file://$(find perseus_description)/meshes/wheel.dae"/>
+    </geometry>
+  </collision>
+</link>
+<link name="${prefix}rear_right_wheel">
+  <!-- <inertial>
+  </inertial> -->
+  <visual>
+      <origin xyz="0.0 0.0  0.0" rpy="0.0 0.0 0.0"/>
+    <geometry>
+      <mesh scale="${0.1/scale_factor} ${0.1/scale_factor}  ${0.1/scale_factor}" filename="file://$(find perseus_description)/meshes/wheel.dae"/>
+    </geometry>
+  </visual>
+  <collision>
+    <origin xyz="0.0 0.0 0.0" rpy="0.0 0.0 0.0"/>
+    <geometry>
+      <mesh scale="${0.1/scale_factor} ${0.1/scale_factor}  ${0.1/scale_factor}" filename="file://$(find perseus_description)/meshes/wheel.dae"/>
+    </geometry>
+  </collision>
+</link>
 </robot>

File: software/ros_ws/src/perseus_description/urdf_old/perseus.materials.xacro (robot description, xacro)
@@ -1,4 +1,4 @@
 <?xml version="1.0"?>
-<robot xmlns:xacro="http://ros.org/wiki/xacro">
+<robot>
   <material name="black">
     <color rgba="0.0 0.0 0.0 1.0"/>

Commit message: refactor: Restore inertial properties for chassis, flange bearing, motor wheels, and wheels

File: software/ros_ws/src/perseus_description/urdf/chassis.urdf.xacro (robot description, xacro)
@@ -2,9 +2,9 @@
 <robot name="chassis" xmlns:xacro="http://ros.org/wiki/xacro">
   <link name="${prefix}chassis">
-    <!-- <inertial>
+    <inertial>
       <origin xyz="0.0 -0.17100473204 0.14732485976" rpy="0 0 0"/>
       <mass value="2.7689940302592726"/>
       <inertia ixx="0.170464" iyy="0.092623" izz="0.224359" ixy="0.0" iyz="0.005411" ixz="-0.0"/>
-    </inertial> -->
+    </inertial>
     <visual>
       <origin xyz="0.0 0.0 0.0" rpy="0 0.0 -${pi/2}"/>

File: software/ros_ws/src/perseus_description/urdf/flange_bearing.urdf.xacro (robot description, xacro)
@@ -3,9 +3,9 @@
 <!-- Flange Bearing -->
 <link name="${prefix}flange_bearing">
-    <!-- <inertial>
-        <origin xyz="0.0 0.0 0.0" rpy="0 0 0"/>
-        <mass value="1.327488734939265"/>
-        <inertia ixx="0.001313" iyy="0.001699" izz="0.000647" ixy="0.0" iyz="0.0" ixz="-0.0"/>
-    </inertial> -->
+    <inertial>
+    <origin xyz="0.0 0.0 0.0" rpy="0 0 0"/>
+    <mass value="1.327488734939265"/>
+    <inertia ixx="0.001313" iyy="0.001699" izz="0.000647" ixy="0.0" iyz="0.0" ixz="-0.0"/>
+    </inertial>
     <visual>
     <origin xyz="0.0 0.0 0.0" rpy="${-pi/2} 0 ${pi/2}"/>
@@ -23,9 +23,9 @@
 <!-- Balance/differential bar -->
 <link name="${prefix}differential_bar">
-    <!-- <inertial>
+    <inertial>
         <origin xyz="0 0 0.0" rpy="0.0 0.0 0.0"/>
         <mass value="0.9172649518127158"/>
         <inertia ixx="0.00036" iyy="0.018339" izz="0.018134" ixy="3e-06" iyz="-0.0" ixz="0.0"/>
-    </inertial> -->
+    </inertial>
     <visual>
     <origin xyz="0.0 0.0 0.0" rpy="${-pi/2} 0 ${-pi/2}"/>

File: software/ros_ws/src/perseus_description/urdf/motor_wheel.urdf.xacro (robot description, xacro)
@@ -2,6 +2,10 @@
 <robot name="motor_wheel" xmlns:xacro="http://www.ros.org/wiki/xacro">
   <link name="${prefix}front_right_motor">
-    <!-- <inertial>
-    </inertial> -->
+    <inertial>
+      <!-- moving origin has no perceivable impact-->
+      <origin xyz="0.0 0.0 0.0" rpy="0.0 0.0 0.0"/>
+      <mass value="5.236579"/>
+      <inertia ixx="0.01" iyy="0.01" izz="0.01" ixy="0.0" iyz="0.0" ixz="0.0"/> <!-- TEMP -->
+    </inertial>
     <visual>
       <origin xyz="0 0.0 0.0" rpy="0.0 0.0 ${pi/2}"/>
@@ -19,6 +23,10 @@
   </link>
   <link name="${prefix}rear_right_motor">
-    <!-- <inertial>
-    </inertial> -->
+    <inertial>
+      <!-- moving origin has no perceivable impact-->
+      <origin xyz="0.0 0.0 0.0" rpy="0.0 0.0 0.0"/>
+      <mass value="5.236579"/>
+      <inertia ixx="0.01" iyy="0.01" izz="0.01" ixy="0.0" iyz="0.0" ixz="0.0"/> <!-- TEMP -->
+    </inertial>
     <visual>
       <origin xyz="0 0.0 0.0" rpy="0.0 0.0 ${pi/2}"/>
@@ -36,6 +44,10 @@
   </link>
   <link name="${prefix}front_left_motor">
-    <!-- <inertial>
-    </inertial> -->
+    <inertial>
+      <!-- moving origin has no perceivable impact-->
+      <origin xyz="0.0 0.0 0.0" rpy="0.0 0.0 0.0"/>
+      <mass value="5.236579"/>
+      <inertia ixx="0.01" iyy="0.01" izz="0.01" ixy="0.0" iyz="0.0" ixz="0.0"/> <!-- TEMP -->
+    </inertial>
     <visual>
       <origin xyz="0 0.0 0.0" rpy="0.0 0.0 ${-pi/2}"/>
@@ -53,6 +65,10 @@
   </link>
   <link name="${prefix}rear_left_motor">
-    <!-- <inertial>
-    </inertial> -->
+    <inertial>
+      <!-- moving origin has no perceivable impact-->
+      <origin xyz="0.0 0.0 0.0" rpy="0.0 0.0 0.0"/>
+      <mass value="5.236579"/>
+      <inertia ixx="0.01" iyy="0.01" izz="0.01" ixy="0.0" iyz="0.0" ixz="0.0"/> <!-- TEMP -->
+    </inertial>
     <visual>
       <origin xyz="0 0.0 0.0" rpy="0.0 0.0 ${-pi/2}"/>

File: software/ros_ws/src/perseus_description/urdf/wheel.urdf.xacro (robot description, xacro)
@@ -2,6 +2,9 @@
 <robot name="wheel" xmlns:xacro="http://ros.org/wiki/xacro">
 <link name="${prefix}front_left_wheel">
-  <!-- <inertial>
-  </inertial> -->
+  <inertial>
+    <origin xyz="0.0 0.0 0.0" rpy="0.0 0.0 0.0"/>
+    <mass value="1.0"/>
+    <inertia ixx="0.04" iyy="0.02" izz="0.02" ixy="0.0" iyz="0.0" ixz="0.0"/>
+  </inertial>
   <visual>
     <origin xyz="0.0 0.0  0.0" rpy="0.0 0.0 ${pi}"/>
@@ -18,6 +21,9 @@
 </link>
 <link name="${prefix}front_right_wheel">
-  <!-- <inertial>
-  </inertial> -->
+  <inertial>
+    <origin xyz="0.0 0.0 0.0" rpy="0.0 0.0 0.0"/>
+    <mass value="1.0"/>
+    <inertia ixx="0.04" iyy="0.02" izz="0.02" ixy="0.0" iyz="0.0" ixz="0.0"/>
+  </inertial>
   <visual>
       <origin xyz="0.0 0.0  0.0" rpy="0.0 0.0 0.0"/>
@@ -34,6 +40,9 @@
 </link>
 <link name="${prefix}rear_left_wheel">
-  <!-- <inertial>
-  </inertial> -->
+  <inertial>
+    <origin xyz="0.0 0.0 0.0" rpy="0.0 0.0 0.0"/>
+    <mass value="1.0"/>
+    <inertia ixx="0.04" iyy="0.02" izz="0.02" ixy="0.0" iyz="0.0" ixz="0.0"/>
+  </inertial>
   <visual>
       <origin xyz="0.0 0.0  0.0" rpy="0.0 0.0 ${pi}"/>
@@ -50,6 +59,9 @@
 </link>
 <link name="${prefix}rear_right_wheel">
-  <!-- <inertial>
-  </inertial> -->
+  <inertial>
+    <origin xyz="0.0 0.0 0.0" rpy="0.0 0.0 0.0"/>
+    <mass value="1.0"/>
+    <inertia ixx="0.04" iyy="0.02" izz="0.02" ixy="0.0" iyz="0.0" ixz="0.0"/>
+  </inertial>
   <visual>
       <origin xyz="0.0 0.0  0.0" rpy="0.0 0.0 0.0"/>
@@ -65,3 +77,107 @@
   </collision>
 </link>
+<gazebo reference="${prefix}front_left_wheel">
+  <!-- TODO: Fix the material tag (this isn't the proper way to do it, and spits out warnings) -->
+  <material>Gazebo/Orange</material>
+  <!-- see http://sdformat.org/spec?ver=1.12&elem=collision -->
+  <collision>
+    <surface>
+        <friction>
+            <ode>
+                <!--
+                In this case, the wheels need lower sideways than forwards coefficients of friction
+                so that the rover can turn (skid steer) -->
+                <!-- forward coefficient of friction -->
+                <mu>0.3</mu>
+                <!-- perpendicular coefficient of friction -->
+                <mu2>1</mu2>
+                <!--
+                However, since mu/mu2 are normally relative to world coordinates,
+                the rover would only be able to turn 90 degrees either way before they swapped, making turning impossible.
+                To solve this, we need to specify the direction that mu/mu2 are relative to.
+                -->
+                <fdir1>1 0 0</fdir1>
+            </ode>
+        </friction>
+    </surface>
+  </collision>
+</gazebo>
+<gazebo reference="${prefix}front_right_wheel">
+  <!-- TODO: Fix the material tag (this isn't the proper way to do it, and spits out warnings) -->
+  <material>Gazebo/Orange</material>
+  <!-- see http://sdformat.org/spec?ver=1.12&elem=collision -->
+  <collision>
+    <surface>
+        <friction>
+            <ode>
+                <!--
+                In this case, the wheels need lower sideways than forwards coefficients of friction
+                so that the rover can turn (skid steer) -->
+                <!-- forward coefficient of friction -->
+                <mu>0.3</mu>
+                <!-- perpendicular coefficient of friction -->
+                <mu2>1</mu2>
+                <!--
+                However, since mu/mu2 are normally relative to world coordinates,
+                the rover would only be able to turn 90 degrees either way before they swapped, making turning impossible.
+                To solve this, we need to specify the direction that mu/mu2 are relative to.
+                -->
+                <fdir1>1 0 0</fdir1>
+            </ode>
+        </friction>
+    </surface>
+  </collision>
+</gazebo>
+<gazebo reference="${prefix}rear_right_wheel">
+  <!-- TODO: Fix the material tag (this isn't the proper way to do it, and spits out warnings) -->
+  <material>Gazebo/Orange</material>
+  <!-- see http://sdformat.org/spec?ver=1.12&elem=collision -->
+  <collision>
+    <surface>
+        <friction>
+            <ode>
+                <!--
+                In this case, the wheels need lower sideways than forwards coefficients of friction
+                so that the rover can turn (skid steer) -->
+                <!-- forward coefficient of friction -->
+                <mu>0.3</mu>
+                <!-- perpendicular coefficient of friction -->
+                <mu2>1</mu2>
+                <!--
+                However, since mu/mu2 are normally relative to world coordinates,
+                the rover would only be able to turn 90 degrees either way before they swapped, making turning impossible.
+                To solve this, we need to specify the direction that mu/mu2 are relative to.
+                -->
+                <fdir1>1 0 0</fdir1>
+            </ode>
+        </friction>
+    </surface>
+  </collision>
+</gazebo>
+<gazebo reference="${prefix}rear_left_wheel">
+  <!-- TODO: Fix the material tag (this isn't the proper way to do it, and spits out warnings) -->
+  <material>Gazebo/Orange</material>
+  <!-- see http://sdformat.org/spec?ver=1.12&elem=collision -->
+  <collision>
+    <surface>
+        <friction>
+            <ode>
+                <!--
+                In this case, the wheels need lower sideways than forwards coefficients of friction
+                so that the rover can turn (skid steer) -->
+                <!-- forward coefficient of friction -->
+                <mu>0.3</mu>
+                <!-- perpendicular coefficient of friction -->
+                <mu2>1</mu2>
+                <!--
+                However, since mu/mu2 are normally relative to world coordinates,
+                the rover would only be able to turn 90 degrees either way before they swapped, making turning impossible.
+                To solve this, we need to specify the direction that mu/mu2 are relative to.
+                -->
+                <fdir1>1 0 0</fdir1>
+            </ode>
+        </friction>
+    </surface>
+  </collision>
+</gazebo>
 </robot>

Commit message: refactor: Update URDF files for chassis and lidar sensor integration

File: software/ros_ws/src/perseus_description/urdf/chassis.urdf.xacro (robot description, xacro)
@@ -21,3 +21,12 @@
     </collision>
   </link>
+  <gazebo reference="${prefix}chassis">
+      <material>Gazebo/Grey</material>
+      <sensor name="imu_sensor" type="imu">
+          <always_on>1</always_on>
+          <update_rate>10</update_rate>
+          <visualize>true</visualize>
+          <topic>imu</topic>
+      </sensor>
+  </gazebo>
 </robot>

File: software/ros_ws/src/perseus_description/urdf/sensors.urdf.xacro (robot description, xacro)
@@ -15,4 +15,5 @@
     </collision>
 </link>
+<!-- Simulating the Livox MID-360 -->
 <gazebo reference="${prefix}laser_frame">
   <material>
@@ -34,4 +35,5 @@
           <max_angle>3.14159</max_angle>
         </horizontal>
+        <!-- Angle Simulating the Livox MID-360 -->
         <vertical>
           <samples>32</samples>
