Commit message: Refactor Nix package definitions for Perseus components
- Updated Nix expressions for `perseus-can-if`, `perseus-description`, `perseus-hardware`, `perseus-input-config`, `perseus-input`, `perseus-payloads`, `perseus-sensors`, `perseus-simulation`, `perseus-teleop`, and `perseus` to improve readability by formatting lists of dependencies.
- Adjusted the `shell.nix` file to enhance the shell hook for ROS 2 completion.
- Modified URDF files for `chassis`, `flange_bearing`, `motor_wheel`, and `wheel` to update inertial properties and mass values for better simulation accuracy.
- Updated `perseus_sim.launch.py` to change the RViz configuration file reference.
- Enhanced RViz configuration in `view.rviz` to improve visualization settings and TF display.

File: software/ros_ws/src/perseus_description/urdf/chassis.urdf.xacro (robot description, xacro)
@@ -2,9 +2,9 @@
 <robot name="chassis" xmlns:xacro="http://ros.org/wiki/xacro">
   <link name="${prefix}chassis">
-    <inertial>
-      <origin xyz="0.0 -0.17100473204 0.14732485976" rpy="0 0 0"/>
-      <mass value="2.7689940302592726"/>
-      <inertia ixx="0.170464" iyy="0.092623" izz="0.224359" ixy="0.0" iyz="0.005411" ixz="-0.0"/>
-    </inertial>
+  <inertial>
+    <origin xyz="0 0 0" rpy="0 0 0"/>
+    <mass value="0.2"/>
+    <inertia ixx="0.00014" iyy="0.00014" izz="0.00025" ixy="0.0" iyz="0.0" ixz="0.0"/>
+  </inertial>
     <visual>
       <origin xyz="0.0 0.0 0.0" rpy="0 0.0 -${pi/2}"/>

File: software/ros_ws/src/perseus_description/urdf/flange_bearing.urdf.xacro (robot description, xacro)
@@ -5,5 +5,5 @@
     <inertial>
     <origin xyz="0.0 0.0 0.0" rpy="0 0 0"/>
-    <mass value="1.327488734939265"/>
+    <mass value="1"/>
     <inertia ixx="0.001313" iyy="0.001699" izz="0.000647" ixy="0.0" iyz="0.0" ixz="-0.0"/>
     </inertial>

File: software/ros_ws/src/perseus_description/urdf/motor_wheel.urdf.xacro (robot description, xacro)
@@ -5,5 +5,5 @@
       <!-- moving origin has no perceivable impact-->
       <origin xyz="0.0 0.0 0.0" rpy="0.0 0.0 0.0"/>
-      <mass value="5.236579"/>
+      <mass value="1"/>
       <inertia ixx="0.01" iyy="0.01" izz="0.01" ixy="0.0" iyz="0.0" ixz="0.0"/> <!-- TEMP -->
     </inertial>
@@ -26,5 +26,5 @@
       <!-- moving origin has no perceivable impact-->
       <origin xyz="0.0 0.0 0.0" rpy="0.0 0.0 0.0"/>
-      <mass value="5.236579"/>
+      <mass value="1"/>
       <inertia ixx="0.01" iyy="0.01" izz="0.01" ixy="0.0" iyz="0.0" ixz="0.0"/> <!-- TEMP -->
     </inertial>
@@ -47,5 +47,5 @@
       <!-- moving origin has no perceivable impact-->
       <origin xyz="0.0 0.0 0.0" rpy="0.0 0.0 0.0"/>
-      <mass value="5.236579"/>
+      <mass value="1"/>
       <inertia ixx="0.01" iyy="0.01" izz="0.01" ixy="0.0" iyz="0.0" ixz="0.0"/> <!-- TEMP -->
     </inertial>
@@ -68,5 +68,5 @@
       <!-- moving origin has no perceivable impact-->
       <origin xyz="0.0 0.0 0.0" rpy="0.0 0.0 0.0"/>
-      <mass value="5.236579"/>
+      <mass value="1"/>
       <inertia ixx="0.01" iyy="0.01" izz="0.01" ixy="0.0" iyz="0.0" ixz="0.0"/> <!-- TEMP -->
     </inertial>

File: software/ros_ws/src/perseus_description/urdf/perseus.urdf.xacro (robot description, xacro)
@@ -99,5 +99,5 @@
       <parent link="${prefix}chassis"/>
       <child link="${prefix}laser_frame"/>
-      <origin xyz="0 0 -0.04" rpy="0 ${PI} 0"/>
+      <origin xyz="0 0 0.23" rpy="0 0.785 0"/>
     </joint>
   </xacro:macro>

File: software/ros_ws/src/perseus_description/urdf/wheel.urdf.xacro (robot description, xacro)
@@ -3,7 +3,7 @@
 <link name="${prefix}front_left_wheel">
   <inertial>
-    <origin xyz="0.0 0.0 0.0" rpy="0.0 0.0 0.0"/>
-    <mass value="1.0"/>
-    <inertia ixx="0.04" iyy="0.02" izz="0.02" ixy="0.0" iyz="0.0" ixz="0.0"/>
+    <origin xyz="0 0 0" rpy="0 0 0"/>
+    <mass value="0.2"/>
+    <inertia ixx="0.00014" iyy="0.00014" izz="0.00025" ixy="0.0" iyz="0.0" ixz="0.0"/>
   </inertial>
   <visual>
@@ -22,7 +22,7 @@
 <link name="${prefix}front_right_wheel">
   <inertial>
-    <origin xyz="0.0 0.0 0.0" rpy="0.0 0.0 0.0"/>
-    <mass value="1.0"/>
-    <inertia ixx="0.04" iyy="0.02" izz="0.02" ixy="0.0" iyz="0.0" ixz="0.0"/>
+    <origin xyz="0 0 0" rpy="0 0 0"/>
+    <mass value="0.2"/>
+    <inertia ixx="0.00014" iyy="0.00014" izz="0.00025" ixy="0.0" iyz="0.0" ixz="0.0"/>
   </inertial>
   <visual>
@@ -41,7 +41,7 @@
 <link name="${prefix}rear_left_wheel">
   <inertial>
-    <origin xyz="0.0 0.0 0.0" rpy="0.0 0.0 0.0"/>
-    <mass value="1.0"/>
-    <inertia ixx="0.04" iyy="0.02" izz="0.02" ixy="0.0" iyz="0.0" ixz="0.0"/>
+    <origin xyz="0 0 0" rpy="0 0 0"/>
+    <mass value="0.2"/>
+    <inertia ixx="0.00014" iyy="0.00014" izz="0.00025" ixy="0.0" iyz="0.0" ixz="0.0"/>
   </inertial>
   <visual>
@@ -60,7 +60,7 @@
 <link name="${prefix}rear_right_wheel">
   <inertial>
-    <origin xyz="0.0 0.0 0.0" rpy="0.0 0.0 0.0"/>
-    <mass value="1.0"/>
-    <inertia ixx="0.04" iyy="0.02" izz="0.02" ixy="0.0" iyz="0.0" ixz="0.0"/>
+    <origin xyz="0 0 0" rpy="0 0 0"/>
+    <mass value="0.2"/>
+    <inertia ixx="0.00014" iyy="0.00014" izz="0.00025" ixy="0.0" iyz="0.0" ixz="0.0"/>
   </inertial>
   <visual>
@@ -78,23 +78,11 @@
 </link>
 <gazebo reference="${prefix}front_left_wheel">
-  <!-- TODO: Fix the material tag (this isn't the proper way to do it, and spits out warnings) -->
   <material>Gazebo/Orange</material>
-  <!-- see http://sdformat.org/spec?ver=1.12&elem=collision -->
   <collision>
     <surface>
         <friction>
             <ode>
-                <!--
-                In this case, the wheels need lower sideways than forwards coefficients of friction
-                so that the rover can turn (skid steer) -->
-                <!-- forward coefficient of friction -->
-                <mu>0.3</mu>
-                <!-- perpendicular coefficient of friction -->
-                <mu2>1</mu2>
-                <!--
-                However, since mu/mu2 are normally relative to world coordinates,
-                the rover would only be able to turn 90 degrees either way before they swapped, making turning impossible.
-                To solve this, we need to specify the direction that mu/mu2 are relative to.
-                -->
+                <mu>0.01</mu>
+                <mu2>0.01</mu2>
                 <fdir1>1 0 0</fdir1>
             </ode>
@@ -104,23 +92,11 @@
 </gazebo>
 <gazebo reference="${prefix}front_right_wheel">
-  <!-- TODO: Fix the material tag (this isn't the proper way to do it, and spits out warnings) -->
   <material>Gazebo/Orange</material>
-  <!-- see http://sdformat.org/spec?ver=1.12&elem=collision -->
   <collision>
     <surface>
         <friction>
             <ode>
-                <!--
-                In this case, the wheels need lower sideways than forwards coefficients of friction
-                so that the rover can turn (skid steer) -->
-                <!-- forward coefficient of friction -->
-                <mu>0.3</mu>
-                <!-- perpendicular coefficient of friction -->
-                <mu2>1</mu2>
-                <!--
-                However, since mu/mu2 are normally relative to world coordinates,
-                the rover would only be able to turn 90 degrees either way before they swapped, making turning impossible.
-                To solve this, we need to specify the direction that mu/mu2 are relative to.
-                -->
+                <mu>0.01</mu>
+                <mu2>0.01</mu2>
                 <fdir1>1 0 0</fdir1>
             </ode>
@@ -130,23 +106,11 @@
 </gazebo>
 <gazebo reference="${prefix}rear_right_wheel">
-  <!-- TODO: Fix the material tag (this isn't the proper way to do it, and spits out warnings) -->
   <material>Gazebo/Orange</material>
-  <!-- see http://sdformat.org/spec?ver=1.12&elem=collision -->
   <collision>
     <surface>
         <friction>
             <ode>
-                <!--
-                In this case, the wheels need lower sideways than forwards coefficients of friction
-                so that the rover can turn (skid steer) -->
-                <!-- forward coefficient of friction -->
-                <mu>0.3</mu>
-                <!-- perpendicular coefficient of friction -->
-                <mu2>1</mu2>
-                <!--
-                However, since mu/mu2 are normally relative to world coordinates,
-                the rover would only be able to turn 90 degrees either way before they swapped, making turning impossible.
-                To solve this, we need to specify the direction that mu/mu2 are relative to.
-                -->
+                <mu>0.01</mu>
+                <mu2>0.01</mu2>
                 <fdir1>1 0 0</fdir1>
             </ode>
@@ -156,23 +120,11 @@
 </gazebo>
 <gazebo reference="${prefix}rear_left_wheel">
-  <!-- TODO: Fix the material tag (this isn't the proper way to do it, and spits out warnings) -->
   <material>Gazebo/Orange</material>
-  <!-- see http://sdformat.org/spec?ver=1.12&elem=collision -->
   <collision>
     <surface>
         <friction>
             <ode>
-                <!--
-                In this case, the wheels need lower sideways than forwards coefficients of friction
-                so that the rover can turn (skid steer) -->
-                <!-- forward coefficient of friction -->
-                <mu>0.3</mu>
-                <!-- perpendicular coefficient of friction -->
-                <mu2>1</mu2>
-                <!--
-                However, since mu/mu2 are normally relative to world coordinates,
-                the rover would only be able to turn 90 degrees either way before they swapped, making turning impossible.
-                To solve this, we need to specify the direction that mu/mu2 are relative to.
-                -->
+                <mu>0.01</mu>
+                <mu2>0.01</mu2>
                 <fdir1>1 0 0</fdir1>
             </ode>

Commit message: refactor: Update URDF files and macros for improved inertia calculations and structure

File: software/ros_ws/src/perseus_description/urdf/chassis.urdf.xacro (robot description, xacro)
@@ -1,9 +1,10 @@
 <?xml version="1.0"?>
 <robot name="chassis" xmlns:xacro="http://ros.org/wiki/xacro">
+  <xacro:property name="chassis_mass" value="2.7689940302592726"/>  <!-- Kg -->
   <link name="${prefix}chassis">
     <inertial>
       <origin xyz="0.0 -0.17100473204 0.14732485976" rpy="0 0 0"/>
-      <mass value="2.7689940302592726"/>
-      <inertia ixx="0.170464" iyy="0.092623" izz="0.224359" ixy="0.0" iyz="0.005411" ixz="-0.0"/>
+      <mass value="${chassis_mass}"/>
+      <xacro:box_inertia m="${chassis_mass}" x="${chassis_length/scale_factor}" y="${chassis_width/scale_factor}" z="${chassis_height/scale_factor}"/>
     </inertial>
     <visual>
@@ -14,8 +15,8 @@
     </visual>
     <collision>
-      <origin xyz="0.0 0.0 0.0" rpy="0 0.0 -${pi/2}"/>
+      <origin xyz="${-chassis_length/scale_factor*0.5} 0.0 ${chassis_height/scale_factor*0.5}" rpy="0 0.0 0"/>
       <!-- Modified to make collision more simple, chassis mesh replaced with box -->
       <geometry>
-        <mesh scale="${0.1/scale_factor} ${0.1/scale_factor}  ${0.1/scale_factor}" filename="file://$(find perseus_description)/meshes/chassis.dae"/>
+        <box size="${chassis_length/scale_factor} ${chassis_width/scale_factor} ${chassis_height/scale_factor}"/>
       </geometry>
     </collision>

File: software/ros_ws/src/perseus_description/urdf/motor_wheel.urdf.xacro (robot description, xacro)
@@ -1,9 +1,13 @@
 <?xml version="1.0"?>
 <robot name="motor_wheel" xmlns:xacro="http://www.ros.org/wiki/xacro">
+  <xacro:property name="motor_mass" value="5.236579"/>  <!-- Kg -->
+  <xacro:property name="collision_motor_length" value="0.1"/>  <!-- m -->
+  <xacro:property name="collision_motor_width" value="0.1"/>  <!-- m -->
+  <xacro:property name="collision_motor_height" value="0.075"/>  <!-- m -->
   <link name="${prefix}front_right_motor">
     <inertial>
       <!-- moving origin has no perceivable impact-->
       <origin xyz="0.0 0.0 0.0" rpy="0.0 0.0 0.0"/>
-      <mass value="5.236579"/>
+      <mass value="${motor_mass}"/>
       <inertia ixx="0.01" iyy="0.01" izz="0.01" ixy="0.0" iyz="0.0" ixz="0.0"/> <!-- TEMP -->
     </inertial>
@@ -16,7 +20,7 @@
     </visual>
     <collision>
-      <origin xyz="-0.3 0.0 0.0" rpy="0.0 0.0 ${pi/2}"/>
+      <origin xyz="0.0 0.0 0.0" rpy="0.0 0.0 ${pi/2}"/>
       <geometry>
-        <mesh scale="${0.1/scale_factor} ${0.1/scale_factor}  ${0.1/scale_factor}" filename="file://$(find perseus_description)/meshes/gearbox.dae"/>
+        <box size="${collision_motor_length/scale_factor} ${collision_motor_width/scale_factor} ${collision_motor_height/scale_factor}" />
       </geometry>
     </collision>
@@ -26,5 +30,5 @@
       <!-- moving origin has no perceivable impact-->
       <origin xyz="0.0 0.0 0.0" rpy="0.0 0.0 0.0"/>
-      <mass value="5.236579"/>
+      <mass value="${motor_mass}"/>
       <inertia ixx="0.01" iyy="0.01" izz="0.01" ixy="0.0" iyz="0.0" ixz="0.0"/> <!-- TEMP -->
     </inertial>
@@ -37,7 +41,7 @@
     </visual>
     <collision>
-      <origin xyz="-0.3 0.0 0.0" rpy="0.0 0.0 ${pi/2}"/>
+      <origin xyz="0.0 0.0 0.0" rpy="0.0 0.0 ${pi/2}"/>
       <geometry>
-        <mesh scale="${0.1/scale_factor} ${0.1/scale_factor}  ${0.1/scale_factor}" filename="file://$(find perseus_description)/meshes/gearbox.dae"/>
+        <box size="${collision_motor_length/scale_factor} ${collision_motor_width/scale_factor} ${collision_motor_height/scale_factor}" />
       </geometry>
     </collision>
@@ -47,5 +51,5 @@
       <!-- moving origin has no perceivable impact-->
       <origin xyz="0.0 0.0 0.0" rpy="0.0 0.0 0.0"/>
-      <mass value="5.236579"/>
+      <mass value="${motor_mass}"/>
       <inertia ixx="0.01" iyy="0.01" izz="0.01" ixy="0.0" iyz="0.0" ixz="0.0"/> <!-- TEMP -->
     </inertial>
@@ -60,5 +64,5 @@
       <origin xyz="0 0.0 0.0" rpy="0.0 0.0 ${-pi/2}"/>
       <geometry>
-        <mesh scale="${0.1/scale_factor} ${0.1/scale_factor}  ${0.1/scale_factor}" filename="file://$(find perseus_description)/meshes/gearbox.dae"/>
+        <box size="${collision_motor_length/scale_factor} ${collision_motor_width/scale_factor} ${collision_motor_height/scale_factor}" />
       </geometry>
     </collision>
@@ -68,5 +72,5 @@
       <!-- moving origin has no perceivable impact-->
       <origin xyz="0.0 0.0 0.0" rpy="0.0 0.0 0.0"/>
-      <mass value="5.236579"/>
+      <mass value="${motor_mass}"/>
       <inertia ixx="0.01" iyy="0.01" izz="0.01" ixy="0.0" iyz="0.0" ixz="0.0"/> <!-- TEMP -->
     </inertial>
@@ -81,5 +85,5 @@
       <origin xyz="0 0.0 0.0" rpy="0.0 0.0 ${-pi/2}"/>
       <geometry>
-        <mesh scale="${0.1/scale_factor} ${0.1/scale_factor}  ${0.1/scale_factor}" filename="file://$(find perseus_description)/meshes/gearbox.dae"/>
+        <box size="${collision_motor_length/scale_factor} ${collision_motor_width/scale_factor} ${collision_motor_height/scale_factor}" />
       </geometry>
     </collision>

File: software/ros_ws/src/perseus_description/urdf/perseus.urdf.xacro (robot description, xacro)
@@ -5,19 +5,28 @@
     <xacro:property name="scale_factor" value="1"/>  <!-- 1 for Perseus and 2 for Perseu_Lite -->
     <xacro:property name="PI" value="3.1415926535897931"/>
+    <!-- Chassis Properties -->
     <xacro:property name="base_mass" value="0.3" /> <!-- arbitrary value for base mass -->
-    <xacro:property name="chassis_width" value="0.1" />
+    <xacro:property name="chassis_width" value="0.45" />
     <xacro:property name="chassis_length" value="0.6" />
-    <xacro:property name="chassis_height" value="0.05" />
+    <xacro:property name="chassis_height" value="0.2" />
     <xacro:property name="chassis_z_offset" value="0.35" /> <!-- Space btw top of beam and the each joint -->
-    <xacro:property name="flange_bearing_z_offset" value="0.1"/>  <!-- 1 for Perseus and 2 for Perseu_Lite -->
+    <!-- Flange Bearing Properties -->
+    <xacro:property name="flange_bearing_z_offset" value="0.1"/>
+    <!-- Rocker Properties -->
     <xacro:property name="rocker_base_distance" value="0.275" />
-    <xacro:property name="rocker_x_offset" value="0.075"/>  <!-- 1 for Perseus and 2 for Perseu_Lite -->
-    <xacro:property name="rocker_y_offset" value="0.05"/>  <!-- 1 for Perseus and 2 for Perseu_Lite -->
-    <xacro:property name="motors_y_offset" value="0.035"/>  <!-- 1 for Perseus and 2 for Perseu_Lite -->
-    <xacro:property name="motors_z_offset" value="-0.25"/>  <!-- 1 for Perseus and 2 for Perseu_Lite -->
-    <xacro:property name="front_motors_x_offset" value="0.3"/>  <!-- 1 for Perseus and 2 for Perseu_Lite -->
-    <xacro:property name="rear_motors_x_offset" value="-0.55"/>  <!-- 1 for Perseus and 2 for Perseu_Lite -->
+    <xacro:property name="rocker_x_offset" value="0.075"/>
+    <xacro:property name="rocker_y_offset" value="0.05"/>
+    <!-- Motors Properties -->
+    <xacro:property name="motors_y_offset" value="0.035"/>
+    <xacro:property name="motors_z_offset" value="-0.25"/>
+    <xacro:property name="front_motors_x_offset" value="0.3"/>
+    <xacro:property name="rear_motors_x_offset" value="-0.55"/>
+    <!-- Wheels Properties -->
     <xacro:property name="wheels_y_offset" value="0.125"/>
+    <xacro:property name="wheel_mass" value="1.0"/>
+    <xacro:property name="wheel_radius" value="0.13"/>
+    <xacro:property name="wheel_length" value="0.15"/>
     <!-- ADD COMPONENTS -->
+    <xacro:include filename="$(find perseus_description)/urdf/inertia_macros.xacro"/>
     <xacro:include filename="$(find perseus_description)/urdf/chassis.urdf.xacro"/>
     <xacro:include filename="$(find perseus_description)/urdf/flange_bearing.urdf.xacro"/>

File: software/ros_ws/src/perseus_description/urdf/rocker.urdf.xacro (robot description, xacro)
@@ -2,6 +2,4 @@
 <robot name="rocker" xmlns:xacro="http://ros.org/wiki/xacro">
   <link name="${prefix}left_rocker">
-    <!-- <inertial>
-    </inertial> -->
     <visual>
       <origin xyz="0.0 0.0 0.0" rpy="0.0 0.0 ${pi}"/>

File: software/ros_ws/src/perseus_description/urdf/wheel.urdf.xacro (robot description, xacro)
@@ -3,7 +3,7 @@
 <link name="${prefix}front_left_wheel">
   <inertial>
-    <origin xyz="0.0 0.0 0.0" rpy="0.0 0.0 0.0"/>
-    <mass value="1.0"/>
-    <inertia ixx="0.04" iyy="0.02" izz="0.02" ixy="0.0" iyz="0.0" ixz="0.0"/>
+    <origin xyz="0.0 0.0  0.0" rpy="0.0 0.0 ${pi}"/>
+    <mass value="${wheel_mass}"/>
+    <xacro:cylinder_inertia m="${wheel_mass}" radius="${wheel_radius}" length="${wheel_length}"/>
   </inertial>
   <visual>
@@ -14,7 +14,7 @@
   </visual>
   <collision>
-    <origin xyz="0.0 0.0 0.0" rpy="0.0 0.0 ${pi}"/>
+    <origin xyz="0.0 0.0 0.0" rpy="${pi/2} 0.0 ${pi}"/>
     <geometry>
-      <mesh scale="${0.1/scale_factor} ${0.1/scale_factor}  ${0.1/scale_factor}" filename="file://$(find perseus_description)/meshes/wheel.dae"/>
+      <cylinder radius="${wheel_radius/scale_factor}" length="${wheel_length/scale_factor}"/>
     </geometry>
   </collision>
@@ -22,7 +22,7 @@
 <link name="${prefix}front_right_wheel">
   <inertial>
-    <origin xyz="0.0 0.0 0.0" rpy="0.0 0.0 0.0"/>
-    <mass value="1.0"/>
-    <inertia ixx="0.04" iyy="0.02" izz="0.02" ixy="0.0" iyz="0.0" ixz="0.0"/>
+    <origin xyz="0.0 0.0  0.0" rpy="0.0 0.0 0.0"/>
+    <mass value="${wheel_mass}"/>
+    <xacro:cylinder_inertia m="${wheel_mass}" radius="${wheel_radius}" length="${wheel_length}"/>
   </inertial>
   <visual>
@@ -33,7 +33,7 @@
   </visual>
   <collision>
-    <origin xyz="0.0 0.0 0.0" rpy="0.0 0.0 0.0"/>
+    <origin xyz="0.0 0.0 0.0" rpy="${pi/2} 0.0 0.0"/>
     <geometry>
-      <mesh scale="${0.1/scale_factor} ${0.1/scale_factor}  ${0.1/scale_factor}" filename="file://$(find perseus_description)/meshes/wheel.dae"/>
+      <cylinder radius="${wheel_radius/scale_factor}" length="${wheel_length/scale_factor}"/>
     </geometry>
   </collision>
@@ -41,7 +41,7 @@
 <link name="${prefix}rear_left_wheel">
   <inertial>
-    <origin xyz="0.0 0.0 0.0" rpy="0.0 0.0 0.0"/>
-    <mass value="1.0"/>
-    <inertia ixx="0.04" iyy="0.02" izz="0.02" ixy="0.0" iyz="0.0" ixz="0.0"/>
+    <origin xyz="0.0 0.0  0.0" rpy="0.0 0.0 ${pi}"/>
+    <mass value="${wheel_mass}"/>
+    <xacro:cylinder_inertia m="${wheel_mass}" radius="${wheel_radius}" length="${wheel_length}"/>
   </inertial>
   <visual>
@@ -52,7 +52,7 @@
   </visual>
   <collision>
-    <origin xyz="0.0 0.0 0.0" rpy="0.0 0.0 ${pi}"/>
+    <origin xyz="0.0 0.0 0.0" rpy="${pi/2} 0.0 ${pi}"/>
     <geometry>
-      <mesh scale="${0.1/scale_factor} ${0.1/scale_factor}  ${0.1/scale_factor}" filename="file://$(find perseus_description)/meshes/wheel.dae"/>
+      <cylinder radius="${wheel_radius/scale_factor}" length="${wheel_length/scale_factor}"/>
     </geometry>
   </collision>
@@ -61,6 +61,6 @@
   <inertial>
     <origin xyz="0.0 0.0 0.0" rpy="0.0 0.0 0.0"/>
-    <mass value="1.0"/>
-    <inertia ixx="0.04" iyy="0.02" izz="0.02" ixy="0.0" iyz="0.0" ixz="0.0"/>
+    <mass value="${wheel_mass}"/>
+    <xacro:cylinder_inertia m="${wheel_mass}" radius="${wheel_radius}" length="${wheel_length}"/>
   </inertial>
   <visual>
@@ -71,7 +71,7 @@
   </visual>
   <collision>
-    <origin xyz="0.0 0.0 0.0" rpy="0.0 0.0 0.0"/>
+    <origin xyz="0.0 0.0 0.0" rpy="${pi/2} 0.0 0.0"/>
     <geometry>
-      <mesh scale="${0.1/scale_factor} ${0.1/scale_factor}  ${0.1/scale_factor}" filename="file://$(find perseus_description)/meshes/wheel.dae"/>
+      <cylinder radius="${wheel_radius/scale_factor}" length="${wheel_length/scale_factor}"/>
     </geometry>
   </collision>
