Commit message: refactor: Update URDF properties and fix inertial definitions for chassis and rocker components

File: software/ros_ws/src/perseus_description/urdf/chassis.urdf.xacro (robot description, xacro)
@@ -4,5 +4,5 @@
   <link name="${prefix}chassis">
     <inertial>
-      <origin xyz="0.0 -0.17100473204 0.14732485976" rpy="0 0 0"/>
+      <origin xyz="${-chassis_length/scale_factor*0.5} 0.0 ${chassis_height/scale_factor*0.5}" rpy="0 0.0 0.0"/>
       <mass value="${chassis_mass}"/>
       <xacro:box_inertia m="${chassis_mass}" x="${chassis_length/scale_factor}" y="${chassis_width/scale_factor}" z="${chassis_height/scale_factor}"/>

File: software/ros_ws/src/perseus_description/urdf/flange_bearing.urdf.xacro (robot description, xacro)
@@ -1,4 +1,7 @@
 <?xml version="1.0"?>
 <robot name="flange_bearing" xmlns:xacro="http://ros.org/wiki/xacro">
+<xacro:property name="bar_length" value="0.22"/>
+<xacro:property name="bar_width" value="0.03"/>
+<xacro:property name="bar_height" value="0.03"/>
 <!-- Flange Bearing -->
 <link name="${prefix}flange_bearing">
@@ -35,7 +38,7 @@
     </visual>
     <collision>
-    <origin xyz="0.0 0.0 -0.01" rpy="0.0 0.0 0.0"/>
+    <origin xyz="0.0 0.0 0.0" rpy="${-pi/2} 0 ${-pi/2}"/>
     <geometry>
-        <mesh scale="${0.1/scale_factor} ${0.1/scale_factor}  ${0.1/scale_factor}" filename="file://$(find perseus_description)/meshes/differential_bar.dae"/>
+        <box size="${bar_length/scale_factor} ${bar_width/scale_factor} ${bar_height/scale_factor}"/>
     </geometry>
     </collision>

File: software/ros_ws/src/perseus_description/urdf/perseus.urdf.xacro (robot description, xacro)
@@ -25,6 +25,6 @@
     <xacro:property name="wheels_y_offset" value="0.125"/>
     <xacro:property name="wheel_mass" value="1.0"/>
-    <xacro:property name="wheel_radius" value="0.13"/>
-    <xacro:property name="wheel_length" value="0.15"/>
+    <xacro:property name="wheel_radius" value="0.15"/>
+    <xacro:property name="wheel_length" value="0.14"/>
     <!-- ADD COMPONENTS -->
     <xacro:include filename="$(find perseus_description)/urdf/inertia_macros.xacro"/>

File: software/ros_ws/src/perseus_description/urdf/rocker.urdf.xacro (robot description, xacro)
@@ -1,31 +1,56 @@
 <?xml version="1.0"?>
 <robot name="rocker" xmlns:xacro="http://ros.org/wiki/xacro">
+  <!-- Rocker properties - Fix negative values -->
+  <xacro:property name="rocker_mass" value="0.5"/>
+  <xacro:property name="rocker_length" value="0.85"/>  <!-- Use positive absolute value -->
+  <xacro:property name="rocker_height" value="0.05"/>  <!-- Use positive value -->
+  <xacro:property name="rocker_width" value="0.03"/>
+  <xacro:property name="rocker_collision_x_offset" value="-0.10"/>
+  <xacro:property name="rocker_collision_z_offset" value="-0.2"/>
+  <!-- LEFT ROCKER LINK -->
   <link name="${prefix}left_rocker">
+    <inertial>
+      <origin xyz="${rocker_collision_x_offset/scale_factor} 0.0 ${rocker_collision_z_offset/scale_factor}" rpy="0.0 0.0 0.0"/>
+      <mass value="${rocker_mass}"/>
+      <xacro:box_inertia m="${rocker_mass}"
+                         x="${rocker_length}"
+                         y="${rocker_width}"
+                         z="${rocker_height}"/>
+    </inertial>
     <visual>
       <origin xyz="0.0 0.0 0.0" rpy="0.0 0.0 ${pi}"/>
       <geometry>
-        <mesh scale="${0.1/scale_factor} ${0.1/scale_factor}  ${0.1/scale_factor}" filename="file://$(find perseus_description)/meshes/rocker_left.dae"/>
+        <mesh scale="${0.1/scale_factor} ${0.1/scale_factor} ${0.1/scale_factor}"
+              filename="file://$(find perseus_description)/meshes/rocker_left.dae"/>
       </geometry>
     </visual>
     <collision>
-      <origin xyz="0.0 0.0 0.0" rpy="0.0 0.0 ${pi}"/>
+      <origin xyz="${rocker_collision_x_offset/scale_factor} 0.0 ${rocker_collision_z_offset/scale_factor}" rpy="0.0 0.0 0.0"/>
       <geometry>
-        <mesh scale="${0.1/scale_factor} ${0.1/scale_factor}  ${0.1/scale_factor}" filename="file://$(find perseus_description)/meshes/rocker_left.dae"/>
+        <box size="${rocker_length/scale_factor} ${rocker_width/scale_factor} ${rocker_height/scale_factor}"/>
       </geometry>
     </collision>
   </link>
+  <!-- RIGHT ROCKER LINK -->
   <link name="${prefix}right_rocker">
-    <!-- <inertial>
-    </inertial> -->
+    <inertial>
+      <origin xyz="${rocker_collision_x_offset/scale_factor} 0.0 ${rocker_collision_z_offset/scale_factor}" rpy="0.0 0.0 0.0"/>
+      <mass value="${rocker_mass}"/>
+      <xacro:box_inertia m="${rocker_mass}"
+                         x="${rocker_length}"
+                         y="${rocker_width}"
+                         z="${rocker_height}"/>
+    </inertial>
     <visual>
       <origin xyz="0.0 0.0 0.0" rpy="0.0 0.0 ${pi}"/>
       <geometry>
-        <mesh scale="${0.1/scale_factor} ${0.1/scale_factor}  ${0.1/scale_factor}" filename="file://$(find perseus_description)/meshes/rocker_right.dae"/>
+        <mesh scale="${0.1/scale_factor} ${0.1/scale_factor} ${0.1/scale_factor}"
+              filename="file://$(find perseus_description)/meshes/rocker_right.dae"/>
       </geometry>
     </visual>
     <collision>
-      <origin xyz="0.0 0.0 0.0" rpy="0.0 0.0 ${pi}"/>
+      <origin xyz="${rocker_collision_x_offset/scale_factor} 0.0 ${rocker_collision_z_offset/scale_factor}" rpy="0.0 0.0 0.0"/>
       <geometry>
-        <mesh scale="${0.1/scale_factor} ${0.1/scale_factor}  ${0.1/scale_factor}" filename="file://$(find perseus_description)/meshes/rocker_right.dae"/>
+        <box size="${rocker_length/scale_factor} ${rocker_width/scale_factor} ${rocker_height/scale_factor}"/>
       </geometry>
     </collision>

Commit message: Refactor chassis properties in URDF files to standardize mass definitions and improve clarity.

File: software/ros_ws/src/perseus_description/urdf/chassis.urdf.xacro (robot description, xacro)
@@ -1,5 +1,4 @@
 <?xml version="1.0"?>
 <robot name="chassis" xmlns:xacro="http://ros.org/wiki/xacro">
-  <xacro:property name="chassis_mass" value="2.7689940302592726"/>  <!-- Kg -->
   <link name="${prefix}chassis">
     <inertial>

File: software/ros_ws/src/perseus_description/urdf/perseus.urdf.xacro (robot description, xacro)
@@ -26,5 +26,5 @@
     <xacro:property name="wheel_length" value="0.14"/>
     <!-- Chassis Properties -->
-    <xacro:property name="base_mass" value="0.3" /> <!-- arbitrary value for base mass -->
+    <xacro:property name="chassis_mass" value="2.7689940302592726"/>  <!-- Kg -->
     <xacro:property name="chassis_width" value="0.45" />
     <xacro:property name="chassis_length" value="0.6" />

Commit message: feat: Update EKF configuration, adjust navigation parameters, and modify launch files for improved sensor integration

File: software/ros_ws/src/perseus_description/urdf/chassis.urdf.xacro (robot description, xacro)
@@ -21,14 +21,3 @@
     </collision>
   </link>
-  <gazebo reference="${prefix}chassis">
-      <material>Gazebo/Grey</material>
-      <sensor name="imu_sensor" type="imu">
-          <always_on>1</always_on>
-          <update_rate>10</update_rate>
-          <visualize>true</visualize>
-          <topic>imu</topic>
-          <!-- Add frame id to imu sensor (achieving correct frame association)-->
-          <gz_frame_id>${prefix}base_link</gz_frame_id>
-      </sensor>
-  </gazebo>
 </robot>
