Commit message: feat: Update camera_d455_gazebo URDF to use 'name' parameter and adjust sensor references

File: software/ros_ws/src/perseus_description/urdf/camera_d455_gazebo.xacro (robot description, xacro)
@@ -1,6 +1,6 @@
 <?xml version="1.0"?>
 <robot xmlns:xacro="http://ros.org/wiki/xacro">
-  <xacro:macro name="camera_d455_gazebo" params="prefix">
-    <gazebo reference="${prefix}camera_color_frame">
+  <xacro:macro name="camera_d455_gazebo" params="name:=camera">
+    <gazebo reference="${name}_color_frame">
       <material>Gazebo/Red</material>
       <sensor name="rgb_camera" type="camera">
@@ -21,34 +21,35 @@
           </clip>
         </camera>
-        <topic>/camera/camera/color/image_raw</topic>
-        <gz_frame_id>${prefix}camera_color_optical_frame</gz_frame_id>
+        <topic>/camera/camera/color/</topic>DingoOz2 hours ago
+        Gazebo's camera sensor type auto-appends /image and /camera_info to whatever you set in . Since the RGB topic is set to /camera/camera/color/image_raw, camera_info will actually publish at /camera/camera/color/image_raw/camera_info. gz_bridge.yaml:47 expects it at /camera/camera/color/camera_info. Same issue applies to all sensor entries in this file (depth, infra1, infra2). Consider setting topics to the base path (e.g. /camera/camera/color) and letting Gazebo append the suffixes, then update the bridge image mappings to match
+        <gz_frame_id>${name}_color_optical_frame</gz_frame_id>
       </sensor>
     </gazebo>
     <!-- Depth Camera -->
-    <gazebo reference="${prefix}camera_depth_frame">
+    <gazebo reference="${name}_depth_frame">
       <sensor name="rgbd_camera" type="rgbd_camera">
-          <pose>0 0 0 0 0 0</pose>
-          <visualize>false</visualize>
-          <update_rate>30</update_rate>
-          <always_on>true</always_on>
-          <camera>
-              <horizontal_fov>1.089</horizontal_fov>
-              <image>
-                  <width>640</width>
-                  <height>480</height>
-              </image>
-              <clip>
-                  <near>0.05</near>
-                  <far>10.0</far>
-              </clip>
-          </camera>
-          <topic>/camera/camera/depth</topic>
-          <gz_frame_id>${prefix}camera_depth_optical_frame</gz_frame_id>
-          <min_depth>0.05</min_depth>
-          <max_depth>10.0</max_depth>
+        <pose>0 0 0 0 0 0</pose>
+        <visualize>false</visualize>
+        <update_rate>30</update_rate>
+        <always_on>true</always_on>
+        <camera>
+          <horizontal_fov>1.089</horizontal_fov>
+          <image>
+            <width>640</width>
+            <height>480</height>
+          </image>
+          <clip>
+            <near>0.05</near>
+            <far>10.0</far>
+          </clip>
+        </camera>
+        <topic>/camera/camera/depth</topic>
+        <gz_frame_id>${name}_depth_optical_frame</gz_frame_id>
+        <min_depth>0.05</min_depth>
+        <max_depth>10.0</max_depth>
       </sensor>
     </gazebo>
     <!-- Left IR Camera -->
-    <gazebo reference="${prefix}camera_infra1_frame">
+    <gazebo reference="${name}_infra1_frame">
       <sensor name="ir_left_camera" type="camera">
         <pose>0 0 0 0 0 0</pose>
@@ -69,9 +70,9 @@
         </camera>
         <topic>/camera/camera/infra1/image_raw</topic>
-        <gz_frame_id>${prefix}camera_infra1_optical_frame</gz_frame_id>
+        <gz_frame_id>${name}_infra1_optical_frame</gz_frame_id>
       </sensor>
     </gazebo>
     <!-- Right IR Camera -->
-    <gazebo reference="${prefix}camera_infra2_frame">
+    <gazebo reference="${name}_infra2_frame">
       <sensor name="ir_right_camera" type="camera">
         <pose>0 0 0 0 0 0</pose>
@@ -92,5 +93,5 @@
         </camera>
         <topic>/camera/camera/infra2/image_raw</topic>
-        <gz_frame_id>${prefix}camera_infra2_optical_frame</gz_frame_id>
+        <gz_frame_id>${name}_infra2_optical_frame</gz_frame_id>
       </sensor>
     </gazebo>

File: software/ros_ws/src/perseus_description/urdf/perseus.urdf.xacro (robot description, xacro)
@@ -95,8 +95,8 @@
       <origin xyz="-0.15 0 0.25" rpy="0 0 0"/>
     </joint>
-  <xacro:sensor_d455 parent="${prefix}chassis" use_nominal_extrinsics="true">
-    <origin xyz="0.055 0.0 0.184" rpy="0 0 0"/>
-  </xacro:sensor_d455>
-  <xacro:camera_d455_gazebo prefix="${prefix}"/>
+    <xacro:sensor_d455 parent="${prefix}chassis" name="camera" use_nominal_extrinsics="true"></xacro:sensor_d455>
+      <origin xyz="0.055 0.0 0.184" rpy="0 0 0"/>
+    </xacro:sensor_d455>
+    <xacro:camera_d455_gazebo name="camera"/>
   </xacro:macro>
 </robot>

Commit message: feat: Update camera topics and frames in URDF and configuration files

File: software/ros_ws/src/perseus_description/urdf/camera_d455_gazebo.xacro (robot description, xacro)
@@ -21,6 +21,5 @@
           </clip>
         </camera>
-        <topic>/camera/camera/color/</topic>DingoOz2 hours ago
-        Gazebo's camera sensor type auto-appends /image and /camera_info to whatever you set in . Since the RGB topic is set to /camera/camera/color/image_raw, camera_info will actually publish at /camera/camera/color/image_raw/camera_info. gz_bridge.yaml:47 expects it at /camera/camera/color/camera_info. Same issue applies to all sensor entries in this file (depth, infra1, infra2). Consider setting topics to the base path (e.g. /camera/camera/color) and letting Gazebo append the suffixes, then update the bridge image mappings to match
+        <topic>/camera/camera/color/image_raw</topic>
         <gz_frame_id>${name}_color_optical_frame</gz_frame_id>
       </sensor>

File: software/ros_ws/src/perseus_description/urdf/perseus.urdf.xacro (robot description, xacro)
@@ -42,9 +42,4 @@
     <xacro:property name="bar_width" value="0.03"/>
     <xacro:property name="bar_height" value="0.03"/>
-    <!-- Depth Camera Properties -->
-    <xacro:property name="camera_mass" value="0.1"/>
-    <xacro:property name="camera_width" value="0.12"/>
-    <xacro:property name="camera_height" value="0.03"/>
-    <xacro:property name="camera_depth" value="0.025"/>
     <!-- 2D and 3D LIDAR Properties -->
     <xacro:property name="laser_2d_mass" value="0.1"/>
@@ -95,5 +90,5 @@
       <origin xyz="-0.15 0 0.25" rpy="0 0 0"/>
     </joint>
-    <xacro:sensor_d455 parent="${prefix}chassis" name="camera" use_nominal_extrinsics="true"></xacro:sensor_d455>
+    <xacro:sensor_d455 parent="${prefix}chassis" name="camera" use_nominal_extrinsics="true">
       <origin xyz="0.055 0.0 0.184" rpy="0 0 0"/>
     </xacro:sensor_d455>

File: software/ros_ws/src/perseus_description/urdf/sensors.urdf.xacro (robot description, xacro)
@@ -122,5 +122,5 @@
         <update_rate>10</update_rate>
         <visualize>true</visualize>
-        <topic>scan_3d/imu</topic>
+        <topic>/scan_3d/imu</topic>
         <!-- Add frame id to imu sensor (achieving correct frame association)-->
         <gz_frame_id>${prefix}livox_frame</gz_frame_id>

Commit message: feat: Update RealSense URDF and configuration for improved topic naming and sensor types

File: software/ros_ws/src/perseus_description/urdf/camera_d455_gazebo.xacro (robot description, xacro)
@@ -3,6 +3,5 @@
   <xacro:macro name="camera_d455_gazebo" params="name:=camera">
     <gazebo reference="${name}_color_frame">
-      <material>Gazebo/Red</material>
-      <sensor name="rgb_camera" type="camera">
+      <sensor name="rgbd_camera" type="rgbd_camera">
         <pose>0 0 0 0 0 0</pose>
         <visualize>true</visualize>
@@ -14,12 +13,11 @@
             <width>640</width>
             <height>480</height>
-            <format>R8G8B8</format>
           </image>
           <clip>
             <near>0.05</near>
-            <far>100</far>
+            <far>10.0</far>
           </clip>
         </camera>
-        <topic>/${name}/${name}/color/image_raw</topic>
+        <topic>/${name}/${name}/color</topic>
         <gz_frame_id>${name}_color_optical_frame</gz_frame_id>
       </sensor>
@@ -27,5 +25,5 @@
     <!-- Depth Camera -->
     <gazebo reference="${name}_depth_frame">
-      <sensor name="rgbd_camera" type="rgbd_camera">
+      <sensor name="depth_camera" type="depth_camera">
         <pose>0 0 0 0 0 0</pose>
         <visualize>false</visualize>
@@ -45,6 +43,4 @@
         <topic>/${name}/${name}/depth</topic>
         <gz_frame_id>${name}_depth_optical_frame</gz_frame_id>
-        <min_depth>0.05</min_depth>
-        <max_depth>10.0</max_depth>
       </sensor>
     </gazebo>
