Commit message: autonomy: update the description with base_footprint

File: software/ros_ws/src/perseus_description/urdf/perseus.urdf.xacro (robot description, xacro)
@@ -7,4 +7,12 @@
     <!-- <xacro:include filename="$(find perseus_description)/urdf/sensors.urdf.xacro"/> -->
     <link name="${prefix}base_link"/>
+    <!--BASE_FOOTPRINT_LINK-->
+    <joint name="base_footprint_joint" type="fixed">
+      <parent link="base_link"/>
+      <child link="base_footprint"/>
+      <origin xyz="0 0 0" rpy="0 0 0"/>
+    </joint>
+    <link name="base_footprint">
+    </link>
     <!-- CHASSIS -->
     <xacro:chassis />

Commit message: autonomy: update the description with base_footprint

File: software/ros_ws/src/perseus_description/urdf/perseus.urdf.xacro (robot description, xacro)
@@ -7,4 +7,12 @@
     <xacro:include filename="$(find perseus_description)/urdf/sensors.urdf.xacro"/>
     <link name="${prefix}base_link"/>
+    <!--BASE_FOOTPRINT_LINK-->
+    <joint name="base_footprint_joint" type="fixed">
+      <parent link="base_link"/>
+      <child link="base_footprint"/>
+      <origin xyz="0 0 0" rpy="0 0 0"/>
+    </joint>
+    <link name="base_footprint">
+    </link>
     <!-- CHASSIS -->
     <xacro:chassis />

Commit message: autonomy: reverted tf tree to base_link from base_footprint

File: software/ros_ws/src/perseus_description/urdf/perseus.urdf.xacro (robot description, xacro)
@@ -7,12 +7,4 @@
     <!-- <xacro:include filename="$(find perseus_description)/urdf/sensors.urdf.xacro"/> -->
     <link name="${prefix}base_link"/>
-    <!--BASE_FOOTPRINT_LINK-->
-    <joint name="base_footprint_joint" type="fixed">
-      <parent link="base_link"/>
-      <child link="base_footprint"/>
-      <origin xyz="0 0 0" rpy="0 0 0"/>
-    </joint>
-    <link name="base_footprint">
-    </link>
     <!-- CHASSIS -->
     <xacro:chassis />

Commit message: autonomy: reverted tf tree to base_link from base_footprint

File: software/ros_ws/src/perseus_description/urdf/perseus.urdf.xacro (robot description, xacro)
@@ -7,12 +7,4 @@
     <xacro:include filename="$(find perseus_description)/urdf/sensors.urdf.xacro"/>
     <link name="${prefix}base_link"/>
-    <!--BASE_FOOTPRINT_LINK-->
-    <joint name="base_footprint_joint" type="fixed">
-      <parent link="base_link"/>
-      <child link="base_footprint"/>
-      <origin xyz="0 0 0" rpy="0 0 0"/>
-    </joint>
-    <link name="base_footprint">
-    </link>
     <!-- CHASSIS -->
     <xacro:chassis />

Commit message: perseus_lite: correct many more references Perseus vs Perseus_lite
Perseus_Lite was created by copying Perseus. Multiple references needed
to be fixed.

File: software/ros_ws/src/perseus_description/urdf/perseus.urdf.xacro (robot description, xacro)
@@ -1,5 +1,5 @@
 <?xml version="1.0"?>
 <robot xmlns:xacro="http://ros.org/wiki/xacro">
-  <xacro:macro name="perseus" params="prefix">
+  <xacro:macro name="perseus_lite" params="prefix">
     <!-- Import components -->
     <xacro:include filename="$(find perseus_description)/urdf/chassis.urdf.xacro"/>

File: software/ros_ws/src/perseus_lite/description/urdf/perseus_lite.urdf.xacro (robot description, xacro)
@@ -1,22 +1,20 @@
 <?xml version="1.0"?>
-<robot xmlns:xacro="http://www.ros.org/wiki/xacro" name="perseus">
+<robot xmlns:xacro="http://www.ros.org/wiki/xacro" name="perseus_lite">
   <xacro:arg name="prefix" default="" />
-  <xacro:arg name="can_bus" default="can0" />
   <xacro:arg name="use_mock_hardware" default="false" />
-  <xacro:arg name="use_legacy_hardware" default="true" />
-  <xacro:property name="use_legacy_hardware" value="$(arg use_legacy_hardware)" />
+  <xacro:arg name="serial_port" default="/dev/ttyUSB0" />
   <xacro:property name="real_hardware_plugin"
-    value="${'perseus_hardware/McbSystemHardware' if use_legacy_hardware else 'perseus_hardware/VescSystemHardware'}" />
+  value="perseus_lite_hardware/ST3215SystemHardware" />
   <xacro:property name="use_mock_hardware" value="$(arg use_mock_hardware)" />
   <xacro:property name="hardware_plugin"
     value="${'mock_components/GenericSystem' if use_mock_hardware else real_hardware_plugin}" />
   <!-- Import URDF description -->
-  <xacro:include filename="$(find perseus_description)/urdf/perseus.urdf.xacro" />
+  <xacro:include filename="$(find perseus_lite_description)/urdf/perseus_lite.urdf.xacro" />
   <!-- Import colours for rviz -->
-  <xacro:include filename="$(find perseus_description)/urdf/perseus.materials.xacro" />
+  <xacro:include filename="$(find perseus_lite_description)/urdf/perseus_lite.materials.xacro" />
   <!-- Import ros2_control description -->
-  <xacro:include filename="$(find perseus_description)/ros2_control/perseus.ros2_control.xacro" />
+  <xacro:include filename="$(find perseus_lite_description)/ros2_control/perseus_lite.ros2_control.xacro" />
   <!-- Instantiate the description and the ROS2 control information -->
-  <xacro:perseus prefix="$(arg prefix)" />
-  <xacro:perseus_ros2_control name="Perseus" prefix="$(arg prefix)" can_bus="$(arg can_bus)" hardware_plugin="${hardware_plugin}"/>
+  <xacro:perseus_lite prefix="$(arg prefix)" />
+  <xacro:perseus_lite_ros2_control name="PerseusLite" prefix="$(arg prefix)" hardware_plugin="${hardware_plugin}" serial_port="$(arg serial_port)"/>
 </robot>

File: software/ros_ws/src/perseus_lite_description/ros2_control/perseus_lite.ros2_control.xacro (robot description, xacro)
@@ -1,10 +1,9 @@
 <?xml version="1.0"?>
 <robot xmlns:xacro="http://www.ros.org/wiki/xacro">
-  <xacro:macro name="perseus_lite_ros2_control" params="name prefix hardware_plugin">
+  <xacro:macro name="perseus_lite_ros2_control" params="name prefix hardware_plugin serial_port">
     <ros2_control name="${name}" type="system">
       <hardware>
         <plugin>${hardware_plugin}</plugin>
-        <!-- Add parameters for ST3215 servo serial connection -->
-        <param name="serial_port">/dev/ttyUSB0</param>
+        <param name="serial_port">${serial_port}</param>
         <param name="baud_rate">115200</param>
       </hardware>
@@ -12,15 +11,13 @@
         <joint name="${prefix}${name}_wheel_joint">
           <param name="id">${id}</param>
-          <!-- ST3215 servo interfaces -->
           <command_interface name="position"/>
           <command_interface name="velocity"/>
           <state_interface name="position"/>
           <state_interface name="velocity"/>
-          <state_interface name="load"/> <!-- ST3215's integrated load sensing -->
-          <!-- ST3215 specific parameters -->
-          <param name="encoder_resolution">4096</param> <!-- 12-bit encoder -->
-          <param name="max_velocity">30.0</param>  <!-- rad/s -->
-          <param name="min_position">-180.0</param>  <!-- degrees -->
-          <param name="max_position">180.0</param>   <!-- degrees -->
+          <state_interface name="load"/>
+          <param name="encoder_resolution">4096</param>
+          <param name="max_velocity">30.0</param>
+          <param name="min_position">-180.0</param>
+          <param name="max_position">180.0</param>
         </joint>
       </xacro:macro>

File: software/ros_ws/src/perseus_lite_description/urdf/perseus_lite.urdf.xacro (robot description, xacro)
@@ -1,12 +1,14 @@
 <?xml version="1.0"?>
 <robot xmlns:xacro="http://ros.org/wiki/xacro">
+  <xacro:arg name="hardware_plugin" default="perseus_lite_hardware/ST3215SystemHardware"/>
+  <xacro:arg name="hardware_type" default="st3215"/>
+  <xacro:arg name="use_mock_hardware" default="false"/>
+  <xacro:arg name="serial_port" default="/dev/ttyUSB0"/>
+  <xacro:include filename="$(find perseus_lite_description)/ros2_control/perseus_lite.ros2_control.xacro" />
   <xacro:macro name="perseus_lite" params="prefix">
-    <!-- Import components -->
     <xacro:include filename="$(find perseus_lite_description)/urdf/chassis.urdf.xacro"/>
     <xacro:include filename="$(find perseus_lite_description)/urdf/rocker.urdf.xacro"/>
-    <!-- Scale factor for Perseus Lite -->
     <xacro:property name="scale" value="0.5"/>
     <link name="${prefix}base_link"/>
-    <!--BASE_FOOTPRINT_LINK-->
     <joint name="base_footprint_joint" type="fixed">
       <parent link="base_link"/>
@@ -16,5 +18,4 @@
     <link name="base_footprint">
     </link>
-    <!-- CHASSIS -->
     <xacro:chassis />
     <joint name="chassis_joint" type="fixed">
@@ -23,13 +24,15 @@
       <child link="${prefix}chassis"/>
     </joint>
-    <!-- ROCKER ARMS -->
-    <!-- LEFT -->
     <xacro:rocker side="left">
       <origin xyz="${-0.275 * scale} ${-0.075 * scale} ${0.05 * scale}" rpy="0.0 0.0 ${-pi/2}"/>
     </xacro:rocker>
-    <!-- RIGHT -->
     <xacro:rocker side="right">
       <origin xyz="${0.275 * scale} ${-0.075 * scale} ${0.05 * scale}" rpy="0.0 0.0 ${-pi/2}"/>
     </xacro:rocker>
+    <xacro:perseus_lite_ros2_control
+      name="PerseusLite"
+      prefix="${prefix}"
+      hardware_plugin="$(arg hardware_plugin)"
+      serial_port="$(arg serial_port)"/>
   </xacro:macro>
 </robot>

Commit message: perseus_lite: Corrected to use diff_drive_base_controller

File: software/ros_ws/src/perseus_description/urdf/perseus.urdf.xacro (robot description, xacro)
@@ -1,5 +1,5 @@
 <?xml version="1.0"?>
 <robot xmlns:xacro="http://ros.org/wiki/xacro">
-  <xacro:macro name="perseus_lite" params="prefix">
+  <xacro:macro name="perseus" params="prefix">
     <!-- Import components -->
     <xacro:include filename="$(find perseus_description)/urdf/chassis.urdf.xacro"/>

File: software/ros_ws/src/perseus_lite_description/ros2_control/perseus_lite.ros2_control.xacro (robot description, xacro)
@@ -8,23 +8,32 @@
         <param name="baud_rate">115200</param>
       </hardware>
-      <xacro:macro name="ros2_control_joint" params="name id">
-        <joint name="${prefix}${name}_wheel_joint">
-          <param name="id">${id}</param>
-          <command_interface name="position"/>
-          <command_interface name="velocity"/>
-          <state_interface name="position"/>
-          <state_interface name="velocity"/>
-          <state_interface name="load"/>
-          <param name="encoder_resolution">4096</param>
-          <param name="max_velocity">30.0</param>
-          <param name="min_position">-180.0</param>
-          <param name="max_position">180.0</param>
-        </joint>
-      </xacro:macro>
-      <!-- Define the four wheel joints -->
-      <xacro:ros2_control_joint name="front_left" id="1"/>
-      <xacro:ros2_control_joint name="front_right" id="2"/>
-      <xacro:ros2_control_joint name="rear_left" id="3"/>
-      <xacro:ros2_control_joint name="rear_right" id="4"/>
+      <joint name="${prefix}front_left_wheel_joint">
+        <command_interface name="velocity"/>
+        <state_interface name="position"/>
+        <state_interface name="velocity"/>
+        <state_interface name="temperature"/>
+        <param name="id">1</param>
+      </joint>
+      <joint name="${prefix}front_right_wheel_joint">
+        <command_interface name="velocity"/>
+        <state_interface name="position"/>
+        <state_interface name="velocity"/>
+        <state_interface name="temperature"/>
+        <param name="id">2</param>
+      </joint>
+      <joint name="${prefix}rear_left_wheel_joint">
+        <command_interface name="velocity"/>
+        <state_interface name="position"/>
+        <state_interface name="velocity"/>
+        <state_interface name="temperature"/>
+        <param name="id">3</param>
+      </joint>
+      <joint name="${prefix}rear_right_wheel_joint">
+        <command_interface name="velocity"/>
+        <state_interface name="position"/>
+        <state_interface name="velocity"/>
+        <state_interface name="temperature"/>
+        <param name="id">4</param>
+      </joint>
     </ros2_control>
   </xacro:macro>

File: software/ros_ws/src/perseus_lite_description/urdf/perseus_lite.urdf.xacro (robot description, xacro)
@@ -1,13 +1,24 @@
 <?xml version="1.0"?>
-<robot xmlns:xacro="http://ros.org/wiki/xacro">
-  <xacro:arg name="hardware_plugin" default="perseus_lite_hardware/ST3215SystemHardware"/>
+<robot xmlns:xacro="http://www.ros.org/wiki/xacro" name="perseus_lite">
+  <!-- Default arguments -->
+  <xacro:arg name="prefix" default="" />
+  <xacro:arg name="use_mock_hardware" default="false" />
+  <xacro:arg name="serial_port" default="/dev/ttyACM0" />
   <xacro:arg name="hardware_type" default="st3215"/>
-  <xacro:arg name="use_mock_hardware" default="false"/>
-  <xacro:arg name="serial_port" default="/dev/ttyUSB0"/>
+  <!-- Hardware plugin selection -->
+  <xacro:property name="real_hardware_plugin" value="perseus_lite_hardware/ST3215SystemHardware" />
+  <xacro:property name="use_mock_hardware" value="$(arg use_mock_hardware)" />
+  <xacro:property name="hardware_plugin"
+    value="${'mock_components/GenericSystem' if use_mock_hardware else real_hardware_plugin}" />
+  <!-- Import dependencies -->
+  <!-- <xacro:include filename="$(find perseus_lite_description)/urdf/perseus_lite.urdf.xacro" /> -->
+  <xacro:include filename="$(find perseus_lite_description)/urdf/chassis.urdf.xacro"/>
+  <xacro:include filename="$(find perseus_lite_description)/urdf/rocker.urdf.xacro"/>
+  <xacro:include filename="$(find perseus_lite_description)/urdf/perseus_lite.materials.xacro" />
   <xacro:include filename="$(find perseus_lite_description)/ros2_control/perseus_lite.ros2_control.xacro" />
+  <!-- Scale for Perseus Lite - DO I NEED THIS?-->
+  <xacro:property name="scale" value="0.5"/>
+  <!-- Main macro definition -->
   <xacro:macro name="perseus_lite" params="prefix">
-    <xacro:include filename="$(find perseus_lite_description)/urdf/chassis.urdf.xacro"/>
-    <xacro:include filename="$(find perseus_lite_description)/urdf/rocker.urdf.xacro"/>
-    <xacro:property name="scale" value="0.5"/>
     <link name="${prefix}base_link"/>
     <joint name="base_footprint_joint" type="fixed">
@@ -30,9 +41,12 @@
       <origin xyz="${0.275 * scale} ${-0.075 * scale} ${0.05 * scale}" rpy="0.0 0.0 ${-pi/2}"/>
     </xacro:rocker>
+    <!-- ROS2 Control -->
     <xacro:perseus_lite_ros2_control
-      name="PerseusLite"
+      name="Perseus_Lite"
       prefix="${prefix}"
-      hardware_plugin="$(arg hardware_plugin)"
+      hardware_plugin="${hardware_plugin}"
       serial_port="$(arg serial_port)"/>
   </xacro:macro>
+  <!-- Instantiate the description -->
+  <xacro:perseus_lite prefix="$(arg prefix)" />
 </robot>

Commit message: Online Aysnc Finally Working!!!

File: software/ros_ws/src/perseus_description/urdf/perseus.urdf.xacro (robot description, xacro)
@@ -7,4 +7,10 @@
     <xacro:include filename="$(find perseus_description)/urdf/sensors.urdf.xacro"/>
     <link name="${prefix}base_link"/>
+    <joint name="base_footprint_joint" type="fixed">
+        <parent link="base_link"/>
+        <child link="base_footprint"/>
+        <origin xyz="0 0 0" rpy="0 0 0"/>
+    </joint>
+    <link name="${prefix}base_footprint"/>
     <!-- CHASSIS -->
     <xacro:chassis />

Commit message: autonomy: launch files and mapping changes (at comp):

File: software/ros_ws/src/perseus_description/urdf/perseus.urdf.xacro (robot description, xacro)
@@ -7,4 +7,10 @@
     <xacro:include filename="$(find perseus_description)/urdf/sensors.urdf.xacro"/>
     <link name="${prefix}base_link"/>
+    <joint name="base_footprint_joint" type="fixed">
+        <parent link="base_link"/>
+        <child link="base_footprint"/>
+        <origin xyz="0 0 0" rpy="0 0 0"/>
+    </joint>
+    <link name="${prefix}base_footprint"/>
     <!-- CHASSIS -->
     <xacro:chassis />

File: software/ros_ws/src/perseus_description/urdf/sensors.urdf.xacro (robot description, xacro)
@@ -47,5 +47,5 @@
         <parent link="${prefix}base_link"/>
         <child link="${prefix}m2m2_lidar_frame"/>
-        <origin xyz="0.2 0.4 0.35" rpy="0 0 -1.57"/>
+        <origin xyz="0.2 0.4 0.35" rpy="0 0 0"/>
     </joint>
     <gazebo reference="${prefix}m2m2_lidar_frame">

Commit message: fix(urdf): correct chassis joint orientation to zero rotation

File: software/ros_ws/src/perseus_description/urdf/perseus.urdf.xacro (robot description, xacro)
@@ -16,5 +16,5 @@
     <xacro:chassis />
     <joint name="${prefix}chassis_joint" type="fixed">
-      <origin xyz="0.21 0.0 0.35" rpy="0.0 0.0 -${pi/2}"/>
+      <origin xyz="0.21 0.0 0.35" rpy="0.0 0.0 0.0"/>
       <parent link="${prefix}base_link"/>
       <child link="${prefix}chassis"/>

Commit message: feat: Add laser sensor integration and update related configurations

File: software/ros_ws/src/perseus_description/urdf/perseus.urdf.xacro (robot description, xacro)
@@ -25,4 +25,5 @@
     <xacro:include filename="$(find perseus_description)/urdf/motor_wheel.urdf.xacro"/>
     <xacro:include filename="$(find perseus_description)/urdf/wheel.urdf.xacro"/>
+    <xacro:include filename="$(find perseus_description)/urdf/sensors.urdf.xacro"/>
     <!-- An empty base_link to attach everything to -->
     <link name="${prefix}base_link"/>
@@ -95,4 +96,9 @@
       <dynamics damping="0.2" friction="0.3"/>
     </joint>
+    <joint name="${prefix}laser_joint" type="fixed">
+      <parent link="${prefix}chassis"/>
+      <child link="${prefix}laser_frame"/>
+      <origin xyz="0 0 0.23" rpy="0 0 0"/>
+    </joint>
   </xacro:macro>
 </robot>

Commit message: fix: Adjust laser joint origin and refine lidar sensor parameters

File: software/ros_ws/src/perseus_description/urdf/perseus.urdf.xacro (robot description, xacro)
@@ -99,5 +99,5 @@
       <parent link="${prefix}chassis"/>
       <child link="${prefix}laser_frame"/>
-      <origin xyz="0 0 0.23" rpy="0 0 0"/>
+      <origin xyz="0 0 -0.04" rpy="0 ${PI} 0"/>
     </joint>
   </xacro:macro>

File: software/ros_ws/src/perseus_description/urdf/sensors.urdf.xacro (robot description, xacro)
@@ -16,10 +16,10 @@
 </link>
 <gazebo reference="${prefix}laser_frame">
-    <material>
+  <material>
     <ambient>0.1 0.1 0.1 1</ambient>
     <diffuse>0.1 0.1 0.1 1</diffuse>
     <specular>0.1 0.1 0.1 1</specular>
-    </material>
-    <sensor name="${prefix}lidar_sensor" type="gpu_lidar">
+  </material>
+  <sensor name="${prefix}lidar_sensor" type="gpu_lidar">
     <topic>scan</topic>
     <update_rate>10</update_rate>
@@ -27,32 +27,25 @@
     <visualize>false</visualize>
     <ray>
-        <scan>
+      <scan>
         <horizontal>
-            <samples>720</samples>
-            <resolution>1</resolution>
-            <min_angle>-3.14159</min_angle>
-            <max_angle>3.14159</max_angle>
+          <samples>720</samples>
+          <resolution>1</resolution>
+          <min_angle>-3.14159</min_angle>
+          <max_angle>3.14159</max_angle>
         </horizontal>
-        <!-- <vertical>
-            <samples>1</samples>
-            <resolution>1</resolution>
-            <min_angle>0</min_angle>
-            <max_angle>0</max_angle>
-        </vertical> -->
         <vertical>
-            <samples>32</samples>
-            <!-- <resolution>1</resolution> -->
-            <min_angle>-0.5353</min_angle>
-            <max_angle>0.1862</max_angle>
+          <samples>32</samples>
+          <min_angle>-0.1222</min_angle>     <!-- –7° in radians -->
+          <max_angle>0.9076</max_angle>      <!-- +52° in radians -->
         </vertical>
-        </scan>
-        <range>
+      </scan>
+      <range>
         <min>0.20</min>
         <max>30.0</max>
         <resolution>0.013</resolution>
-        </range>
+      </range>
     </ray>
     <gz_frame_id>laser_frame</gz_frame_id>
-    </sensor>
+  </sensor>
 </gazebo>
 </robot>

Commit message: feat: update laser joint origin and visualization parameters for improved alignment and clarity

File: software/ros_ws/src/perseus_description/urdf/perseus.urdf.xacro (robot description, xacro)
@@ -99,5 +99,5 @@
       <parent link="${prefix}chassis"/>
       <child link="${prefix}laser_frame"/>
-      <origin xyz="0 0 0.23" rpy="0 0.785 0"/>
+      <origin xyz="0 0 -0.035" rpy="0 ${PI} 0"/>
     </joint>
   </xacro:macro>

Commit message: feat: integrate 2D LIDAR support and update configurations in simulation

File: software/ros_ws/src/perseus_description/urdf/perseus.urdf.xacro (robot description, xacro)
@@ -103,8 +103,13 @@
       <origin xyz="0 0 -0.035" rpy="0 ${PI} 0"/>
     </joint>
+    <joint name="${prefix}laser_2d_joint" type="fixed">
+      <parent link="${prefix}chassis"/>
+      <child link="${prefix}laser_2d_frame"/>
+      <origin xyz="-0.15 0 0.25" rpy="0 0 0"/>
+    </joint>
     <joint name="${prefix}camera_joint" type="fixed">
         <parent link="${prefix}chassis"/>
         <child link="${prefix}camera_link"/>
-        <origin xyz="0.01 0 0.2" rpy="0 0 0"/>
+        <origin xyz="0.01 0 0.18" rpy="0 0 0"/>
     </joint>
   </xacro:macro>

File: software/ros_ws/src/perseus_description/urdf/sensors.urdf.xacro (robot description, xacro)
@@ -1,4 +1,5 @@
 <?xml version="1.0"?>
 <robot name="lidar" xmlns:xacro="http://ros.org/wiki/xacro">
+<!-- 3D LIDAR (Existing - Livox MID-360) -->
 <link name="${prefix}laser_frame">
     <visual>
@@ -15,4 +16,21 @@
     </collision>
 </link>
+<!-- 2D LIDAR -->
+<link name="${prefix}laser_2d_frame">
+    <visual>
+        <origin xyz="0 0 0"/>
+        <geometry>
+            <cylinder radius="0.04" length="0.04"/>
+        </geometry>
+        <material name="blue">
+            <color rgba="0.0 0.0 1.0 1.0"/>
+        </material>
+    </visual>
+    <collision>
+        <geometry>
+            <cylinder radius="0.04" length="0.04"/>
+        </geometry>
+    </collision>
+</link>
 <!-- Simulating the Livox MID-360 -->
 <gazebo reference="${prefix}laser_frame">
@@ -25,5 +43,5 @@
     <topic>scan</topic>
     <update_rate>50</update_rate>
-    <always_on>true</always_on>
+    <always_on>false</always_on>
     <visualize>false</visualize>
     <ray>
@@ -51,3 +69,39 @@
   </sensor>
 </gazebo>
+<!-- 2D LIDAR SENSOR (Traditional 2D Laser Scanner) -->
+<gazebo reference="${prefix}laser_2d_frame">
+  <material>
+    <ambient>0.0 0.0 1.0 1</ambient>
+    <diffuse>0.0 0.0 1.0 1</diffuse>
+    <specular>0.0 0.0 1.0 1</specular>
+  </material>
+  <sensor name="${prefix}laser_2d_sensor" type="gpu_lidar">
+    <topic>scan_2d</topic>
+    <update_rate>50</update_rate>
+    <always_on>true</always_on>
+    <visualize>false</visualize>
+    <ray>
+      <scan>
+        <horizontal>
+          <samples>720</samples>
+          <resolution>1</resolution>
+          <min_angle>-3.14159</min_angle>
+          <max_angle>3.14159</max_angle>
+        </horizontal>
+        <!-- Single horizontal plane for 2D scanning -->
+        <vertical>
+          <samples>1</samples>
+          <min_angle>0.0</min_angle>
+          <max_angle>0.0</max_angle>
+        </vertical>
+      </scan>
+      <range>
+        <min>0.10</min>
+        <max>25.0</max>
+        <resolution>0.01</resolution>
+      </range>
+    </ray>
+    <gz_frame_id>laser_2d_frame</gz_frame_id>
+  </sensor>
+</gazebo>
 </robot>
