Commit message: Reorder base_link and base_footprint definitions for improved structure and clarity in URDF file

File: software/ros_ws/src/perseus_description/urdf/perseus.urdf.xacro (robot description, xacro)
@@ -65,14 +65,14 @@
     <!-- An empty base_link to attach everything to -->
     <link name="${prefix}base_link"/>
-    <joint name="base_footprint_joint" type="fixed">
-        <parent link="base_link"/>
-        <child link="base_footprint"/>
-        <origin xyz="0 0 0" rpy="0 0 0"/>
-    </joint>
-    <link name="${prefix}base_footprint"/>
     <joint name="${prefix}chassis_joint" type="fixed"> <!-- Joint Connect base_link and chassis -->
       <origin xyz="0 0.0 ${chassis_z_offset}" rpy="0.0 0.0 0.0"/>
       <parent link="${prefix}base_link"/>
       <child link="${prefix}chassis"/>
+    </joint>
+    <link name="${prefix}base_footprint"/>
+    <joint name="base_footprint_joint" type="fixed">
+        <parent link="${prefix}chassis"/>
+        <child link="${prefix}base_footprint"/>
+        <origin xyz="0 0 0" rpy="0 0 0"/>
     </joint>
     <!-- ADD 2 ROCKERS (INCLUDING 4 MOTORS + 4 WHEELS) -->

Commit message: undo base_footprint changes

File: software/ros_ws/src/perseus_description/urdf/perseus.urdf.xacro (robot description, xacro)
@@ -72,5 +72,5 @@
     <link name="${prefix}base_footprint"/>
     <joint name="base_footprint_joint" type="fixed">
-        <parent link="${prefix}chassis"/>
+        <parent link="${prefix}base_link"/>
         <child link="${prefix}base_footprint"/>
         <origin xyz="0 0 0" rpy="0 0 0"/>

Commit message: feat: update navigation parameters for improved robot control and adjust URDF joint origin

File: software/ros_ws/src/perseus_description/urdf/perseus.urdf.xacro (robot description, xacro)
@@ -66,5 +66,5 @@
     <link name="${prefix}base_link"/>
     <joint name="${prefix}chassis_joint" type="fixed"> <!-- Joint Connect base_link and chassis -->
-      <origin xyz="0 0.0 ${chassis_z_offset}" rpy="0.0 0.0 0.0"/>
+      <origin xyz="${chassis_length} 0.0 ${chassis_z_offset}" rpy="0.0 0.0 0.0"/>
       <parent link="${prefix}base_link"/>
       <child link="${prefix}chassis"/>

Commit message: feat: Adjust laser and camera joint positions in URDF file

File: software/ros_ws/src/perseus_description/urdf/perseus.urdf.xacro (robot description, xacro)
@@ -87,5 +87,5 @@
       <parent link="${prefix}chassis"/>
       <child link="${prefix}livox_frame"/>
-      <origin xyz="-0.27 -0.04 -0.04" rpy="0 ${pi} ${pi}"/>
+      <origin xyz="-0.193 -0.047 -0.03375" rpy="0 ${pi} ${pi}"/>
     </joint>
     <joint name="${prefix}laser_2d_joint" type="fixed">
@@ -97,5 +97,5 @@
         <parent link="${prefix}chassis"/>
         <child link="${prefix}camera_link"/>
-        <origin xyz="0.145 0 0.34" rpy="0 0.174533 0"/>
+        <origin xyz="0.055 0 0.184" rpy="0 0.174533 0"/>
     </joint>
   </xacro:macro>

Commit message: feat: Update joint origin and rotation for laser and lidar sensors

File: software/ros_ws/src/perseus_description/urdf/perseus.urdf.xacro (robot description, xacro)
@@ -87,5 +87,5 @@
       <parent link="${prefix}chassis"/>
       <child link="${prefix}livox_frame"/>
-      <origin xyz="-0.173 -0.047 -0.03375" rpy="0 ${pi} ${pi}"/>
+      <origin xyz="-0.173 0.047 -0.04375" rpy="0 ${pi} ${pi/2}"/>
     </joint>
     <joint name="${prefix}laser_2d_joint" type="fixed">

File: software/ros_ws/src/perseus_description/urdf/sensors.urdf.xacro (robot description, xacro)
@@ -9,5 +9,5 @@
     </inertial>
     <visual>
-        <origin xyz="0 0.0 -0.02" rpy="${pi/2} 0.0 0.0"/>
+        <origin xyz="0 0.0 -0.02" rpy="${pi/2} 0.0 ${pi}"/>
         <geometry>
             <mesh scale="1.0 1.0  1.0" filename="file://$(find perseus_description)/meshes/mid-360.dae"/>

Commit message: feat: Update camera joint rotation in URDF file

File: software/ros_ws/src/perseus_description/urdf/perseus.urdf.xacro (robot description, xacro)
@@ -97,5 +97,5 @@
         <parent link="${prefix}chassis"/>
         <child link="${prefix}camera_link"/>
-        <origin xyz="0.055 0 0.184" rpy="0 0.174533 0"/>
+        <origin xyz="0.055 0 0.184" rpy="0 0.0 0"/>
     </joint>
   </xacro:macro>

Commit message: refactor: remove pointcloud to laserscan converter node from launch file

File: software/ros_ws/src/perseus_description/urdf/perseus.urdf.xacro (robot description, xacro)
@@ -91,5 +91,5 @@
     </joint>
     <xacro:sensor_d455 parent="${prefix}chassis" name="camera" use_nominal_extrinsics="true">
-      <origin xyz="0.055 0.0 0.184" rpy="0 0 0"/>
+      <origin xyz="0.055 0.0 0.184" rpy="0 ${pi/18} 0"/>
     </xacro:sensor_d455>
     <xacro:camera_d455_gazebo name="camera"/>
