Commit message: feat: update camera depth integration and adjust joint parameters for improved alignment

File: software/ros_ws/src/perseus/urdf/perseus.urdf.xacro (robot description, xacro)
@@ -10,8 +10,6 @@
   <!-- Import ros2_control description -->
   <xacro:include filename="$(find perseus_description)/ros2_control/perseus.ros2_control.xacro" />
-  <xacro:include filename="$(find perseus_description)/urdf/camera_depth.urdf.xacro" />
   <!-- Instantiate the description and the ROS2 control information -->
   <xacro:perseus prefix="$(arg prefix)" />
-  <xacro:camera_depth prefix="$(arg prefix)" />
   <xacro:perseus_ros2_control name="Perseus" prefix="$(arg prefix)" can_bus="$(arg can_bus)" hardware_plugin="$(arg hardware_plugin)"/>
 </robot>

File: software/ros_ws/src/perseus_description/urdf/camera_depth.urdf.xacro (robot description, xacro)
@@ -3,11 +3,6 @@
 <!-- <box size="0.020 0.07 0.03"/>  -->
 <robot name="camera_depth" xmlns:xacro="http://ros.org/wiki/xacro">
-  <xacro:macro name="camera_depth" params="prefix:=^">
-    <joint name="camera_joint" type="fixed">
-        <parent link="base_link"/>
-        <child link="camera_link"/>
-        <origin xyz="0.220 0 0.4" rpy="0 0 0"/>
-    </joint>
-    <link name="camera_link">
+  <xacro:macro name="camera_depth" params="prefix">
+    <link name="${prefix}camera_link">
         <visual>
             <geometry>
@@ -17,11 +12,11 @@
         </visual>
     </link>
-    <joint name="camera_optical_joint" type="fixed">
-        <parent link="camera_link"/>
-        <child link="camera_link_optical"/>
+    <joint name="${prefix}camera_optical_joint" type="fixed">
+        <parent link="${prefix}camera_link"/>
+        <child link="${prefix}camera_link_optical"/>
         <origin xyz="0 0 0" rpy="0 0 0"/>
     </joint>
-    <link name="camera_link_optical"></link>
-    <gazebo reference="camera_link">
+    <link name="${prefix}camera_link_optical"></link>
+    <gazebo reference="${prefix}camera_link">
         <material>Gazebo/Red</material>
         <sensor name="rgbd_camera" type="rgbd_camera">
@@ -41,5 +36,5 @@
                 </clip>
             </camera>
-            <gz_frame_id>camera_link_optical</gz_frame_id>
+            <gz_frame_id>${prefix}camera_link_optical</gz_frame_id>
             <min_depth>0.05</min_depth>
             <max_depth>100.0</max_depth>

File: software/ros_ws/src/perseus_description/urdf/perseus.urdf.xacro (robot description, xacro)
@@ -26,8 +26,10 @@
     <xacro:include filename="$(find perseus_description)/urdf/wheel.urdf.xacro"/>
     <xacro:include filename="$(find perseus_description)/urdf/sensors.urdf.xacro"/>
+    <xacro:include filename="$(find perseus_description)/urdf/camera_depth.urdf.xacro" />
+    <!-- <xacro:camera_depth prefix="$(prefix)" /> -->
     <!-- An empty base_link to attach everything to -->
     <link name="${prefix}base_link"/>
     <joint name="${prefix}chassis_joint" type="fixed"> <!-- Joint Connect base_link and chassis -->
-      <origin xyz="0 0.0 ${chassis_z_offset/scale_factor}" rpy="0.0 0.0 0.0"/>
+      <origin xyz="0.3 0.0 ${chassis_z_offset/scale_factor}" rpy="0 0.0 0.0"/>
       <parent link="${prefix}base_link"/>
       <child link="${prefix}chassis"/>
@@ -101,4 +103,9 @@
       <origin xyz="0 0 -0.035" rpy="0 ${PI} 0"/>
     </joint>
+    <joint name="${prefix}camera_joint" type="fixed">
+        <parent link="${prefix}chassis"/>
+        <child link="${prefix}camera_link"/>
+        <origin xyz="0.01 0 0.2" rpy="0 0 0"/>
+    </joint>
   </xacro:macro>
 </robot>
