File: hardware/post-landing-breakout/post-landing-breakout.kicad_sch (KiCad schematic)
At the start: 42 parts, among them J1 DE9_Socket, J2 XT90, J3 DE9_Socket, J4 RSBL85, J6 Smol_Brain_Board, Q1 MMBT3906, SW1 SW_Slide_DPDT, U1 LM2596S-5

Commit message: feat: Changed mounting holes to 3mm, rounded corners
Parts:
- H1, H2, H3, H4, H5: footprint MountingHole:MountingHole_2.5mm_Pad_TopBottom -> MountingHole:MountingHole_3mm_Pad_TopBottom
Changed lines of the file:
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@@
 			)
 		)
-		(property "Footprint" "MountingHole:MountingHole_2.5mm_Pad_TopBottom"
+		(property "Footprint" "MountingHole:MountingHole_3mm_Pad_TopBottom"
 			(at 19.05 147.32 0)
 			(hide yes)
@@
 			)
 		)
-		(property "Footprint" "MountingHole:MountingHole_2.5mm_Pad_TopBottom"
+		(property "Footprint" "MountingHole:MountingHole_3mm_Pad_TopBottom"
 			(at 19.05 142.24 0)
 			(hide yes)
@@
 			)
 		)
-		(property "Footprint" "MountingHole:MountingHole_2.5mm_Pad_TopBottom"
+		(property "Footprint" "MountingHole:MountingHole_3mm_Pad_TopBottom"
 			(at 19.05 152.4 0)
 			(hide yes)
@@
 			)
 		)
-		(property "Footprint" "MountingHole:MountingHole_2.5mm_Pad_TopBottom"
+		(property "Footprint" "MountingHole:MountingHole_3mm_Pad_TopBottom"
 			(at 19.05 132.08 0)
 			(hide yes)
@@
 			)
 		)
-		(property "Footprint" "MountingHole:MountingHole_2.5mm_Pad_TopBottom"
+		(property "Footprint" "MountingHole:MountingHole_3mm_Pad_TopBottom"
 			(at 19.05 137.16 0)
 			(hide yes)

Commit message: fix: Changed mounting holes to 3.2mm
Parts:
- H1, H2, H3, H4, H5: footprint MountingHole:MountingHole_3mm_Pad_TopBottom -> MountingHole:MountingHole_3.2mm_M3_Pad_Via
Changed lines of the file:
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@@
 			)
 		)
-		(property "Footprint" "MountingHole:MountingHole_3mm_Pad_TopBottom"
+		(property "Footprint" "MountingHole:MountingHole_3.2mm_M3_Pad_Via"
 			(at 19.05 147.32 0)
 			(hide yes)
@@
 			)
 		)
-		(property "Footprint" "MountingHole:MountingHole_3mm_Pad_TopBottom"
+		(property "Footprint" "MountingHole:MountingHole_3.2mm_M3_Pad_Via"
 			(at 19.05 142.24 0)
 			(hide yes)
@@
 			)
 		)
-		(property "Footprint" "MountingHole:MountingHole_3mm_Pad_TopBottom"
+		(property "Footprint" "MountingHole:MountingHole_3.2mm_M3_Pad_Via"
 			(at 19.05 152.4 0)
 			(hide yes)
@@
 			)
 		)
-		(property "Footprint" "MountingHole:MountingHole_3mm_Pad_TopBottom"
+		(property "Footprint" "MountingHole:MountingHole_3.2mm_M3_Pad_Via"
 			(at 19.05 132.08 0)
 			(hide yes)
@@
 			)
 		)
-		(property "Footprint" "MountingHole:MountingHole_3mm_Pad_TopBottom"
+		(property "Footprint" "MountingHole:MountingHole_3.2mm_M3_Pad_Via"
 			(at 19.05 137.16 0)
 			(hide yes)
