File: hardware/SR_deplotables_control_board/sr ir sensor.kicad_pcb (KiCad board)
At the start: 2 copper layers, 34.2 x 35 mm, 26 parts, among them J1 Conn_01x12_Pin, J2 Conn_01x02_Pin, J3 Conn_01x07_Pin, Q3 2N7002, Q4 2N7002, U1 MCP3002, U2 DRV8833PW

Commit message: cleaned up control board pcb
Other:
- board text added: "3.3v"
- board text added: "5v"
- board text added: "GND"
Changed lines of the file:
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@@
 			(outputformat 1)
 			(mirror no)
-			(drillshape 1)
+			(drillshape 0)
 			(scaleselection 1)
-			(outputdirectory "")
+			(outputdirectory "manufacture/")
 		)
 	)
@@
 		(layer "Edge.Cuts")
 	)
+	(gr_text "GND\n"
+		(at 131.5 106.5 0)
+		(layer "F.SilkS" knockout)
+		(effects
+			(font
+				(size 1.5 1.5)
+				(thickness 0.3)
+				(bold yes)
+			)
+			(justify left bottom)
+		)
+	)
+	(gr_text "GND"
+		(at 134 80 0)
+		(layer "F.SilkS" knockout)
+		(effects
+			(font
+				(size 1.5 1.5)
+				(thickness 0.3)
+				(bold yes)
+			)
+			(justify left bottom)
+		)
+	)
+	(gr_text "3.3v"
+		(at 110 79 0)
+		(layer "F.SilkS" knockout)
+		(effects
+			(font
+				(size 1.5 1.5)
+				(thickness 0.3)
+				(bold yes)
+			)
+			(justify left bottom)
+		)
+	)
+	(gr_text "5v"
+		(at 109.5 105.5 0)
+		(layer "F.SilkS" knockout)
+		(effects
+			(font
+				(size 1.5 1.5)
+				(thickness 0.3)
+				(bold yes)
+			)
+			(justify left bottom)
+		)
+	)
 	(segment
