File: hardware/SR_deplotables_control_board/sr deployables control board.kicad_sch (KiCad schematic)
At the start: 26 parts, among them J1 Conn_01x12_Pin, J2 Conn_01x02_Pin, J3 Conn_01x07_Pin, Q3 2N7002, Q4 2N7002, U1 MCP3002, U2 DRV8833PW

Commit message: feat: Cleanup files and start redesign
Parts:
- J1: symbol Connector:Conn_01x12_Pin -> Connector_Generic:Conn_01x12
Connections:
- net +3.3V: now also J1.12 (Pin_12); no longer J1.1 (Pin_1)
- net +5V: now also J1.11 (Pin_11); no longer J1.2 (Pin_2)
- net AIN1: now also J1.4 (Pin_4); no longer J1.9 (Pin_9)
- net AIN2: now also J1.3 (Pin_3); no longer J1.10 (Pin_10)
- net CLK: now also J1.9 (Pin_9); no longer J1.4 (Pin_4)
- net CS: now also J1.10 (Pin_10); no longer J1.3 (Pin_3)
- net GATE1: now also J1.6 (Pin_6); no longer J1.7 (Pin_7)
- net GATE2: now also J1.5 (Pin_5); no longer J1.8 (Pin_8)
- net GND: now also J1.1 (Pin_1); no longer J1.12 (Pin_12)
- net MISO: now also J1.8 (Pin_8); no longer J1.5 (Pin_5)
- net MOSI: now also J1.7 (Pin_7); no longer J1.6 (Pin_6)
- net SWITCH: now also J1.2 (Pin_2); no longer J1.11 (Pin_11)
