File: hardware/light-tower-controlboard/control-board/control-board.kicad_sch (KiCad schematic)
At the start: 8 parts, among them J1 DE9, J2 VIN, J5 Conn_01x02

Commit message: finalised design and ready for manufacture
Parts:
- removed J2: VIN, Library:TerminalBlock_4Ucon_1x02_P3.50mm_Horizontal, symbol Library:Screw_Terminal_01x02
- removed TP1: GND, TestPoint:TestPoint_Pad_D4.0mm, symbol Connector:TestPoint
- removed TP2: LED_VOUT, TestPoint:TestPoint_Pad_D4.0mm, symbol Connector:TestPoint
- added H1, H2, H3, H4: MountingHole_Pad, MountingHole:MountingHole_3mm_Pad, symbol Library:MountingHole_Pad
- added J2, J6: Conn_01x20, Connector_PinSocket_2.54mm:PinSocket_1x20_P2.54mm_Vertical, symbol Connector_Generic:Conn_01x20
- added J4: ~, Connector_AMASS:AMASS_XT30U-F_1x02_P5.0mm_Vertical, symbol Library:XT_Connector
- J5: value Conn_01x02 -> LED_SIG
- U1: footprint (none) -> Library:LM2596_reg_module
Connections:
- net GND: now also H1.1, H2.1, H3.1, H4.1, J2.1 (Pin_1), J4.1 (-), J6.1 (Pin_1)
- net VCC: now also PCB1.1 (VCC), J2.20 (Pin_20)
- net CAN_L: now reaches J1.1, J1.2, PCB1.8 (CAN_L)
- net CAN_L: now also J2.13 (Pin_13)
- net CAN_H: now reaches J1.7, J1.8, PCB1.7 (CAN_H)
- net CAN_H: now also J2.14 (Pin_14)
- net at PCB1.10 (A2): now also J2.11 (Pin_11)
- net at PCB1.11 (A3): now also J2.10 (Pin_10)
- net at PCB1.12 (A4): now also J2.9 (Pin_9)
- net at PCB1.13 (A5): now also J2.8 (Pin_8)
- net at PCB1.14 (A6): now also J2.7 (Pin_7)
- net at PCB1.15 (A7): now also J2.6 (Pin_6)
- net at PCB1.16 (A8): now also J2.5 (Pin_5)
- net at PCB1.17 (A9): now also J2.4 (Pin_4)
- net at PCB1.18 (A10): now also J2.3 (Pin_3)
- net at PCB1.19 (IO12): now also J2.2 (Pin_2)
- net at PCB1.2 (LED_DOUT): now also J2.19 (Pin_19)
- net at PCB1.21 (3V3): now also J6.20 (Pin_20)
- net at PCB1.22 (IO13): now also J6.19 (Pin_19)
- net at PCB1.23 (IO14): now also J6.18 (Pin_18)
- net at PCB1.24 (IO21): now also J6.17 (Pin_17)
- net at PCB1.25 (IO47): now also J6.16 (Pin_16)
- net at PCB1.26 (IO48): now also J6.15 (Pin_15)
- net at PCB1.27 (IO45): now also J6.14 (Pin_14)
- net at PCB1.28 (IO37): now also J6.13 (Pin_13)
- net at PCB1.29 (IO38): now also J6.12 (Pin_12)
- net at PCB1.3 (UART0_TX): now also J2.18 (Pin_18)
- net at PCB1.30 (IO39): now also J6.11 (Pin_11)
- net at PCB1.31 (IO40): now also J6.10 (Pin_10)
- net at PCB1.32 (IO41): now also J6.9 (Pin_9)
- net at PCB1.33 (IO42): now also J6.8 (Pin_8)
- net at PCB1.34 (IO16): now also J6.7 (Pin_7)
- net LED_SIG: now reaches J5.1 (Pin_1), J5.2 (Pin_2), PCB1.35 (IO15)
- net LED_SIG: now also J6.6 (Pin_6)
- net at PCB1.36 (CAN_RX): now also J6.5 (Pin_5)
- net at PCB1.37 (CAN_TX): now also J6.4 (Pin_4)
- net at PCB1.38 (I2C_SDA): now also J6.3 (Pin_3)
- net at PCB1.39 (I2C_SCK): now also J6.2 (Pin_2)
- net at PCB1.4 (UART0_RX): now also J2.17 (Pin_17)
- net at PCB1.5 (UART1_TX): now also J2.16 (Pin_16)
- net at PCB1.6 (UART1_RX): now also J2.15 (Pin_15)
- net at PCB1.9 (A1): now also J2.12 (Pin_12)
- net +5V renamed VBUS
- net VBUS: now also J4.2 (+); no longer PCB1.1 (VCC)
- no-connect marks 39 -> 5
Other:
- note added: "In"
- note added: "Out"
- note added: "Power"
- note added: "regulator"
- moved on the sheet: J1, J3, J5, U1
