Commit message: wip: Add MoveIt Servo integration and configuration for arm control, and WIP Simulation

File: software/ros_ws/src/perseus_payloads/config/arm.ros2_control.xacro (robot description, xacro)
@@ -1,9 +1,14 @@
 <?xml version="1.0"?>
 <robot xmlns:xacro="http://www.ros.org/wiki/xacro">
-    <xacro:macro name="arm_ros2_control" params="name initial_positions_file">
+    <xacro:macro name="arm_ros2_control" params="name initial_positions_file use_mock_hardware:=false">
         <xacro:property name="initial_positions" value="${xacro.load_yaml(initial_positions_file)['initial_positions']}"/>
         <ros2_control name="${name}" type="system">
             <hardware>
-                <plugin>perseus_payloads/PerseusArmHardware</plugin>
+                <xacro:if value="${use_mock_hardware}">
+                  <plugin>mock_components/GenericSystem</plugin>
+                </xacro:if>
+                <xacro:unless value="${use_mock_hardware}">
+                  <plugin>perseus_payloads/PerseusArmHardware</plugin>
+                </xacro:unless>
             </hardware>
             <joint name="shoulder_pan">

File: software/ros_ws/src/perseus_payloads/config/arm.urdf.xacro (robot description, xacro)
@@ -2,8 +2,9 @@
 <robot xmlns:xacro="http://www.ros.org/wiki/xacro" name="arm">
     <xacro:arg name="initial_positions_file" default="initial_positions.yaml" />
+    <xacro:arg name="use_mock_hardware" default="true" />
     <!-- Import arm urdf file -->
     <xacro:include filename="$(find perseus_payloads)/src/moveit/arm.urdf" />
     <!-- Import control_xacro -->
     <xacro:include filename="arm.ros2_control.xacro" />
-    <xacro:arm_ros2_control name="FakeSystem" initial_positions_file="$(arg initial_positions_file)"/>
+    <xacro:arm_ros2_control name="FakeSystem" initial_positions_file="$(arg initial_positions_file)" use_mock_hardware="$(arg use_mock_hardware)"/>
 </robot>

Commit message: chore: fix Perseus Arm hardware interface with updated CAN addressing, actuator message.

File: software/ros_ws/src/perseus_payloads/config/arm.ros2_control.xacro (robot description, xacro)
@@ -12,4 +12,12 @@
                 </xacro:unless>
             </hardware>
+            <joint name="shoulder_tilt">
+                <command_interface name="position"/>
+                <command_interface name="velocity"/>
+                <state_interface name="position">
+                  <param name="initial_value">${initial_positions['shoulder_tilt']}</param>
+                </state_interface>
+                <state_interface name="velocity"/>
+            </joint>
             <joint name="shoulder_pan">
                 <command_interface name="position"/>
@@ -17,12 +25,4 @@
                 <state_interface name="position">
                   <param name="initial_value">${initial_positions['shoulder_pan']}</param>
-                </state_interface>
-                <state_interface name="velocity"/>
-            </joint>
-            <joint name="shoulder_tilt">
-                <command_interface name="position"/>
-                <command_interface name="velocity"/>
-                <state_interface name="position">
-                  <param name="initial_value">${initial_positions['shoulder_tilt']}</param>
                 </state_interface>
                 <state_interface name="velocity"/>

File: software/ros_ws/src/perseus_payloads/src/moveit/arm.urdf (robot description, URDF)
Before this commit: robot arm, 8 links, 7 joints
Joints:
- joint elbow: limit lower=-3.14 upper=3.14 effort=8.0 velocity=2.0 -> lower=-3.14159 upper=3.14159 effort=8.0 velocity=2.0
- joint shoulder_pan: limit lower=-3.14 upper=3.14 effort=10.0 velocity=2.0 -> lower=-3.14159 upper=3.14159 effort=10.0 velocity=2.0
- joint wrist_roll: limit lower=-3.14 upper=3.14 effort=5.0 velocity=3.0 -> lower=-3.14159 upper=3.14159 effort=10.0 velocity=2.0

Commit message: feat: Add fake_dof joint and reconfigure end-effector

File: software/ros_ws/src/perseus_payloads/config/arm.ros2_control.xacro (robot description, xacro)
@@ -52,4 +52,12 @@
                 <state_interface name="velocity"/>
             </joint>
+            <joint name="fake_dof">
+                <command_interface name="position"/>
+                <command_interface name="velocity"/>
+                <state_interface name="position">
+                  <param name="initial_value">${initial_positions['fake_dof']}</param>
+                </state_interface>
+                <state_interface name="velocity"/>
+            </joint>
         </ros2_control>
     </xacro:macro>

File: software/ros_ws/src/perseus_payloads/src/moveit/arm.urdf (robot description, URDF)
Before this commit: robot arm, 8 links, 7 joints
Links:
- added link fake_dof_link, mass 0.001; collision sphere radius=0.005; visual sphere radius=0.005
Joints:
- added joint fake_dof: type revolute, parent wrist_roll_link, child fake_dof_link, origin xyz=0 0 0.028 rpy=0 0 0, axis 1 0 0, limit lower=-0.5 upper=0.5 effort=1.0 velocity=1.0
- joint end_effector_mount: origin xyz=0 0 0.028 rpy=0 0 0 -> xyz=0 0 0 rpy=0 0 0; parent wrist_roll_link -> fake_dof_link
