Commit message: feat: fixarm MoveIt configuration  and keyboard teleoperation

File: software/ros_ws/src/perseus_payloads/src/moveit/arm.urdf (robot description, URDF)
Before this commit: robot arm, 7 links, 6 joints
Links:
- added link forearm_tip, mass 0.001; collision sphere radius=0.01; visual sphere radius=0.01
- link end_effector: mass None -> 0.05
- link forearm: mass None -> 0.5
- link plate: mass None -> 0.5
- link shoulder_arm: mass None -> 0.6
- link shoulder_base: mass None -> 0.8
- link wrist_pitch_link: mass None -> 0.2
- link wrist_roll_link: mass None -> 0.15
Joints:
- added joint forearm_tip_joint: type fixed, parent forearm, child forearm_tip, origin xyz=0 0 0.558 rpy=0 0 0
- joint elbow: limit lower=-2.62 upper=2.62 effort=8.0 velocity=2.0 -> lower=-3.14 upper=3.14 effort=8.0 velocity=2.0; origin xyz=0 0 0.3 rpy=0 0 0 -> xyz=0 -0.03 0.275 rpy=0 0 0
- joint end_effector_mount: parent wrist_roll_link -> wrist_pitch_link
- joint shoulder_pan: limit effort=10.0 velocity=2.0 -> lower=-3.14 upper=3.14 effort=10.0 velocity=2.0; type continuous -> revolute
- joint wrist_roll: limit effort=5.0 velocity=3.0 -> lower=-3.14 upper=3.14 effort=5.0 velocity=3.0; type continuous -> revolute

Commit message: refactor: switch arm kinematics solver to KDL

File: software/ros_ws/src/perseus_payloads/src/moveit/arm.urdf (robot description, URDF)
Before this commit: robot arm, 8 links, 7 joints
Joints:
- joint end_effector_mount: parent wrist_pitch_link -> wrist_roll_link

Commit message: feat: Implement continuous RSBL servo position tracking with rollover handling

File: software/ros_ws/src/perseus_payloads/src/moveit/arm.urdf (robot description, URDF)
Before this commit: robot arm, 9 links, 8 joints
Joints:
- joint fake_dof: limit lower=-0.5 upper=0.5 effort=1.0 velocity=1.0 -> lower=-1.57 upper=1.57 effort=1.0 velocity=1.0
