Commit message: feat: Add calibration node and update Perseus Lite hardware and mapping autotune
Add calibration_node for mapping autotune, improve maneuver executor,
update Perseus Lite URDF/ros2_control/hardware interface, and wire
autotune into autonomy launch.

File: software/ros_ws/src/perseus_lite/urdf/perseus_lite.urdf.xacro (robot description, xacro)
@@ -5,4 +5,5 @@
   <xacro:arg name="serial_port" default="/dev/ttyACM0" />
   <xacro:arg name="baud_rate" default="1000000" />
+  <xacro:arg name="servo_max_rpm" default="112.8" />
   <!-- Import URDF description -->
   <xacro:include filename="$(find perseus_lite_description)/urdf/perseus_lite.urdf.xacro" />
@@ -18,4 +19,5 @@
     hardware_plugin="$(arg hardware_plugin)"
     serial_port="$(arg serial_port)"
-    baud_rate="$(arg baud_rate)"/>
+    baud_rate="$(arg baud_rate)"
+    servo_max_rpm="$(arg servo_max_rpm)"/>
 </robot>

File: software/ros_ws/src/perseus_lite_description/ros2_control/perseus_lite.ros2_control.xacro (robot description, xacro)
@@ -1,5 +1,5 @@
 <?xml version="1.0"?>
 <robot xmlns:xacro="http://www.ros.org/wiki/xacro">
-  <xacro:macro name="perseus_lite_ros2_control" params="name prefix hardware_plugin serial_port baud_rate">
+  <xacro:macro name="perseus_lite_ros2_control" params="name prefix hardware_plugin serial_port baud_rate servo_max_rpm">
     <ros2_control name="${name}" type="system">
       <hardware>
@@ -7,4 +7,5 @@
         <param name="serial_port">${serial_port}</param>
         <param name="baud_rate">${baud_rate}</param>
+        <param name="servo_max_rpm">${servo_max_rpm}</param>
       </hardware>
       <joint name="${prefix}front_left_wheel_joint">
