Commit message: perseus_lite: alignment of launch and yaml with perseus
perseus_lite: added debug info to serial commands

perseus_lite: reorder node launch sequence

ros_ws(nix): Updated nix packaging

File: software/ros_ws/src/perseus_lite_description/ros2_control/perseus_lite.ros2_control.xacro (robot description, xacro)
@@ -1,10 +1,10 @@
 <?xml version="1.0"?>
 <robot xmlns:xacro="http://www.ros.org/wiki/xacro">
-  <xacro:macro name="perseus_lite_ros2_control" params="name prefix hardware_plugin serial_port">
+  <xacro:macro name="perseus_lite_ros2_control" params="name prefix hardware_plugin serial_port baud_rate">
     <ros2_control name="${name}" type="system">
       <hardware>
         <plugin>${hardware_plugin}</plugin>
         <param name="serial_port">${serial_port}</param>
-        <param name="baud_rate">115200</param>
+        <param name="baud_rate">${baud_rate}</param>
       </hardware>
       <joint name="${prefix}front_left_wheel_joint">

File: software/ros_ws/src/perseus_lite_description/urdf/perseus_lite.urdf.xacro (robot description, xacro)
@@ -1,52 +1,26 @@
 <?xml version="1.0"?>
-<robot xmlns:xacro="http://www.ros.org/wiki/xacro" name="perseus_lite">
-  <!-- Default arguments -->
-  <xacro:arg name="prefix" default="" />
-  <xacro:arg name="use_mock_hardware" default="false" />
-  <xacro:arg name="serial_port" default="/dev/ttyACM0" />
-  <xacro:arg name="hardware_type" default="st3215"/>
-  <!-- Hardware plugin selection -->
-  <xacro:property name="real_hardware_plugin" value="perseus_lite_hardware/ST3215SystemHardware" />
-  <xacro:property name="use_mock_hardware" value="$(arg use_mock_hardware)" />
-  <xacro:property name="hardware_plugin"
-    value="${'mock_components/GenericSystem' if use_mock_hardware else real_hardware_plugin}" />
-  <!-- Import dependencies -->
-  <!-- <xacro:include filename="$(find perseus_lite_description)/urdf/perseus_lite.urdf.xacro" /> -->
-  <xacro:include filename="$(find perseus_lite_description)/urdf/chassis.urdf.xacro"/>
-  <xacro:include filename="$(find perseus_lite_description)/urdf/rocker.urdf.xacro"/>
-  <xacro:include filename="$(find perseus_lite_description)/urdf/perseus_lite.materials.xacro" />
-  <xacro:include filename="$(find perseus_lite_description)/ros2_control/perseus_lite.ros2_control.xacro" />
-  <!-- Scale for Perseus Lite - DO I NEED THIS?-->
-  <xacro:property name="scale" value="0.5"/>
-  <!-- Main macro definition -->
+<robot xmlns:xacro="http://ros.org/wiki/xacro">
   <xacro:macro name="perseus_lite" params="prefix">
+    <!-- Import components -->
+    <xacro:include filename="$(find perseus_lite_description)/urdf/chassis.urdf.xacro"/>
+    <xacro:include filename="$(find perseus_lite_description)/urdf/rocker.urdf.xacro"/>
+    <!-- <xacro:include filename="$(find perseus_lite_description)/urdf/sensors.urdf.xacro"/> -->
     <link name="${prefix}base_link"/>
-    <joint name="base_footprint_joint" type="fixed">
-      <parent link="base_link"/>
-      <child link="base_footprint"/>
-      <origin xyz="0 0 0" rpy="0 0 0"/>
-    </joint>
-    <link name="base_footprint">
-    </link>
+    <!-- CHASSIS -->
     <xacro:chassis />
-    <joint name="chassis_joint" type="fixed">
-      <origin xyz="${0.21 * scale} 0.0 ${0.35 * scale}" rpy="0.0 0.0 -${pi/2}"/>
+    <joint name="${prefix}chassis_joint" type="fixed">
+      <origin xyz="0.21 0.0 0.35" rpy="0.0 0.0 -${pi/2}"/>
       <parent link="${prefix}base_link"/>
       <child link="${prefix}chassis"/>
     </joint>
+    <!-- ROCKER ARMS -->
+    <!-- LEFT -->
     <xacro:rocker side="left">
-      <origin xyz="${-0.275 * scale} ${-0.075 * scale} ${0.05 * scale}" rpy="0.0 0.0 ${-pi/2}"/>
+      <origin xyz="-0.275 -0.075 0.05" rpy="0.0 0.0 ${-pi/2}"/>
     </xacro:rocker>
+    <!-- RIGHT -->
     <xacro:rocker side="right">
-      <origin xyz="${0.275 * scale} ${-0.075 * scale} ${0.05 * scale}" rpy="0.0 0.0 ${-pi/2}"/>
+      <origin xyz="0.275 -0.075 0.05" rpy="0.0 0.0 ${-pi/2}"/>
     </xacro:rocker>
-    <!-- ROS2 Control -->
-    <xacro:perseus_lite_ros2_control
-      name="Perseus_Lite"
-      prefix="${prefix}"
-      hardware_plugin="${hardware_plugin}"
-      serial_port="$(arg serial_port)"/>
   </xacro:macro>
-  <!-- Instantiate the description -->
-  <xacro:perseus_lite prefix="$(arg prefix)" />
 </robot>

File: software/ros_ws/src/perseus_lite_description/urdf/wheel.urdf.xacro (robot description, xacro)
@@ -34,4 +34,16 @@
       <dynamics damping="0.5" friction="0.5"/>
     </joint>
+  <transmission name="${prefix}${end}_${side}_wheel_trans">
+    <type>transmission_interface/SimpleTransmission</type>
+      <joint name="${prefix}${end}_${side}_wheel_joint">
+        <command_interface name="velocity"/>
+        <state_interface name="position"/>
+        <state_interface name="velocity"/>
+        <state_interface name="temperature"/>
+      </joint>
+      <actuator name="${prefix}${end}_${side}_wheel_motor">
+        <mechanical_reduction>1.0</mechanical_reduction>
+      </actuator>
+    </transmission>
   </xacro:macro>
 </robot>

Commit message: persues_lite: tweaks to the URDF

File: software/ros_ws/src/perseus_lite_description/ros2_control/perseus_lite.ros2_control.xacro (robot description, xacro)
@@ -13,5 +13,5 @@
         <state_interface name="velocity"/>
         <state_interface name="temperature"/>
-        <param name="id">1</param>
+        <param name="id">3</param>
       </joint>
       <joint name="${prefix}front_right_wheel_joint">
@@ -20,5 +20,5 @@
         <state_interface name="velocity"/>
         <state_interface name="temperature"/>
-        <param name="id">2</param>
+        <param name="id">4</param>
       </joint>
       <joint name="${prefix}rear_left_wheel_joint">
@@ -27,5 +27,5 @@
         <state_interface name="velocity"/>
         <state_interface name="temperature"/>
-        <param name="id">3</param>
+        <param name="id">2</param>
       </joint>
       <joint name="${prefix}rear_right_wheel_joint">
@@ -34,5 +34,5 @@
         <state_interface name="velocity"/>
         <state_interface name="temperature"/>
-        <param name="id">4</param>
+        <param name="id">1</param>
       </joint>
     </ros2_control>

File: software/ros_ws/src/perseus_lite_description/urdf/wheel.urdf.xacro (robot description, xacro)
@@ -24,5 +24,5 @@
     <joint name="${prefix}${end}_${side}_wheel_joint" type="continuous">
       <xacro:if value="${side == 'left'}">
-        <axis xyz="0 1 0" rpy="0 0 0"/>
+        <axis xyz="0 -1 0" rpy="0 0 0"/>
       </xacro:if>
       <xacro:if value="${side == 'right'}">

Commit message: fix: Address code review findings across hardware, CI, and launch files
Hardware interface (perseus_lite_hardware):
- Implement a real serial read timeout: the old steady_timer was never
  awaited, so read_some() could block the comm thread forever on a wedged
  servo or unplugged adapter
- Fix temperature state reading the voltage register (0x3E) instead of
  the temperature register (0x3F)
- Hold the serial mutex across the full request/response transaction so
  controller writes cannot interleave mid-exchange
- Make inverted servo IDs a hardware parameter (inverted_servo_ids,
  default 2,3) instead of hardcoding them in the protocol header
- Remove dead code: unused update_servo_states(), never-started
  _io_thread, duplicated protocol constants
- Extract packet parsing into testable protocol::extract_packets() and
  protocol::parse_status_payload(); add 18 unit tests (47 total)

CI / fork hygiene:
- Fix is-main gate that still checked ROAR-QUTRC/perseus-v2, disabling
  main-branch automation on this fork; gate docs deploy on its secret
- Run colcon test across all packages so new test suites are picked up
  automatically; rely on colcon test-result for failure detection
- Add advisory cppcheck static-analysis job
- Update README title/badge, vision config comment, and home-manager
  flake path from perseus-v2 to perseus-lite; document why the cube
  detector model downloads from upstream releases

Launch/config:
- Add lidar_port launch argument instead of hardcoded /dev/ttyUSB0
- Make the TwistStamped frame_id a parameter on the xbox controller

Build hygiene:
- Standardize -Wshadow across in-house C++ packages; add C++20 and
  warnings to perseus_autonomy_bridge and perseus_bt_nodes
- Document the package versioning scheme
- Ignore .claude/ session data; log fixed defects in ERRORS.md

File: software/ros_ws/src/perseus_lite_description/ros2_control/perseus_lite.ros2_control.xacro (robot description, xacro)
@@ -1,5 +1,5 @@
 <?xml version="1.0"?>
 <robot xmlns:xacro="http://www.ros.org/wiki/xacro">
-  <xacro:macro name="perseus_lite_ros2_control" params="name prefix hardware_plugin serial_port baud_rate">
+  <xacro:macro name="perseus_lite_ros2_control" params="name prefix hardware_plugin serial_port baud_rate inverted_servo_ids:='2,3'">
     <ros2_control name="${name}" type="system">
       <hardware>
@@ -7,4 +7,6 @@
         <param name="serial_port">${serial_port}</param>
         <param name="baud_rate">${baud_rate}</param>
+        <!-- Left-side servos drive mirrored, so their velocity is inverted -->
+        <param name="inverted_servo_ids">${inverted_servo_ids}</param>
       </hardware>
       <joint name="${prefix}front_left_wheel_joint">
