File: hardware/rover-control-board-v2/HV_smart_switch.kicad_sch (KiCad schematic)
At the start: 26 parts, among them Q3 Q_NMOS_DGS, Q4 Q_PMOS_DGS, U2 BTH50015

Commit message: Started protection circuits
Parts:
- removed C6: 10nF, symbol Device:C
- removed D3: RED, symbol Device:LED
- removed JP1, JP2: ADDR, Jumper:SolderJumper-3_P1.3mm_Open_Pad1.0x1.5mm, symbol Jumper:SolderJumper_3_Open
- removed Q3: Q_NMOS_DGS, symbol Transistor_FET:Q_NMOS_DGS
- removed Q4: Q_PMOS_DGS, symbol Transistor_FET:Q_PMOS_DGS
- removed R17: 10R, symbol Device:R
- removed U1: (no value), footprints:LM82, symbol component_library:LM82
- removed U2: BTH50015, Package_SO:Infineon_PG-TSDSO-14-22, symbol component_library:BTH50015
- added C: 10nF, symbol Device:C
- added D: RED, symbol Device:LED
- added Q: Q_PMOS_DGS, symbol Transistor_FET:Q_PMOS_DGS
- added Q: Q_NMOS_DGS, symbol Transistor_FET:Q_NMOS_DGS
- added R: 10R, symbol Device:R
- added U: BTH50015, Package_SO:Infineon_PG-TSDSO-14-22, symbol component_library:BTH50015
Connections:
- net GND: now also C.2, Q.3 (S), U.1 (GND)
- net PRE_EN: now also D.2 (A)
- net PWR_IN: now also R.1, U.4 (DEN), U.9 (VS)
- net PWR_OUT: now also Q.3 (S), U.5 (OUT), U.6 (OUT), U.7 (OUT), U.8 (OUT)
- net i_sense: now also C.1
- net at R4.1: now also Q.1 (D)
- net at R3.1, R4.2: now also Q.2 (G)
- net at R5.2, R6.2: now also Q.2 (G)
- net at R8.2, R9.1: now also U.2 (IS)
- net at R7.2: now also D.1 (K)
- net at R2.2, R3.2: now also Q.1 (D), R.2
- net at R10.1: now also U.3 (IN)
- no-connect marks 5 -> 0

Commit message: Channels routed, temp bus pending
Parts:
- removed C, C2, C4: 10nF, symbol Device:C
- removed C3, C5: 100nF, symbol Device:C
- removed D2: GREEN, symbol Device:LED
- removed R10, R9: 1k, symbol Device:R
- removed R11, R13, R8: 10k, symbol Device:R
- removed R12: 500k, symbol Device:R
- removed U: BTH50015, Package_SO:Infineon_PG-TSDSO-14-22, symbol component_library:BTH50015
- added C45, C46, C48: 10nF, symbol Device:C
- added C47, C49, C56: 100nF, symbol Device:C
- added D34: RED, symbol Device:LED
- added D35, D37: ESD5Zxx, Diode_SMD:D_SOD-523, symbol Diode:ESD5Zxx
- added D36: GREEN, symbol Device:LED
- added J18: TEMP_PROBE, symbol Connector_Generic:Conn_01x02
- added JP13, JP14: ADDR, Jumper:SolderJumper-3_P1.3mm_Open_Pad1.0x1.5mm, symbol Jumper:SolderJumper_3_Open
- added Q12: Q_NMOS, symbol Device:Q_NMOS
- added R78, R80, R81, R83, R86: 10k, symbol Device:R
- added R79: 100R, symbol Device:R
- added R82, R84: 1k, symbol Device:R
- added R85: 500k, symbol Device:R
- added U15: (no value), footprints:LM82, symbol component_library:LM82
- added U16: BTH50015, Package_SO:Infineon_PG-TSDSO-14-22, symbol component_library:BTH50015
Connections:
- net CTRL: now also D36.2 (A), R84.2
- net GND: now also C45.2, C46.2, C47.2, C48.2, C49.2, C56.1, D35.2 (A), D37.2 (A), JP13.3 (B), JP14.3 (B), Q12.S, R80.2, R82.2, R83.1, R86.1, U15.7 (GND), U15.8 (GND), U16.1 (GND)
- net PWR_IN: now also C46.1, C47.1, U16.4 (DEN), U16.9 (VS)
- net PWR_OUT: now also C48.1, C49.1, R85.2, U16.5 (OUT), U16.6 (OUT), U16.7 (OUT), U16.8 (OUT)
- net V_sense: now also D37.1 (K), R85.1, R86.2
- net i_sense: now also C45.1, D35.1 (K), R81.1
- new net: Q12.G, R79.1, R80.1
- new net: D36.1 (K), R83.2
- new net: J18.1 (Pin_1), U15.4 (D-)
- new net: J18.2 (Pin_2), U15.3 (D+)
- new net: JP13.2 (C), U15.10 (ADDR0)
- new net: JP14.2 (C), U15.6 (ADDR1)
- new net: Q12.D, R78.1
- new net: D34.1 (K), R78.2
- new net: R84.1, U16.3 (IN)
- new net: R81.2, R82.1, U16.2 (IS)
- new net 3V3: C56.2, D34.2 (A), JP13.1 (A), JP14.1 (A), U15.2 (VCC)
- new net SCLK: U15.14 (SCLK)
- new net SDATA: U15.12 (SDATA)
- new net TEMP_ALARM_: R79.2, U15.16 (T_ALARM)
- new net TEMP_INT_: U15.11 (INT_)
- no-connect marks 0 -> 5
Other:
- note added: "1x02 pin header"
- note added: "5v varient needed"
- note added: "OVER TEMP"
- note added: "Use 2N3906 for external temp probe"
- note removed: "Add TVS"
- note removed: "Add TVS or Opto Coupler"
- note removed: "Check to make sure ADC of SBB has enough resolution"

Commit message: Bus routed
Parts:
- renumbered C56 to C53, C45 to C54, C46 to C55, C47 to C56, C48 to C57, C49 to C58, D to D39, D34 to D40, D35 to D41, D36 to D42, D37 to D43, J18 to J16, Q to Q22, Q to Q23, Q12 to Q24, R7 to R113, R5 to R114, R6 to R115, R to R116, R2 to R117, R3 to R118, R4 to R119, R78 to R120, R79 to R121, R80 to R122, R81 to R123, R82 to R124, R83 to R125, R84 to R126, R85 to R127, R86 to R128, U15 to U17, U16 to U18

Commit message: revamping channel switches
Parts:
- renumbered C53 to C47, C54 to C48, C55 to C49, C56 to C50, C57 to C51, C58 to C52, J16 to J17, R113 to R112, R114 to R113, R115 to R114, R116 to R115, R117 to R116, R118 to R117, R119 to R118, R120 to R119, R121 to R120, R122 to R121, R123 to R122, R124 to R123, R125 to R124, R126 to R125, R127 to R126, R128 to R127, U17 to U16, U18 to U17

Commit message: Minor fixes and sanity checks
Parts:
- removed C48, C51: 10nF, symbol Device:C
- removed C50, C52: 100nF, symbol Device:C
- removed D41, D43: ESD5Zxx, Diode_SMD:D_SOD-523, symbol Diode:ESD5Zxx
- removed D42: GREEN, symbol Device:LED
- removed R122, R124, R127: 10k, symbol Device:R
- removed R123, R125: 1k, symbol Device:R
- removed R126: 500k, symbol Device:R
- removed U17: BTH50015, Package_SO:Infineon_PG-TSDSO-14-22, symbol component_library:BTH50015
- added C46: 100nF, symbol Device:C
- added C47: 0.1uF, symbol Device:C
- added C48: C_Polarized, Capacitor_SMD:CP_Elec_10x10.5, symbol Device:C_Polarized
- added D36: GREEN, symbol Device:LED
- added D37: ESD5Zxx, Diode_SMD:D_SOD-523, symbol Diode:ESD5Zxx
- added F8: Blade, symbol Device:Fuse
- added Q31: CSD19533Q5A, Package_TO_SOT_SMD:TDSON-8-1, symbol Transistor_FET:CSD19533Q5A
- added R109, R111: 10k, symbol Device:R
- added R110: 500k, symbol Device:R
- added U23: LTC7001, Package_SO:MSOP-10-1EP_3x3mm_P0.5mm_EP1.68x1.88mm, symbol component_library:LTC7001
- added U24: ACS37003, Package_SO:SOIC-16W_7.5x10.3mm_P1.27mm, symbol component_library:ACS37003
- C49: value 10nF -> 100nF
- renumbered C47 to C45, D39 to D34, D40 to D35, J17 to J18, Q22 to Q28, Q23 to Q29, Q24 to Q30, R113 to R100, R114 to R101, R115 to R102, R116 to R103, R117 to R104, R118 to R105, R119 to R106, R120 to R107, R121 to R108, R112 to R99, U16 to U22
Connections:
- net 3V3: now also C49.2, U24.13 (VCC)
- net CTRL: now also D36.2 (A), U23.4 (INP)
- net GND: now also C49.1, C46.1, C48.2, D37.2 (A), R109.1, R111.1, U23.11 (PAD), U23.2 (VCCUV), U23.3 (GND), U23.5 (OVLO), U24.16 (GND); no longer C49.2
- net PWR_IN: now also C48.1, Q31.5 (D); no longer C49.1
- net PWR_OUT: now also F8.1, R110.2
- net V_sense: now also D37.1 (K), R110.1, R111.2
- net TEMP_INT_: no longer names the net of U22.11 (INT_)
- new net: C46.2, U23.1 (VCC)
- new net: Q31.1 (S), Q31.2 (S), Q31.3 (S), U24.1 (IP+), U24.2 (IP+), U24.3 (IP+), U24.4 (IP+)
- new net: F8.2, U24.5 (IP-), U24.6 (IP-), U24.7 (IP-), U24.8 (IP-)
- new net: D36.1 (K), R109.2
- new net: C47.1, U23.9 (BST)
- new net: C47.2, U23.8 (TS)
- new net: Q31.4 (G), U23.6 (TGDN), U23.7 (TGUP)
- new net VIOUT: U24.12 (VIOUT)
- new net VI_VREF: U24.11 (VREF)
- no-connect marks 5 -> 11
Other:
- note removed: "5v varient needed"
- note removed: "High precision needed"
