File: hardware/rover-control-board-v2/aux1_smart_switch.kicad_sch (KiCad schematic)
At the start: 23 parts, among them Q3 Q_NMOS_DGS, Q4 Q_PMOS_DGS, U2 BTH50015

Commit message: Buses added
Parts:
- removed C6: 10nF, symbol Device:C
- removed D3: RED, symbol Device:LED
- removed Q3: Q_NMOS_DGS, symbol Transistor_FET:Q_NMOS_DGS
- removed Q4: Q_PMOS_DGS, symbol Transistor_FET:Q_PMOS_DGS
- removed R17: 10R, symbol Device:R
- removed U2: BTH50015, Package_SO:Infineon_PG-TSDSO-14-22, symbol component_library:BTH50015
- added C: 10nF, symbol Device:C
- added D: RED, symbol Device:LED
- added Q: Q_NMOS_DGS, symbol Transistor_FET:Q_NMOS_DGS
- added Q: Q_PMOS_DGS, symbol Transistor_FET:Q_PMOS_DGS
- added R: 10R, symbol Device:R
- added U: BTH50015, Package_SO:Infineon_PG-TSDSO-14-22, symbol component_library:BTH50015
Connections:
- net GND: now also C.2, Q.3 (S), U.1 (GND)
- net PRE_EN: now also D.2 (A)
- net PWR_IN: now also R.1, U.4 (DEN), U.9 (VS)
- net PWR_OUT: now also Q.3 (S), U.5 (OUT), U.6 (OUT), U.7 (OUT), U.8 (OUT)
- net i_sense: now also C.1
- net at R4.1: now also Q.1 (D)
- net at R3.1, R4.2: now also Q.2 (G)
- net at R5.2, R6.2: now also Q.2 (G)
- net at R8.2, R9.1: now also U.2 (IS)
- net at R7.2: now also D.1 (K)
- net at R2.2, R3.2: now also Q.1 (D), R.2
- net at R10.1: now also U.3 (IN)

Commit message: Channels routed, temp bus pending
Parts:
- removed C, C2, C4: 10nF, symbol Device:C
- removed C3, C5: 100nF, symbol Device:C
- removed D2: GREEN, symbol Device:LED
- removed R10, R9: 1k, symbol Device:R
- removed R11, R13, R8: 10k, symbol Device:R
- removed R12: 500k, symbol Device:R
- removed U: BTH50015, Package_SO:Infineon_PG-TSDSO-14-22, symbol component_library:BTH50015
- added C20, C21, C23: 10nF, symbol Device:C
- added C22, C24, C51: 100nF, symbol Device:C
- added D14: RED, symbol Device:LED
- added D15, D17: ESD5Zxx, Diode_SMD:D_SOD-523, symbol Diode:ESD5Zxx
- added D16: GREEN, symbol Device:LED
- added J13: TEMP_PROBE, symbol Connector_Generic:Conn_01x02
- added JP3, JP4: ADDR, Jumper:SolderJumper-3_P1.3mm_Open_Pad1.0x1.5mm, symbol Jumper:SolderJumper_3_Open
- added Q7: Q_NMOS, symbol Device:Q_NMOS
- added R33, R35, R36, R38, R41: 10k, symbol Device:R
- added R34: 100R, symbol Device:R
- added R37, R39: 1k, symbol Device:R
- added R40: 500k, symbol Device:R
- added U5: (no value), footprints:LM82, symbol component_library:LM82
- added U6: BTH50015, Package_SO:Infineon_PG-TSDSO-14-22, symbol component_library:BTH50015
Connections:
- net CTRL: now also D16.2 (A), R39.2
- net GND: now also C20.2, C21.2, C22.2, C23.2, C24.2, C51.1, D15.2 (A), D17.2 (A), JP3.3 (B), JP4.3 (B), Q7.S, R35.2, R37.2, R38.1, R41.1, U5.7 (GND), U5.8 (GND), U6.1 (GND)
- net PWR_IN: now also C21.1, C22.1, U6.4 (DEN), U6.9 (VS)
- net PWR_OUT: now also C23.1, C24.1, R40.2, U6.5 (OUT), U6.6 (OUT), U6.7 (OUT), U6.8 (OUT)
- net V_sense: now also D17.1 (K), R40.1, R41.2
- net i_sense: now also C20.1, D15.1 (K), R36.1
- new net: Q7.G, R34.1, R35.1
- new net: D14.1 (K), R33.2
- new net: J13.1 (Pin_1), U5.4 (D-)
- new net: J13.2 (Pin_2), U5.3 (D+)
- new net: JP3.2 (C), U5.10 (ADDR0)
- new net: JP4.2 (C), U5.6 (ADDR1)
- new net: R36.2, R37.1, U6.2 (IS)
- new net: Q7.D, R33.1
- new net: R39.1, U6.3 (IN)
- new net: D16.1 (K), R38.2
- new net 3V3: C51.2, D14.2 (A), JP3.1 (A), JP4.1 (A), U5.2 (VCC)
- new net SCLK: U5.14 (SCLK)
- new net SDATA: U5.12 (SDATA)
- new net TEMP_ALARM_: R34.2, U5.16 (T_ALARM)
- new net TEMP_INT_: U5.11 (INT_)
- no-connect marks 0 -> 5
Other:
- note added: "1x02 pin header"
- note added: "5v varient needed"
- note added: "OVER TEMP"
- note added: "Use 2N3906 for external temp probe"
- note removed: "Add TVS"
- note removed: "Add TVS or Opto Coupler"
- note removed: "Check to make sure ADC of SBB has enough resolution"

Commit message: Bus routed
Parts:
- renumbered C51 to C22, C20 to C23, C21 to C24, C22 to C25, C23 to C26, C24 to C27, D to D10, D14 to D11, D15 to D12, D16 to D13, D17 to D14, J13 to J11, Q to Q6, Q to Q7, Q7 to Q8, R7 to R30, R5 to R31, R6 to R32, R to R33, R2 to R34, R3 to R35, R4 to R36, R33 to R37, R34 to R38, R35 to R39, R36 to R40, R37 to R41, R38 to R42, R39 to R43, R40 to R44, R41 to R45, U5 to U7, U6 to U8

Commit message: revamping channel switches
Parts:
- renumbered C22 to C16, C23 to C17, C24 to C18, C25 to C19, C26 to C20, C27 to C21, J11 to J12, R30 to R29, R31 to R30, R32 to R31, R33 to R32, R34 to R33, R35 to R34, R36 to R35, R37 to R36, R38 to R37, R39 to R38, R40 to R39, R41 to R40, R42 to R41, R43 to R42, R44 to R43, R45 to R44, U7 to U6, U8 to U7

Commit message: Minor fixes and sanity checks
Parts:
- removed C17, C18: 10nF, symbol Device:C
- removed C19: 100nF, symbol Device:C
- removed D12, D14: ESD5Zxx, Diode_SMD:D_SOD-523, symbol Diode:ESD5Zxx
- removed D13: GREEN, symbol Device:LED
- removed R39, R44: 10k, symbol Device:R
- removed R40: 1k, symbol Device:R
- removed U7: BTH50015, Package_SO:Infineon_PG-TSDSO-14-22, symbol component_library:BTH50015
- added C22: C_Polarized, Capacitor_SMD:CP_Elec_10x10.5, symbol Device:C_Polarized
- added C23: 100nF, symbol Device:C
- added D12: GREEN, symbol Device:LED
- added D13: ESD5Zxx, Diode_SMD:D_SOD-523, symbol Diode:ESD5Zxx
- added F2: Blade, symbol Device:Fuse
- added Q10: CSD19533Q5A, Package_TO_SOT_SMD:TDSON-8-1, symbol Transistor_FET:CSD19533Q5A
- added U8: LTC7001, Package_SO:MSOP-10-1EP_3x3mm_P0.5mm_EP1.68x1.88mm, symbol component_library:LTC7001
- added U9: ACS37003, Package_SO:SOIC-16W_7.5x10.3mm_P1.27mm, symbol component_library:ACS37003
- C20: value 10nF -> 100nF
- C21: value 100nF -> 0.1uF
- R42: value 1k -> 500k
- R43: value 500k -> 10k
- renumbered C16 to C19, J12 to J13, Q6 to Q7, Q7 to Q8, Q8 to Q9, R29 to R31, R30 to R32, R31 to R33, R32 to R34, R33 to R35, R34 to R36, R35 to R37, R36 to R38, R37 to R39, R38 to R40, U6 to U7
Connections:
- net 3V3: now also C23.2, U9.13 (VCC)
- net CTRL: now also D12.2 (A), U8.4 (INP); no longer R42.2
- net GND: now also C20.1, R43.1, C22.2, C23.1, D13.2 (A), U8.11 (PAD), U8.2 (VCCUV), U8.3 (GND), U8.5 (OVLO), U9.16 (GND); no longer C20.2, C21.2
- net PWR_IN: now also C22.1, Q10.5 (D)
- net PWR_OUT: now also R42.2, F2.1; no longer C20.1, C21.1, R43.2
- net V_sense: now also R42.1, R43.2, D13.1 (K); no longer R43.1
- net at R41.2: now also D12.1 (K)
- net TEMP_INT_: no longer names the net of U7.11 (INT_)
- new net: Q10.1 (S), Q10.2 (S), Q10.3 (S), U9.1 (IP+), U9.2 (IP+), U9.3 (IP+), U9.4 (IP+)
- new net: Q10.4 (G), U8.6 (TGDN), U8.7 (TGUP)
- new net: F2.2, U9.5 (IP-), U9.6 (IP-), U9.7 (IP-), U9.8 (IP-)
- new net: C21.1, U8.9 (BST)
- new net: C21.2, U8.8 (TS)
- new net: C20.2, U8.1 (VCC)
- new net VIOUT: U9.12 (VIOUT)
- new net VI_VREF: U9.11 (VREF)
- no-connect marks 5 -> 11
Other:
- note removed: "5v varient needed"
- note removed: "High precision needed"
