File: hardware/rover-control-board-v2/aux2_smart_switch.kicad_sch (KiCad schematic)
At the start: 23 parts, among them Q3 Q_NMOS_DGS, Q4 Q_PMOS_DGS, U2 BTH50015

Commit message: Buses added
Parts:
- removed C6: 10nF, symbol Device:C
- removed D3: RED, symbol Device:LED
- removed Q3: Q_NMOS_DGS, symbol Transistor_FET:Q_NMOS_DGS
- removed Q4: Q_PMOS_DGS, symbol Transistor_FET:Q_PMOS_DGS
- removed R17: 10R, symbol Device:R
- removed U2: BTH50015, Package_SO:Infineon_PG-TSDSO-14-22, symbol component_library:BTH50015
- added C: 10nF, symbol Device:C
- added D: RED, symbol Device:LED
- added Q: Q_PMOS_DGS, symbol Transistor_FET:Q_PMOS_DGS
- added Q: Q_NMOS_DGS, symbol Transistor_FET:Q_NMOS_DGS
- added R: 10R, symbol Device:R
- added U: BTH50015, Package_SO:Infineon_PG-TSDSO-14-22, symbol component_library:BTH50015
Connections:
- net GND: now also C.2, Q.3 (S), U.1 (GND)
- net PRE_EN: now also D.2 (A)
- net PWR_IN: now also R.1, U.4 (DEN), U.9 (VS)
- net PWR_OUT: now also Q.3 (S), U.5 (OUT), U.6 (OUT), U.7 (OUT), U.8 (OUT)
- net i_sense: now also C.1
- net at R4.1: now also Q.1 (D)
- net at R3.1, R4.2: now also Q.2 (G)
- net at R5.2, R6.2: now also Q.2 (G)
- net at R8.2, R9.1: now also U.2 (IS)
- net at R7.2: now also D.1 (K)
- net at R2.2, R3.2: now also Q.1 (D), R.2
- net at R10.1: now also U.3 (IN)

Commit message: Channels routed, temp bus pending
Parts:
- removed C, C2, C4: 10nF, symbol Device:C
- removed C3, C5: 100nF, symbol Device:C
- removed D2: GREEN, symbol Device:LED
- removed R10, R9: 1k, symbol Device:R
- removed R11, R13, R8: 10k, symbol Device:R
- removed R12: 500k, symbol Device:R
- removed U: BTH50015, Package_SO:Infineon_PG-TSDSO-14-22, symbol component_library:BTH50015
- added C25, C26, C28: 10nF, symbol Device:C
- added C27, C29, C52: 100nF, symbol Device:C
- added D18: RED, symbol Device:LED
- added D19, D21: ESD5Zxx, Diode_SMD:D_SOD-523, symbol Diode:ESD5Zxx
- added D20: GREEN, symbol Device:LED
- added J14: TEMP_PROBE, symbol Connector_Generic:Conn_01x02
- added JP5, JP6: ADDR, Jumper:SolderJumper-3_P1.3mm_Open_Pad1.0x1.5mm, symbol Jumper:SolderJumper_3_Open
- added Q8: Q_NMOS, symbol Device:Q_NMOS
- added R42, R44, R45, R47, R50: 10k, symbol Device:R
- added R43: 100R, symbol Device:R
- added R46, R48: 1k, symbol Device:R
- added R49: 500k, symbol Device:R
- added U7: (no value), footprints:LM82, symbol component_library:LM82
- added U8: BTH50015, Package_SO:Infineon_PG-TSDSO-14-22, symbol component_library:BTH50015
Connections:
- net CTRL: now also D20.2 (A), R48.2
- net GND: now also C25.2, C26.2, C27.2, C28.2, C29.2, C52.1, D19.2 (A), D21.2 (A), JP5.3 (B), JP6.3 (B), Q8.S, R44.2, R46.2, R47.1, R50.1, U7.7 (GND), U7.8 (GND), U8.1 (GND)
- net PWR_IN: now also C26.1, C27.1, U8.4 (DEN), U8.9 (VS)
- net PWR_OUT: now also C28.1, C29.1, R49.2, U8.5 (OUT), U8.6 (OUT), U8.7 (OUT), U8.8 (OUT)
- net V_sense: now also D21.1 (K), R49.1, R50.2
- net i_sense: now also C25.1, D19.1 (K), R45.1
- new net: Q8.G, R43.1, R44.1
- new net: D20.1 (K), R47.2
- new net: JP5.2 (C), U7.10 (ADDR0)
- new net: R45.2, R46.1, U8.2 (IS)
- new net: JP6.2 (C), U7.6 (ADDR1)
- new net: Q8.D, R42.1
- new net: R48.1, U8.3 (IN)
- new net: J14.2 (Pin_2), U7.3 (D+)
- new net: J14.1 (Pin_1), U7.4 (D-)
- new net: D18.1 (K), R42.2
- new net 3V3: C52.2, D18.2 (A), JP5.1 (A), JP6.1 (A), U7.2 (VCC)
- new net SCLK: U7.14 (SCLK)
- new net SDATA: U7.12 (SDATA)
- new net TEMP_ALARM_: R43.2, U7.16 (T_ALARM)
- new net TEMP_INT_: U7.11 (INT_)
- no-connect marks 0 -> 5
Other:
- note added: "1x02 pin header"
- note added: "5v varient needed"
- note added: "OVER TEMP"
- note added: "Use 2N3906 for external temp probe"
- note removed: "Add TVS"
- note removed: "Add TVS or Opto Coupler"
- note removed: "Check to make sure ADC of SBB has enough resolution"

Commit message: Bus routed
Parts:
- renumbered C52 to C28, C25 to C29, C26 to C30, C27 to C31, C28 to C32, C29 to C33, D to D15, D18 to D16, D19 to D17, D20 to D18, D21 to D19, J14 to J12, Q to Q10, Q8 to Q11, Q to Q9, R7 to R46, R5 to R47, R6 to R48, R to R49, R2 to R50, R3 to R51, R4 to R52, R42 to R53, R43 to R54, R44 to R55, R45 to R56, R46 to R57, R47 to R58, R48 to R59, R49 to R60, R50 to R61, U8 to U10, U7 to U9

Commit message: revamping channel switches
Parts:
- renumbered C28 to C22, C29 to C23, C30 to C24, C31 to C25, C32 to C26, C33 to C27, J12 to J13, R46 to R45, R47 to R46, R48 to R47, R49 to R48, R50 to R49, R51 to R50, R52 to R51, R53 to R52, R54 to R53, R55 to R54, R56 to R55, R57 to R56, R58 to R57, R59 to R58, R60 to R59, R61 to R60, U9 to U8, U10 to U9

Commit message: Minor fixes and sanity checks
Parts:
- removed C23, C24: 10nF, symbol Device:C
- removed C27: 100nF, symbol Device:C
- removed D18: GREEN, symbol Device:LED
- removed D19: ESD5Zxx, Diode_SMD:D_SOD-523, symbol Diode:ESD5Zxx
- removed R57, R60: 10k, symbol Device:R
- removed R58: 1k, symbol Device:R
- removed R59: 500k, symbol Device:R
- removed U9: BTH50015, Package_SO:Infineon_PG-TSDSO-14-22, symbol component_library:BTH50015
- added C27: C_Polarized, Capacitor_SMD:CP_Elec_10x10.5, symbol Device:C_Polarized
- added C28: 100nF, symbol Device:C
- added D16: GREEN, symbol Device:LED
- added F3: Blade, symbol Device:Fuse
- added Q14: CSD19533Q5A, Package_TO_SOT_SMD:TDSON-8-1, symbol Transistor_FET:CSD19533Q5A
- added R54: 10k, symbol Device:R
- added U11: LTC7001, Package_SO:MSOP-10-1EP_3x3mm_P0.5mm_EP1.68x1.88mm, symbol component_library:LTC7001
- added U12: ACS37003, Package_SO:SOIC-16W_7.5x10.3mm_P1.27mm, symbol component_library:ACS37003
- C26: value 10nF -> 0.1uF
- R55: value 10k -> 500k
- R56: value 1k -> 10k
- renumbered C22 to C24, D15 to D14, D16 to D15, J13 to J14, Q9 to Q11, Q10 to Q12, Q11 to Q13, R45 to R44, R46 to R45, R47 to R46, R48 to R47, R49 to R48, R50 to R49, R51 to R50, R52 to R51, R53 to R52, R54 to R53, U8 to U10
Connections:
- net i_sense is gone; now on net V_sense: D17.1 (K), R55.1
- net 3V3: now also C28.2, U12.13 (VCC)
- net CTRL: now also D16.2 (A), U11.4 (INP)
- net GND: now also C25.1, R56.1, C27.2, C28.1, R54.1, U11.11 (PAD), U11.2 (VCCUV), U11.3 (GND), U11.5 (OVLO), U12.16 (GND); no longer C25.2, C26.2, R56.2
- net PWR_IN: now also C27.1, Q14.5 (D); no longer C25.1
- net PWR_OUT: now also R55.2, F3.1; no longer C26.1
- net V_sense: now also R56.2
- net TEMP_INT_: no longer names the net of U10.11 (INT_)
- new net: C26.1, U11.9 (BST)
- new net: C26.2, U11.8 (TS)
- new net: Q14.1 (S), Q14.2 (S), Q14.3 (S), U12.1 (IP+), U12.2 (IP+), U12.3 (IP+), U12.4 (IP+)
- new net: Q14.4 (G), U11.6 (TGDN), U11.7 (TGUP)
- new net: C25.2, U11.1 (VCC)
- new net: F3.2, U12.5 (IP-), U12.6 (IP-), U12.7 (IP-), U12.8 (IP-)
- new net: D16.1 (K), R54.2
- new net VIOUT: U12.12 (VIOUT)
- new net VI_VREF: U12.11 (VREF)
- no-connect marks 5 -> 11
Other:
- note removed: "5v varient needed"
- note removed: "High precision needed"
