File: hardware/rover-control-board-v2/drive2_smart_switch.kicad_sch (KiCad schematic)
At the start: 23 parts, among them Q3 Q_NMOS_DGS, Q4 Q_PMOS_DGS, U2 BTH50015

Commit message: Buses added
Parts:
- removed C6: 10nF, symbol Device:C
- removed D3: RED, symbol Device:LED
- removed Q3: Q_NMOS_DGS, symbol Transistor_FET:Q_NMOS_DGS
- removed Q4: Q_PMOS_DGS, symbol Transistor_FET:Q_PMOS_DGS
- removed R17: 10R, symbol Device:R
- removed U2: BTH50015, Package_SO:Infineon_PG-TSDSO-14-22, symbol component_library:BTH50015
- added C: 10nF, symbol Device:C
- added D: RED, symbol Device:LED
- added Q: Q_PMOS_DGS, symbol Transistor_FET:Q_PMOS_DGS
- added Q: Q_NMOS_DGS, symbol Transistor_FET:Q_NMOS_DGS
- added R: 10R, symbol Device:R
- added U: BTH50015, Package_SO:Infineon_PG-TSDSO-14-22, symbol component_library:BTH50015
Connections:
- net GND: now also C.2, Q.3 (S), U.1 (GND)
- net PRE_EN: now also D.2 (A)
- net PWR_IN: now also R.1, U.4 (DEN), U.9 (VS)
- net PWR_OUT: now also Q.3 (S), U.5 (OUT), U.6 (OUT), U.7 (OUT), U.8 (OUT)
- net i_sense: now also C.1
- net at R4.1: now also Q.1 (D)
- net at R3.1, R4.2: now also Q.2 (G)
- net at R5.2, R6.2: now also Q.2 (G)
- net at R8.2, R9.1: now also U.2 (IS)
- net at R7.2: now also D.1 (K)
- net at R2.2, R3.2: now also Q.1 (D), R.2
- net at R10.1: now also U.3 (IN)

Commit message: Channels routed, temp bus pending
Parts:
- removed C, C2, C4: 10nF, symbol Device:C
- removed C3, C5: 100nF, symbol Device:C
- removed D2: GREEN, symbol Device:LED
- removed R10, R9: 1k, symbol Device:R
- removed R11, R13, R8: 10k, symbol Device:R
- removed R12: 500k, symbol Device:R
- removed U: BTH50015, Package_SO:Infineon_PG-TSDSO-14-22, symbol component_library:BTH50015
- added C35, C36, C38: 10nF, symbol Device:C
- added C37, C39, C54: 100nF, symbol Device:C
- added D26: RED, symbol Device:LED
- added D27, D29: ESD5Zxx, Diode_SMD:D_SOD-523, symbol Diode:ESD5Zxx
- added D28: GREEN, symbol Device:LED
- added J16: TEMP_PROBE, symbol Connector_Generic:Conn_01x02
- added JP10, JP9: ADDR, Jumper:SolderJumper-3_P1.3mm_Open_Pad1.0x1.5mm, symbol Jumper:SolderJumper_3_Open
- added Q10: Q_NMOS, symbol Device:Q_NMOS
- added R60, R62, R63, R65, R68: 10k, symbol Device:R
- added R61: 100R, symbol Device:R
- added R64, R66: 1k, symbol Device:R
- added R67: 500k, symbol Device:R
- added U11: (no value), footprints:LM82, symbol component_library:LM82
- added U12: BTH50015, Package_SO:Infineon_PG-TSDSO-14-22, symbol component_library:BTH50015
Connections:
- net CTRL: now also D28.2 (A), R66.2
- net GND: now also C35.2, C36.2, C37.2, C38.2, C39.2, C54.1, D27.2 (A), D29.2 (A), JP10.3 (B), JP9.3 (B), Q10.S, R62.2, R64.2, R65.1, R68.1, U11.7 (GND), U11.8 (GND), U12.1 (GND)
- net PWR_IN: now also C36.1, C37.1, U12.4 (DEN), U12.9 (VS)
- net PWR_OUT: now also C38.1, C39.1, R67.2, U12.5 (OUT), U12.6 (OUT), U12.7 (OUT), U12.8 (OUT)
- net V_sense: now also D29.1 (K), R67.1, R68.2
- net i_sense: now also C35.1, D27.1 (K), R63.1
- new net: R63.2, R64.1, U12.2 (IS)
- new net: J16.1 (Pin_1), U11.4 (D-)
- new net: J16.2 (Pin_2), U11.3 (D+)
- new net: R66.1, U12.3 (IN)
- new net: D28.1 (K), R65.2
- new net: JP9.2 (C), U11.10 (ADDR0)
- new net: JP10.2 (C), U11.6 (ADDR1)
- new net: Q10.G, R61.1, R62.1
- new net: Q10.D, R60.1
- new net: D26.1 (K), R60.2
- new net 3V3: C54.2, D26.2 (A), JP10.1 (A), JP9.1 (A), U11.2 (VCC)
- new net SCLK: U11.14 (SCLK)
- new net SDATA: U11.12 (SDATA)
- new net TEMP_ALARM_: R61.2, U11.16 (T_ALARM)
- new net TEMP_INT_: U11.11 (INT_)
- no-connect marks 0 -> 5
Other:
- note added: "1x02 pin header"
- note added: "5v varient needed"
- note added: "OVER TEMP"
- note added: "Use 2N3906 for external temp probe"
- note removed: "Add TVS"
- note removed: "Add TVS or Opto Coupler"
- note removed: "Check to make sure ADC of SBB has enough resolution"

Commit message: Bus routed
Parts:
- removed D: RED, symbol Device:LED
- removed Q: Q_PMOS_DGS, symbol Transistor_FET:Q_PMOS_DGS
- removed Q: Q_NMOS_DGS, symbol Transistor_FET:Q_NMOS_DGS
- removed R, R2: 10R, symbol Device:R
- removed R3, R4: 1k, symbol Device:R
- removed R5: 100, symbol Device:R
- removed R6: 4.7k, symbol Device:R
- removed R7: 10k, symbol Device:R
- added D25: RED, symbol Device:LED
- added Q15: Q_NMOS_DGS, symbol Transistor_FET:Q_NMOS_DGS
- added Q16: Q_PMOS_DGS, symbol Transistor_FET:Q_PMOS_DGS
- added R78: 10k, symbol Device:R
- added R79: 100, symbol Device:R
- added R80: 4.7k, symbol Device:R
- added R81, R82: 10R, symbol Device:R
- added R83, R84: 1k, symbol Device:R
- renumbered C54 to C40, C35 to C41, C36 to C42, C37 to C43, C38 to C44, C39 to C45, J16 to J14, Q10 to Q17, R60 to R85, R61 to R86, R62 to R87, R63 to R88, R64 to R89, R65 to R90, R66 to R91, R67 to R92, R68 to R93, U11 to U13, U12 to U14
Connections:
- net GND: now also Q15.3 (S), R78.1, R80.1
- net PRE_EN: now also D25.2 (A), R79.1
- net PWR_IN: now also R81.1, R82.1
- net PWR_OUT: now also Q16.3 (S)
- new net: Q15.2 (G), R79.2, R80.2
- new net: Q15.1 (D), R84.1
- new net: Q16.2 (G), R83.1, R84.2
- new net: D25.1 (K), R78.2
- new net: Q16.1 (D), R81.2, R82.2, R83.2

Commit message: revamping channel switches
Parts:
- renumbered C40 to C34, C41 to C35, C42 to C36, C43 to C37, C44 to C38, C45 to C39, J14 to J15, R78 to R77, R79 to R78, R80 to R79, R81 to R80, R82 to R81, R83 to R82, R84 to R83, R85 to R84, R86 to R85, R87 to R86, R88 to R87, R89 to R88, R90 to R89, R91 to R90, R92 to R91, R93 to R92, U13 to U12, U14 to U13

Commit message: Minor fixes and sanity checks
Parts:
- removed C37, C39: 100nF, symbol Device:C
- removed D27, D29: ESD5Zxx, Diode_SMD:D_SOD-523, symbol Diode:ESD5Zxx
- removed D28: GREEN, symbol Device:LED
- removed R87, R89, R92: 10k, symbol Device:R
- removed R88, R90: 1k, symbol Device:R
- removed R91: 500k, symbol Device:R
- removed U13: BTH50015, Package_SO:Infineon_PG-TSDSO-14-22, symbol component_library:BTH50015
- added C37: C_Polarized, Capacitor_SMD:CP_Elec_10x10.5, symbol Device:C_Polarized
- added D24: GREEN, symbol Device:LED
- added D25: ESD5Zxx, Diode_SMD:D_SOD-523, symbol Diode:ESD5Zxx
- added F5: Blade, symbol Device:Fuse
- added Q22: CSD19533Q5A, Package_TO_SOT_SMD:TDSON-8-1, symbol Transistor_FET:CSD19533Q5A
- added R80, R82: 10k, symbol Device:R
- added R81: 500k, symbol Device:R
- added U17: LTC7001, Package_SO:MSOP-10-1EP_3x3mm_P0.5mm_EP1.68x1.88mm, symbol component_library:LTC7001
- added U18: ACS37003, Package_SO:SOIC-16W_7.5x10.3mm_P1.27mm, symbol component_library:ACS37003
- C35, C38: value 10nF -> 100nF
- C36: value 10nF -> 0.1uF
- renumbered D25 to D22, D26 to D23, J15 to J16, Q15 to Q19, Q16 to Q20, Q17 to Q21, R77 to R70, R78 to R71, R79 to R72, R80 to R73, R81 to R74, R82 to R75, R83 to R76, R84 to R77, R85 to R78, R86 to R79, U12 to U16
Connections:
- net i_sense is gone; now on net GND: C35.1
- net 3V3: now also C38.2, U18.13 (VCC)
- net CTRL: now also D24.2 (A), U17.4 (INP)
- net GND: now also C38.1, C37.2, D25.2 (A), R80.1, R82.1, U17.11 (PAD), U17.2 (VCCUV), U17.3 (GND), U17.5 (OVLO), U18.16 (GND); no longer C35.2, C36.2, C38.2
- net PWR_IN: now also C37.1, Q22.5 (D); no longer C36.1
- net PWR_OUT: now also F5.1, R81.2; no longer C38.1
- net V_sense: now also D25.1 (K), R81.1, R82.2
- net TEMP_INT_: no longer names the net of U16.11 (INT_)
- new net: Q22.1 (S), Q22.2 (S), Q22.3 (S), U18.1 (IP+), U18.2 (IP+), U18.3 (IP+), U18.4 (IP+)
- new net: F5.2, U18.5 (IP-), U18.6 (IP-), U18.7 (IP-), U18.8 (IP-)
- new net: D24.1 (K), R80.2
- new net: C36.1, U17.9 (BST)
- new net: C36.2, U17.8 (TS)
- new net: Q22.4 (G), U17.6 (TGDN), U17.7 (TGUP)
- new net: C35.2, U17.1 (VCC)
- new net VIOUT: U18.12 (VIOUT)
- new net VI_VREF: U18.11 (VREF)
- no-connect marks 5 -> 11
Other:
- note removed: "5v varient needed"
- note removed: "High precision needed"
