File: hardware/rover-control-board-v2/ext_smart_switch.kicad_sch (KiCad schematic)
At the start: 23 parts, among them Q3 Q_NMOS_DGS, Q4 Q_PMOS_DGS, U2 BTH50015

Commit message: Buses added
Parts:
- removed C6: 10nF, symbol Device:C
- removed D3: RED, symbol Device:LED
- removed Q3: Q_NMOS_DGS, symbol Transistor_FET:Q_NMOS_DGS
- removed Q4: Q_PMOS_DGS, symbol Transistor_FET:Q_PMOS_DGS
- removed R17: 10R, symbol Device:R
- removed U2: BTH50015, Package_SO:Infineon_PG-TSDSO-14-22, symbol component_library:BTH50015
- added C: 10nF, symbol Device:C
- added D: RED, symbol Device:LED
- added Q: Q_PMOS_DGS, symbol Transistor_FET:Q_PMOS_DGS
- added Q: Q_NMOS_DGS, symbol Transistor_FET:Q_NMOS_DGS
- added R: 10R, symbol Device:R
- added U: BTH50015, Package_SO:Infineon_PG-TSDSO-14-22, symbol component_library:BTH50015
Connections:
- net GND: now also C.2, Q.3 (S), U.1 (GND)
- net PRE_EN: now also D.2 (A)
- net PWR_IN: now also R.1, U.4 (DEN), U.9 (VS)
- net PWR_OUT: now also Q.3 (S), U.5 (OUT), U.6 (OUT), U.7 (OUT), U.8 (OUT)
- net i_sense: now also C.1
- net at R4.1: now also Q.1 (D)
- net at R3.1, R4.2: now also Q.2 (G)
- net at R5.2, R6.2: now also Q.2 (G)
- net at R8.2, R9.1: now also U.2 (IS)
- net at R7.2: now also D.1 (K)
- net at R2.2, R3.2: now also Q.1 (D), R.2
- net at R10.1: now also U.3 (IN)

Commit message: Channels routed, temp bus pending
Parts:
- removed C, C2, C4: 10nF, symbol Device:C
- removed C3, C5: 100nF, symbol Device:C
- removed D2: GREEN, symbol Device:LED
- removed R10, R9: 1k, symbol Device:R
- removed R11, R13, R8: 10k, symbol Device:R
- removed R12: 500k, symbol Device:R
- removed U: BTH50015, Package_SO:Infineon_PG-TSDSO-14-22, symbol component_library:BTH50015
- added C40, C41, C43: 10nF, symbol Device:C
- added C42, C44, C55: 100nF, symbol Device:C
- added D30: RED, symbol Device:LED
- added D31, D33: ESD5Zxx, Diode_SMD:D_SOD-523, symbol Diode:ESD5Zxx
- added D32: GREEN, symbol Device:LED
- added J17: TEMP_PROBE, symbol Connector_Generic:Conn_01x02
- added JP11, JP12: ADDR, Jumper:SolderJumper-3_P1.3mm_Open_Pad1.0x1.5mm, symbol Jumper:SolderJumper_3_Open
- added Q11: Q_NMOS, symbol Device:Q_NMOS
- added R69, R71, R72, R74, R77: 10k, symbol Device:R
- added R70: 100R, symbol Device:R
- added R73, R75: 1k, symbol Device:R
- added R76: 500k, symbol Device:R
- added U13: (no value), footprints:LM82, symbol component_library:LM82
- added U14: BTH50015, Package_SO:Infineon_PG-TSDSO-14-22, symbol component_library:BTH50015
Connections:
- net CTRL: now also D32.2 (A), R75.2
- net GND: now also C40.2, C41.2, C42.2, C43.2, C44.2, C55.1, D31.2 (A), D33.2 (A), JP11.3 (B), JP12.3 (B), Q11.S, R71.2, R73.2, R74.1, R77.1, U13.7 (GND), U13.8 (GND), U14.1 (GND)
- net PWR_IN: now also C41.1, C42.1, U14.4 (DEN), U14.9 (VS)
- net PWR_OUT: now also C43.1, C44.1, R76.2, U14.5 (OUT), U14.6 (OUT), U14.7 (OUT), U14.8 (OUT)
- net V_sense: now also D33.1 (K), R76.1, R77.2
- net i_sense: now also C40.1, D31.1 (K), R72.1
- new net: D30.1 (K), R69.2
- new net: R72.2, R73.1, U14.2 (IS)
- new net: Q11.D, R69.1
- new net: Q11.G, R70.1, R71.1
- new net: D32.1 (K), R74.2
- new net: R75.1, U14.3 (IN)
- new net: JP11.2 (C), U13.10 (ADDR0)
- new net: JP12.2 (C), U13.6 (ADDR1)
- new net: J17.1 (Pin_1), U13.4 (D-)
- new net: J17.2 (Pin_2), U13.3 (D+)
- new net 3V3: C55.2, D30.2 (A), JP11.1 (A), JP12.1 (A), U13.2 (VCC)
- new net SCLK: U13.14 (SCLK)
- new net SDATA: U13.12 (SDATA)
- new net TEMP_ALARM_: R70.2, U13.16 (T_ALARM)
- new net TEMP_INT_: U13.11 (INT_)
- no-connect marks 0 -> 5
Other:
- note added: "1x02 pin header"
- note added: "5v varient needed"
- note added: "OVER TEMP"
- note added: "Use 2N3906 for external temp probe"
- note removed: "Add TVS"
- note removed: "Add TVS or Opto Coupler"
- note removed: "Check to make sure ADC of SBB has enough resolution"

Commit message: Bus routed
Parts:
- renumbered C55 to C46, C40 to C47, C41 to C48, C42 to C49, C43 to C50, C44 to C51, D to D30, D30 to D31, D31 to D32, D32 to D33, D33 to D34, J17 to J15, Q to Q18, Q to Q19, Q11 to Q20, R4 to R100, R69 to R101, R70 to R102, R71 to R103, R72 to R104, R73 to R105, R74 to R106, R75 to R107, R76 to R108, R77 to R109, R7 to R94, R5 to R95, R6 to R96, R to R97, R2 to R98, R3 to R99, U13 to U15, U14 to U16

Commit message: revamping channel switches
Parts:
- renumbered C46 to C40, C47 to C41, C48 to C42, C49 to C43, C50 to C44, C51 to C45, J15 to J16, R101 to R100, R102 to R101, R103 to R102, R104 to R103, R105 to R104, R106 to R105, R107 to R106, R108 to R107, R109 to R108, R94 to R93, R95 to R94, R96 to R95, R97 to R96, R98 to R97, R99 to R98, R100 to R99, U15 to U14, U16 to U15

Commit message: Minor fixes and sanity checks
Parts:
- removed C42, C44: 10nF, symbol Device:C
- removed C45: 100nF, symbol Device:C
- removed D32, D34: ESD5Zxx, Diode_SMD:D_SOD-523, symbol Diode:ESD5Zxx
- removed D33: GREEN, symbol Device:LED
- removed R103, R105, R108: 10k, symbol Device:R
- removed R104, R106: 1k, symbol Device:R
- removed R107: 500k, symbol Device:R
- removed U15: BTH50015, Package_SO:Infineon_PG-TSDSO-14-22, symbol component_library:BTH50015
- added C40: 100nF, symbol Device:C
- added C42: C_Polarized, Capacitor_SMD:CP_Elec_10x10.5, symbol Device:C_Polarized
- added D28: GREEN, symbol Device:LED
- added D29: ESD5Zxx, Diode_SMD:D_SOD-523, symbol Diode:ESD5Zxx
- added F6: Blade, symbol Device:Fuse
- added Q26: CSD19533Q5A, Package_TO_SOT_SMD:TDSON-8-1, symbol Transistor_FET:CSD19533Q5A
- added R93, R95: 10k, symbol Device:R
- added R94: 500k, symbol Device:R
- added U20: LTC7001, Package_SO:MSOP-10-1EP_3x3mm_P0.5mm_EP1.68x1.88mm, symbol component_library:LTC7001
- added U21: ACS37003, Package_SO:SOIC-16W_7.5x10.3mm_P1.27mm, symbol component_library:ACS37003
- C41: value 10nF -> 0.1uF
- renumbered C40 to C39, D30 to D26, D31 to D27, J16 to J17, Q18 to Q23, Q19 to Q24, Q20 to Q25, R93 to R83, R94 to R84, R95 to R85, R96 to R86, R97 to R87, R98 to R88, R99 to R89, R100 to R90, R101 to R91, R102 to R92, U14 to U19
Connections:
- net 3V3: now also C43.2, U21.13 (VCC)
- net CTRL: now also D28.2 (A), U20.4 (INP)
- net GND: now also C43.1, C40.1, C42.2, D29.2 (A), R93.1, R95.1, U20.11 (PAD), U20.2 (VCCUV), U20.3 (GND), U20.5 (OVLO), U21.16 (GND); no longer C41.2, C43.2
- net PWR_IN: now also C42.1, Q26.5 (D); no longer C43.1
- net PWR_OUT: now also F6.1, R94.2
- net V_sense: now also D29.1 (K), R94.1, R95.2
- net TEMP_INT_: no longer names the net of U19.11 (INT_)
- net i_sense: no longer names the net of C41.1
- net i_sense: now also U20.9 (BST)
- new net: Q26.1 (S), Q26.2 (S), Q26.3 (S), U21.1 (IP+), U21.2 (IP+), U21.3 (IP+), U21.4 (IP+)
- new net: Q26.4 (G), U20.6 (TGDN), U20.7 (TGUP)
- new net: C40.2, U20.1 (VCC)
- new net: C41.2, U20.8 (TS)
- new net: F6.2, U21.5 (IP-), U21.6 (IP-), U21.7 (IP-), U21.8 (IP-)
- new net: D28.1 (K), R93.2
- new net VIOUT: U21.12 (VIOUT)
- new net VI_VREF: U21.11 (VREF)
- no-connect marks 5 -> 11
Other:
- note removed: "5v varient needed"
- note removed: "High precision needed"
