File: hardware/rover-control-board-v2/rover-control-board-v2.kicad_pcb (KiCad board)
At the start: 2 copper layers, 0 parts

Commit message: Added photovoltaic gate driver and ESD protection
Parts:
- added G***: LOGO, LOGO, F.Cu at (133.2, 86.2)
