File: hardware/rover-control-board-v2/rover-control-board-v2.kicad_pcb (KiCad board)
At the start: 2 copper layers, 101 parts, among them J10 M8 receptacle, J11 Contactor, J12 TEMP_PROBE, J13 XT90, J14 EXT_I_SENSE, J15 XT90_PWR, J3 XT90_REG_OUT, J5 XT90_REG_RET, J6 CAN1, J7 CAN1, J8 CAN1, J9 M8 receptacle, Q2 CSD19533Q5A, Q6 CSD19533Q5A, Q7 Q_PMOS_GDS, U10 MCP3427x-xUN, U11 MCP3427x-xUN, U4 LM82, U6 ACS37003, U7 VOM1271T, U9 MCP3427x-xUN

Commit message: Initial component placement, finalising schematic
Parts:
- removed J3: XT90_REG_OUT, footprints:AMASS_XT90-F_1x02_P11.00mm_Vertical
- removed J5: XT90_REG_RET, footprints:AMASS_XT90-F_1x02_P11.00mm_Vertical
- removed RED1: 5991110147F, LED_SMD:LED_0805_2012Metric
- added C1: 4.7nF, Capacitor_SMD:C_0603_1608Metric, F.Cu at (-21.1, 62.6)
- added C15: 100nF, Capacitor_SMD:C_0603_1608Metric, F.Cu at (-21.1, 65.1)
- added C16: 1uF, Capacitor_SMD:C_0603_1608Metric, F.Cu at (-21.1, 67.6)
- added C21: 22uF, Capacitor_SMD:C_0603_1608Metric, F.Cu at (-21.1, 70.2)
- added C22: 22uF, Capacitor_SMD:C_0603_1608Metric, F.Cu at (-21.1, 72.7)
- added C23: 100nF, Capacitor_SMD:C_0603_1608Metric, F.Cu at (-36.8, 45.6)
- added C24: C_Polarized, Capacitor_SMD:CP_Elec_10x10.5, F.Cu at (-50.3, 42.7)
- added C25: 100nF, Capacitor_SMD:C_0603_1608Metric, F.Cu at (-36.8, 48.1)
- added C26: 100nF, Capacitor_SMD:C_0603_1608Metric, F.Cu at (-79.6, 90.3)
- added C27: 100nF, Capacitor_SMD:C_0603_1608Metric, F.Cu at (-36.8, 50.6)
- added C28: C_Polarized, Capacitor_SMD:CP_Elec_10x10.5, F.Cu at (-93.2, 87.5)
- added C29: 100nF, Capacitor_SMD:C_0603_1608Metric, F.Cu at (-79.6, 92.8)
- added C30: 100nF, Capacitor_SMD:C_0603_1608Metric, F.Cu at (-79.6, 95.3)
- added C31: 100nF, Capacitor_SMD:C_0603_1608Metric, F.Cu at (-79.6, 45.6)
- added C32: C_Polarized, Capacitor_SMD:CP_Elec_10x10.5, F.Cu at (-93.2, 42.7)
- added C33: 100nF, Capacitor_SMD:C_0603_1608Metric, F.Cu at (-79.6, 48.1)
- added C34: 100nF, Capacitor_SMD:C_0603_1608Metric, F.Cu at (-79.6, 50.6)
- added F2: Blade, Fuse:Fuseholder_Keystone_3555-2, F.Cu at (-53.7, 20.4)
- added F3: Blade, Fuse:Fuseholder_Keystone_3555-2, F.Cu at (-96.5, 65.1)
- added F4: Blade, Fuse:Fuseholder_Keystone_3555-2, F.Cu at (-96.5, 20.4)
- added F7: 2A, Fuse:Fuse_2920_7451Metric_Pad2.10x5.45mm_HandSolder, F.Cu at (-36.6, 98.3)
- added GREEN3: 350-599, LED_SMD:LED_0805_2012Metric, F.Cu at (-41.6, 50.3)
- added GREEN4: 350-599, LED_SMD:LED_0805_2012Metric, F.Cu at (-84.5, 95.0)
- added GREEN5: 350-599, LED_SMD:LED_0805_2012Metric, F.Cu at (-84.5, 50.3)
- added J13: TEMP_PROBE, Connector_JST:JST_XH_B2B-XH-A_1x02_P2.50mm_Vertical, F.Cu at (-23.1, 39.5)
- added J14: TEMP_PROBE, Connector_JST:JST_XH_B2B-XH-A_1x02_P2.50mm_Vertical, F.Cu at (-66.0, 84.2)
- added J16: TEMP_PROBE, Connector_JST:JST_XH_B2B-XH-A_1x02_P2.50mm_Vertical, F.Cu at (-66.0, 39.5)
- added JP10: ADDR2, Jumper:SolderJumper-3_P1.3mm_Open_Pad1.0x1.5mm, F.Cu at (-46.7, 54.4)
- added JP11: ADDR1, Jumper:SolderJumper-3_P1.3mm_Open_Pad1.0x1.5mm, F.Cu at (-89.5, 95.3)
- added JP12: ADDR2, Jumper:SolderJumper-3_P1.3mm_Open_Pad1.0x1.5mm, F.Cu at (-89.5, 99.1)
- added JP13: ADDR, Jumper:SolderJumper-3_P1.3mm_Open_Pad1.0x1.5mm, F.Cu at (-35.9, 86.2)
- added JP14: ADDR, Jumper:SolderJumper-3_P1.3mm_Open_Pad1.0x1.5mm, F.Cu at (-35.9, 90.1)
- added JP15: ADDR1, Jumper:SolderJumper-3_P1.3mm_Open_Pad1.0x1.5mm, F.Cu at (-89.5, 50.5)
- added JP16: ADDR2, Jumper:SolderJumper-3_P1.3mm_Open_Pad1.0x1.5mm, F.Cu at (-89.5, 54.4)
- added JP9: ADDR1, Jumper:SolderJumper-3_P1.3mm_Open_Pad1.0x1.5mm, F.Cu at (-46.7, 50.5)
- added MP1: Redcube Press Fit, footprints:MP_Wurth_WP-BUFU_7461097, F.Cu at (88.1, 49.7)
- added MP2: Redcube Press Fit, footprints:MP_Wurth_WP-BUFU_7461097, F.Cu at (100.6, 49.6)
- added MP3: Redcube Press Fit, footprints:MP_Wurth_WP-BUFU_7461097, F.Cu at (92.7, 135.8)
- added MP4: Redcube Press Fit, footprints:MP_Wurth_WP-BUFU_7461097, F.Cu at (135.5, 134.8)
- added MP5: Redcube Press Fit, footprints:MP_Wurth_WP-BUFU_7461097, F.Cu at (172.4, 134.6)
- added MP6: Redcube Press Fit, footprints:MP_Wurth_WP-BUFU_7461097, F.Cu at (204.3, 134.1)
- added PRE1: 5991110147F, LED_SMD:LED_0805_2012Metric, F.Cu at (79.0, 133.2)
- added PRE2: 5991110147F, LED_SMD:LED_0805_2012Metric, F.Cu at (8.20, 1.02)
- added PRE3: 5991110147F, LED_SMD:LED_0805_2012Metric, F.Cu at (8.20, 6.06)
- added PRE4: 5991110147F, LED_SMD:LED_0805_2012Metric, F.Cu at (1.75, 1.02)
- added Q1: NMOS_GDS, Package_TO_SOT_SMD:SOT-223, F.Cu at (82.9, 126.0)
- added Q10: Q_PMOS_GDS, Package_TO_SOT_SMD:TO-252-2, F.Cu at (-31.8, 40.3)
- added Q11: CSD19533Q5A, Package_TO_SOT_SMD:TDSON-8-1, F.Cu at (-53.6, 52.1)
- added Q12: NMOS_GDS, Package_TO_SOT_SMD:SOT-223, F.Cu at (-64.7, 93.3)
- added Q13: PMOS, Package_TO_SOT_SMD:SOT-323_SC-70, F.Cu at (-98.6, 101.9)
- added Q14: Q_PMOS_GDS, Package_TO_SOT_SMD:TO-252-2, F.Cu at (-74.7, 85.0)
- added Q15: CSD19533Q5A, Package_TO_SOT_SMD:TDSON-8-1, F.Cu at (-96.5, 96.9)
- added Q16: NMOS_GDS, Package_TO_SOT_SMD:SOT-223, F.Cu at (-64.7, 48.5)
- added Q17: PMOS, Package_TO_SOT_SMD:SOT-323_SC-70, F.Cu at (-98.6, 57.2)
- added Q18: Q_PMOS_GDS, Package_TO_SOT_SMD:TO-252-2, F.Cu at (-74.7, 40.3)
- added Q19: CSD19533Q5A, Package_TO_SOT_SMD:TDSON-8-1, F.Cu at (-96.5, 52.1)
- added Q3: NMOS_GDS, Package_TO_SOT_SMD:SOT-223, F.Cu at (-37.0, 106.0)
- added Q4: Q_PMOS_GDS, Package_TO_SOT_SMD:TO-252-2, F.Cu at (83.8, 134.7)
- added Q5: PMOS, Package_TO_SOT_SMD:SOT-323_SC-70, F.Cu at (72.6, 162.4)
- added Q8: NMOS_GDS, Package_TO_SOT_SMD:SOT-223, F.Cu at (-21.8, 48.5)
- added Q9: PMOS, Package_TO_SOT_SMD:SOT-323_SC-70, F.Cu at (-55.8, 57.2)
- added R3: 62R, Capacitor_SMD:C_0603_1608Metric, F.Cu at (-21.1, 75.2)
- added R32: 10k, Resistor_SMD:R_0603_1608Metric, F.Cu at (-36.8, 53.1)
- added R33: 100R, Resistor_SMD:R_0603_1608Metric, F.Cu at (-36.8, 55.6)
- added R34: 10R, footprints:RES_PWR263S-35-10R0F, F.Cu at (-48.0, 30.4)
- added R35: 4.7k, Resistor_SMD:R_0603_1608Metric, F.Cu at (-36.8, 58.1)
- added R36: 10k, Resistor_SMD:R_0603_1608Metric, F.Cu at (-32.7, 45.6)
- added R37: 1k, Resistor_SMD:R_0603_1608Metric, F.Cu at (-32.7, 48.1)
- added R38: 1k, Resistor_SMD:R_0603_1608Metric, F.Cu at (-32.7, 50.6)
- added R39: 100R, Resistor_SMD:R_0603_1608Metric, F.Cu at (-32.7, 53.1)
- added R4: 62R, Capacitor_SMD:C_0603_1608Metric, F.Cu at (-21.1, 77.7)
- added R40: 10k, Resistor_SMD:R_0603_1608Metric, F.Cu at (-32.7, 55.6)
- added R41: 10k, Resistor_SMD:R_0603_1608Metric, F.Cu at (-32.7, 58.1)
- added R42: 200R, Resistor_SMD:R_0603_1608Metric, F.Cu at (-28.7, 45.6)
- added R43: 10k, Resistor_SMD:R_0603_1608Metric, F.Cu at (-79.6, 97.8)
- added R44: 20k, Resistor_SMD:R_0603_1608Metric, F.Cu at (-28.7, 48.1)
- added R45: 1k, Resistor_SMD:R_0603_1608Metric, F.Cu at (-28.7, 50.6)
- added R46: 100R, Resistor_SMD:R_0603_1608Metric, F.Cu at (-79.6, 100.4)
- added R47: 10R, footprints:RES_PWR263S-35-10R0F, F.Cu at (-90.9, 75.2)
- added R48: 4.7k, Resistor_SMD:R_0603_1608Metric, F.Cu at (-79.6, 102.9)
- added R49: 10k, Resistor_SMD:R_0603_1608Metric, F.Cu at (-75.6, 90.3)
- added R50: 1k, Resistor_SMD:R_0603_1608Metric, F.Cu at (-75.6, 92.8)
- added R51: 1k, Resistor_SMD:R_0603_1608Metric, F.Cu at (-75.6, 95.3)
- added R52: 100R, Resistor_SMD:R_0603_1608Metric, F.Cu at (-75.6, 97.8)
- added R53: 10k, Resistor_SMD:R_0603_1608Metric, F.Cu at (-75.6, 100.4)
- added R54: 10k, Resistor_SMD:R_0603_1608Metric, F.Cu at (-75.6, 102.9)
- added R55: 200R, Resistor_SMD:R_0603_1608Metric, F.Cu at (-71.6, 90.3)
- added R56: 20k, Resistor_SMD:R_0603_1608Metric, F.Cu at (-71.6, 92.8)
- added R57: 1k, Resistor_SMD:R_0603_1608Metric, F.Cu at (-71.6, 95.3)
- added R58: 10k, Resistor_SMD:R_0603_1608Metric, F.Cu at (-79.6, 53.1)
- added R59: 100R, Resistor_SMD:R_0603_1608Metric, F.Cu at (-79.6, 55.6)
- added R60: 10R, footprints:RES_PWR263S-35-10R0F, F.Cu at (-90.9, 30.4)
- added R61: 4.7k, Resistor_SMD:R_0603_1608Metric, F.Cu at (-79.6, 58.1)
- added R62: 10k, Resistor_SMD:R_0603_1608Metric, F.Cu at (-75.6, 45.6)
- added R63: 1k, Resistor_SMD:R_0603_1608Metric, F.Cu at (-75.6, 48.1)
- added R64: 1k, Resistor_SMD:R_0603_1608Metric, F.Cu at (-75.6, 50.6)
- added R65: 100R, Resistor_SMD:R_0603_1608Metric, F.Cu at (-75.6, 53.1)
- added R66: 10k, Resistor_SMD:R_0603_1608Metric, F.Cu at (-75.6, 55.6)
- added R67: 10k, Resistor_SMD:R_0603_1608Metric, F.Cu at (-75.6, 58.1)
- added R68: 200R, Resistor_SMD:R_0603_1608Metric, F.Cu at (-71.6, 45.6)
- added R69: 20k, Resistor_SMD:R_0603_1608Metric, F.Cu at (-71.6, 48.1)
- added R70: 1k, Resistor_SMD:R_0603_1608Metric, F.Cu at (-71.6, 50.6)
- added RED4: 5991110147F, LED_SMD:LED_0805_2012Metric, F.Cu at (-41.6, 56.4)
- added RED6: 5991110147F, LED_SMD:LED_0805_2012Metric, F.Cu at (-84.5, 101.1)
- added RED8: 5991110147F, LED_SMD:LED_0805_2012Metric, F.Cu at (-84.5, 56.4)
- added U12: MCP1792x-5002xDB, Package_TO_SOT_SMD:SOT-223-3_TabPin2, F.Cu at (-52.8, 88.7)
- added U13: LM82, footprints:LM82, F.Cu at (-21.5, 27.4)
- added U14: VOM1271T, Package_SO:SOP-4_3.8x4.1mm_P2.54mm, F.Cu at (-22.5, 55.5)
- added U15: ACS37003, Package_SO:SOIC-16W_7.5x10.3mm_P1.27mm, F.Cu at (-32.3, 30.2)
- added U16: LM82, footprints:LM82, F.Cu at (-64.4, 72.1)
- added U17: D3V3M1U2S9-7, Diode_SMD:D_SOD-882, F.Cu at (-52.4, 56.6)
- added U18: VOM1271T, Package_SO:SOP-4_3.8x4.1mm_P2.54mm, F.Cu at (-65.3, 100.2)
- added U19: ACS37003, Package_SO:SOIC-16W_7.5x10.3mm_P1.27mm, F.Cu at (-75.2, 75.0)
- added U20: D3V3M1U2S9-7, Diode_SMD:D_SOD-882, F.Cu at (-95.3, 101.4)
- added U21: LM82, footprints:LM82, F.Cu at (-64.4, 27.4)
- added U22: VOM1271T, Package_SO:SOP-4_3.8x4.1mm_P2.54mm, F.Cu at (-65.3, 55.5)
- added U23: ACS37003, Package_SO:SOIC-16W_7.5x10.3mm_P1.27mm, F.Cu at (-75.2, 30.2)
- added U24: D3V3M1U2S9-7, Diode_SMD:D_SOD-882, F.Cu at (-95.3, 56.6)
- added U3: ADC128D818, Package_SO:TSSOP-16_4.4x5mm_P0.65mm, F.Cu at (-43.1, 87.8)
- C4: value 0.1uF -> 100nF; footprint Capacitor_SMD:C_0402_1005Metric -> Capacitor_SMD:C_0603_1608Metric
- JP1: value ADDR -> ADDR1
- JP2: value ADDR -> ADDR2
- R19, R96: value 100 -> 100R
- R6: value 50k -> 20k
- R8: footprint Resistor_SMD:R_0402_1005Metric -> Capacitor_SMD:C_0603_1608Metric
- U1: value ~ -> max6496
- U10, U11, U9: value MCP3427x-xUN -> MCP3427T-E/UN; footprint Package_SO:MSOP-10_3x3mm_P0.5mm -> Package_SO:SOP-4_3.8x4.1mm_P2.54mm
- U2, U8: value ~ -> D3V3M1U2S9-7
- U7: footprint footprints:SOIC254P695X242-4N -> Package_SO:SOP-4_3.8x4.1mm_P2.54mm
- moved J13 261.7 mm to (-208.1, 140.6)
- moved R1 260.9 mm to (-197.9, 48.2)
- moved R10 260.9 mm to (-197.9, 63.3)
- moved R2 260.9 mm to (-197.9, 50.7)
- moved R5 260.9 mm to (-197.9, 53.2)
- moved R6 260.9 mm to (-197.9, 55.8)
- moved R7 260.9 mm to (-197.9, 58.3)
- moved R9 260.9 mm to (-197.9, 60.8)
- moved 3V1 260.9 mm to (-189.8, 49.0)
- moved 3V3_IND1 260.9 mm to (-201.6, 66.1)
- moved 3V3_IND2 260.9 mm to (-201.6, 69.1)
- moved 3V3_IND4 260.9 mm to (-201.6, 75.2)
- moved C11 260.9 mm to (-170.1, 17.1)
- moved C12 260.9 mm to (-170.1, 19.6)
- moved C13 260.9 mm to (-170.1, 22.1)
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- renumbered 3V3_IND3 to PWR_IND3
Connections:
- net /JMP_PWR renamed Net-(3V3_IND4-A)
- R21 pad 2: Net-(J14-Pin_3) -> Net-(Q4-D)
- R23 pad 2: Net-(J14-Pin_3) -> Net-(Q4-D)
Other:
- board outline added: 150 x 100 mm
- copper layers 2 -> 4

Commit message: More placements
Parts:
- moved 3V1 278.4 mm to (88.4, 59.4)
- moved 3V3_IND1 278.4 mm to (76.6, 76.4)
- moved 3V3_IND2 278.4 mm to (76.6, 79.5)
- moved 3V3_IND4 278.4 mm to (76.6, 85.5)
- moved C2 278.4 mm to (76.4, 58.6)
- moved C20 278.4 mm to (76.4, 71.1)
- moved C3 278.4 mm to (76.4, 61.1)
- moved C4 278.4 mm to (88.4, 86.1)
- moved C44 278.4 mm to (102.5, 58.6)
- moved C5 278.4 mm to (76.4, 63.6)
- moved C50 278.4 mm to (76.4, 73.6)
- moved C6 278.4 mm to (76.4, 66.1)
- moved C7 278.4 mm to (76.4, 68.6)
- moved D2 278.4 mm to (94.5, 59.6)
- moved D3 278.4 mm to (94.5, 64.2)
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