File: hardware/rover-control-board-v2/current_adc.kicad_sch (KiCad schematic)
At the start: 15 parts, among them U10 MCP3427x-xUN, U11 MCP3427x-xUN, U9 MCP3427x-xUN

Commit message: BOM
Parts:
- C11, C8, C9: digikey_part_num (none) -> 311-1344-1-ND
- C12, C13, C19: digikey_part_num (none) -> 399-C0603X103K1RAC3121CT-ND
Changed lines of the file:
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@@
+			)
+		)
+		(property "digikey_part_num" "399-C0603X103K1RAC3121CT-ND"
+			(at 266.7 104.14 0)
+			(hide yes)
+			(show_name no)
+			(do_not_autoplace no)
+			(effects
+				(font
+					(size 1.27 1.27)
+				)
 			)
 		)
@@
 			)
 		)
+		(property "digikey_part_num" "399-C0603X103K1RAC3121CT-ND"
+			(at 146.05 104.14 0)
+			(hide yes)
+			(show_name no)
+			(do_not_autoplace no)
+			(effects
+				(font
+					(size 1.27 1.27)
+				)
+			)
+		)
 		(pin "2"
 		)
@@
 			)
 		)
+		(property "digikey_part_num" "311-1344-1-ND"
+			(at 194.31 104.14 0)
+			(hide yes)
+			(show_name no)
+			(do_not_autoplace no)
+			(effects
+				(font
+					(size 1.27 1.27)
+				)
+			)
+		)
 		(pin "2"
 		)
@@
 			)
 		)
+		(property "digikey_part_num" "311-1344-1-ND"
+			(at 256.54 104.14 0)
+			(hide yes)
+			(show_name no)
+			(do_not_autoplace no)
+			(effects
+				(font
+					(size 1.27 1.27)
+				)
+			)
+		)
 		(pin "2"
 		)
@@
 			)
 		)
+		(property "digikey_part_num" "399-C0603X103K1RAC3121CT-ND"
+			(at 204.47 104.14 0)
+			(hide yes)
+			(show_name no)
+			(do_not_autoplace no)
+			(effects
+				(font
+					(size 1.27 1.27)
+				)
+			)
+		)
 		(pin "2"
 		)
@@
 			(at 135.89 104.14 0)
 			(hide yes)
+			(show_name no)
+			(do_not_autoplace no)
+			(effects
+				(font
+					(size 1.27 1.27)
+				)
+			)
+		)
+		(property "digikey_part_num" "311-1344-1-ND"
+			(at 135.89 104.14 0)
+			(hide yes)

Commit message: Finished BOM
Parts:
- U10, U11, U9: value MCP3427x-xUN -> MCP3427T-E/UN; footprint Package_SO:MSOP-10_3x3mm_P0.5mm -> Package_SO:SOP-4_3.8x4.1mm_P2.54mm; digikey_part_num (none) -> 150-MCP3427T-E/UNCT-ND
Changed lines of the file:
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@@
 			)
 		)
-		(property "Value" "MCP3427x-xUN"
+		(property "Value" "MCP3427T-E/UN"
 			(at 258.6833 110.49 0)
 			(show_name no)
@@
 			)
 		)
-		(property "Footprint" "Package_SO:MSOP-10_3x3mm_P0.5mm"
+		(property "Footprint" "Package_SO:SOP-4_3.8x4.1mm_P2.54mm"
 			(at 276.86 129.54 0)
 			(hide yes)
@@
 		)
 		(property "Description" "16-Bit, Multi-Channel ΔΣ Analog-to-Digital Converter with I2C Interface and On-Board Reference, MSOP-10"
+			(at 256.54 120.65 0)
+			(hide yes)
+			(show_name no)
+			(do_not_autoplace no)
+			(effects
+				(font
+					(size 1.27 1.27)
+				)
+			)
+		)
+		(property "digikey_part_num" "150-MCP3427T-E/UNCT-ND"
 			(at 256.54 120.65 0)
 			(hide yes)
@@
 			)
 		)
-		(property "Value" "MCP3427x-xUN"
+		(property "Value" "MCP3427T-E/UN"
 			(at 196.4533 110.49 0)
 			(show_name no)
@@
 			)
 		)
-		(property "Footprint" "Package_SO:MSOP-10_3x3mm_P0.5mm"
+		(property "Footprint" "Package_SO:SOP-4_3.8x4.1mm_P2.54mm"
 			(at 214.63 129.54 0)
 			(hide yes)
@@
 		)
 		(property "Description" "16-Bit, Multi-Channel ΔΣ Analog-to-Digital Converter with I2C Interface and On-Board Reference, MSOP-10"
+			(at 194.31 120.65 0)
+			(hide yes)
+			(show_name no)
+			(do_not_autoplace no)
+			(effects
+				(font
+					(size 1.27 1.27)
+				)
+			)
+		)
+		(property "digikey_part_num" "150-MCP3427T-E/UNCT-ND"
 			(at 194.31 120.65 0)
 			(hide yes)
@@
 			)
 		)
-		(property "Value" "MCP3427x-xUN"
+		(property "Value" "MCP3427T-E/UN"
 			(at 138.0333 110.49 0)
 			(show_name no)
@@
 			)
 		)
-		(property "Footprint" "Package_SO:MSOP-10_3x3mm_P0.5mm"
+		(property "Footprint" "Package_SO:SOP-4_3.8x4.1mm_P2.54mm"
 			(at 156.21 129.54 0)
 			(hide yes)
@@
 			(at 135.89 120.65 0)
 			(hide yes)
+			(show_name no)
+			(do_not_autoplace no)
+			(effects
+				(font
+					(size 1.27 1.27)
+				)
+			)
+		)
+		(property "digikey_part_num" "150-MCP3427T-E/UNCT-ND"
+			(at 135.89 120.65 0)
+			(hide yes)
