File: hardware/rover-control-board-v2/rover-control-board-v2.kicad_sch (KiCad schematic)
At the start: 55 parts, among them J10 M8 receptacle, J11 Contactor, J15 XT90_PWR, J2 RET, J4 OUT, J6 CAN1, J7 CAN1, J8 CAN1, J9 M8 receptacle, Q2 CSD19533Q5A, Q7 Q_PMOS_GDS, U1 max6496, U3 MC74HCT595ADTR2G

Commit message: Finished BOM
Parts:
- U3: digikey_part_num (none) -> MC74HCT595ADTR2GOSCT-ND
- U8: value (none) -> D3V3M1U2S9-7; digikey_part_num (none) -> 31-D3V3M1U2S9-7CT-ND
- VR1: Manufacturer URL (none) -> https://www.lcsc.com/product-detail/C780769.html?s_z=n_q_AP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; digikey_part_num (none) -> AP63203WU-7DICT-ND
Changed lines of the file:
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@@
 			)
 		)
-		(property "Value" ""
+		(property "Value" "D3V3M1U2S9-7"
 			(at 30.48 139.7 0)
 			(show_name no)
@@
 			)
 		)
+		(property "digikey_part_num" "31-D3V3M1U2S9-7CT-ND"
+			(at 30.48 139.7 0)
+			(hide yes)
+			(show_name no)
+			(do_not_autoplace no)
+			(effects
+				(font
+					(size 1.27 1.27)
+				)
+			)
+		)
 		(pin "2"
 		)
@@
 			)
 		)
+		(property "digikey_part_num" "MC74HCT595ADTR2GOSCT-ND"
+			(at 196.85 100.33 0)
+			(hide yes)
+			(show_name no)
+			(do_not_autoplace no)
+			(effects
+				(font
+					(size 1.27 1.27)
+				)
+			)
+		)
 		(pin "13"
 		)
@@
 			(at 67.31 204.47 0)
 			(hide yes)
+			(show_name no)
+			(do_not_autoplace no)
+			(effects
+				(font
+					(size 1.27 1.27)
+				)
+			)
+		)
+		(property "Manufacturer URL" "https://www.lcsc.com/product-detail/C780769.html?s_z=n_q_AP63203WU-7&spm=wm.fly.bg.0.xh&lcsc_vid=T1UMUVNVEQUMUQEDQFYPXgBWQ1BfAlYDRAUPAVxRElUxVlNeQFlcV1ZVR1BeUzsOAxUeFF5JWBYZEEoKFBINSQcJGk4%3D"
+			(at 67.31 204.47 0)
+			(hide yes)
+			(show_name no)
+			(do_not_autoplace no)
+			(effects
+				(font
+					(size 1.27 1.27)
+				)
+			)
+		)
+		(property "digikey_part_num" "AP63203WU-7DICT-ND"
+			(at 67.31 204.47 0)
+			(hide yes)

Commit message: Initial component placement, finalising schematic
Parts:
- removed U3: MC74HCT595ADTR2G, Package_SO:TSSOP-16_4.4x5mm_P0.65mm, symbol component_library:MC74HCT595ADTR2G
- added C15: 100nF, Capacitor_SMD:C_0603_1608Metric, symbol Device:C
- added C16: 1uF, Capacitor_SMD:C_0603_1608Metric, symbol Device:C
- added C21, C22: 22uF, Capacitor_SMD:C_0603_1608Metric, symbol Device:C
- added JP13, JP14: ADDR, Jumper:SolderJumper-3_P1.3mm_Open_Pad1.0x1.5mm, symbol Jumper:SolderJumper_3_Open
- added MP4, MP5, MP6: Redcube Press Fit, footprints:MP_Wurth_WP-BUFU_7461097, symbol component_library:Redcube Press Fit
- added U12: MCP1792x-5002xDB, Package_TO_SOT_SMD:SOT-223-3_TabPin2, symbol Regulator_Linear:MCP1792x-5002xDB
- added U3: ADC128D818, Package_SO:TSSOP-16_4.4x5mm_P0.65mm, symbol Analog_ADC:ADC128D818
Connections:
- net 3V3: now also C15.2, C16.1, JP13.1 (A), JP14.1 (A), U3.5 (V+)
- net GND: now also C15.1, C16.2, C21.2, C22.2, JP13.3 (B), JP14.3 (B), U12.2 (GND), U3.4 (GND)
- net JMP_PWR: now also C21.1, U12.1 (VI); no longer 3V3_IND4.2 (A), D3.2 (A)
- net TEMP_INT: no longer PCB1.19 (IO12)
- net V_channel_mux: no longer names the net of PCB1.10 (A2)
- net channel_mux_addr0: no longer names the net of PCB1.12 (A4)
- net channel_mux_addr1: no longer names the net of PCB1.13 (A5)
- net channel_mux_addr2: no longer names the net of PCB1.14 (A6)
- new net: 3V3_IND4.2 (A), C22.1, D3.2 (A), U12.3 (VO)
- new net: JP14.2 (C), U3.7 (A0)
- new net: JP13.2 (C), U3.8 (A1)
- new net power_bus_2/PWR_OUT: MP4.1
- new net power_bus_3/PWR_OUT: MP5.1
- new net power_bus_4/PWR_OUT: MP6.1
- no-connect marks 25 -> 26
Other:
- added sheet power_bus_2 (power_bus_channel.kicad_sch)
- added sheet power_bus_3 (power_bus_channel.kicad_sch)
- added sheet power_bus_4 (power_bus_channel.kicad_sch)
- note added: "Protect against 48v overwhelming SBB if 12s used"
- note removed: "JUMP WILL SEND 48V TO SBB!!! Put inline 10-5v reg"
- moved on the sheet: 3V3_IND4, C3, D2, D3, MP3, PCB1, R11, R12, R2
