File: hardware/enc-encoder/enc-encoder.kicad_sch (KiCad schematic)
At the start: 0 parts

Commit message: Initial component placement
Parts:
- added 3V3, GND1, VBUS1, VCC1: Testpoint, TestPoint:TestPoint_Pad_D2.0mm, symbol Connector:TestPoint
- added C10, C11, C12, C13, C14, C15, C16, C17, C3, C7, C8, C9: 100nF, Capacitor_SMD:C_0603_1608Metric, symbol Device:C
- added C18, C19, C20, C21: 4.7uF, Capacitor_SMD:C_0603_1608Metric, symbol Device:C
- added C4: 10uF, Capacitor_SMD:C_0603_1608Metric, symbol Device:C
- added C5, C6: 22uF, Capacitor_SMD:C_0603_1608Metric, symbol Device:C
- added D1, D4: DSS14UTR, Diode_SMD:D_SOD-123F, symbol Device:D_Schottky
- added D2, D7: PESD1, Diode_SMD:D_SOD-882, symbol Device:D_TVS
- added D6: ESDA5V3L, Package_TO_SOT_SMD:SOT-416, symbol Power_Protection:RCLAMP0502B
- added F1: 500mA PTC fuse, Fuse:Fuse_1812_4532Metric, symbol Device:Fuse
- added F2: 500mA fast-blow fuse, Fuse:Fuse_0603_1608Metric, symbol Device:Fuse
- added J1: USB_C_Receptacle, Connector_USB:USB_C_Receptacle_Amphenol_12401610E4-2A, symbol Connector:USB_C_Receptacle
- added L1: HPC4018NF-4R7M, Inductor_SMD:L_Taiyo-Yuden_MD-4040, symbol Device:L
- added L2: 3.3uH, Inductor_SMD:L_0805_2012Metric_Pad1.05x1.20mm_HandSolder, symbol Device:L
- added R1, R2: 5.1k, symbol Device:R
- added R10: 10k, Resistor_SMD:R_0402_1005Metric, symbol Device:R
- added R11, R16, R9: 10k, Resistor_SMD:R_0603_1608Metric, symbol Device:R
- added R3: 33, symbol Device:R
- added R8: 470R, Resistor_SMD:R_0603_1608Metric, symbol Device:R
- added STATUS1: 16347, LED_SMD:LED_WS2812B_PLCC4_5.0x5.0mm_P3.2mm, symbol LED:WS2812B
- added SW1: SW_DIP_x03, symbol Switch:SW_DIP_x03
- added U1: RP2350A, Package_DFN_QFN:QFN-60-1EP_7x7mm_P0.4mm_EP3.4x3.4mm, symbol MCU_RaspberryPi:RP2350A
- added U2: W25Q128JVS, Package_SO:SOIC-8_5.3x5.3mm_P1.27mm, symbol Memory_Flash:W25Q128JVS
- added U3: SP3485CN, Package_SO:SOIC-8_3.9x4.9mm_P1.27mm, symbol Interface_UART:SP3485CN
- added VR1: AP63203WU-7, Package_TO_SOT_SMD:TSOT-23-6, symbol Regulator_Switching:AP63203WU
- added Y1: Crystal_GND24, symbol Device:Crystal_GND24
Connections:
- new net: L2.2, U1.48 (VREG_LX)
- new net: J1.B5 (CC2), R2.1
- new net: C4.1, F1.1, F2.2, R10.1, VCC1.1, VR1.3 (IN)
- new net: C7.1, R10.2, VR1.2 (EN)
- new net: R8.2, STATUS1.4 (DIN)
- new net: C19.1, R3.1, U1.46 (VREG_AVDD)
- new net: J1.A5 (CC1), R1.1
- new net: D1.1 (K), F1.2
- new net: C3.1, L1.1, VR1.5 (SW)
- new net: C3.2, VR1.6 (BST)
- new net: D4.1 (K), F2.1
- new net: Y1.2 (G), Y1.4 (G)
- new net +1V1: C16.1, C17.1, C18.1, C21.1, L2.1, U1.23 (DVDD), U1.39 (DVDD), U1.50 (VREG_FB), U1.6 (DVDD)
- new net 3V3: 3V3.1, C10.1, C11.1, C12.1, C13.1, C14.1, C15.1, C20.1, C5.1, C6.1, C8.1, C9.1, L1.2, R3.2, STATUS1.1 (VDD), U1.1 (IOVDD), U1.11 (IOVDD), U1.20 (IOVDD), U1.30 (IOVDD), U1.38 (IOVDD), U1.44 (ADC_AVDD), U1.45 (IOVDD), U1.49 (VREG_VIN), U1.53 (USB_OTP_VDD), U1.54 (QSPI_IOVDD), VR1.1 (FB)
- new net GND: C10.2, C11.2, C12.2, C13.2, C14.2, C15.2, C16.2, C17.2, C18.2, C19.2, C20.2, C21.2, C4.2, C5.2, C6.2, C7.2, C8.2, C9.2, D2.2 (A2), D6.3 (A), D7.2 (A2), GND1.1, J1.A1 (GND), J1.A12 (GND), J1.B1 (GND), J1.B12 (GND), J1.S1 (SHIELD), R1.2, R11.2, R16.2, R2.2, R9.2, STATUS1.3 (VSS), U1.47 (VREG_PGND), U1.61 (GND), VR1.4 (GND)
- new net LED_DOUT: STATUS1.2 (DOUT)
- new net USB_D_N: D6.1 (K1), J1.A7 (D-), J1.B7 (D-)
- new net USB_D_P: D6.2 (K2), J1.A6 (D+), J1.B6 (D+)
- new net VBUS: D2.1 (A1), D4.2 (A), J1.A4 (VBUS), J1.A9 (VBUS), J1.B4 (VBUS), J1.B9 (VBUS), VBUS1.1
- new net VIN: D1.2 (A), D7.1 (A1)
- new net uC_LED: R16.1, R8.1
- no-connect marks 0 -> 10
Other:
- note added: "2.5ms startup delay"
- note added: "5V 3A"
- note added: "Iout: 1A Max"
- note added: "Power supply"
- note added: "VIN: 3.8 - 32V"
- title: (none) -> Magnetic Angle Sensor

Commit message: Additions and cleanup
Parts:
- removed C11, C12, C13, C14, C15, C16, C17, C8, C9: 100nF, Capacitor_SMD:C_0603_1608Metric, symbol Device:C
- removed C18, C19, C20, C21: 4.7uF, Capacitor_SMD:C_0603_1608Metric, symbol Device:C
- removed L2: 3.3uH, Inductor_SMD:L_0805_2012Metric_Pad1.05x1.20mm_HandSolder, symbol Device:L
- removed R3: 33, symbol Device:R
- removed SW1: SW_DIP_x03, symbol Switch:SW_DIP_x03
- removed U1: RP2350A, Package_DFN_QFN:QFN-60-1EP_7x7mm_P0.4mm_EP3.4x3.4mm, symbol MCU_RaspberryPi:RP2350A
- removed U2: W25Q128JVS, Package_SO:SOIC-8_5.3x5.3mm_P1.27mm, symbol Memory_Flash:W25Q128JVS
- removed U3: SP3485CN, Package_SO:SOIC-8_3.9x4.9mm_P1.27mm, symbol Interface_UART:SP3485CN
- removed Y1: Crystal_GND24, symbol Device:Crystal_GND24
- added C23: 100nF, Capacitor_SMD:C_0603_1608Metric, symbol Device:C
- added C24: 100n, Capacitor_SMD:C_0603_1608Metric, symbol Capacitor:C_100n_50V_0603
- added D3: SM712_SOT23, Package_TO_SOT_SMD:SOT-23, symbol Diode:SM712_SOT23
- added H1, H2, H3, H4: M3, MountingHole:MountingHole_3.2mm_M3_DIN965_Pad, symbol Mechanical:MountingHole_Pad
- added J2: SM03B-SRSS-TB, Connector_JST:JST_SH_SM03B-SRSS-TB_1x03-1MP_P1.00mm_Horizontal, symbol Connector_Generic_MountingPin:Conn_01x03_MountingPin
- added J3, J4: OQ0232510000G, ConnectorsOther:AnyTek_OQ_3.81mm_90_2P_TriangleKeyLock, symbol Connector_Generic:Conn_01x02
- added R17, R19: 330, Resistor_SMD:R_0603_1608Metric, symbol Device:R
- added R18: 120, Resistor_SMD:R_0603_1608Metric, symbol Device:R
- added U4: (no value), Package_SO:SOIC-8_3.9x4.9mm_P1.27mm, symbol component_library:AS5600
- added U5: (no value), footprints:SW_218-4LPSTR, symbol component_library:4_DIP
- added U6: SP3485CN, Package_SO:SOIC-8_3.9x4.9mm_P1.27mm, symbol Interface_UART:SP3485CN
Connections:
- net 3V3: now also C23.1, U4.1 (VDD5V), U4.2 (VDD3V)
- net GND: now also C23.2, C24.2, D3.3 (common), H1.1, H2.1, H3.1, H4.1, J2.2 (Pin_2), J2.MP (MountPin), J3.2 (Pin_2), R19.2, U4.4 (GND), U6.5 (GND)
- new net: D3.1 (A1), J4.2 (Pin_2), R18.2, R19.1, U6.7 (B)
- new net: D3.2 (A2), J4.1 (Pin_1), R17.2, R18.1, U6.6 (A)
- new net +3V3: C24.1, J3.1 (Pin_1), R17.1, U6.8 (VCC)
- new net RP_SWCLK: J2.1 (Pin_1)
- new net RP_SWDIO: J2.3 (Pin_3)
- new net RS485_DIR: U6.2 (~{RE}), U6.3 (DE)
- new net RS485_RX: U6.1 (RO)
- new net RS485_TX: U6.4 (DI)
Other:
- added sheet rp2350 (rp2350a.kicad_sch)
- note added: "/RE LOW enables receiver DE HIGH enables transmitter"
- note added: "0.25 W"
- note added: "DEBUG INTERFACE"
- note added: "Failsafe Bias: V_AB = 3.3 * 60/(330 + 60 + 330) = 275 mV Idle differential v is ~275mV, above +-200mV used by RS-485"
- note added: "Termination resistor"
- moved on the sheet: 3V3, C10, C3, C4, C5, C6, C7, D1, D2, D4, D6, D7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
